File: KiCad files/Test PCBs/CNLJS_test_LEDice_dual/CNLJS_test_LEDice_dual.kicad_pcb (KiCad board)
At the start: 2 copper layers, 99.8 x 99.8 mm, 25 parts, among them J1 Conn_01x03_Male, U1 WS2812-4020_dual, U10 WS2812-4020_dual, U11 WS2812-4020_dual, U12 WS2812-4020_dual, U13 WS2812-4020_dual, U14 WS2812-4020_dual, U15 WS2812-4020_dual, U16 WS2812-4020_dual, U17 WS2812-4020_dual, U18 WS2812-4020_dual, U19 WS2812-4020_dual, U2 WS2812-4020_dual, U20 WS2812-4020_dual, U21 WS2812-4020_dual, U22 WS2812-4020_dual, U23 WS2812-4020_dual, U3 WS2812-4020_dual, U4 WS2812-4020_dual, U5 WS2812-4020_dual, U6 WS2812-4020_dual, U7 WS2812-4020_dual, U8 WS2812-4020_dual, U9 WS2812-4020_dual

Commit message: test_1
Parts:
- added G***: LOGO, test_library:test1, F.Cu at (146.1, 89.6)
- added U24: WS2812-4020_dual, Josip_global:WS2812-4020-dual-6mm_bezMaske, B.Cu at (180.3, 26.7)
- added U25: WS2812-4020_dual, Josip_global:WS2812-4020-dual-6mm_bezMaske, B.Cu at (192.5, 22.2)
- added U26: WS2812-4020_dual, Josip_global:WS2812-4020-dual-6mm_bezMaske, B.Cu at (204.3, 23.8)
- added U27: WS2812-4020_dual, Josip_global:WS2812-4020-dual-6mm_bezMaske, B.Cu at (212.7, 32.5)
- added U28: WS2812-4020_dual, Josip_global:WS2812-4020-dual-6mm_bezMaske, B.Cu at (213.9, 44.7)
- added U29: WS2812-4020_dual, Josip_global:WS2812-4020-dual-6mm_bezMaske, B.Cu at (209.0, 57.1)
- added U30: WS2812-4020_dual, Josip_global:WS2812-4020-dual-6mm_bezMaske, B.Cu at (199.2, 68.4)
- added U31: WS2812-4020_dual, Josip_global:WS2812-4020-dual-6mm_bezMaske, B.Cu at (186.7, 77.7)
- added U32: WS2812-4020_dual, Josip_global:WS2812-4020-dual-6mm_bezMaske, B.Cu at (173.2, 85.0)
- added U33: WS2812-4020_dual, Josip_global:WS2812-4020-dual-6mm_bezMaske, B.Cu at (163.0, 89.5)
- added U34: WS2812-4020_dual, Josip_global:WS2812-4020-dual-6mm_bezMaske, B.Cu at (175.0, 94.5)
- added U35: WS2812-4020_dual, Josip_global:WS2812-4020-dual-6mm_bezMaske, B.Cu at (188.2, 101.9)
- added U36: WS2812-4020_dual, Josip_global:WS2812-4020-dual-6mm_bezMaske, B.Cu at (195.0, 89.6)
- added U37: WS2812-4020_dual, Josip_global:WS2812-4020-dual-6mm_bezMaske, B.Cu at (203.1, 81.6)
- added U38: WS2812-4020_dual, Josip_global:WS2812-4020-dual-6mm_bezMaske, B.Cu at (151.3, 115.6)
- added U39: WS2812-4020_dual, Josip_global:WS2812-4020-dual-6mm_bezMaske, B.Cu at (211.0, 89.5)
- added U40: WS2812-4020_dual, Josip_global:WS2812-4020-dual-6mm_bezMaske, B.Cu at (146.9, 105.7)
- added U41: WS2812-4020_dual, Josip_global:WS2812-4020-dual-6mm_bezMaske, B.Cu at (203.1, 97.5)
- added U42: WS2812-4020_dual, Josip_global:WS2812-4020-dual-6mm_bezMaske, B.Cu at (141.8, 117.5)
- added U43: WS2812-4020_dual, Josip_global:WS2812-4020-dual-6mm_bezMaske, B.Cu at (200.3, 111.2)
- added U44: WS2812-4020_dual, Josip_global:WS2812-4020-dual-6mm_bezMaske, B.Cu at (134.4, 130.6)
- added U45: WS2812-4020_dual, Josip_global:WS2812-4020-dual-6mm_bezMaske, B.Cu at (209.7, 122.8)
- added U46: WS2812-4020_dual, Josip_global:WS2812-4020-dual-6mm_bezMaske, B.Cu at (146.9, 137.6)
- added U47: WS2812-4020_dual, Josip_global:WS2812-4020-dual-6mm_bezMaske, B.Cu at (214.1, 135.0)
- added U48: WS2812-4020_dual, Josip_global:WS2812-4020-dual-6mm_bezMaske, B.Cu at (154.9, 145.7)
- added U49: WS2812-4020_dual, Josip_global:WS2812-4020-dual-6mm_bezMaske, B.Cu at (212.5, 146.8)
- added U50: WS2812-4020_dual, Josip_global:WS2812-4020-dual-6mm_bezMaske, B.Cu at (146.9, 153.7)
- added U51: WS2812-4020_dual, Josip_global:WS2812-4020-dual-6mm_bezMaske, B.Cu at (203.8, 155.2)
- added U52: WS2812-4020_dual, Josip_global:WS2812-4020-dual-6mm_bezMaske, B.Cu at (138.9, 145.7)
- added U53: WS2812-4020_dual, Josip_global:WS2812-4020-dual-6mm_bezMaske, B.Cu at (191.7, 156.4)
- added U54: WS2812-4020_dual, Josip_global:WS2812-4020-dual-6mm_bezMaske, B.Cu at (125.1, 142.8)
- added U55: WS2812-4020_dual, Josip_global:WS2812-4020-dual-6mm_bezMaske, B.Cu at (179.3, 151.5)
- added U56: WS2812-4020_dual, Josip_global:WS2812-4020-dual-6mm_bezMaske, B.Cu at (113.6, 152.1)
- added U57: WS2812-4020_dual, Josip_global:WS2812-4020-dual-6mm_bezMaske, B.Cu at (167.9, 141.6)
- added U58: WS2812-4020_dual, Josip_global:WS2812-4020-dual-6mm_bezMaske, B.Cu at (101.4, 156.6)
- added U59: WS2812-4020_dual, Josip_global:WS2812-4020-dual-6mm_bezMaske, B.Cu at (158.6, 129.1)
- added U60: WS2812-4020_dual, Josip_global:WS2812-4020-dual-6mm_bezMaske, B.Cu at (89.5, 154.9)
- added U61: WS2812-4020_dual, Josip_global:WS2812-4020-dual-6mm_bezMaske, B.Cu at (81.1, 146.3)
- added U62: WS2812-4020_dual, Josip_global:WS2812-4020-dual-6mm_bezMaske, B.Cu at (79.9, 134.1)
- added U63: WS2812-4020_dual, Josip_global:WS2812-4020-dual-6mm_bezMaske, B.Cu at (84.9, 121.8)
- added U64: WS2812-4020_dual, Josip_global:WS2812-4020-dual-6mm_bezMaske, B.Cu at (94.7, 110.4)
- added U65: WS2812-4020_dual, Josip_global:WS2812-4020-dual-6mm_bezMaske, B.Cu at (107.1, 101.1)
- added U66: WS2812-4020_dual, Josip_global:WS2812-4020-dual-6mm_bezMaske, B.Cu at (120.7, 93.7)
- added U67: WS2812-4020_dual, Josip_global:WS2812-4020-dual-6mm_bezMaske, B.Cu at (130.8, 89.5)
- added U68: WS2812-4020_dual, Josip_global:WS2812-4020-dual-6mm_bezMaske, B.Cu at (118.9, 84.2)
- added U69: WS2812-4020_dual, Josip_global:WS2812-4020-dual-6mm_bezMaske, B.Cu at (122.8, 65.5)
- added U70: WS2812-4020_dual, Josip_global:WS2812-4020-dual-6mm_bezMaske, B.Cu at (114.9, 57.5)
- added U71: WS2812-4020_dual, Josip_global:WS2812-4020-dual-6mm_bezMaske, B.Cu at (106.8, 49.4)
- added U72: WS2812-4020_dual, Josip_global:WS2812-4020-dual-6mm_bezMaske, B.Cu at (98.8, 41.5)
- added U73: WS2812-4020_dual, Josip_global:WS2812-4020-dual-6mm_bezMaske, B.Cu at (170.9, 65.5)
- added U74: WS2812-4020_dual, Josip_global:WS2812-4020-dual-6mm_bezMaske, B.Cu at (179.0, 57.5)
- added U75: WS2812-4020_dual, Josip_global:WS2812-4020-dual-6mm_bezMaske, B.Cu at (187.0, 49.4)
- added U76: WS2812-4020_dual, Josip_global:WS2812-4020-dual-6mm_bezMaske, B.Cu at (195.0, 41.4)
- added U77: WS2812-4020_dual, Josip_global:WS2812-4020-dual-6mm_bezMaske, B.Cu at (170.9, 113.6)
- added U78: WS2812-4020_dual, Josip_global:WS2812-4020-dual-6mm_bezMaske, B.Cu at (179.0, 121.6)
- added U79: WS2812-4020_dual, Josip_global:WS2812-4020-dual-6mm_bezMaske, B.Cu at (187.0, 129.6)
- added U80: WS2812-4020_dual, Josip_global:WS2812-4020-dual-6mm_bezMaske, B.Cu at (195.0, 137.6)
- added U81: WS2812-4020_dual, Josip_global:WS2812-4020-dual-6mm_bezMaske, B.Cu at (122.9, 113.6)
- added U82: WS2812-4020_dual, Josip_global:WS2812-4020-dual-6mm_bezMaske, B.Cu at (114.9, 121.6)
- added U83: WS2812-4020_dual, Josip_global:WS2812-4020-dual-6mm_bezMaske, B.Cu at (106.8, 129.6)
- added U84: WS2812-4020_dual, Josip_global:WS2812-4020-dual-6mm_bezMaske, B.Cu at (98.8, 137.6)
- U1, U2, U3, U4, U5, U6, U7: moved to B.Cu
- U10, U11, U12, U13, U8, U9: footprint Josip_global:WS2812-4020-dual-8mm_bezMaske -> Josip_global:WS2812-4020-dual-6mm_bezMaske; moved to B.Cu
- U14, U15, U16, U17, U18: footprint Josip_global:WS2812-4020-dual-10mm_bezMaske -> Josip_global:WS2812-4020-dual-6mm_bezMaske; moved to B.Cu
- U19, U20, U21, U22, U23: footprint Josip_global:WS2812-4020-dual-12mm_bezMaske -> Josip_global:WS2812-4020-dual-6mm_bezMaske; moved to B.Cu
- moved U7 134.3 mm to (84.3, 56.1), turned to 180 degrees
- moved U6 109.5 mm to (93.5, 67.6), turned to 180 degrees
- moved U17 109.2 mm to (81.3, 31.9), turned to 180 degrees
- moved U23 92.1 mm to (114.5, 27.3), turned to 180 degrees
- moved U5 84.2 mm to (105.7, 76.9), turned to 180 degrees
- moved U15 80.8 mm to (79.8, 43.9), turned to 180 degrees
- moved U3 76.5 mm to (90.8, 81.7)
- moved U21 75.7 mm to (102.2, 22.4), turned to 180 degrees
- moved U4 74.3 mm to (98.8, 89.7), turned to 180 degrees
- moved U18 74.3 mm to (147.0, 25.4), turned to 180 degrees
- moved U2 71.4 mm to (82.8, 89.7)
- moved U8 69.0 mm to (125.9, 37.1), turned to 180 degrees
- moved U13 68.6 mm to (159.4, 48.2), turned to 180 degrees
- moved U19 61.1 mm to (90.0, 23.6), turned to 180 degrees
- moved U9 56.9 mm to (135.2, 49.6), turned to 180 degrees
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Connections:
- U13 pad 5: unconnected-(U13-Pad5) -> Net-(U13-Pad5)
- U14 pad 1: Net-(R1-Pad2) -> Net-(U13-Pad5)
- U15 pad 1: Net-(U14-Pad5) -> Net-(U7-Pad5)
- U16 pad 1: Net-(U15-Pad5) -> Net-(U14-Pad5)
- U17 pad 1: Net-(U16-Pad5) -> Net-(U15-Pad5)
- U18 pad 1: Net-(U17-Pad5) -> Net-(U16-Pad5)
- U18 pad 5: unconnected-(U18-Pad5) -> Net-(U18-Pad5)
- U19 pad 1: Net-(R1-Pad2) -> Net-(U17-Pad5)
- U20 pad 1: Net-(U19-Pad5) -> Net-(U18-Pad5)
- U21 pad 1: Net-(U20-Pad5) -> Net-(U19-Pad5)
- U22 pad 1: Net-(U21-Pad5) -> Net-(U20-Pad5)
- U23 pad 1: Net-(U22-Pad5) -> Net-(U21-Pad5)
- U23 pad 5: unconnected-(U23-Pad5) -> Net-(U23-Pad5)
- U7 pad 5: unconnected-(U7-Pad5) -> Net-(U7-Pad5)
- U8 pad 1: Net-(R1-Pad2) -> Net-(U23-Pad5)
Routing:
- net VDD: track 785.2 -> 0.00 mm
- net (no net): track 380.6 -> 0.00 mm
- net Net-(R1-Pad2): track 109.0 -> 0.00 mm
- net GND: track 85.2 -> 0.00 mm, vias 46 -> 0
- net Net-(U22-Pad5): track 33.8 -> 0.00 mm
- net Net-(U20-Pad5): track 32.3 -> 0.00 mm
- net Net-(U21-Pad5): track 32.1 -> 0.00 mm
- net Net-(U17-Pad5): track 30.4 -> 0.00 mm
- net Net-(U19-Pad5): track 30.3 -> 0.00 mm
- net Net-(U16-Pad5): track 29.5 -> 0.00 mm
- net Net-(U12-Pad5): track 28.3 -> 0.00 mm
- net Net-(U15-Pad5): track 27.6 -> 0.00 mm
- net Net-(U11-Pad5): track 26.9 -> 0.00 mm
- net Net-(U14-Pad5): track 26.9 -> 0.00 mm
- net Net-(U10-Pad5): track 26.3 -> 0.00 mm
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- removed copper zone on B.Cu, net GND
Other:
- board size 99.8 x 99.8 mm -> 150 x 150 mm
- board text removed: "GND"
- board text removed: "IN"
- board text removed: "JLCJLCJLCJLC"
- board text removed: "VDD"

Commit message: layout
Parts:
- removed the G*** at (146.1, 89.6)
- added G***: LOGO, Library:pozadina_v2, F.Cu at (146.7, 89.3)
- added R2: 470, Resistor_SMD:R_0805_2012Metric, F.Cu at (253.8, 62.3)
- added R3: 470, Resistor_SMD:R_0805_2012Metric, F.Cu at (253.8, 65.2)
- added R4: 470, Resistor_SMD:R_0805_2012Metric, F.Cu at (258.2, 67.5)
- added U85: WS2812-4020_dual, Josip_global:WS2812-4020-single-6mm_bezMaske, F.Cu at (140.3, 83.1)
- added U86: WS2812-4020_dual, Josip_global:WS2812-4020-single-6mm_bezMaske, F.Cu at (146.9, 83.1)
- added U87: WS2812-4020_dual, Josip_global:WS2812-4020-single-6mm_bezMaske, F.Cu at (153.5, 83.1)
- added U88: WS2812-4020_dual, Josip_global:WS2812-4020-single-6mm_bezMaske, F.Cu at (153.5, 89.7)
- added U89: WS2812-4020_dual, Josip_global:WS2812-4020-single-6mm_bezMaske, F.Cu at (146.9, 89.8)
- added U90: WS2812-4020_dual, Josip_global:WS2812-4020-single-6mm_bezMaske, F.Cu at (140.3, 89.7)
- added U91: WS2812-4020_dual, Josip_global:WS2812-4020-single-6mm_bezMaske, F.Cu at (140.3, 96.3)
- added U92: WS2812-4020_dual, Josip_global:WS2812-4020-single-6mm_bezMaske, F.Cu at (146.9, 96.3)
- added U93: WS2812-4020_dual, Josip_global:WS2812-4020-single-6mm_bezMaske, F.Cu at (153.5, 96.3)
- J1: value Conn_01x03_Male -> Conn_01x06_Male; footprint Connector_PinHeader_2.54mm:PinHeader_1x03_P2.54mm_Vertical -> Connector_PinHeader_2.54mm:PinHeader_1x06_P2.54mm_Horizontal
- U1, U10, U11, U12, U13, U14, U15, U16, U17, U18, U19, U2, U20, U21, U22, U23, U24, U25, U26, U27, U28, U29, U3, U30, U31, U32, U33, U34, U35, U36, U37, U38, U39, U4, U40, U41, U42, U43, U44, U45, U46, U47, U48, U49, U5, U50, U51, U52, U53, U54, U55, U56, U57, U58, U59, U6, U60, U61, U62, U63, U64, U65, U66, U67, U68, U69, U7, U70, U71, U72, U73, U74, U75, U76, U77, U78, U79, U8, U80, U81, U82, U83, U84, U9: footprint Josip_global:WS2812-4020-dual-6mm_bezMaske -> Josip_global:WS2812-4020-dual-7mm_bezMaske; moved to F.Cu
- moved R1 191.8 mm to (261.6, 51.0)
- moved J1 184.8 mm to (253.9, 34.5)
- moved U16 104.7 mm to (104.4, 132.2), turned to 0 degrees
- moved U7 97.6 mm to (181.9, 54.7)
- moved U15 86.9 mm to (111.9, 124.7), turned to 0 degrees
- moved U6 81.1 mm to (174.4, 62.2)
- moved U14 80.6 mm to (119.4, 117.2), turned to 0 degrees
- moved U12 80.1 mm to (189.4, 132.2), turned to 0 degrees
- moved U22 79.5 mm to (89.9, 25.2)
- moved U27 76.6 mm to (141.4, 60.4), turned to 0 degrees
- moved U34 75.0 mm to (203.6, 25.2), turned to 0 degrees
- moved U26 74.9 mm to (133.6, 48.4), turned to 0 degrees
- moved U20 74.4 mm to (81.2, 43.4), turned to 90 degrees
- moved U35 72.9 mm to (211.1, 32.7), turned to -45 degrees
- moved U33 72.0 mm to (192.9, 24.0), turned to 0 degrees
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Connections:
- J1 pad 3: GND -> Net-(J1-Pad3)
- U15 pad 1: Net-(U7-Pad5) -> Net-(U14-Pad5)
- U16 pad 1: Net-(U14-Pad5) -> Net-(U15-Pad5)
- U16 pad 5: Net-(U16-Pad5) -> unconnected-(U16-Pad5)
- U17 pad 1: Net-(U15-Pad5) -> Net-(R2-Pad2)
- U18 pad 1: Net-(U16-Pad5) -> Net-(U17-Pad5)
- U19 pad 1: Net-(U17-Pad5) -> Net-(U18-Pad5)
- U20 pad 1: Net-(U18-Pad5) -> Net-(U19-Pad5)
- U21 pad 1: Net-(U19-Pad5) -> Net-(U20-Pad5)
- U22 pad 1: Net-(U20-Pad5) -> Net-(U21-Pad5)
- U23 pad 1: Net-(U21-Pad5) -> Net-(U22-Pad5)
- U24 pad 1: Net-(U22-Pad5) -> Net-(U23-Pad5)
- U38 pad 1: Net-(U38-Pad1) -> Net-(U37-Pad5)
- U39 pad 1: Net-(U37-Pad5) -> Net-(U38-Pad5)
- U40 pad 1: Net-(U38-Pad5) -> Net-(U39-Pad5)
- U41 pad 1: Net-(U39-Pad5) -> Net-(U40-Pad5)
- U42 pad 1: Net-(U40-Pad5) -> Net-(U41-Pad5)
- U43 pad 1: Net-(U41-Pad5) -> Net-(U42-Pad5)
- U44 pad 1: Net-(U42-Pad5) -> Net-(U43-Pad5)
- U45 pad 1: Net-(U43-Pad5) -> Net-(U44-Pad5)
- U46 pad 1: Net-(U44-Pad5) -> Net-(U45-Pad5)
- U47 pad 1: Net-(U45-Pad5) -> Net-(U46-Pad5)
- U48 pad 1: Net-(U46-Pad5) -> Net-(U47-Pad5)
- U49 pad 1: Net-(U47-Pad5) -> Net-(U48-Pad5)
- U50 pad 1: Net-(U48-Pad5) -> Net-(U49-Pad5)
- U51 pad 1: Net-(U49-Pad5) -> Net-(U50-Pad5)
- U52 pad 1: Net-(U50-Pad5) -> Net-(U51-Pad5)
- U53 pad 1: Net-(U51-Pad5) -> Net-(U52-Pad5)
- U54 pad 1: Net-(U52-Pad5) -> Net-(U53-Pad5)
- U55 pad 1: Net-(U53-Pad5) -> Net-(U54-Pad5)
- U56 pad 1: Net-(U54-Pad5) -> Net-(U55-Pad5)
- U57 pad 1: Net-(U55-Pad5) -> Net-(U56-Pad5)
- U58 pad 1: Net-(U56-Pad5) -> Net-(U57-Pad5)
- U59 pad 1: Net-(U57-Pad5) -> Net-(U58-Pad5)
- U59 pad 5: Net-(U38-Pad1) -> Net-(U59-Pad5)
- U60 pad 1: Net-(U58-Pad5) -> Net-(U59-Pad5)
- U68 pad 5: Net-(U68-Pad5) -> unconnected-(U68-Pad5)
- U69 pad 1: Net-(U68-Pad5) -> Net-(R3-Pad2)
- U8 pad 1: Net-(U23-Pad5) -> Net-(U7-Pad5)
Routing:
- net (no net): track 0.00 -> 82.5 mm
- net Net-(U20-Pad5): track 0.00 -> 18.6 mm
- net Net-(U66-Pad5): track 0.00 -> 12.6 mm
- net Net-(U19-Pad5): track 0.00 -> 11.7 mm
- net Net-(U18-Pad5): track 0.00 -> 10.4 mm
- net Net-(U67-Pad5): track 0.00 -> 8.97 mm
- net Net-(U17-Pad5): track 0.00 -> 6.19 mm

Commit message: update
Parts:
- turned U24 to 180 degrees
Routing:
- net (no net): track 82.5 -> 147.2 mm
- net Net-(U24-Pad5): track 0.00 -> 21.7 mm
- net Net-(U22-Pad5): track 0.00 -> 17.4 mm
- net Net-(U23-Pad5): track 0.00 -> 17.0 mm
- net Net-(U21-Pad5): track 0.00 -> 15.7 mm

Commit message: update
Parts:
- U1, U10, U11, U12, U13, U14, U15, U16, U17, U18, U19, U2, U20, U21, U22, U23, U24, U25, U26, U27, U28, U29, U3, U30, U31, U32, U33, U34, U35, U36, U37, U38, U39, U4, U40, U41, U42, U43, U44, U45, U46, U47, U48, U49, U5, U50, U51, U52, U53, U54, U55, U56, U57, U58, U59, U6, U60, U61, U62, U63, U64, U65, U66, U67, U68, U69, U7, U70, U71, U72, U73, U74, U75, U76, U77, U78, U79, U8, U80, U81, U82, U83, U84, U9: footprint Josip_global:WS2812-4020-dual-7mm_bezMaske -> test_library:WS2812-4020-dual-7mm_bezMaske
- U85, U86, U87, U88, U89, U90, U91, U92, U93: footprint Josip_global:WS2812-4020-single-6mm_bezMaske -> test_library:WS2812-4020-single-6mm_bezMaske
- turned U91 to -45 degrees
- turned U93 to 45 degrees

Commit message: route
Parts:
- removed the G*** at (146.7, 89.3)
- added C1: 0-50 pF, Capacitor_SMD:C_0805_2012Metric, F.Cu at (259.9, 105.1)
- added C2: 100n, Capacitor_SMD:C_0805_2012Metric, F.Cu at (270.2, 97.6)
- added C3: 0-50 pF, Capacitor_SMD:C_0805_2012Metric, F.Cu at (251.7, 122.8)
- added C4: 100n, Capacitor_SMD:C_0805_2012Metric, F.Cu at (264.4, 105.1)
- added C5: 0-50 pF, Capacitor_SMD:C_0805_2012Metric, F.Cu at (259.9, 102.1)
- added C6: 100n, Capacitor_SMD:C_0805_2012Metric, F.Cu at (264.4, 102.1)
- added G***: LOGO, Library:pozadina_v3, F.Cu at (149.3, 90.3)
- added J2: Conn_01x14_Male, Connector_PinHeader_2.54mm:PinHeader_1x14_P2.54mm_Horizontal, F.Cu at (246.6, 86.0)
- added TP1: TestPoint, test_library:TP_11mm_strelicaLijevo, B.Cu at (80.9, 105.0)
- added TP2: TestPoint, test_library:TP_11mm_kvacica, B.Cu at (80.9, 89.7)
- added TP3: TestPoint, test_library:TP_11mm_strelicaDesno, B.Cu at (80.9, 69.7)
- added U94: TTP223-BA6, Package_TO_SOT_SMD:SOT-23-6, F.Cu at (246.8, 123.5)
- added U95: TTP223-BA6, Package_TO_SOT_SMD:SOT-23-6, F.Cu at (265.4, 98.4)
- added U96: TTP223-BA6, Package_TO_SOT_SMD:SOT-23-6, F.Cu at (260.2, 98.4)
- moved R2 138.4 mm to (116.0, 74.9), turned to 180 degrees
- moved R1 131.0 mm to (131.9, 69.3), turned to 90 degrees
- moved U12 7.53 mm to (194.8, 137.4), turned to 90 degrees
- moved U10 7.50 mm to (179.8, 122.4), turned to 90 degrees
- moved U11 7.50 mm to (187.3, 129.9), turned to -90 degrees
- moved U9 7.50 mm to (172.3, 114.9), turned to -90 degrees
- moved U5 7.44 mm to (172.5, 64.8), turned to -90 degrees
- moved U8 7.38 mm to (195.0, 42.4), turned to -90 degrees
- moved U6 7.30 mm to (179.9, 57.4), turned to 90 degrees
- moved U7 7.30 mm to (187.4, 49.9), turned to -90 degrees
- moved U16 7.14 mm to (99.5, 137.4)
- moved U13 7.14 mm to (122.0, 114.9)
- moved U14 7.14 mm to (114.5, 122.4)
- moved U15 7.14 mm to (107.0, 129.9)
- moved U2 7.00 mm to (114.5, 57.2), turned to -90 degrees
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Routing:
- net (no net): track 147.2 -> 1059.0 mm
- net Net-(U8-Pad5): track 0.00 -> 108.4 mm
- net Net-(U4-Pad5): track 0.00 -> 84.0 mm
- net Net-(U12-Pad5): track 0.00 -> 47.6 mm
- net Net-(U49-Pad5): track 0.00 -> 20.1 mm
- net Net-(U32-Pad5): track 0.00 -> 19.5 mm
- net Net-(U56-Pad5): track 0.00 -> 19.0 mm
- net Net-(U5-Pad5): track 0.00 -> 18.3 mm
- net Net-(U31-Pad5): track 0.00 -> 17.8 mm
- net Net-(U10-Pad5): track 0.00 -> 17.3 mm
- net Net-(U62-Pad5): track 0.00 -> 17.1 mm
- net Net-(U57-Pad5): track 0.00 -> 16.8 mm
- net Net-(U59-Pad5): track 0.00 -> 16.5 mm
- net Net-(U2-Pad5): track 0.00 -> 16.4 mm
- net Net-(U6-Pad5): track 0.00 -> 16.3 mm
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- added copper zone on B.Cu, net GND
- added copper zone on F.Cu, net GND
Other:
- board text added: "1"

Commit message: update
Parts:
- renumbered U13 to U1, U6 to U10, U7 to U11, U8 to U12, U1 to U13, U2 to U14, U3 to U15, U4 to U16, U14 to U2, U15 to U3, U16 to U4, U9 to U5, U10 to U6, U11 to U7, U12 to U8, U87 to U85, U85 to U87, U90 to U88, U91 to U89, U5 to U9, U92 to U90, U93 to U91, U88 to U92, U89 to U93
Connections:
- U1 pad 1: Net-(U12-Pad5) -> Net-(R1-Pad2)
- U12 pad 5: Net-(U8-Pad5) -> Net-(U12-Pad5)
- U13 pad 1: Net-(R1-Pad2) -> Net-(U12-Pad5)
- U16 pad 5: Net-(U4-Pad5) -> unconnected-(U16-Pad5)
- U4 pad 5: unconnected-(U16-Pad5) -> Net-(U4-Pad5)
- U5 pad 1: Net-(U8-Pad5) -> Net-(U4-Pad5)
- U8 pad 5: Net-(U12-Pad5) -> Net-(U8-Pad5)
- U85 pad 1: Net-(U86-Pad5) -> Net-(R4-Pad2)
- U87 pad 1: Net-(R4-Pad2) -> Net-(U86-Pad4)
- U9 pad 1: Net-(U4-Pad5) -> Net-(U8-Pad5)
Routing:
- net unconnected-(U16-Pad5): track 0.00 -> 84.0 mm
- net Net-(U4-Pad5): track 84.0 -> 0.00 mm
- net Net-(U12-Pad5): track 47.6 -> 116.6 mm
- net Net-(U8-Pad5): track 108.4 -> 47.6 mm
- net (no net): track 1059.0 -> 1024.6 mm
- net VDD: track 1.10 -> 19.8 mm
- net GND: track 0.00 -> 15.8 mm
- net Net-(R1-Pad2): track 8.20 -> 0.00 mm
