File: KiCad files/Test PCBs/CNLJS_test_LEDice_dual/CNLJS_test_LEDice_dual.kicad_sch (KiCad schematic)
At the start: 25 parts, among them J1 Conn_01x03_Male, U1 WS2812-4020_dual, U10 WS2812-4020_dual, U11 WS2812-4020_dual, U12 WS2812-4020_dual, U13 WS2812-4020_dual, U14 WS2812-4020_dual, U15 WS2812-4020_dual, U16 WS2812-4020_dual, U17 WS2812-4020_dual, U18 WS2812-4020_dual, U19 WS2812-4020_dual, U2 WS2812-4020_dual, U20 WS2812-4020_dual, U21 WS2812-4020_dual, U22 WS2812-4020_dual, U23 WS2812-4020_dual, U3 WS2812-4020_dual, U4 WS2812-4020_dual, U5 WS2812-4020_dual, U6 WS2812-4020_dual, U7 WS2812-4020_dual, U8 WS2812-4020_dual, U9 WS2812-4020_dual

Commit message: test_1
Parts:
- added U24, U25, U26, U27, U28, U29, U30, U31, U32, U33, U34, U35, U36, U37, U38, U39, U40, U41, U42, U43, U44, U45, U46, U47, U48, U49, U50, U51, U52, U53, U54, U55, U56, U57, U58, U59, U60, U61, U62, U63, U64, U65, U66, U67, U68, U69, U70, U71, U72, U73, U74, U75, U76, U77, U78, U79, U80, U81, U82, U83, U84: WS2812-4020_dual, Josip_global:WS2812-4020-dual-6mm_bezMaske, symbol Josip_symbol_global:WS2812-4020_dual
- U10, U11, U12, U13, U8, U9: footprint Josip_global:WS2812-4020-dual-8mm_bezMaske -> Josip_global:WS2812-4020-dual-6mm_bezMaske
- U14, U15, U16, U17, U18: footprint Josip_global:WS2812-4020-dual-10mm_bezMaske -> Josip_global:WS2812-4020-dual-6mm_bezMaske
- U19, U20, U21, U22, U23: footprint Josip_global:WS2812-4020-dual-12mm_bezMaske -> Josip_global:WS2812-4020-dual-6mm_bezMaske
Connections:
- net GND: now also U24.4 (VSS), U25.4 (VSS), U26.4 (VSS), U27.4 (VSS), U28.4 (VSS), U29.4 (VSS), U30.4 (VSS), U31.4 (VSS), U32.4 (VSS), U33.4 (VSS), U34.4 (VSS), U35.4 (VSS), U36.4 (VSS), U37.4 (VSS), U38.4 (VSS), U39.4 (VSS), U40.4 (VSS), U41.4 (VSS), U42.4 (VSS), U43.4 (VSS), U44.4 (VSS), U45.4 (VSS), U46.4 (VSS), U47.4 (VSS), U48.4 (VSS), U49.4 (VSS), U50.4 (VSS), U51.4 (VSS), U52.4 (VSS), U53.4 (VSS), U54.4 (VSS), U55.4 (VSS), U56.4 (VSS), U57.4 (VSS), U58.4 (VSS), U59.4 (VSS), U60.4 (VSS), U61.4 (VSS), U62.4 (VSS), U63.4 (VSS), U64.4 (VSS), U65.4 (VSS), U66.4 (VSS), U67.4 (VSS), U68.4 (VSS), U69.4 (VSS), U70.4 (VSS), U71.4 (VSS), U72.4 (VSS), U73.4 (VSS), U74.4 (VSS), U75.4 (VSS), U76.4 (VSS), U77.4 (VSS), U78.4 (VSS), U79.4 (VSS), U80.4 (VSS), U81.4 (VSS), U82.4 (VSS), U83.4 (VSS), U84.4 (VSS)
- net VDD: now also U24.2 (VDD), U25.2 (VDD), U26.2 (VDD), U27.2 (VDD), U28.2 (VDD), U29.2 (VDD), U30.2 (VDD), U31.2 (VDD), U32.2 (VDD), U33.2 (VDD), U34.2 (VDD), U35.2 (VDD), U36.2 (VDD), U37.2 (VDD), U38.2 (VDD), U39.2 (VDD), U40.2 (VDD), U41.2 (VDD), U42.2 (VDD), U43.2 (VDD), U44.2 (VDD), U45.2 (VDD), U46.2 (VDD), U47.2 (VDD), U48.2 (VDD), U49.2 (VDD), U50.2 (VDD), U51.2 (VDD), U52.2 (VDD), U53.2 (VDD), U54.2 (VDD), U55.2 (VDD), U56.2 (VDD), U57.2 (VDD), U58.2 (VDD), U59.2 (VDD), U60.2 (VDD), U61.2 (VDD), U62.2 (VDD), U63.2 (VDD), U64.2 (VDD), U65.2 (VDD), U66.2 (VDD), U67.2 (VDD), U68.2 (VDD), U69.2 (VDD), U70.2 (VDD), U71.2 (VDD), U72.2 (VDD), U73.2 (VDD), U74.2 (VDD), U75.2 (VDD), U76.2 (VDD), U77.2 (VDD), U78.2 (VDD), U79.2 (VDD), U80.2 (VDD), U81.2 (VDD), U82.2 (VDD), U83.2 (VDD), U84.2 (VDD)
- net at U7.5 (DOUT): now also U15.1 (DIN)
- net at U16.5 (DOUT): now also U18.1 (DIN); no longer U17.1 (DIN)
- net at U17.5 (DOUT): now also U19.1 (DIN); no longer U18.1 (DIN)
- net at U22.1 (DIN): now also U20.5 (DOUT); no longer U21.5 (DOUT)
- net at U22.5 (DOUT): now also U24.1 (DIN); no longer U23.1 (DIN)
- net at U20.1 (DIN): now also U18.5 (DOUT); no longer U19.5 (DOUT)
- net at U14.5 (DOUT): now also U16.1 (DIN); no longer U15.1 (DIN)
- net at U21.1 (DIN): now also U19.5 (DOUT); no longer U20.5 (DOUT)
- net at U15.5 (DOUT): now also U17.1 (DIN); no longer U16.1 (DIN)
- net at U23.5 (DOUT): now also U8.1 (DIN)
- net at U13.5 (DOUT): now also U14.1 (DIN)
- new net: U42.5 (DOUT), U44.1 (DIN)
- new net: U44.5 (DOUT), U46.1 (DIN)
- new net: U53.5 (DOUT), U55.1 (DIN)
- new net: U55.5 (DOUT), U57.1 (DIN)
- new net: U26.5 (DOUT), U27.1 (DIN)
- new net: U27.5 (DOUT), U28.1 (DIN)
- new net: U39.5 (DOUT), U41.1 (DIN)
- new net: U41.5 (DOUT), U43.1 (DIN)
- new net: U34.5 (DOUT), U35.1 (DIN)
- new net: U35.5 (DOUT), U36.1 (DIN)
- new net: R1.2, U1.1 (DIN)
- new net: U62.5 (DOUT), U63.1 (DIN)
- new net: U63.5 (DOUT), U64.1 (DIN)
- new net: U79.5 (DOUT), U80.1 (DIN)
- new net: U80.5 (DOUT), U81.1 (DIN)
- new net: U48.5 (DOUT), U50.1 (DIN)
- new net: U50.5 (DOUT), U52.1 (DIN)
- new net: U38.5 (DOUT), U40.1 (DIN)
- new net: U40.5 (DOUT), U42.1 (DIN)
- new net: U30.5 (DOUT), U31.1 (DIN)
- new net: U31.5 (DOUT), U32.1 (DIN)
- new net: U28.5 (DOUT), U29.1 (DIN)
- new net: U52.5 (DOUT), U54.1 (DIN)
- new net: U81.5 (DOUT), U82.1 (DIN)
- new net: U82.5 (DOUT), U83.1 (DIN)
- new net: U46.5 (DOUT), U48.1 (DIN)
- new net: U57.5 (DOUT), U59.1 (DIN)
- new net: U38.1 (DIN), U59.5 (DOUT)
- new net: U47.5 (DOUT), U49.1 (DIN)
- new net: U49.5 (DOUT), U51.1 (DIN)
- new net: U25.5 (DOUT), U26.1 (DIN)
- new net: U75.5 (DOUT), U76.1 (DIN)
- new net: U76.5 (DOUT), U77.1 (DIN)
- new net: U72.5 (DOUT), U73.1 (DIN)
- new net: U73.5 (DOUT), U74.1 (DIN)
- new net: U24.5 (DOUT), U25.1 (DIN)
- new net: U64.5 (DOUT), U65.1 (DIN)
- new net: U58.5 (DOUT), U60.1 (DIN)
- new net: U60.5 (DOUT), U61.1 (DIN)
- new net: U78.5 (DOUT), U79.1 (DIN)
- new net: U37.5 (DOUT), U39.1 (DIN)
- new net: U67.5 (DOUT), U68.1 (DIN)
- new net: U68.5 (DOUT), U69.1 (DIN)
- new net: U33.5 (DOUT), U34.1 (DIN)
- new net: U51.5 (DOUT), U53.1 (DIN)
- new net: U29.5 (DOUT), U30.1 (DIN)
- new net: U69.5 (DOUT), U70.1 (DIN)
- new net: U70.5 (DOUT), U71.1 (DIN)
- new net: U65.5 (DOUT), U66.1 (DIN)
- new net: U36.5 (DOUT), U37.1 (DIN)
- new net: U21.5 (DOUT), U23.1 (DIN)
- new net: U71.5 (DOUT), U72.1 (DIN)
- new net: U54.5 (DOUT), U56.1 (DIN)
- new net: U56.5 (DOUT), U58.1 (DIN)
- new net: U43.5 (DOUT), U45.1 (DIN)
- new net: U45.5 (DOUT), U47.1 (DIN)
- new net: U66.5 (DOUT), U67.1 (DIN)
- new net: U32.5 (DOUT), U33.1 (DIN)
- new net: U77.5 (DOUT), U78.1 (DIN)
- new net: U83.5 (DOUT), U84.1 (DIN)
- new net: U74.5 (DOUT), U75.1 (DIN)
- new net: U61.5 (DOUT), U62.1 (DIN)
- no-connect marks 4 -> 0
Other:
- moved on the sheet: J1, R1, U1, U2, U3, U4, U5, U6, U7

Commit message: layout
Parts:
- removed J1: Conn_01x03_Male, Connector_PinHeader_2.54mm:PinHeader_1x03_P2.54mm_Vertical, symbol Connector:Conn_01x03_Male
- removed U8, U9: WS2812-4020_dual, Josip_global:WS2812-4020-dual-6mm_bezMaske, symbol Josip_symbol_global:WS2812-4020_dual
- added J1: (no value), symbol Connector:Conn_01x06_Male
- added R2, R3, R4: 470, Resistor_SMD:R_0805_2012Metric, symbol Device:R_Small
- added U15, U17, U85, U86, U87, U88, U89, U90, U91, U92, U93: WS2812-4020_dual, symbol Josip_symbol_global:WS2812-4020_dual
- U1, U10, U11, U12, U13, U14, U16, U18, U19, U2, U20, U21, U22, U23, U24, U25, U26, U27, U28, U29, U3, U30, U31, U32, U33, U34, U35, U36, U37, U38, U39, U4, U40, U41, U42, U43, U44, U45, U46, U47, U48, U49, U5, U50, U51, U52, U6, U7: footprint Josip_global:WS2812-4020-dual-6mm_bezMaske -> (none)
- U53, U54, U55, U56, U57, U58, U59, U60, U61, U62, U63, U64, U65, U66, U67, U68, U69, U70, U71, U72, U73, U74, U75, U76, U77, U78, U79, U80, U81, U82, U83, U84: footprint Josip_global:WS2812-4020-dual-6mm_bezMaske -> Josip_global:WS2812-4020-dual-7mm_bezMaske
- U8: renamed from U15; footprint Josip_global:WS2812-4020-dual-6mm_bezMaske -> (none)
- U9: renamed from U17; footprint Josip_global:WS2812-4020-dual-6mm_bezMaske -> (none)
Connections:
- net GND: now also J1.6 (Pin_6), U15.4 (VSS), U17.4 (VSS), U85.4 (VSS), U86.4 (VSS), U87.4 (VSS), U88.4 (VSS), U89.4 (VSS), U90.4 (VSS), U91.4 (VSS), U92.4 (VSS), U93.4 (VSS)
- net VDD: now also J1.1 (Pin_1), U15.2 (VDD), U17.2 (VDD), U85.2 (VDD), U86.2 (VDD), U87.2 (VDD), U88.2 (VDD), U89.2 (VDD), U90.2 (VDD), U91.2 (VDD), U92.2 (VDD), U93.2 (VDD)
- net at U42.5 (DOUT): now also U43.1 (DIN); no longer U44.1 (DIN)
- net at U44.5 (DOUT): now also U45.1 (DIN); no longer U46.1 (DIN)
- net at U53.5 (DOUT): now also U54.1 (DIN); no longer U55.1 (DIN)
- net at U55.5 (DOUT): now also U56.1 (DIN); no longer U57.1 (DIN)
- net at U39.5 (DOUT): now also U40.1 (DIN); no longer U41.1 (DIN)
- net at U41.5 (DOUT): now also U42.1 (DIN); no longer U43.1 (DIN)
- net at U50.1 (DIN): now also U49.5 (DOUT); no longer U48.5 (DOUT)
- net at U50.5 (DOUT): now also U51.1 (DIN); no longer U52.1 (DIN)
- net at U38.5 (DOUT): now also U39.1 (DIN); no longer U40.1 (DIN)
- net at U40.5 (DOUT): now also U41.1 (DIN); no longer U42.1 (DIN)
- net at U22.1 (DIN): now also U21.5 (DOUT); no longer U20.5 (DOUT)
- net at U22.5 (DOUT): now also U23.1 (DIN); no longer U24.1 (DIN)
- net at U16.1 (DIN): now also U15.5 (DOUT); no longer U14.5 (DOUT)
- net at U16.5 (DOUT): no longer U18.1 (DIN)
- net at U52.5 (DOUT): now also U53.1 (DIN); no longer U54.1 (DIN)
- net at U46.5 (DOUT): now also U47.1 (DIN); no longer U48.1 (DIN)
- net at U57.5 (DOUT): now also U58.1 (DIN); no longer U59.1 (DIN)
- net at U59.5 (DOUT): now also U60.1 (DIN); no longer U38.1 (DIN)
- net at U47.5 (DOUT): now also U48.1 (DIN); no longer U49.1 (DIN)
- net at U58.5 (DOUT): now also U59.1 (DIN); no longer U60.1 (DIN)
- net at U18.5 (DOUT): now also U19.1 (DIN); no longer U20.1 (DIN)
- net at R1.1: now also J1.2 (Pin_2)
- net at U37.5 (DOUT): now also U38.1 (DIN); no longer U39.1 (DIN)
- net at U69.1 (DIN): now also R3.2; no longer U68.5 (DOUT)
- net at U10.1 (DIN): now also U9.5 (DOUT)
- net at U51.5 (DOUT): now also U52.1 (DIN); no longer U53.1 (DIN)
- net at U23.5 (DOUT): now also U24.1 (DIN)
- net at U54.5 (DOUT): now also U55.1 (DIN); no longer U56.1 (DIN)
- net at U56.5 (DOUT): now also U57.1 (DIN); no longer U58.1 (DIN)
- net at U43.5 (DOUT): now also U44.1 (DIN); no longer U45.1 (DIN)
- net at U45.5 (DOUT): now also U46.1 (DIN); no longer U47.1 (DIN)
- net at U19.5 (DOUT): now also U20.1 (DIN); no longer U21.1 (DIN)
- new net: U87.5 (DOUT), U88.1 (DIN)
- new net: U88.5 (DOUT), U89.1 (DIN)
- new net: U92.5 (DOUT), U93.1 (DIN)
- new net: U20.5 (DOUT), U21.1 (DIN)
- new net: U48.5 (DOUT), U49.1 (DIN)
- new net: U14.5 (DOUT), U15.1 (DIN)
- new net: J1.3 (Pin_3), R2.1
- new net: R2.2, U17.1 (DIN)
- new net: J1.4 (Pin_4), R3.1
- new net: J1.5 (Pin_5), R4.1
- new net: U86.5 (DOUT), U87.1 (DIN)
- new net: U85.5 (DOUT), U86.1 (DIN)
- new net: U89.5 (DOUT), U90.1 (DIN)
- new net: U90.5 (DOUT), U91.1 (DIN)
- new net: U91.5 (DOUT), U92.1 (DIN)
- new net: U17.5 (DOUT), U18.1 (DIN)
- new net: R4.2, U85.1 (DIN)
- no-connect marks 0 -> 2
Other:
- note added: "cilj (16 polja)"
- note added: "kocka"
- note added: "početna polja"
- note added: "putanja"
- moved on the sheet: R1, U1, U2, U3, U4, U5, U6, U7, U8, U9

Commit message: update
Parts:
- J1: value (none) -> Conn_01x06_Male; footprint (none) -> Connector_PinHeader_2.54mm:PinHeader_1x06_P2.54mm_Horizontal
- U53, U54, U55, U56, U57, U58, U59, U60, U61, U62, U63, U64, U65, U66, U67, U68, U69, U70, U71, U72, U73, U74, U75, U76, U77, U78, U79, U80, U81, U82, U83, U84: footprint Josip_global:WS2812-4020-dual-7mm_bezMaske -> (none)

Commit message: route
Parts:
- added C1, C3, C5: 0-50 pF, Capacitor_SMD:C_0805_2012Metric, symbol Device:C_Small
- added C2, C4, C6: 100n, Capacitor_SMD:C_0805_2012Metric, symbol Device:C_Small
- added J2: Conn_01x14_Male, Connector_PinHeader_2.54mm:PinHeader_1x14_P2.54mm_Horizontal, symbol Connector:Conn_01x14_Male
- added TP1: TestPoint, test_library:TP_11mm_strelicaLijevo, symbol Connector:TestPoint
- added TP2: TestPoint, test_library:TP_11mm_kvacica, symbol Connector:TestPoint
- added TP3: TestPoint, test_library:TP_11mm_strelicaDesno, symbol Connector:TestPoint
- added U94, U95, U96: TTP223-BA6, Package_TO_SOT_SMD:SOT-23-6, symbol ttp223-ba6:TTP223-BA6
- U1, U10, U11, U12, U13, U14, U15, U16, U17, U18, U19, U2, U20, U21, U22, U23, U24, U25, U26, U27, U28, U29, U3, U30, U31, U32, U33, U34, U35, U36, U37, U38, U39, U4, U40, U41, U42, U43, U44, U45, U46, U47, U48, U49, U5, U50, U51, U52, U53, U54, U55, U56, U57, U58, U59, U6, U60, U61, U62, U63, U64, U65, U66, U67, U68, U69, U7, U70, U71, U72, U73, U74, U75, U76, U77, U78, U79, U8, U80, U81, U82, U83, U84, U9: footprint (none) -> test_library:WS2812-4020-dual-7mm_bezMaske
- U85, U86, U87, U88, U89, U90, U91, U92, U93: footprint (none) -> test_library:WS2812-4020-single-6mm_bezMaske
Connections:
- net GND: now also C1.2, C2.2, C3.2, C4.2, C5.2, C6.2, J2.14 (Pin_14), U94.2 (VSS), U95.2 (VSS), U96.2 (VSS)
- new net: C5.1, TP3.1, U96.3 (I)
- new net: C1.1, TP1.1, U94.3 (I)
- new net: C3.1, TP2.1, U95.3 (I)
- new net +5V: C2.1, C4.1, C6.1, J2.1 (Pin_1), U94.5 (VDD), U95.5 (VDD), U96.5 (VDD)
- new net TP1: J2.2 (Pin_2), U94.1 (Q)
- new net TP10: J2.11 (Pin_11)
- new net TP11: J2.12 (Pin_12)
- new net TP12: J2.13 (Pin_13)
- new net TP2: J2.3 (Pin_3), U95.1 (Q)
- new net TP3: J2.4 (Pin_4), U96.1 (Q)
- new net TP4: J2.5 (Pin_5)
- new net TP5: J2.6 (Pin_6)
- new net TP6: J2.7 (Pin_7)
- new net TP7: J2.8 (Pin_8)
- new net TP8: J2.9 (Pin_9)
- new net TP9: J2.10 (Pin_10)
- no-connect marks 2 -> 9

Commit message: update
Parts:
- U1: renamed from U13; footprint test_library:WS2812-4020-dual-7mm_bezMaske -> (none)
- U10: renamed from U6; value WS2812-4020_dual -> (none); footprint test_library:WS2812-4020-dual-7mm_bezMaske -> (none)
- U11: renamed from U7; value WS2812-4020_dual -> (none); footprint test_library:WS2812-4020-dual-7mm_bezMaske -> (none)
- U12: renamed from U8; value WS2812-4020_dual -> (none); footprint test_library:WS2812-4020-dual-7mm_bezMaske -> (none)
- U13: renamed from U1; value WS2812-4020_dual -> (none); footprint test_library:WS2812-4020-dual-7mm_bezMaske -> (none)
- U14: renamed from U2; value WS2812-4020_dual -> (none); footprint test_library:WS2812-4020-dual-7mm_bezMaske -> (none)
- U15: renamed from U3; value WS2812-4020_dual -> (none); footprint test_library:WS2812-4020-dual-7mm_bezMaske -> (none)
- U16: renamed from U4; value WS2812-4020_dual -> (none); footprint test_library:WS2812-4020-dual-7mm_bezMaske -> (none)
- U17, U18, U19, U20, U21, U22, U23, U24, U25, U26, U27, U28, U29, U30, U31, U32, U33, U34, U35, U36, U37, U38, U39, U40, U41, U42, U43, U44, U45, U46, U47, U48, U49, U50, U51, U52, U53, U54, U55, U56, U57, U58, U59, U60, U61, U62, U63, U64, U65, U66, U67, U68, U69, U70, U71, U72, U73, U74, U75, U76, U77, U78, U79, U80, U81, U82, U83, U84: footprint test_library:WS2812-4020-dual-7mm_bezMaske -> (none)
- U2: renamed from U14; value WS2812-4020_dual -> (none); footprint test_library:WS2812-4020-dual-7mm_bezMaske -> (none)
- U3: renamed from U15; value WS2812-4020_dual -> (none); footprint test_library:WS2812-4020-dual-7mm_bezMaske -> (none)
- U4: renamed from U16; value WS2812-4020_dual -> (none); footprint test_library:WS2812-4020-dual-7mm_bezMaske -> (none)
- U5: renamed from U9; value WS2812-4020_dual -> (none); footprint test_library:WS2812-4020-dual-7mm_bezMaske -> (none)
- U6: renamed from U10; value WS2812-4020_dual -> (none); footprint test_library:WS2812-4020-dual-7mm_bezMaske -> (none)
- U7: renamed from U11; value WS2812-4020_dual -> (none); footprint test_library:WS2812-4020-dual-7mm_bezMaske -> (none)
- U8: renamed from U12; value WS2812-4020_dual -> (none); footprint test_library:WS2812-4020-dual-7mm_bezMaske -> (none)
- U85: value WS2812-4020_dual -> (none); symbol Josip_symbol_global:WS2812-4020_dual -> Symbol_test:WS2812-4020_single
- U86, U87, U88, U89, U90, U91, U92, U93: symbol Josip_symbol_global:WS2812-4020_dual -> Symbol_test:WS2812-4020_single
- U9: renamed from U5; value WS2812-4020_dual -> (none); footprint test_library:WS2812-4020-dual-7mm_bezMaske -> (none)
Connections:
- net at U13.1 (DIN): now also U12.5 (DOUT); no longer R1.2
- net at U88.1 (DIN): now also U87.4 (VSS); no longer U87.5 (DOUT)
- net at U89.1 (DIN): now also U88.4 (VSS); no longer U88.5 (DOUT)
- net at U4.5 (DOUT): now also U5.1 (DIN)
- net at U93.1 (DIN): now also U92.4 (VSS); no longer U92.5 (DOUT)
- net at U87.1 (DIN): now also U86.4 (VSS); no longer U86.5 (DOUT)
- net at U86.1 (DIN): now also U85.4 (VSS); no longer U85.5 (DOUT)
- net at U90.1 (DIN): now also U89.4 (VSS); no longer U89.5 (DOUT)
- net at U91.1 (DIN): now also U90.4 (VSS); no longer U90.5 (DOUT)
- net at U1.1 (DIN): now also R1.2; no longer U8.5 (DOUT)
- net at U92.1 (DIN): now also U91.4 (VSS); no longer U91.5 (DOUT)
- net at U9.1 (DIN): now also U8.5 (DOUT); no longer U16.5 (DOUT)
Other:
- moved on the sheet: U1, U10, U11, U12, U13, U14, U15, U16, U2, U3, U4, U5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
