File: KiCad files/FieldBoard/FieldBoard.kicad_pcb (KiCad board)
At the start: 2 copper layers, 150 x 150 mm, 151 parts, among them J1 Conn_01x05_Male, J2 Conn_01x05_Male, J3 Conn_01x06_Male, J4 Conn_01x05_Male, J5 Conn_01x05_Male, U1 TTP223-BA6, U10 TTP223-BA6, U11 TTP223-BA6, U12 TTP223-BA6, U2 TTP223-BA6, U3 TTP223-BA6, U4 TTP223-BA6, U5 TTP223-BA6, U6 TTP223-BA6, U7 TTP223-BA6, U8 TTP223-BA6, U9 TTP223-BA6

Commit message: layout
Parts:
- moved POS75 319.3 mm to (97.5, 155.0)
- moved POS77 311.8 mm to (78.9, 146.3), turned to -45 degrees
- moved POS34 302.5 mm to (90.7, 66.2), turned to -90 degrees
- moved POS81 296.2 mm to (102.0, 102.7), turned to -90 degrees
- moved R2 292.0 mm to (84.6, 107.6), turned to 0 degrees
- moved POS36 291.0 mm to (77.5, 43.2)
- moved POS80 285.5 mm to (90.6, 112.5), turned to 135 degrees
- moved POS74 282.2 mm to (109.6, 150.5)
- moved POS38 280.1 mm to (86.4, 25.0), turned to -135 degrees
- moved POS78 277.0 mm to (77.4, 135.5), turned to 90 degrees
- moved POS76 277.0 mm to (86.5, 153.9), turned to -45 degrees
- moved R4 276.6 mm to (111.6, 77.3)
- moved R1 275.9 mm to (121.4, 74.9)
- moved POS79 266.8 mm to (82.1, 123.5), turned to 135 degrees
- moved POS41 263.2 mm to (120.7, 37.1)
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Routing:
- net (no net): track 0.00 -> 202.7 mm
- net Net-(POS4-Pad5): track 0.00 -> 104.2 mm
- net Net-(POS38-Pad5): track 0.00 -> 22.8 mm
- net Net-(POS3-Pad5): track 0.00 -> 15.3 mm
- net Net-(POS1-Pad5): track 0.00 -> 15.2 mm
- net Net-(POS2-Pad5): track 0.00 -> 15.0 mm
- net Net-(POS34-Pad5): track 0.00 -> 14.9 mm
- net Net-(POS37-Pad5): track 0.00 -> 14.0 mm
- net Net-(POS36-Pad5): track 0.00 -> 12.7 mm
- net Net-(POS33-Pad5): track 0.00 -> 12.3 mm
- net Net-(POS35-Pad5): track 0.00 -> 10.9 mm
- net Net-(POS17-Pad5): track 0.00 -> 8.64 mm
- net Net-(POS39-Pad5): track 0.00 -> 8.03 mm
- net /Finish (16LEDs)/Finish-LEDs: track 0.00 -> 7.53 mm
- net /Start (16LEDs)/Start-LEDs: track 0.00 -> 5.10 mm

Commit message: update
Parts:
- moved POS21 106.2 mm to (136.6, 37.1), turned to 45 degrees
- moved R2 35.5 mm to (81.9, 72.2)
- moved POS17 22.6 mm to (90.5, 78.2), turned to 45 degrees
- moved POS19 22.5 mm to (90.6, 100.8), turned to 135 degrees
- moved POS62 0.34 mm to (209.6, 135.2), turned to 0 degrees
- moved POS52 0.10 mm to (209.7, 43.2), turned to 0 degrees
- moved POS49 0.10 mm to (190.1, 23.8)
- turned POS60 to 45 degrees
- turned POS61 to 45 degrees
- turned POS33 to -135 degrees
- turned POS18 to -45 degrees
- turned POS20 to 180 degrees
- turned POS38 to 180 degrees
- turned POS41 to 0 degrees
- turned POS42 to 0 degrees
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Routing:
- net (no net): track 202.7 -> 736.9 mm
- net Net-(POS20-Pad5): track 0.00 -> 148.6 mm
- net Net-(POS65-Pad5): track 0.00 -> 19.8 mm
- net Net-(POS63-Pad5): track 0.00 -> 17.4 mm
- net Net-(POS53-Pad5): track 0.00 -> 17.4 mm
- net Net-(POS76-Pad5): track 0.00 -> 17.3 mm
- net Net-(POS49-Pad5): track 0.00 -> 17.3 mm
- net Net-(POS74-Pad5): track 0.00 -> 17.1 mm
- net Net-(POS51-Pad5): track 0.00 -> 16.5 mm
- net Net-(POS41-Pad5): track 0.00 -> 13.9 mm
- net Net-(POS54-Pad5): track 0.00 -> 13.9 mm
- net Net-(POS52-Pad5): track 0.00 -> 12.8 mm
- net Net-(POS50-Pad5): track 0.00 -> 12.5 mm
- net Net-(POS46-Pad5): track 0.00 -> 12.3 mm
- net Net-(POS55-Pad5): track 0.00 -> 11.9 mm
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- added copper zone on B.Cu, net GND

Commit message: layout
Parts:
- moved POS23 146.3 mm to (132.6, 37.0), turned to 45 degrees
- moved POS24 127.8 mm to (143.8, 48.4), turned to 90 degrees
- moved POS22 126.2 mm to (143.8, 37.1), turned to -135 degrees
- moved POS25 44.5 mm to (229.9, 66.1)
- moved POS21 18.5 mm to (155.1, 37.0), turned to -45 degrees
- moved R2 0.87 mm to (81.2, 72.7)
- moved POS13 0.10 mm to (118.6, 114.5), turned to 0 degrees
- moved POS10 0.10 mm to (176.6, 122.0), turned to 0 degrees
- turned POS11 to 0 degrees
- turned POS12 to 0 degrees
- turned POS14 to 0 degrees
- turned POS15 to 0 degrees
- turned POS16 to 0 degrees
- turned POS34 to -135 degrees
- turned POS35 to -135 degrees
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Routing:
- net VDD: track 0.00 -> 390.3 mm, vias 0 -> 153
- net (no net): track 736.9 -> 1059.7 mm
- net Net-(POS8-Pad5): track 0.00 -> 110.4 mm
- net Net-(POS12-Pad5): track 0.00 -> 101.9 mm
- net Net-(POS20-Pad5): track 148.6 -> 179.3 mm
- net Net-(POS10-Pad5): track 0.00 -> 14.3 mm
- net Net-(POS11-Pad5): track 0.00 -> 13.7 mm
- net Net-(POS10-Pad1): track 0.00 -> 13.6 mm
- net Net-(POS53-Pad5): track 17.4 -> 5.17 mm
- net Net-(POS15-Pad5): track 0.00 -> 12.0 mm
- net Net-(POS13-Pad5): track 0.00 -> 11.7 mm
- net Net-(POS14-Pad5): track 0.00 -> 11.5 mm
- net Net-(POS7-Pad5): track 0.00 -> 11.3 mm
- net Net-(POS6-Pad5): track 0.00 -> 11.2 mm
- net Net-(POS34-Pad5): track 14.9 -> 4.35 mm
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- added copper zone on F.Cu, net VDD
