File: KiCad files/FieldBoard/FieldBoard.kicad_pcb (KiCad board)
At the start: 2 copper layers, 150 x 150 mm, 146 parts, among them U1 TTP223-BA6, U10 TTP223-BA6, U11 TTP223-BA6, U12 TTP223-BA6, U2 TTP223-BA6, U3 TTP223-BA6, U4 TTP223-BA6, U5 TTP223-BA6, U6 TTP223-BA6, U7 TTP223-BA6, U8 TTP223-BA6, U9 TTP223-BA6

Commit message: update
Parts:
- moved LED7 0.90 mm to (136.9, 95.6)
- moved LED8 0.90 mm to (136.9, 89.6)
Changed lines of the file:
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@@
   )
   (footprint "LED_SMD:LED_WS2812B_PLCC4_5.0x5.0mm_P3.2mm" (layer "F.Cu")
-    (at 137.800004 95.608851)
+    (at 136.9 95.608851)
     (descr "https://cdn-shop.adafruit.com/datasheets/WS2812B.pdf")
     (tags "LED RGB NeoPixel")
@@
   )
   (footprint "LED_SMD:LED_WS2812B_PLCC4_5.0x5.0mm_P3.2mm" (layer "F.Cu")
-    (at 137.800004 89.558851)
+    (at 136.9 89.558851)
     (descr "https://cdn-shop.adafruit.com/datasheets/WS2812B.pdf")
     (tags "LED RGB NeoPixel")
@@
     )
   )
-  (gr_arc (start 154.788425 98.154422) (mid 154.1 99.9) (end 152.3789 100.647521) (layer "F.SilkS") (width 0.3))
   (gr_arc (start 78.9 66.5) (mid 82.435534 67.964466) (end 83.9 71.5) (layer "F.SilkS") (width 0.3))
-  (gr_line (start 154.847521 81.0211) (end 154.788425 98.154422) (layer "F.SilkS") (width 0.3))
-  (gr_arc (start 152.354422 78.611575) (mid 154.1 79.3) (end 154.847521 81.0211) (layer "F.SilkS") (width 0.3))
-  (gr_arc (start 135.245578 100.588425) (mid 133.5 99.9) (end 132.752479 98.1789) (layer "F.SilkS") (width 0.3))
   (gr_line (start 69.1 113.1) (end 78.9 113.064466) (layer "F.SilkS") (width 0.3))
-  (gr_line (start 135.2211 78.652479) (end 152.354422 78.611575) (layer "F.SilkS") (width 0.3))
   (gr_line (start 78.9 66.5) (end 69.1 66.5) (layer "F.SilkS") (width 0.3))
   (gr_arc (start 83.9 108.064466) (mid 82.435534 111.6) (end 78.9 113.064466) (layer "F.SilkS") (width 0.3))
-  (gr_arc (start 132.811575 81.145578) (mid 133.5 79.4) (end 135.2211 78.652479) (layer "F.SilkS") (width 0.3))
   (gr_line (start 83.9 108.064466) (end 83.9 71.5) (layer "F.SilkS") (width 0.3))
-  (gr_line (start 135.245578 100.588425) (end 152.3789 100.647521) (layer "F.SilkS") (width 0.3))
-  (gr_line (start 132.811575 81.145578) (end 132.752479 98.1789) (layer "F.SilkS") (width 0.3))
   (gr_arc (start 68.857864 34.657864) (mid 74.715728 20.515728) (end 88.857864 14.657864) (layer "Edge.Cuts") (width 0.1))
   (gr_arc (start 218.857864 144.657864) (mid 213 158.8) (end 198.857864 164.657864) (layer "Edge.Cuts") (width 0.1))

Commit message: update
Parts:
- removed C1, C13, C14, C15, C19, C2, C20, C21, C3, C7, C8, C9: 100n, Capacitor_SMD:C_0603_1608Metric
- removed C10, C11, C12, C16, C17, C18, C22, C23, C24, C4, C5, C6: 0-50 pF, Capacitor_SMD:C_0603_1608Metric
- removed TP1, TP10, TP4, TP7: TestPoint, FieldBoard_footprint:TP_11mm_strelicaLijevo
- removed TP11, TP2, TP5, TP8: TestPoint, FieldBoard_footprint:TP_11mm_kvacica
- removed TP12, TP3, TP6, TP9: TestPoint, FieldBoard_footprint:TP_11mm_strelicaDesno
- removed U1, U10, U11, U12, U2, U3, U4, U5, U6, U7, U8, U9: TTP223-BA6, Package_TO_SOT_SMD:SOT-23-6
- added J1: Conn_01x02, TerminalBlock_Phoenix:TerminalBlock_Phoenix_MKDS-1,5-2-5.08_1x02_P5.08mm_Horizontal, B.Cu at (242.1, 77.5)
- added J2: Conn_01x05_Male, Connector_PinHeader_2.54mm:PinHeader_1x05_P2.54mm_Vertical, B.Cu at (222.4, 72.6)
- R1, R2, R3, R4: moved to F.Cu
- moved R2 20.3 mm to (93.0, 72.2), turned to -90 degrees
- moved R1 11.7 mm to (126.0, 62.9)
- moved R3 9.84 mm to (139.4, 78.0), turned to -90 degrees
- moved R4 4.17 mm to (108.6, 74.4), turned to 0 degrees
- moved POS29 0.11 mm to (132.4, 141.8), turned to 0 degrees
- moved POS21 0.10 mm to (155.1, 37.1), turned to 0 degrees
- moved POS18 0.10 mm to (90.6, 89.5), turned to 0 degrees
- moved POS34 0.10 mm to (90.6, 66.2), turned to 0 degrees
- moved POS17 0.10 mm to (90.6, 78.2), turned to 0 degrees
- moved POS31 0.07 mm to (155.0, 141.8), turned to 0 degrees
- moved POS23 0.07 mm to (132.6, 37.1), turned to 0 degrees
- turned POS25 to 0 degrees
- turned POS30 to 0 degrees
- turned POS22 to 0 degrees
- turned POS26 to 0 degrees
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- renumbered POS1 to FIN1, POS10 to FIN10, POS11 to FIN11, POS12 to FIN12, POS13 to FIN13, POS14 to FIN14, POS15 to FIN15, POS16 to FIN16, POS2 to FIN2, POS3 to FIN3, POS4 to FIN4, POS5 to FIN5, POS6 to FIN6, POS7 to FIN7, POS8 to FIN8, POS9 to FIN9
Connections:
- LED1 pad 2: unconnected-(LED1-Pad2) -> Net-(LED1-Pad2)
- LED1 pad 4: unconnected-(LED1-Pad4) -> /Cube (9LEDs)/Cube-LEDs
- LED2 pad 2: unconnected-(LED2-Pad2) -> Net-(LED2-Pad2)
- LED2 pad 4: unconnected-(LED2-Pad4) -> Net-(LED1-Pad2)
- LED3 pad 2: unconnected-(LED3-Pad2) -> Net-(LED3-Pad2)
- LED3 pad 4: unconnected-(LED3-Pad4) -> Net-(LED2-Pad2)
- LED4 pad 2: unconnected-(LED4-Pad2) -> Net-(LED4-Pad2)
- LED4 pad 4: unconnected-(LED4-Pad4) -> Net-(LED3-Pad2)
- LED5 pad 2: unconnected-(LED5-Pad2) -> Net-(LED5-Pad2)
- LED5 pad 4: unconnected-(LED5-Pad4) -> Net-(LED4-Pad2)
- LED6 pad 2: unconnected-(LED6-Pad2) -> Net-(LED6-Pad2)
- LED6 pad 4: unconnected-(LED6-Pad4) -> Net-(LED5-Pad2)
- LED7 pad 2: unconnected-(LED7-Pad2) -> Net-(LED7-Pad2)
- LED7 pad 4: unconnected-(LED7-Pad4) -> Net-(LED6-Pad2)
- LED8 pad 2: unconnected-(LED8-Pad2) -> Net-(LED8-Pad2)
- LED8 pad 4: unconnected-(LED8-Pad4) -> Net-(LED7-Pad2)
- LED9 pad 4: unconnected-(LED9-Pad4) -> Net-(LED8-Pad2)
- POS24 pad 2: unconnected-(POS24-Pad2) -> Net-(POS24-Pad2)
- POS25 pad 2: unconnected-(POS25-Pad2) -> Net-(POS25-Pad2)
- POS25 pad 4: unconnected-(POS25-Pad4) -> Net-(POS24-Pad2)
- POS26 pad 2: unconnected-(POS26-Pad2) -> Net-(POS26-Pad2)
- POS26 pad 4: unconnected-(POS26-Pad4) -> Net-(POS25-Pad2)
- POS27 pad 2: unconnected-(POS27-Pad2) -> Net-(POS27-Pad2)
- POS27 pad 4: unconnected-(POS27-Pad4) -> Net-(POS26-Pad2)
- POS28 pad 2: unconnected-(POS28-Pad2) -> Net-(POS28-Pad2)
- POS28 pad 4: unconnected-(POS28-Pad4) -> Net-(POS27-Pad2)
- POS29 pad 2: unconnected-(POS29-Pad2) -> Net-(POS29-Pad2)
- POS29 pad 4: unconnected-(POS29-Pad4) -> Net-(POS28-Pad2)
- POS30 pad 2: unconnected-(POS30-Pad2) -> Net-(POS30-Pad2)
- POS30 pad 4: unconnected-(POS30-Pad4) -> Net-(POS29-Pad2)
- POS31 pad 2: unconnected-(POS31-Pad2) -> Net-(POS31-Pad2)
- POS31 pad 4: unconnected-(POS31-Pad4) -> Net-(POS30-Pad2)
- POS32 pad 4: unconnected-(POS32-Pad4) -> Net-(POS31-Pad2)
- POS33 pad 2: unconnected-(POS33-Pad2) -> Net-(POS33-Pad2)
- POS33 pad 4: unconnected-(POS33-Pad4) -> /Positions (52LEDs)/Positions-LEDs
- POS34 pad 2: unconnected-(POS34-Pad2) -> Net-(POS34-Pad2)
- POS34 pad 4: unconnected-(POS34-Pad4) -> Net-(POS33-Pad2)
- POS35 pad 2: unconnected-(POS35-Pad2) -> Net-(POS35-Pad2)
- POS35 pad 4: unconnected-(POS35-Pad4) -> Net-(POS34-Pad2)
- POS36 pad 2: unconnected-(POS36-Pad2) -> Net-(POS36-Pad2)
- POS36 pad 4: unconnected-(POS36-Pad4) -> Net-(POS35-Pad2)
- POS37 pad 2: unconnected-(POS37-Pad2) -> Net-(POS37-Pad2)
- POS37 pad 4: unconnected-(POS37-Pad4) -> Net-(POS36-Pad2)
- POS38 pad 2: unconnected-(POS38-Pad2) -> Net-(POS38-Pad2)
- POS38 pad 4: unconnected-(POS38-Pad4) -> Net-(POS37-Pad2)
- POS39 pad 2: unconnected-(POS39-Pad2) -> Net-(POS39-Pad2)
- POS39 pad 4: unconnected-(POS39-Pad4) -> Net-(POS38-Pad2)
- POS40 pad 2: unconnected-(POS40-Pad2) -> Net-(POS40-Pad2)
- POS40 pad 4: unconnected-(POS40-Pad4) -> Net-(POS39-Pad2)
- POS41 pad 2: unconnected-(POS41-Pad2) -> Net-(POS41-Pad2)
- POS41 pad 4: unconnected-(POS41-Pad4) -> Net-(POS40-Pad2)
- POS42 pad 2: unconnected-(POS42-Pad2) -> Net-(POS42-Pad2)
- POS42 pad 4: unconnected-(POS42-Pad4) -> Net-(POS41-Pad2)
- POS43 pad 2: unconnected-(POS43-Pad2) -> Net-(POS43-Pad2)
- POS43 pad 4: unconnected-(POS43-Pad4) -> Net-(POS42-Pad2)
- POS44 pad 2: unconnected-(POS44-Pad2) -> Net-(POS44-Pad2)
- POS44 pad 4: unconnected-(POS44-Pad4) -> Net-(POS43-Pad2)
- POS45 pad 2: unconnected-(POS45-Pad2) -> Net-(POS45-Pad2)
- POS45 pad 4: unconnected-(POS45-Pad4) -> Net-(POS44-Pad2)
- POS46 pad 2: unconnected-(POS46-Pad2) -> Net-(POS46-Pad2)
- POS46 pad 4: unconnected-(POS46-Pad4) -> Net-(POS45-Pad2)
- POS47 pad 2: unconnected-(POS47-Pad2) -> Net-(POS47-Pad2)
- POS47 pad 4: unconnected-(POS47-Pad4) -> Net-(POS46-Pad2)
- POS48 pad 2: unconnected-(POS48-Pad2) -> Net-(POS48-Pad2)
- POS48 pad 4: unconnected-(POS48-Pad4) -> Net-(POS47-Pad2)
- POS49 pad 2: unconnected-(POS49-Pad2) -> Net-(POS49-Pad2)
- POS49 pad 4: unconnected-(POS49-Pad4) -> Net-(POS48-Pad2)
- POS50 pad 2: unconnected-(POS50-Pad2) -> Net-(POS50-Pad2)
- POS50 pad 4: unconnected-(POS50-Pad4) -> Net-(POS49-Pad2)
- POS51 pad 2: unconnected-(POS51-Pad2) -> Net-(POS51-Pad2)
- POS51 pad 4: unconnected-(POS51-Pad4) -> Net-(POS50-Pad2)
- POS52 pad 2: unconnected-(POS52-Pad2) -> Net-(POS52-Pad2)
- POS52 pad 4: unconnected-(POS52-Pad4) -> Net-(POS51-Pad2)
- POS53 pad 2: unconnected-(POS53-Pad2) -> Net-(POS53-Pad2)
- POS53 pad 4: unconnected-(POS53-Pad4) -> Net-(POS52-Pad2)
- POS54 pad 2: unconnected-(POS54-Pad2) -> Net-(POS54-Pad2)
- POS54 pad 4: unconnected-(POS54-Pad4) -> Net-(POS53-Pad2)
- POS55 pad 2: unconnected-(POS55-Pad2) -> Net-(POS55-Pad2)
- POS55 pad 4: unconnected-(POS55-Pad4) -> Net-(POS54-Pad2)
- POS56 pad 2: unconnected-(POS56-Pad2) -> Net-(POS56-Pad2)
- POS56 pad 4: unconnected-(POS56-Pad4) -> Net-(POS55-Pad2)
- POS57 pad 2: unconnected-(POS57-Pad2) -> Net-(POS57-Pad2)
- POS57 pad 4: unconnected-(POS57-Pad4) -> Net-(POS56-Pad2)
- POS58 pad 2: unconnected-(POS58-Pad2) -> Net-(POS58-Pad2)
- POS58 pad 4: unconnected-(POS58-Pad4) -> Net-(POS57-Pad2)
- POS59 pad 2: unconnected-(POS59-Pad2) -> Net-(POS59-Pad2)
- POS59 pad 4: unconnected-(POS59-Pad4) -> Net-(POS58-Pad2)
- POS60 pad 2: unconnected-(POS60-Pad2) -> Net-(POS60-Pad2)
- POS60 pad 4: unconnected-(POS60-Pad4) -> Net-(POS59-Pad2)
- POS61 pad 2: unconnected-(POS61-Pad2) -> Net-(POS61-Pad2)
- POS61 pad 4: unconnected-(POS61-Pad4) -> Net-(POS60-Pad2)
- POS62 pad 2: unconnected-(POS62-Pad2) -> Net-(POS62-Pad2)
- POS62 pad 4: unconnected-(POS62-Pad4) -> Net-(POS61-Pad2)
- POS63 pad 2: unconnected-(POS63-Pad2) -> Net-(POS63-Pad2)
- POS63 pad 4: unconnected-(POS63-Pad4) -> Net-(POS62-Pad2)
- POS64 pad 2: unconnected-(POS64-Pad2) -> Net-(POS64-Pad2)
- POS64 pad 4: unconnected-(POS64-Pad4) -> Net-(POS63-Pad2)
- POS65 pad 2: unconnected-(POS65-Pad2) -> Net-(POS65-Pad2)
- POS65 pad 4: unconnected-(POS65-Pad4) -> Net-(POS64-Pad2)
- POS66 pad 2: unconnected-(POS66-Pad2) -> Net-(POS66-Pad2)
- POS66 pad 4: unconnected-(POS66-Pad4) -> Net-(POS65-Pad2)
- POS67 pad 2: unconnected-(POS67-Pad2) -> Net-(POS67-Pad2)
- POS67 pad 4: unconnected-(POS67-Pad4) -> Net-(POS66-Pad2)
- POS68 pad 2: unconnected-(POS68-Pad2) -> Net-(POS68-Pad2)
- POS68 pad 4: unconnected-(POS68-Pad4) -> Net-(POS67-Pad2)
- POS69 pad 2: unconnected-(POS69-Pad2) -> Net-(POS69-Pad2)
- POS69 pad 4: unconnected-(POS69-Pad4) -> Net-(POS68-Pad2)
- POS70 pad 2: unconnected-(POS70-Pad2) -> Net-(POS70-Pad2)
- POS70 pad 4: unconnected-(POS70-Pad4) -> Net-(POS69-Pad2)
- POS71 pad 2: unconnected-(POS71-Pad2) -> Net-(POS71-Pad2)
- POS71 pad 4: unconnected-(POS71-Pad4) -> Net-(POS70-Pad2)
- POS72 pad 2: unconnected-(POS72-Pad2) -> Net-(POS72-Pad2)
- POS72 pad 4: unconnected-(POS72-Pad4) -> Net-(POS71-Pad2)
- POS73 pad 2: unconnected-(POS73-Pad2) -> Net-(POS73-Pad2)
- POS73 pad 4: unconnected-(POS73-Pad4) -> Net-(POS72-Pad2)
- POS74 pad 2: unconnected-(POS74-Pad2) -> Net-(POS74-Pad2)
- POS74 pad 4: unconnected-(POS74-Pad4) -> Net-(POS73-Pad2)
- POS75 pad 2: unconnected-(POS75-Pad2) -> Net-(POS75-Pad2)
- POS75 pad 4: unconnected-(POS75-Pad4) -> Net-(POS74-Pad2)
- POS76 pad 2: unconnected-(POS76-Pad2) -> Net-(POS76-Pad2)
- POS76 pad 4: unconnected-(POS76-Pad4) -> Net-(POS75-Pad2)
- POS77 pad 2: unconnected-(POS77-Pad2) -> Net-(POS77-Pad2)
- POS77 pad 4: unconnected-(POS77-Pad4) -> Net-(POS76-Pad2)
- POS78 pad 2: unconnected-(POS78-Pad2) -> Net-(POS78-Pad2)
- POS78 pad 4: unconnected-(POS78-Pad4) -> Net-(POS77-Pad2)
- POS79 pad 2: unconnected-(POS79-Pad2) -> Net-(POS79-Pad2)
- POS79 pad 4: unconnected-(POS79-Pad4) -> Net-(POS78-Pad2)
- POS80 pad 2: unconnected-(POS80-Pad2) -> Net-(POS80-Pad2)
- POS80 pad 4: unconnected-(POS80-Pad4) -> Net-(POS79-Pad2)
- POS81 pad 2: unconnected-(POS81-Pad2) -> Net-(POS81-Pad2)
- POS81 pad 4: unconnected-(POS81-Pad4) -> Net-(POS80-Pad2)
- POS82 pad 2: unconnected-(POS82-Pad2) -> Net-(POS82-Pad2)
- POS82 pad 4: unconnected-(POS82-Pad4) -> Net-(POS81-Pad2)
- POS83 pad 2: unconnected-(POS83-Pad2) -> Net-(POS83-Pad2)
- POS83 pad 4: unconnected-(POS83-Pad4) -> Net-(POS82-Pad2)
- POS84 pad 4: unconnected-(POS84-Pad4) -> Net-(POS83-Pad2)
- R1 pad 1: unconnected-(R1-Pad1) -> Net-(J2-Pad1)
- R2 pad 1: unconnected-(R2-Pad1) -> Net-(J2-Pad2)
- R3 pad 1: unconnected-(R3-Pad1) -> Net-(J2-Pad3)
- R4 pad 1: unconnected-(R4-Pad1) -> Net-(J2-Pad4)
Other:
- board size 150 x 150 mm -> 150.1 x 150.1 mm

Commit message: layout v1
Parts:
- LED1, LED2, LED3, LED4, LED5, LED6, LED7, LED8, LED9: footprint LED_SMD:LED_WS2812B_PLCC4_5.0x5.0mm_P3.2mm -> FieldBoard_footprint:WS2812-mini
- moved J1 118.4 mm to (126.0, 100.9), turned to -90 degrees
- moved J2 96.5 mm to (126.3, 80.9), turned to 0 degrees
- moved R2 19.3 mm to (112.2, 74.4), turned to 180 degrees
- moved R4 13.3 mm to (121.3, 78.4), turned to 180 degrees
- moved R1 8.81 mm to (121.9, 70.7)
- moved R3 8.05 mm to (131.4, 78.9)
- moved LED1 0.90 mm to (137.8, 83.6), turned to 180 degrees
- moved LED7 0.90 mm to (137.8, 95.6)
- moved LED8 0.90 mm to (137.8, 89.6), turned to 180 degrees
- moved POS67 0.14 mm to (166.9, 141.7), turned to -90 degrees
- moved LED5 0.10 mm to (149.8, 95.6)
- moved POS47 0.10 mm to (166.9, 37.1), turned to -90 degrees
- moved POS68 0.10 mm to (157.2, 130.4), turned to -90 degrees
- moved POS54 0.10 mm to (196.4, 66.2), turned to 90 degrees
- moved POS77 0.05 mm to (78.8, 146.3), turned to -90 degrees
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- renumbered POS20 to POS17, POS19 to POS18, POS18 to POS19, POS17 to POS20, POS24 to POS21, POS23 to POS22, POS22 to POS23, POS21 to POS24, POS28 to POS25, POS27 to POS26, POS26 to POS27, POS25 to POS28, POS32 to POS29, POS31 to POS30, POS30 to POS31, POS29 to POS32
Connections:
- J2 pad 1: Net-(J2-Pad1) -> GND
- J2 pad 2: Net-(J2-Pad2) -> Net-(R4-Pad1)
- J2 pad 4: Net-(J2-Pad4) -> Net-(R2-Pad1)
- J2 pad 5: GND -> Net-(R1-Pad1)
- POS17 pad 2: Net-(POS20-Pad2) -> Net-(POS17-Pad2)
- POS17 pad 4: Net-(POS19-Pad2) -> /Start (16LEDs)/Start-LEDs
- POS18 pad 2: Net-(POS19-Pad2) -> Net-(POS18-Pad2)
- POS18 pad 4: Net-(POS18-Pad2) -> Net-(POS17-Pad2)
- POS19 pad 2: Net-(POS18-Pad2) -> Net-(POS19-Pad2)
- POS19 pad 4: Net-(POS17-Pad2) -> Net-(POS18-Pad2)
- POS20 pad 2: Net-(POS17-Pad2) -> Net-(POS20-Pad2)
- POS20 pad 4: /Start (16LEDs)/Start-LEDs -> Net-(POS19-Pad2)
- POS21 pad 2: Net-(POS24-Pad2) -> Net-(POS21-Pad2)
- POS21 pad 4: Net-(POS23-Pad2) -> Net-(POS20-Pad2)
- POS22 pad 2: Net-(POS23-Pad2) -> Net-(POS22-Pad2)
- POS22 pad 4: Net-(POS22-Pad2) -> Net-(POS21-Pad2)
- POS23 pad 2: Net-(POS22-Pad2) -> Net-(POS23-Pad2)
- POS23 pad 4: Net-(POS21-Pad2) -> Net-(POS22-Pad2)
- POS24 pad 2: Net-(POS21-Pad2) -> Net-(POS24-Pad2)
- POS24 pad 4: Net-(POS20-Pad2) -> Net-(POS23-Pad2)
- POS25 pad 2: Net-(POS28-Pad2) -> Net-(POS25-Pad2)
- POS25 pad 4: Net-(POS27-Pad2) -> Net-(POS24-Pad2)
- POS26 pad 2: Net-(POS27-Pad2) -> Net-(POS26-Pad2)
- POS26 pad 4: Net-(POS26-Pad2) -> Net-(POS25-Pad2)
- POS27 pad 2: Net-(POS26-Pad2) -> Net-(POS27-Pad2)
- POS27 pad 4: Net-(POS25-Pad2) -> Net-(POS26-Pad2)
- POS28 pad 2: Net-(POS25-Pad2) -> Net-(POS28-Pad2)
- POS28 pad 4: Net-(POS24-Pad2) -> Net-(POS27-Pad2)
- POS29 pad 2: unconnected-(POS32-Pad2) -> Net-(POS29-Pad2)
- POS29 pad 4: Net-(POS31-Pad2) -> Net-(POS28-Pad2)
- POS30 pad 2: Net-(POS31-Pad2) -> Net-(POS30-Pad2)
- POS30 pad 4: Net-(POS30-Pad2) -> Net-(POS29-Pad2)
- POS31 pad 2: Net-(POS30-Pad2) -> Net-(POS31-Pad2)
- POS31 pad 4: Net-(POS29-Pad2) -> Net-(POS30-Pad2)
- POS32 pad 2: Net-(POS29-Pad2) -> unconnected-(POS32-Pad2)
- POS32 pad 4: Net-(POS28-Pad2) -> Net-(POS31-Pad2)
- R1 pad 1: Net-(J2-Pad1) -> Net-(R1-Pad1)
- R2 pad 1: Net-(J2-Pad2) -> Net-(R2-Pad1)
- R2 pad 2: /Start (16LEDs)/Start-LEDs -> /Positions (52LEDs)/Positions-LEDs
- R4 pad 1: Net-(J2-Pad4) -> Net-(R4-Pad1)
- R4 pad 2: /Positions (52LEDs)/Positions-LEDs -> /Start (16LEDs)/Start-LEDs
Routing:
- net GND: track 0.00 -> 169.5 mm, vias 0 -> 93
- net Net-(POS20-Pad2): track 0.00 -> 156.1 mm
- net Net-(POS28-Pad2): track 0.00 -> 148.1 mm
- net Net-(POS24-Pad2): track 0.00 -> 147.5 mm
- net Net-(FIN12-Pad2): track 0.00 -> 102.8 mm
- net Net-(FIN8-Pad2): track 0.00 -> 101.8 mm
- net Net-(FIN4-Pad2): track 0.00 -> 100.3 mm
- net /Start (16LEDs)/Start-LEDs: track 0.00 -> 24.4 mm
- net Net-(POS54-Pad2): track 0.00 -> 18.9 mm
- net Net-(POS72-Pad2): track 0.00 -> 18.2 mm
- net Net-(POS53-Pad2): track 0.00 -> 18.0 mm
- net Net-(POS17-Pad2): track 0.00 -> 17.9 mm
- net Net-(POS46-Pad2): track 0.00 -> 17.3 mm
- net Net-(POS29-Pad2): track 0.00 -> 17.3 mm
- net Net-(POS71-Pad2): track 0.00 -> 16.9 mm
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- added copper zone on B.Cu, net GND
- added copper zone on F.Cu, net VDD
Other:
- board text added: "JLCJLCJLCJLC"
- board text added: "v1"

Commit message: Update FieldBoard.kicad_pcb
Routing:
- net VDD: track 10.7 -> 0.00 mm
Changed lines of the file:
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@@
   (via (at 122.9 116.1) (size 0.8) (drill 0.4) (layers "F.Cu" "B.Cu") (net 1))
   (via (at 196.8 23.4) (size 0.8) (drill 0.4) (layers "F.Cu" "B.Cu") (net 1))
-  (segment (start 126.005 100.855) (end 129.355 100.855) (width 2.54) (layer "F.Cu") (net 2))
-  (segment (start 126.005 100.855) (end 123.045 100.855) (width 2.54) (layer "F.Cu") (net 2))
-  (segment (start 126.005 100.855) (end 126.005 98.105) (width 2.54) (layer "F.Cu") (net 2))
-  (segment (start 126.005 100.855) (end 126.005 102.495) (width 2.54) (layer "F.Cu") (net 2))
   (segment (start 131.4 81.9) (end 133.99 84.49) (width 0.3556) (layer "F.Cu") (net 3))
   (segment (start 131.4 79.725) (end 131.4 81.9) (width 0.3556) (layer "F.Cu") (net 3))
@@
   (segment (start 123.3 84.4) (end 120.7 81.8) (width 0.3556) (layer "F.Cu") (net 103))
   (zone (net 2) (net_name "VDD") (layer "F.Cu") (hatch edge 0.508)
+    (connect_pads yes (clearance 0.508))
+    (min_thickness 0.254) (filled_areas_thickness no)
+    (fill yes (thermal_gap 0.508) (thermal_bridge_width 0.508))
+    (polygon
+      (pts
+        (xy 130.8 103.2)
+        (xy 120.8 103.2)
+        (xy 120.8 98.2)
+        (xy 130.8 98.2)
+      )
+    )
+  )
+  (zone (net 2) (net_name "VDD") (layer "F.Cu") (hatch edge 0.508)
     (connect_pads (clearance 0.508))
     (min_thickness 0.254) (filled_areas_thickness no)
@@
       )
     )
+  )
+  (zone (net 1) (net_name "GND") (layer "B.Cu") (hatch edge 0.508)
+    (connect_pads yes (clearance 0.508))
+    (min_thickness 0.254) (filled_areas_thickness no)
+    (fill yes (thermal_gap 0.508) (thermal_bridge_width 0.508))
+    (polygon
+      (pts
+        (xy 130.8 108.6)
+        (xy 120.8 108.6)
+        (xy 120.8 103.6)
+        (xy 130.8 103.6)
+      )
+    )
