File: KiCad files/FieldBoard/Touchpads.kicad_sch (KiCad schematic)
At the start: 48 parts, among them U1 TTP223-BA6, U10 TTP223-BA6, U11 TTP223-BA6, U12 TTP223-BA6, U2 TTP223-BA6, U3 TTP223-BA6, U5 TTP223-BA6, U6 TTP223-BA6, U7 TTP223-BA6, U8 TTP223-BA6, U9 TTP223-BA6

Commit message: update
Parts:
- TP1, TP10, TP11, TP12, TP2, TP3, TP4, TP5, TP6, TP7, TP8, TP9: footprint test_library:TP_11mm_strelicaLijevo -> (none)
- U4: value (none) -> TTP223-BA6
Changed lines of the file:
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@@
       (effects (font (size 1.27 1.27)) (justify left) hide)
     )
-    (property "Footprint" "test_library:TP_11mm_strelicaLijevo" (id 2) (at 188.595 111.76 0)
+    (property "Footprint" "" (id 2) (at 188.595 111.76 0)
       (effects (font (size 1.27 1.27)) hide)
     )
@@
       (effects (font (size 1.27 1.27)) (justify left) hide)
     )
-    (property "Footprint" "test_library:TP_11mm_strelicaLijevo" (id 2) (at 140.335 55.245 0)
+    (property "Footprint" "" (id 2) (at 140.335 55.245 0)
       (effects (font (size 1.27 1.27)) hide)
     )
@@
       (effects (font (size 1.27 1.27)) (justify left) hide)
     )
-    (property "Footprint" "test_library:TP_11mm_strelicaLijevo" (id 2) (at 90.805 111.76 0)
+    (property "Footprint" "" (id 2) (at 90.805 111.76 0)
       (effects (font (size 1.27 1.27)) hide)
     )
@@
       (effects (font (size 1.27 1.27)) (justify left) hide)
     )
-    (property "Footprint" "test_library:TP_11mm_strelicaLijevo" (id 2) (at 91.44 55.245 0)
+    (property "Footprint" "" (id 2) (at 91.44 55.245 0)
       (effects (font (size 1.27 1.27)) hide)
     )
@@
     (in_bom yes) (on_board yes)
     (property "Reference" "U4" (id 0) (at 97.79 42.545 0))
-    (property "Value" "" (id 1) (at 102.235 55.88 0))
+    (property "Value" "TTP223-BA6" (id 1) (at 102.235 55.88 0))
     (property "Footprint" "" (id 2) (at 102.235 55.245 0)
       (effects (font (size 1.27 1.27)) hide)
@@
       (effects (font (size 1.27 1.27)) (justify left) hide)
     )
-    (property "Footprint" "test_library:TP_11mm_strelicaLijevo" (id 2) (at 139.7 85.09 0)
+    (property "Footprint" "" (id 2) (at 139.7 85.09 0)
       (effects (font (size 1.27 1.27)) hide)
     )
@@
       (effects (font (size 1.27 1.27)) (justify left) hide)
     )
-    (property "Footprint" "test_library:TP_11mm_strelicaLijevo" (id 2) (at 139.065 141.605 0)
+    (property "Footprint" "" (id 2) (at 139.065 141.605 0)
       (effects (font (size 1.27 1.27)) hide)
     )
@@
       (effects (font (size 1.27 1.27)) (justify left) hide)
     )
-    (property "Footprint" "test_library:TP_11mm_strelicaLijevo" (id 2) (at 187.96 141.605 0)
+    (property "Footprint" "" (id 2) (at 187.96 141.605 0)
       (effects (font (size 1.27 1.27)) hide)
     )
@@
       (effects (font (size 1.27 1.27)) (justify left) hide)
     )
-    (property "Footprint" "test_library:TP_11mm_strelicaLijevo" (id 2) (at 90.805 85.09 0)
+    (property "Footprint" "" (id 2) (at 90.805 85.09 0)
       (effects (font (size 1.27 1.27)) hide)
     )
@@
       (effects (font (size 1.27 1.27)) (justify left) hide)
     )
-    (property "Footprint" "test_library:TP_11mm_strelicaLijevo" (id 2) (at 90.17 141.605 0)
+    (property "Footprint" "" (id 2) (at 90.17 141.605 0)
       (effects (font (size 1.27 1.27)) hide)
     )
@@
       (effects (font (size 1.27 1.27)) (justify left) hide)
     )
-    (property "Footprint" "test_library:TP_11mm_strelicaLijevo" (id 2) (at 189.23 55.245 0)
+    (property "Footprint" "" (id 2) (at 189.23 55.245 0)
       (effects (font (size 1.27 1.27)) hide)
     )
@@
       (effects (font (size 1.27 1.27)) (justify left) hide)
     )
-    (property "Footprint" "test_library:TP_11mm_strelicaLijevo" (id 2) (at 188.595 85.09 0)
+    (property "Footprint" "" (id 2) (at 188.595 85.09 0)
       (effects (font (size 1.27 1.27)) hide)
     )
@@
       (effects (font (size 1.27 1.27)) (justify left) hide)
     )
-    (property "Footprint" "test_library:TP_11mm_strelicaLijevo" (id 2) (at 139.7 111.76 0)
-      (effects (font (size 1.27 1.27)) hide)
-    )
+    (property "Footprint" "" (id 2) (at 139.7 111.76 0)
+      (effects (font (size 1.27 1.27)) hide)
+    )

Commit message: update
Parts:
- U1, U10, U11, U12, U2, U3, U4, U5, U6, U7, U8, U9: footprint (none) -> Package_TO_SOT_SMD:SOT-23-6
Changed lines of the file:
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@@
     (property "Reference" "U1" (id 0) (at 96.52 128.905 0))
     (property "Value" "TTP223-BA6" (id 1) (at 100.965 142.24 0))
-    (property "Footprint" "" (id 2) (at 100.965 141.605 0)
+    (property "Footprint" "Package_TO_SOT_SMD:SOT-23-6" (id 2) (at 100.965 141.605 0)
       (effects (font (size 1.27 1.27)) hide)
     )
@@
     (property "Reference" "U9" (id 0) (at 194.31 128.905 0))
     (property "Value" "TTP223-BA6" (id 1) (at 198.755 142.24 0))
-    (property "Footprint" "" (id 2) (at 198.755 141.605 0)
+    (property "Footprint" "Package_TO_SOT_SMD:SOT-23-6" (id 2) (at 198.755 141.605 0)
       (effects (font (size 1.27 1.27)) hide)
     )
@@
     (property "Reference" "U6" (id 0) (at 146.05 72.39 0))
     (property "Value" "TTP223-BA6" (id 1) (at 150.495 85.725 0))
-    (property "Footprint" "" (id 2) (at 150.495 85.09 0)
+    (property "Footprint" "Package_TO_SOT_SMD:SOT-23-6" (id 2) (at 150.495 85.09 0)
       (effects (font (size 1.27 1.27)) hide)
     )
@@
     (property "Reference" "U8" (id 0) (at 146.685 42.545 0))
     (property "Value" "TTP223-BA6" (id 1) (at 151.13 55.88 0))
-    (property "Footprint" "" (id 2) (at 151.13 55.245 0)
+    (property "Footprint" "Package_TO_SOT_SMD:SOT-23-6" (id 2) (at 151.13 55.245 0)
       (effects (font (size 1.27 1.27)) hide)
     )
@@
     (property "Reference" "U10" (id 0) (at 194.945 72.39 0))
     (property "Value" "TTP223-BA6" (id 1) (at 199.39 85.725 0))
-    (property "Footprint" "" (id 2) (at 199.39 85.09 0)
+    (property "Footprint" "Package_TO_SOT_SMD:SOT-23-6" (id 2) (at 199.39 85.09 0)
       (effects (font (size 1.27 1.27)) hide)
     )
@@
     (property "Reference" "U7" (id 0) (at 146.05 99.06 0))
     (property "Value" "TTP223-BA6" (id 1) (at 150.495 112.395 0))
-    (property "Footprint" "" (id 2) (at 150.495 111.76 0)
+    (property "Footprint" "Package_TO_SOT_SMD:SOT-23-6" (id 2) (at 150.495 111.76 0)
       (effects (font (size 1.27 1.27)) hide)
     )
@@
     (property "Reference" "U11" (id 0) (at 194.945 99.06 0))
     (property "Value" "TTP223-BA6" (id 1) (at 199.39 112.395 0))
-    (property "Footprint" "" (id 2) (at 199.39 111.76 0)
+    (property "Footprint" "Package_TO_SOT_SMD:SOT-23-6" (id 2) (at 199.39 111.76 0)
       (effects (font (size 1.27 1.27)) hide)
     )
@@
     (property "Reference" "U4" (id 0) (at 97.79 42.545 0))
     (property "Value" "TTP223-BA6" (id 1) (at 102.235 55.88 0))
-    (property "Footprint" "" (id 2) (at 102.235 55.245 0)
+    (property "Footprint" "Package_TO_SOT_SMD:SOT-23-6" (id 2) (at 102.235 55.245 0)
       (effects (font (size 1.27 1.27)) hide)
     )
@@
     (property "Reference" "U2" (id 0) (at 97.155 72.39 0))
     (property "Value" "TTP223-BA6" (id 1) (at 101.6 85.725 0))
-    (property "Footprint" "" (id 2) (at 101.6 85.09 0)
+    (property "Footprint" "Package_TO_SOT_SMD:SOT-23-6" (id 2) (at 101.6 85.09 0)
       (effects (font (size 1.27 1.27)) hide)
     )
@@
     (property "Reference" "U5" (id 0) (at 145.415 128.905 0))
     (property "Value" "TTP223-BA6" (id 1) (at 149.86 142.24 0))
-    (property "Footprint" "" (id 2) (at 149.86 141.605 0)
+    (property "Footprint" "Package_TO_SOT_SMD:SOT-23-6" (id 2) (at 149.86 141.605 0)
       (effects (font (size 1.27 1.27)) hide)
     )
@@
     (property "Reference" "U3" (id 0) (at 97.155 99.06 0))
     (property "Value" "TTP223-BA6" (id 1) (at 101.6 112.395 0))
-    (property "Footprint" "" (id 2) (at 101.6 111.76 0)
+    (property "Footprint" "Package_TO_SOT_SMD:SOT-23-6" (id 2) (at 101.6 111.76 0)
       (effects (font (size 1.27 1.27)) hide)
     )
@@
     (property "Reference" "U12" (id 0) (at 195.58 42.545 0))
     (property "Value" "TTP223-BA6" (id 1) (at 200.025 55.88 0))
-    (property "Footprint" "" (id 2) (at 200.025 55.245 0)
-      (effects (font (size 1.27 1.27)) hide)
-    )
+    (property "Footprint" "Package_TO_SOT_SMD:SOT-23-6" (id 2) (at 200.025 55.245 0)
+      (effects (font (size 1.27 1.27)) hide)
+    )

Commit message: update
Parts:
- TP1: renamed from TP4; footprint (none) -> FieldBoard_footprint:TP_11mm_strelicaLijevo
- TP10: renamed from TP1; footprint (none) -> FieldBoard_footprint:TP_11mm_strelicaLijevo
- TP11: renamed from TP5; footprint (none) -> FieldBoard_footprint:TP_11mm_kvacica
- TP12: renamed from TP9; footprint (none) -> FieldBoard_footprint:TP_11mm_strelicaDesno
- TP2: renamed from TP8; footprint (none) -> FieldBoard_footprint:TP_11mm_kvacica
- TP3: renamed from TP12; footprint (none) -> FieldBoard_footprint:TP_11mm_strelicaDesno
- TP4: renamed from TP2; footprint (none) -> FieldBoard_footprint:TP_11mm_kvacica
- TP5: renamed from TP6; footprint (none) -> FieldBoard_footprint:TP_11mm_strelicaDesno
- TP6: renamed from TP10; footprint (none) -> FieldBoard_footprint:TP_11mm_strelicaLijevo
- TP7: renamed from TP3; footprint (none) -> FieldBoard_footprint:TP_11mm_strelicaDesno
- TP8: renamed from TP7; footprint (none) -> FieldBoard_footprint:TP_11mm_strelicaLijevo
- TP9: renamed from TP11; footprint (none) -> FieldBoard_footprint:TP_11mm_kvacica
- renumbered C8 to C1, C2 to C10, C10 to C11, C18 to C12, C7 to C13, C15 to C14, C23 to C15, C3 to C16, C11 to C17, C19 to C18, C5 to C19, C16 to C2, C13 to C20, C1 to C22, C9 to C23, C17 to C24, C24 to C3, C12 to C5, C20 to C6, C6 to C7, C14 to C8, C22 to C9, U4 to U1, U1 to U10, U5 to U11, U9 to U12, U8 to U2, U12 to U3, U2 to U4, U6 to U5, U10 to U6, U3 to U7, U7 to U8, U11 to U9

Commit message: update
Parts:
- C1, C10, C11, C12, C13, C14, C15, C16, C17, C18, C19, C2, C20, C21, C22, C23, C24, C3, C4, C5, C6, C7, C8, C9: footprint Capacitor_SMD:C_0805_2012Metric -> Capacitor_SMD:C_0603_1608Metric
- TP4: footprint FieldBoard_footprint:TP_11mm_kvacica -> FieldBoard_footprint:TP_11mm_strelicaLijevo
- TP5: footprint FieldBoard_footprint:TP_11mm_strelicaDesno -> FieldBoard_footprint:TP_11mm_kvacica
- TP6: footprint FieldBoard_footprint:TP_11mm_strelicaLijevo -> FieldBoard_footprint:TP_11mm_strelicaDesno
- TP7: footprint FieldBoard_footprint:TP_11mm_strelicaDesno -> FieldBoard_footprint:TP_11mm_strelicaLijevo
- TP8: footprint FieldBoard_footprint:TP_11mm_strelicaLijevo -> FieldBoard_footprint:TP_11mm_kvacica
- TP9: footprint FieldBoard_footprint:TP_11mm_kvacica -> FieldBoard_footprint:TP_11mm_strelicaDesno
Changed lines of the file:
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@@
       (effects (font (size 1.27 1.27)) (justify left))
     )
-    (property "Footprint" "Capacitor_SMD:C_0805_2012Metric" (id 2) (at 163.83 109.22 0)
+    (property "Footprint" "Capacitor_SMD:C_0603_1608Metric" (id 2) (at 163.83 109.22 0)
       (effects (font (size 1.27 1.27)) hide)
     )
@@
       (effects (font (size 1.27 1.27)) (justify left))
     )
-    (property "Footprint" "Capacitor_SMD:C_0805_2012Metric" (id 2) (at 212.725 82.55 0)
+    (property "Footprint" "Capacitor_SMD:C_0603_1608Metric" (id 2) (at 212.725 82.55 0)
       (effects (font (size 1.27 1.27)) hide)
     )
@@
       (effects (font (size 1.27 1.27)) (justify left))
     )
-    (property "Footprint" "Capacitor_SMD:C_0805_2012Metric" (id 2) (at 114.935 82.55 0)
+    (property "Footprint" "Capacitor_SMD:C_0603_1608Metric" (id 2) (at 114.935 82.55 0)
       (effects (font (size 1.27 1.27)) hide)
     )
@@
       (effects (font (size 1.27 1.27)) (justify left) hide)
     )
-    (property "Footprint" "FieldBoard_footprint:TP_11mm_kvacica" (id 2) (at 188.595 111.76 0)
+    (property "Footprint" "FieldBoard_footprint:TP_11mm_strelicaDesno" (id 2) (at 188.595 111.76 0)
       (effects (font (size 1.27 1.27)) hide)
     )
@@
       (effects (font (size 1.27 1.27)) (justify left))
     )
-    (property "Footprint" "Capacitor_SMD:C_0805_2012Metric" (id 2) (at 190.5 59.69 0)
+    (property "Footprint" "Capacitor_SMD:C_0603_1608Metric" (id 2) (at 190.5 59.69 0)
       (effects (font (size 1.27 1.27)) hide)
     )
@@
       (effects (font (size 1.27 1.27)) (justify left))
     )
-    (property "Footprint" "Capacitor_SMD:C_0805_2012Metric" (id 2) (at 140.97 89.535 0)
+    (property "Footprint" "Capacitor_SMD:C_0603_1608Metric" (id 2) (at 140.97 89.535 0)
       (effects (font (size 1.27 1.27)) hide)
     )
@@
       (effects (font (size 1.27 1.27)) (justify left))
     )
-    (property "Footprint" "Capacitor_SMD:C_0805_2012Metric" (id 2) (at 91.44 146.05 0)
+    (property "Footprint" "Capacitor_SMD:C_0603_1608Metric" (id 2) (at 91.44 146.05 0)
       (effects (font (size 1.27 1.27)) hide)
     )
@@
       (effects (font (size 1.27 1.27)) (justify left) hide)
     )
-    (property "Footprint" "FieldBoard_footprint:TP_11mm_strelicaDesno" (id 2) (at 90.805 111.76 0)
+    (property "Footprint" "FieldBoard_footprint:TP_11mm_strelicaLijevo" (id 2) (at 90.805 111.76 0)
       (effects (font (size 1.27 1.27)) hide)
     )
@@
       (effects (font (size 1.27 1.27)) (justify left))
     )
-    (property "Footprint" "Capacitor_SMD:C_0805_2012Metric" (id 2) (at 92.075 89.535 0)
+    (property "Footprint" "Capacitor_SMD:C_0603_1608Metric" (id 2) (at 92.075 89.535 0)
       (effects (font (size 1.27 1.27)) hide)
     )
@@
       (effects (font (size 1.27 1.27)) (justify left))
     )
-    (property "Footprint" "Capacitor_SMD:C_0805_2012Metric" (id 2) (at 140.335 146.05 0)
+    (property "Footprint" "Capacitor_SMD:C_0603_1608Metric" (id 2) (at 140.335 146.05 0)
       (effects (font (size 1.27 1.27)) hide)
     )
@@
       (effects (font (size 1.27 1.27)) (justify left) hide)
     )
-    (property "Footprint" "FieldBoard_footprint:TP_11mm_strelicaDesno" (id 2) (at 139.7 85.09 0)
+    (property "Footprint" "FieldBoard_footprint:TP_11mm_kvacica" (id 2) (at 139.7 85.09 0)
       (effects (font (size 1.27 1.27)) hide)
     )
@@
       (effects (font (size 1.27 1.27)) (justify left))
     )
-    (property "Footprint" "Capacitor_SMD:C_0805_2012Metric" (id 2) (at 189.865 116.205 0)
+    (property "Footprint" "Capacitor_SMD:C_0603_1608Metric" (id 2) (at 189.865 116.205 0)
       (effects (font (size 1.27 1.27)) hide)
     )
@@
       (effects (font (size 1.27 1.27)) (justify left))
     )
-    (property "Footprint" "Capacitor_SMD:C_0805_2012Metric" (id 2) (at 92.075 116.205 0)
+    (property "Footprint" "Capacitor_SMD:C_0603_1608Metric" (id 2) (at 92.075 116.205 0)
       (effects (font (size 1.27 1.27)) hide)
     )
@@
       (effects (font (size 1.27 1.27)) (justify left))
     )
-    (property "Footprint" "Capacitor_SMD:C_0805_2012Metric" (id 2) (at 115.57 52.705 0)
+    (property "Footprint" "Capacitor_SMD:C_0603_1608Metric" (id 2) (at 115.57 52.705 0)
       (effects (font (size 1.27 1.27)) hide)
     )
@@
       (effects (font (size 1.27 1.27)) (justify left))
     )
-    (property "Footprint" "Capacitor_SMD:C_0805_2012Metric" (id 2) (at 163.195 139.065 0)
+    (property "Footprint" "Capacitor_SMD:C_0603_1608Metric" (id 2) (at 163.195 139.065 0)
       (effects (font (size 1.27 1.27)) hide)
     )
@@
       (effects (font (size 1.27 1.27)) (justify left))
     )
-    (property "Footprint" "Capacitor_SMD:C_0805_2012Metric" (id 2) (at 212.725 109.22 0)
+    (property "Footprint" "Capacitor_SMD:C_0603_1608Metric" (id 2) (at 212.725 109.22 0)
       (effects (font (size 1.27 1.27)) hide)
     )
@@
       (effects (font (size 1.27 1.27)) (justify left))
     )
-    (property "Footprint" "Capacitor_SMD:C_0805_2012Metric" (id 2) (at 189.865 89.535 0)
+    (property "Footprint" "Capacitor_SMD:C_0603_1608Metric" (id 2) (at 189.865 89.535 0)
       (effects (font (size 1.27 1.27)) hide)
     )
@@
       (effects (font (size 1.27 1.27)) (justify left))
     )
-    (property "Footprint" "Capacitor_SMD:C_0805_2012Metric" (id 2) (at 92.71 59.69 0)
+    (property "Footprint" "Capacitor_SMD:C_0603_1608Metric" (id 2) (at 92.71 59.69 0)
       (effects (font (size 1.27 1.27)) hide)
     )
@@
       (effects (font (size 1.27 1.27)) (justify left))
     )
-    (property "Footprint" "Capacitor_SMD:C_0805_2012Metric" (id 2) (at 114.3 139.065 0)
+    (property "Footprint" "Capacitor_SMD:C_0603_1608Metric" (id 2) (at 114.3 139.065 0)
       (effects (font (size 1.27 1.27)) hide)
     )
@@
       (effects (font (size 1.27 1.27)) (justify left))
     )
-    (property "Footprint" "Capacitor_SMD:C_0805_2012Metric" (id 2) (at 114.935 109.22 0)
+    (property "Footprint" "Capacitor_SMD:C_0603_1608Metric" (id 2) (at 114.935 109.22 0)
       (effects (font (size 1.27 1.27)) hide)
     )
@@
       (effects (font (size 1.27 1.27)) (justify left))
     )
-    (property "Footprint" "Capacitor_SMD:C_0805_2012Metric" (id 2) (at 140.97 116.205 0)
+    (property "Footprint" "Capacitor_SMD:C_0603_1608Metric" (id 2) (at 140.97 116.205 0)
       (effects (font (size 1.27 1.27)) hide)
     )
@@
       (effects (font (size 1.27 1.27)) (justify left) hide)
     )
-    (property "Footprint" "FieldBoard_footprint:TP_11mm_kvacica" (id 2) (at 90.805 85.09 0)
+    (property "Footprint" "FieldBoard_footprint:TP_11mm_strelicaLijevo" (id 2) (at 90.805 85.09 0)
       (effects (font (size 1.27 1.27)) hide)
     )
@@
       (effects (font (size 1.27 1.27)) (justify left))
     )
-    (property "Footprint" "Capacitor_SMD:C_0805_2012Metric" (id 2) (at 212.09 139.065 0)
+    (property "Footprint" "Capacitor_SMD:C_0603_1608Metric" (id 2) (at 212.09 139.065 0)
       (effects (font (size 1.27 1.27)) hide)
     )
@@
       (effects (font (size 1.27 1.27)) (justify left))
     )
-    (property "Footprint" "Capacitor_SMD:C_0805_2012Metric" (id 2) (at 189.23 146.05 0)
+    (property "Footprint" "Capacitor_SMD:C_0603_1608Metric" (id 2) (at 189.23 146.05 0)
       (effects (font (size 1.27 1.27)) hide)
     )
@@
       (effects (font (size 1.27 1.27)) (justify left))
     )
-    (property "Footprint" "Capacitor_SMD:C_0805_2012Metric" (id 2) (at 141.605 59.69 0)
+    (property "Footprint" "Capacitor_SMD:C_0603_1608Metric" (id 2) (at 141.605 59.69 0)
       (effects (font (size 1.27 1.27)) hide)
     )
@@
       (effects (font (size 1.27 1.27)) (justify left))
     )
-    (property "Footprint" "Capacitor_SMD:C_0805_2012Metric" (id 2) (at 164.465 52.705 0)
+    (property "Footprint" "Capacitor_SMD:C_0603_1608Metric" (id 2) (at 164.465 52.705 0)
       (effects (font (size 1.27 1.27)) hide)
     )
@@
       (effects (font (size 1.27 1.27)) (justify left))
     )
-    (property "Footprint" "Capacitor_SMD:C_0805_2012Metric" (id 2) (at 163.83 82.55 0)
+    (property "Footprint" "Capacitor_SMD:C_0603_1608Metric" (id 2) (at 163.83 82.55 0)
       (effects (font (size 1.27 1.27)) hide)
     )
@@
       (effects (font (size 1.27 1.27)) (justify left))
     )
-    (property "Footprint" "Capacitor_SMD:C_0805_2012Metric" (id 2) (at 213.36 52.705 0)
+    (property "Footprint" "Capacitor_SMD:C_0603_1608Metric" (id 2) (at 213.36 52.705 0)
       (effects (font (size 1.27 1.27)) hide)
     )
@@
       (effects (font (size 1.27 1.27)) (justify left) hide)
     )
-    (property "Footprint" "FieldBoard_footprint:TP_11mm_strelicaLijevo" (id 2) (at 188.595 85.09 0)
+    (property "Footprint" "FieldBoard_footprint:TP_11mm_strelicaDesno" (id 2) (at 188.595 85.09 0)
       (effects (font (size 1.27 1.27)) hide)
     )
@@
       (effects (font (size 1.27 1.27)) (justify left) hide)
     )
-    (property "Footprint" "FieldBoard_footprint:TP_11mm_strelicaLijevo" (id 2) (at 139.7 111.76 0)
-      (effects (font (size 1.27 1.27)) hide)
-    )
+    (property "Footprint" "FieldBoard_footprint:TP_11mm_kvacica" (id 2) (at 139.7 111.76 0)
+      (effects (font (size 1.27 1.27)) hide)
+    )
