File: KiCad files/FieldBoard/FieldBoard.kicad_sch (KiCad schematic)
At the start: 6 parts, among them J1 Conn_01x06_Male, J2 Conn_01x14_Male

Commit message: update
Other:
- note added: "TO-DO: - konektor napajanja koji može podnijeti 5A"
Changed lines of the file:
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@@
     (effects (font (size 3 3) (thickness 0.6) bold) (justify left bottom))
+  )
+  (text "TO-DO:\n- konektor napajanja koji može podnijeti 5A"
+    (at 26.67 155.575 0)
+    (effects (font (size 2 2)) (justify left bottom))
   )
   (symbol (lib_id "Device:R_Small") (at 95.885 76.835 90) (unit 1)
@@
     )
     (path "/3c394a32-751f-48ca-bfb7-93be96f92c8f/f2afdb2f-9391-4cec-901b-85a93e07430a"
-      (reference "TP1") (unit 1) (value "TestPoint") (footprint "test_library:TP_11mm_strelicaLijevo")
+      (reference "TP1") (unit 1) (value "TestPoint") (footprint "")
     )
     (path "/3c394a32-751f-48ca-bfb7-93be96f92c8f/b7003926-dbb6-4145-b1f6-ce1e250c690e"
-      (reference "TP2") (unit 1) (value "TestPoint") (footprint "test_library:TP_11mm_strelicaLijevo")
+      (reference "TP2") (unit 1) (value "TestPoint") (footprint "")
     )
     (path "/3c394a32-751f-48ca-bfb7-93be96f92c8f/32b8f6ef-fe19-448e-9bc3-c4baa1834ea8"
-      (reference "TP3") (unit 1) (value "TestPoint") (footprint "test_library:TP_11mm_strelicaLijevo")
+      (reference "TP3") (unit 1) (value "TestPoint") (footprint "")
     )
     (path "/3c394a32-751f-48ca-bfb7-93be96f92c8f/46ecad93-7ca1-492e-9bc1-1fa9dd1841d7"
-      (reference "TP4") (unit 1) (value "TestPoint") (footprint "test_library:TP_11mm_strelicaLijevo")
+      (reference "TP4") (unit 1) (value "TestPoint") (footprint "")
     )
     (path "/3c394a32-751f-48ca-bfb7-93be96f92c8f/870929b6-85bb-4730-9a37-375aca8976b5"
-      (reference "TP5") (unit 1) (value "TestPoint") (footprint "test_library:TP_11mm_strelicaLijevo")
+      (reference "TP5") (unit 1) (value "TestPoint") (footprint "")
     )
     (path "/3c394a32-751f-48ca-bfb7-93be96f92c8f/73bec328-37c2-4c57-a553-1220bb0b1d05"
-      (reference "TP6") (unit 1) (value "TestPoint") (footprint "test_library:TP_11mm_strelicaLijevo")
+      (reference "TP6") (unit 1) (value "TestPoint") (footprint "")
     )
     (path "/3c394a32-751f-48ca-bfb7-93be96f92c8f/ff893075-9c8c-4519-96bc-8b15a5dac4e0"
-      (reference "TP7") (unit 1) (value "TestPoint") (footprint "test_library:TP_11mm_strelicaLijevo")
+      (reference "TP7") (unit 1) (value "TestPoint") (footprint "")
     )
     (path "/3c394a32-751f-48ca-bfb7-93be96f92c8f/24aa5ff9-83a8-4975-8ea5-f494562f1d6a"
-      (reference "TP8") (unit 1) (value "TestPoint") (footprint "test_library:TP_11mm_strelicaLijevo")
+      (reference "TP8") (unit 1) (value "TestPoint") (footprint "")
     )
     (path "/3c394a32-751f-48ca-bfb7-93be96f92c8f/9ff9c206-726c-4a69-8e07-75ee55bef344"
-      (reference "TP9") (unit 1) (value "TestPoint") (footprint "test_library:TP_11mm_strelicaLijevo")
+      (reference "TP9") (unit 1) (value "TestPoint") (footprint "")
     )
     (path "/3c394a32-751f-48ca-bfb7-93be96f92c8f/fe012903-350c-4138-a0e8-16353361383f"
-      (reference "TP10") (unit 1) (value "TestPoint") (footprint "test_library:TP_11mm_strelicaLijevo")
+      (reference "TP10") (unit 1) (value "TestPoint") (footprint "")
     )
     (path "/3c394a32-751f-48ca-bfb7-93be96f92c8f/19f429a6-677f-43f6-89a3-19c6b6e5c5d9"
-      (reference "TP11") (unit 1) (value "TestPoint") (footprint "test_library:TP_11mm_strelicaLijevo")
+      (reference "TP11") (unit 1) (value "TestPoint") (footprint "")
     )
     (path "/3c394a32-751f-48ca-bfb7-93be96f92c8f/fd82520f-2b71-4935-a276-f713db092349"
-      (reference "TP12") (unit 1) (value "TestPoint") (footprint "test_library:TP_11mm_strelicaLijevo")
+      (reference "TP12") (unit 1) (value "TestPoint") (footprint "")
     )
     (path "/3c394a32-751f-48ca-bfb7-93be96f92c8f/06f97ced-c48a-4269-9d29-bc99f1061eb7"
-      (reference "U1") (unit 1) (value "TTP223-BA6") (footprint "")
+      (reference "U1") (unit 1) (value "TTP223-BA6") (footprint "Package_TO_SOT_SMD:SOT-23-6")
     )
     (path "/3c394a32-751f-48ca-bfb7-93be96f92c8f/925bf12b-6fa0-46cc-b8cf-9908bdd19f62"
-      (reference "U2") (unit 1) (value "TTP223-BA6") (footprint "")
+      (reference "U2") (unit 1) (value "TTP223-BA6") (footprint "Package_TO_SOT_SMD:SOT-23-6")
     )
     (path "/3c394a32-751f-48ca-bfb7-93be96f92c8f/d20fab24-e6a4-4d9a-868f-35fc04ed6fad"
-      (reference "U3") (unit 1) (value "TTP223-BA6") (footprint "")
+      (reference "U3") (unit 1) (value "TTP223-BA6") (footprint "Package_TO_SOT_SMD:SOT-23-6")
     )
     (path "/3c394a32-751f-48ca-bfb7-93be96f92c8f/5452c99d-37eb-4314-b287-192c3dbd8d70"
-      (reference "U4") (unit 1) (value "TTP223-BA6") (footprint "")
+      (reference "U4") (unit 1) (value "TTP223-BA6") (footprint "Package_TO_SOT_SMD:SOT-23-6")
     )
     (path "/3c394a32-751f-48ca-bfb7-93be96f92c8f/c0954bcb-eabf-43b0-8054-76f817450d4f"
-      (reference "U5") (unit 1) (value "TTP223-BA6") (footprint "")
+      (reference "U5") (unit 1) (value "TTP223-BA6") (footprint "Package_TO_SOT_SMD:SOT-23-6")
     )
     (path "/3c394a32-751f-48ca-bfb7-93be96f92c8f/0959f30e-a2ed-4fa9-84e8-dd4d25983cd0"
-      (reference "U6") (unit 1) (value "TTP223-BA6") (footprint "")
+      (reference "U6") (unit 1) (value "TTP223-BA6") (footprint "Package_TO_SOT_SMD:SOT-23-6")
     )
     (path "/3c394a32-751f-48ca-bfb7-93be96f92c8f/3aaed85b-d72d-4ce0-aef2-dc7077b0318f"
-      (reference "U7") (unit 1) (value "TTP223-BA6") (footprint "")
+      (reference "U7") (unit 1) (value "TTP223-BA6") (footprint "Package_TO_SOT_SMD:SOT-23-6")
     )
     (path "/3c394a32-751f-48ca-bfb7-93be96f92c8f/0e58e455-439d-4805-baaf-ede6598932da"
-      (reference "U8") (unit 1) (value "TTP223-BA6") (footprint "")
+      (reference "U8") (unit 1) (value "TTP223-BA6") (footprint "Package_TO_SOT_SMD:SOT-23-6")
     )
     (path "/3c394a32-751f-48ca-bfb7-93be96f92c8f/078ce96e-f0cd-4cb5-af0d-6097edbfb4d1"
-      (reference "U9") (unit 1) (value "TTP223-BA6") (footprint "")
+      (reference "U9") (unit 1) (value "TTP223-BA6") (footprint "Package_TO_SOT_SMD:SOT-23-6")
     )
     (path "/3c394a32-751f-48ca-bfb7-93be96f92c8f/25837a02-67b0-47d4-81db-722246363686"
-      (reference "U10") (unit 1) (value "TTP223-BA6") (footprint "")
+      (reference "U10") (unit 1) (value "TTP223-BA6") (footprint "Package_TO_SOT_SMD:SOT-23-6")
     )
     (path "/3c394a32-751f-48ca-bfb7-93be96f92c8f/441f897f-85a6-4754-a83f-523cd4afad80"
-      (reference "U11") (unit 1) (value "TTP223-BA6") (footprint "")
+      (reference "U11") (unit 1) (value "TTP223-BA6") (footprint "Package_TO_SOT_SMD:SOT-23-6")
     )
     (path "/3c394a32-751f-48ca-bfb7-93be96f92c8f/e8eec3c4-31ef-44d3-8525-b9849bd323ca"
-      (reference "U12") (unit 1) (value "TTP223-BA6") (footprint "")
-    )
-  )
+      (reference "U12") (unit 1) (value "TTP223-BA6") (footprint "Package_TO_SOT_SMD:SOT-23-6")
+    )
+  )

Commit message: update
Parts:
- removed J2: Conn_01x14_Male, symbol Connector:Conn_01x14_Male
- added J2, J3, J4, J5: Conn_01x05_Male, Connector_PinHeader_2.54mm:PinHeader_1x05_P2.54mm_Vertical, symbol Connector:Conn_01x05_Male
- J1: footprint (none) -> Connector_PinHeader_2.54mm:PinHeader_1x06_P2.54mm_Vertical
- R1, R2, R3, R4: footprint (none) -> Resistor_SMD:R_0805_2012Metric
Connections:
- net +5V: now also J2.1 (Pin_1), J3.1 (Pin_1), J4.1 (Pin_1), J5.1 (Pin_1)
- net GND: now also J2.5 (Pin_5), J3.5 (Pin_5), J4.5 (Pin_5), J5.5 (Pin_5)
- net Touchpads (12)/TP1: now also J2.2 (Pin_2)
- net Touchpads (12)/TP10: now also J5.2 (Pin_2)
- net Touchpads (12)/TP11: now also J5.3 (Pin_3)
- net Touchpads (12)/TP12: now also J5.4 (Pin_4)
- net Touchpads (12)/TP2: now also J2.3 (Pin_3)
- net Touchpads (12)/TP3: now also J2.4 (Pin_4)
- net Touchpads (12)/TP4: now also J3.2 (Pin_2)
- net Touchpads (12)/TP5: now also J3.3 (Pin_3)
- net Touchpads (12)/TP6: now also J3.4 (Pin_4)
- net Touchpads (12)/TP7: now also J4.2 (Pin_2)
- net Touchpads (12)/TP8: now also J4.3 (Pin_3)
- net Touchpads (12)/TP9: now also J4.4 (Pin_4)

Commit message: update
Parts:
- renumbered J2 to J1, J3 to J2, J1 to J3
Other:
- note added: "TO-DO: - konektor napajanja koji može podnijeti 5A - dodati rupe"
- note removed: "TO-DO: - konektor napajanja koji može podnijeti 5A"

Commit message: update
Parts:
- removed J1, J2, J4, J5: Conn_01x05_Male, Connector_PinHeader_2.54mm:PinHeader_1x05_P2.54mm_Vertical, symbol Connector:Conn_01x05_Male
- removed J3: Conn_01x06_Male, Connector_PinHeader_2.54mm:PinHeader_1x06_P2.54mm_Vertical, symbol Connector:Conn_01x06_Male
- added J1, J10, J11, J12, J13, J14, J15, J16, J17, J18, J19, J2, J20, J21, J22, J23, J24, J25, J26, J3, J4, J5, J6, J8, J9: Conn_01x01_Male, symbol Connector:Conn_01x01_Male
- added J7: (no value), symbol Connector:Conn_01x01_Male
- R1, R2, R3, R4: footprint Resistor_SMD:R_0805_2012Metric -> Resistor_SMD:R_0603_1608Metric
Connections:
- net +5V: now also J12.1 (Pin_1), J17.1 (Pin_1), J22.1 (Pin_1), J7.1 (Pin_1)
- net GND: now also J11.1 (Pin_1), J16.1 (Pin_1), J21.1 (Pin_1), J26.1 (Pin_1), J6.1 (Pin_1)
- net Touchpads (12)/TP1: now also J8.1 (Pin_1)
- net Touchpads (12)/TP10: now also J23.1 (Pin_1)
- net Touchpads (12)/TP11: now also J24.1 (Pin_1)
- net Touchpads (12)/TP12: now also J25.1 (Pin_1)
- net Touchpads (12)/TP2: now also J9.1 (Pin_1)
- net Touchpads (12)/TP3: now also J10.1 (Pin_1)
- net Touchpads (12)/TP4: now also J13.1 (Pin_1)
- net Touchpads (12)/TP5: now also J14.1 (Pin_1)
- net Touchpads (12)/TP6: now also J15.1 (Pin_1)
- net Touchpads (12)/TP7: now also J18.1 (Pin_1)
- net Touchpads (12)/TP8: now also J19.1 (Pin_1)
- net Touchpads (12)/TP9: now also J20.1 (Pin_1)
- net VDD: now also J1.1 (Pin_1)
- net at R1.1: now also J2.1 (Pin_1)
- net at R3.1: now also J4.1 (Pin_1)
- net at R2.1: now also J3.1 (Pin_1)
- net at R4.1: now also J5.1 (Pin_1)

Commit message: v2
Parts:
- J1, J10, J11, J12, J13, J14, J15, J16, J17, J18, J19, J2, J20, J21, J22, J23, J24, J25, J26, J3, J4, J5, J6, J8, J9: footprint (none) -> FieldBoard_footprint:ConnectionPad
- J7: value (none) -> Conn_01x01_Male; footprint (none) -> FieldBoard_footprint:ConnectionPad

Commit message: update
Parts:
- removed J1, J10, J11, J12, J13, J14, J15, J16, J17, J18, J19, J2, J20, J21, J22, J23, J24, J25, J26, J3, J4, J5, J6, J7, J8, J9: Conn_01x01_Male, FieldBoard_footprint:ConnectionPad, symbol Connector:Conn_01x01_Male

Commit message: update
Parts:
- added J1: (no value), symbol Connector_Generic:Conn_01x02
- added J2: (no value), symbol Connector:Conn_01x05_Male
Connections:
- net GND: now also J1.2 (Pin_2), J2.5 (Pin_5)
- net VDD: now also J1.1 (Pin_1)
- net at R1.1: now also J2.1 (Pin_1)
- net at R3.1: now also J2.3 (Pin_3)
- net at R2.1: now also J2.2 (Pin_2)
- net at R4.1: now also J2.4 (Pin_4)
Other:
- removed sheet Touchpads (12)
- note removed: "Touchpads"

Commit message: layout v1
Parts:
- J1: value (none) -> Conn_01x02; footprint (none) -> TerminalBlock_Phoenix:TerminalBlock_Phoenix_MKDS-1,5-2-5.08_1x02_P5.08mm_Horizontal
- J2: value (none) -> Conn_01x05_Male; footprint (none) -> Connector_PinHeader_2.54mm:PinHeader_1x05_P2.54mm_Vertical
Connections:
- net GND: now also J2.1 (Pin_1); no longer J2.5 (Pin_5)
- net Positions (52LEDs)/Positions-LEDs: now also R2.2; no longer R4.2
- net Start (16LEDs)/Start-LEDs: now also R4.2; no longer R2.2
- net at R1.1: now also J2.5 (Pin_5); no longer J2.1 (Pin_1)
- net at R2.1: now also J2.4 (Pin_4); no longer J2.2 (Pin_2)
- net at R4.1: now also J2.2 (Pin_2); no longer J2.4 (Pin_4)
Other:
- moved on the sheet: J1
