File: KiCad files/FieldBoard/FieldBoard.kicad_sch (KiCad schematic)
At the start: 6 parts, among them J1 Conn_01x02, J2 Conn_01x05_Male

Commit message: up
Other:
- note added: "TO-DO: - dodati rupe"
- note removed: "TO-DO: - konektor napajanja koji može podnijeti 5A - dodati rupe"
Changed lines of the file:
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@@
     (effects (font (size 3 3) (thickness 0.6) bold) (justify left bottom))
   )
-  (text "TO-DO:\n- konektor napajanja koji može podnijeti 5A\n- dodati rupe"
-    (at 26.67 155.575 0)
+  (text "TO-DO:\n- dodati rupe" (at 26.67 155.575 0)
     (effects (font (size 2 2)) (justify left bottom))
   )
@@
       (effects (font (size 1.27 1.27)) hide)
     )
-    (property "Value" "" (id 1) (at 95.25 55.4792 0))
+    (property "Value" "PWR_FLAG" (id 1) (at 95.25 55.4792 0))
     (property "Footprint" "" (id 2) (at 95.25 59.055 0)
       (effects (font (size 1.27 1.27)) hide)
