File: KiCad files/FieldBoard/Finish.kicad_sch (KiCad schematic)
At the start: 16 parts

Commit message: update
Parts:
- POS1, POS16: footprint (none) -> FieldBoard_footprint:WS2812-4020-dual-7mm_bezMaske
- POS10: renamed from POS4; footprint (none) -> FieldBoard_footprint:WS2812-4020-dual-7mm_bezMaske
- POS11: renamed from POS6; footprint (none) -> FieldBoard_footprint:WS2812-4020-dual-7mm_bezMaske
- POS12: renamed from POS8; footprint (none) -> FieldBoard_footprint:WS2812-4020-dual-7mm_bezMaske
- POS13: renamed from POS10; footprint (none) -> FieldBoard_footprint:WS2812-4020-dual-7mm_bezMaske
- POS14: renamed from POS12; footprint (none) -> FieldBoard_footprint:WS2812-4020-dual-7mm_bezMaske
- POS15: renamed from POS14; footprint (none) -> FieldBoard_footprint:WS2812-4020-dual-7mm_bezMaske
- POS2: renamed from POS3; footprint (none) -> FieldBoard_footprint:WS2812-4020-dual-7mm_bezMaske
- POS3: renamed from POS5; footprint (none) -> FieldBoard_footprint:WS2812-4020-dual-7mm_bezMaske
- POS4: renamed from POS7; footprint (none) -> FieldBoard_footprint:WS2812-4020-dual-7mm_bezMaske
- POS5: renamed from POS9; footprint (none) -> FieldBoard_footprint:WS2812-4020-dual-7mm_bezMaske
- POS6: renamed from POS11; footprint (none) -> FieldBoard_footprint:WS2812-4020-dual-7mm_bezMaske
- POS7: renamed from POS13; footprint (none) -> FieldBoard_footprint:WS2812-4020-dual-7mm_bezMaske
- POS8: renamed from POS15; footprint (none) -> FieldBoard_footprint:WS2812-4020-dual-7mm_bezMaske
- POS9: renamed from POS2; footprint (none) -> FieldBoard_footprint:WS2812-4020-dual-7mm_bezMaske

Commit message: v2
Parts:
- POS1, POS10, POS11, POS12, POS13, POS14, POS16, POS2, POS3, POS4, POS5, POS6, POS7, POS8, POS9: footprint FieldBoard_footprint:WS2812-4020-dual-7mm_bezMaske -> LED_SMD:LED_WS2812B_PLCC4_5.0x5.0mm_P3.2mm; symbol FieldBoard_symbol:WS2812-4020_dual -> LED:WS2812B
- POS15: value WS2812-4020_dual -> (none); footprint FieldBoard_footprint:WS2812-4020-dual-7mm_bezMaske -> LED_SMD:LED_WS2812B_PLCC4_5.0x5.0mm_P3.2mm; symbol FieldBoard_symbol:WS2812-4020_dual -> LED:WS2812B
Connections:
- net Finish-LEDs: now also POS1.4 (DIN); no longer POS1.1 (DIN)
- net GND: now also POS1.3 (VSS), POS10.3 (VSS), POS11.3 (VSS), POS12.3 (VSS), POS13.3 (VSS), POS14.3 (VSS), POS15.3 (VSS), POS16.3 (VSS), POS2.3 (VSS), POS3.3 (VSS), POS4.3 (VSS), POS5.3 (VSS), POS6.3 (VSS), POS7.3 (VSS), POS8.3 (VSS), POS9.3 (VSS); no longer POS1.4 (VSS), POS10.4 (VSS), POS11.4 (VSS), POS12.4 (VSS), POS13.4 (VSS), POS14.4 (VSS), POS15.4 (VSS), POS16.4 (VSS), POS2.4 (VSS), POS3.4 (VSS), POS4.4 (VSS), POS5.4 (VSS), POS6.4 (VSS), POS7.4 (VSS), POS8.4 (VSS), POS9.4 (VSS)
- net VDD: now also POS1.1 (VDD), POS10.1 (VDD), POS11.1 (VDD), POS12.1 (VDD), POS13.1 (VDD), POS14.1 (VDD), POS15.1 (VDD), POS16.1 (VDD), POS2.1 (VDD), POS3.1 (VDD), POS4.1 (VDD), POS5.1 (VDD), POS6.1 (VDD), POS7.1 (VDD), POS8.1 (VDD), POS9.1 (VDD); no longer POS1.2 (VDD), POS10.2 (VDD), POS11.2 (VDD), POS12.2 (VDD), POS13.2 (VDD), POS14.2 (VDD), POS15.2 (VDD), POS16.2 (VDD), POS2.2 (VDD), POS3.2 (VDD), POS4.2 (VDD), POS5.2 (VDD), POS6.2 (VDD), POS7.2 (VDD), POS8.2 (VDD), POS9.2 (VDD)
- new net: POS13.2 (DOUT), POS14.4 (DIN)
- new net: POS12.2 (DOUT), POS13.4 (DIN)
- new net: POS7.2 (DOUT), POS8.4 (DIN)
- new net: POS6.2 (DOUT), POS7.4 (DIN)
- new net: POS2.2 (DOUT), POS3.4 (DIN)
- new net: POS1.2 (DOUT), POS2.4 (DIN)
- new net: POS8.2 (DOUT), POS9.4 (DIN)
- new net: POS10.2 (DOUT), POS11.4 (DIN)
- new net: POS10.4 (DIN), POS9.2 (DOUT)
- new net: POS15.2 (DOUT), POS16.4 (DIN)
- new net: POS14.2 (DOUT), POS15.4 (DIN)
- new net: POS11.2 (DOUT), POS12.4 (DIN)
- new net: POS5.2 (DOUT), POS6.4 (DIN)
- new net: POS4.2 (DOUT), POS5.4 (DIN)
- new net: POS3.2 (DOUT), POS4.4 (DIN)

Commit message: update
Parts:
- FIN15: renamed from POS15; value (none) -> WS2812-4020_dual
- renumbered POS1 to FIN1, POS10 to FIN10, POS11 to FIN11, POS12 to FIN12, POS13 to FIN13, POS14 to FIN14, POS16 to FIN16, POS2 to FIN2, POS3 to FIN3, POS4 to FIN4, POS5 to FIN5, POS6 to FIN6, POS7 to FIN7, POS8 to FIN8, POS9 to FIN9
Changed lines of the file:
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@@
   (symbol (lib_id "LED:WS2812B") (at 155.575 97.79 0) (unit 1)
     (in_bom yes) (on_board yes)
-    (property "Reference" "POS13" (id 0) (at 150.495 90.17 0))
+    (property "Reference" "FIN13" (id 0) (at 150.495 90.17 0))
     (property "Value" "WS2812-4020_dual" (id 1) (at 165.735 105.41 0)
       (effects (font (size 1.27 1.27)) hide)
@@
   (symbol (lib_id "LED:WS2812B") (at 196.215 66.675 0) (unit 1)
     (in_bom yes) (on_board yes)
-    (property "Reference" "POS7" (id 0) (at 191.135 59.055 0))
+    (property "Reference" "FIN7" (id 0) (at 191.135 59.055 0))
     (property "Value" "WS2812-4020_dual" (id 1) (at 206.375 74.295 0)
       (effects (font (size 1.27 1.27)) hide)
@@
   (symbol (lib_id "LED:WS2812B") (at 94.615 66.675 0) (unit 1)
     (in_bom yes) (on_board yes)
-    (property "Reference" "POS2" (id 0) (at 89.535 59.055 0))
+    (property "Reference" "FIN2" (id 0) (at 89.535 59.055 0))
     (property "Value" "WS2812-4020_dual" (id 1) (at 104.775 74.295 0)
       (effects (font (size 1.27 1.27)) hide)
@@
   (symbol (lib_id "LED:WS2812B") (at 216.535 66.675 0) (unit 1)
     (in_bom yes) (on_board yes)
-    (property "Reference" "POS8" (id 0) (at 211.455 59.055 0))
+    (property "Reference" "FIN8" (id 0) (at 211.455 59.055 0))
     (property "Value" "WS2812-4020_dual" (id 1) (at 226.695 74.295 0)
       (effects (font (size 1.27 1.27)) hide)
@@
   (symbol (lib_id "LED:WS2812B") (at 94.615 97.79 0) (unit 1)
     (in_bom yes) (on_board yes)
-    (property "Reference" "POS10" (id 0) (at 89.535 90.17 0))
+    (property "Reference" "FIN10" (id 0) (at 89.535 90.17 0))
     (property "Value" "WS2812-4020_dual" (id 1) (at 104.775 105.41 0)
       (effects (font (size 1.27 1.27)) hide)
@@
   (symbol (lib_id "LED:WS2812B") (at 216.535 97.79 0) (unit 1)
     (in_bom yes) (on_board yes)
-    (property "Reference" "POS16" (id 0) (at 211.455 90.17 0))
+    (property "Reference" "FIN16" (id 0) (at 211.455 90.17 0))
     (property "Value" "WS2812-4020_dual" (id 1) (at 226.695 105.41 0)
       (effects (font (size 1.27 1.27)) hide)
@@
   (symbol (lib_id "LED:WS2812B") (at 196.215 97.79 0) (unit 1)
     (in_bom yes) (on_board yes)
-    (property "Reference" "POS15" (id 0) (at 191.135 90.17 0))
-    (property "Value" "" (id 1) (at 206.375 105.41 0)
+    (property "Reference" "FIN15" (id 0) (at 191.135 90.17 0))
+    (property "Value" "WS2812-4020_dual" (id 1) (at 206.375 105.41 0)
       (effects (font (size 1.27 1.27)) hide)
     )
@@
   (symbol (lib_id "LED:WS2812B") (at 135.255 97.79 0) (unit 1)
     (in_bom yes) (on_board yes)
-    (property "Reference" "POS12" (id 0) (at 130.175 90.17 0))
+    (property "Reference" "FIN12" (id 0) (at 130.175 90.17 0))
     (property "Value" "WS2812-4020_dual" (id 1) (at 145.415 105.41 0)
       (effects (font (size 1.27 1.27)) hide)
@@
   (symbol (lib_id "LED:WS2812B") (at 114.935 97.79 0) (unit 1)
     (in_bom yes) (on_board yes)
-    (property "Reference" "POS11" (id 0) (at 109.855 90.17 0))
+    (property "Reference" "FIN11" (id 0) (at 109.855 90.17 0))
     (property "Value" "WS2812-4020_dual" (id 1) (at 125.095 105.41 0)
       (effects (font (size 1.27 1.27)) hide)
@@
   (symbol (lib_id "LED:WS2812B") (at 74.295 97.79 0) (unit 1)
     (in_bom yes) (on_board yes)
-    (property "Reference" "POS9" (id 0) (at 69.215 90.17 0))
+    (property "Reference" "FIN9" (id 0) (at 69.215 90.17 0))
     (property "Value" "WS2812-4020_dual" (id 1) (at 84.455 105.41 0)
       (effects (font (size 1.27 1.27)) hide)
@@
   (symbol (lib_id "LED:WS2812B") (at 155.575 66.675 0) (unit 1)
     (in_bom yes) (on_board yes)
-    (property "Reference" "POS5" (id 0) (at 150.495 59.055 0))
+    (property "Reference" "FIN5" (id 0) (at 150.495 59.055 0))
     (property "Value" "WS2812-4020_dual" (id 1) (at 165.735 74.295 0)
       (effects (font (size 1.27 1.27)) hide)
@@
   (symbol (lib_id "LED:WS2812B") (at 74.295 66.675 0) (unit 1)
     (in_bom yes) (on_board yes)
-    (property "Reference" "POS1" (id 0) (at 69.215 59.055 0))
+    (property "Reference" "FIN1" (id 0) (at 69.215 59.055 0))
     (property "Value" "WS2812-4020_dual" (id 1) (at 84.455 74.295 0)
       (effects (font (size 1.27 1.27)) hide)
@@
   (symbol (lib_id "LED:WS2812B") (at 135.255 66.675 0) (unit 1)
     (in_bom yes) (on_board yes)
-    (property "Reference" "POS4" (id 0) (at 130.175 59.055 0))
+    (property "Reference" "FIN4" (id 0) (at 130.175 59.055 0))
     (property "Value" "WS2812-4020_dual" (id 1) (at 145.415 74.295 0)
       (effects (font (size 1.27 1.27)) hide)
@@
   (symbol (lib_id "LED:WS2812B") (at 175.895 97.79 0) (unit 1)
     (in_bom yes) (on_board yes)
-    (property "Reference" "POS14" (id 0) (at 170.815 90.17 0))
+    (property "Reference" "FIN14" (id 0) (at 170.815 90.17 0))
     (property "Value" "WS2812-4020_dual" (id 1) (at 186.055 105.41 0)
       (effects (font (size 1.27 1.27)) hide)
@@
   (symbol (lib_id "LED:WS2812B") (at 114.935 66.675 0) (unit 1)
     (in_bom yes) (on_board yes)
-    (property "Reference" "POS3" (id 0) (at 109.855 59.055 0))
+    (property "Reference" "FIN3" (id 0) (at 109.855 59.055 0))
     (property "Value" "WS2812-4020_dual" (id 1) (at 125.095 74.295 0)
       (effects (font (size 1.27 1.27)) hide)
@@
   (symbol (lib_id "LED:WS2812B") (at 175.895 66.675 0) (unit 1)
     (in_bom yes) (on_board yes)
-    (property "Reference" "POS6" (id 0) (at 170.815 59.055 0))
+    (property "Reference" "FIN6" (id 0) (at 170.815 59.055 0))
     (property "Value" "WS2812-4020_dual" (id 1) (at 186.055 74.295 0)
       (effects (font (size 1.27 1.27)) hide)

Commit message: update
Parts:
- FIN1, FIN10, FIN11, FIN12, FIN13, FIN14, FIN15, FIN16, FIN2, FIN3, FIN4, FIN5, FIN6, FIN7, FIN8, FIN9: footprint LED_SMD:LED_WS2812B_PLCC4_5.0x5.0mm_P3.2mm -> FieldBoard_footprint:LED_WS2812B_PLCC4_5.0x5.0mm_P3.2mm
Changed lines of the file:
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@@
       (effects (font (size 1.27 1.27)) hide)
     )
-    (property "Footprint" "LED_SMD:LED_WS2812B_PLCC4_5.0x5.0mm_P3.2mm" (id 2) (at 156.845 105.41 0)
+    (property "Footprint" "FieldBoard_footprint:LED_WS2812B_PLCC4_5.0x5.0mm_P3.2mm" (id 2) (at 156.845 105.41 0)
       (effects (font (size 1.27 1.27)) (justify left top) hide)
     )
@@
       (effects (font (size 1.27 1.27)) hide)
     )
-    (property "Footprint" "LED_SMD:LED_WS2812B_PLCC4_5.0x5.0mm_P3.2mm" (id 2) (at 197.485 74.295 0)
+    (property "Footprint" "FieldBoard_footprint:LED_WS2812B_PLCC4_5.0x5.0mm_P3.2mm" (id 2) (at 197.485 74.295 0)
       (effects (font (size 1.27 1.27)) (justify left top) hide)
     )
@@
       (effects (font (size 1.27 1.27)) hide)
     )
-    (property "Footprint" "LED_SMD:LED_WS2812B_PLCC4_5.0x5.0mm_P3.2mm" (id 2) (at 95.885 74.295 0)
+    (property "Footprint" "FieldBoard_footprint:LED_WS2812B_PLCC4_5.0x5.0mm_P3.2mm" (id 2) (at 95.885 74.295 0)
       (effects (font (size 1.27 1.27)) (justify left top) hide)
     )
@@
       (effects (font (size 1.27 1.27)) hide)
     )
-    (property "Footprint" "LED_SMD:LED_WS2812B_PLCC4_5.0x5.0mm_P3.2mm" (id 2) (at 217.805 74.295 0)
+    (property "Footprint" "FieldBoard_footprint:LED_WS2812B_PLCC4_5.0x5.0mm_P3.2mm" (id 2) (at 217.805 74.295 0)
       (effects (font (size 1.27 1.27)) (justify left top) hide)
     )
@@
       (effects (font (size 1.27 1.27)) hide)
     )
-    (property "Footprint" "LED_SMD:LED_WS2812B_PLCC4_5.0x5.0mm_P3.2mm" (id 2) (at 95.885 105.41 0)
+    (property "Footprint" "FieldBoard_footprint:LED_WS2812B_PLCC4_5.0x5.0mm_P3.2mm" (id 2) (at 95.885 105.41 0)
       (effects (font (size 1.27 1.27)) (justify left top) hide)
     )
@@
       (effects (font (size 1.27 1.27)) hide)
     )
-    (property "Footprint" "LED_SMD:LED_WS2812B_PLCC4_5.0x5.0mm_P3.2mm" (id 2) (at 217.805 105.41 0)
+    (property "Footprint" "FieldBoard_footprint:LED_WS2812B_PLCC4_5.0x5.0mm_P3.2mm" (id 2) (at 217.805 105.41 0)
       (effects (font (size 1.27 1.27)) (justify left top) hide)
     )
@@
       (effects (font (size 1.27 1.27)) hide)
     )
-    (property "Footprint" "LED_SMD:LED_WS2812B_PLCC4_5.0x5.0mm_P3.2mm" (id 2) (at 197.485 105.41 0)
+    (property "Footprint" "FieldBoard_footprint:LED_WS2812B_PLCC4_5.0x5.0mm_P3.2mm" (id 2) (at 197.485 105.41 0)
       (effects (font (size 1.27 1.27)) (justify left top) hide)
     )
@@
       (effects (font (size 1.27 1.27)) hide)
     )
-    (property "Footprint" "LED_SMD:LED_WS2812B_PLCC4_5.0x5.0mm_P3.2mm" (id 2) (at 136.525 105.41 0)
+    (property "Footprint" "FieldBoard_footprint:LED_WS2812B_PLCC4_5.0x5.0mm_P3.2mm" (id 2) (at 136.525 105.41 0)
       (effects (font (size 1.27 1.27)) (justify left top) hide)
     )
@@
       (effects (font (size 1.27 1.27)) hide)
     )
-    (property "Footprint" "LED_SMD:LED_WS2812B_PLCC4_5.0x5.0mm_P3.2mm" (id 2) (at 116.205 105.41 0)
+    (property "Footprint" "FieldBoard_footprint:LED_WS2812B_PLCC4_5.0x5.0mm_P3.2mm" (id 2) (at 116.205 105.41 0)
       (effects (font (size 1.27 1.27)) (justify left top) hide)
     )
@@
       (effects (font (size 1.27 1.27)) hide)
     )
-    (property "Footprint" "LED_SMD:LED_WS2812B_PLCC4_5.0x5.0mm_P3.2mm" (id 2) (at 75.565 105.41 0)
+    (property "Footprint" "FieldBoard_footprint:LED_WS2812B_PLCC4_5.0x5.0mm_P3.2mm" (id 2) (at 75.565 105.41 0)
       (effects (font (size 1.27 1.27)) (justify left top) hide)
     )
@@
       (effects (font (size 1.27 1.27)) hide)
     )
-    (property "Footprint" "LED_SMD:LED_WS2812B_PLCC4_5.0x5.0mm_P3.2mm" (id 2) (at 156.845 74.295 0)
+    (property "Footprint" "FieldBoard_footprint:LED_WS2812B_PLCC4_5.0x5.0mm_P3.2mm" (id 2) (at 156.845 74.295 0)
       (effects (font (size 1.27 1.27)) (justify left top) hide)
     )
@@
       (effects (font (size 1.27 1.27)) hide)
     )
-    (property "Footprint" "LED_SMD:LED_WS2812B_PLCC4_5.0x5.0mm_P3.2mm" (id 2) (at 75.565 74.295 0)
+    (property "Footprint" "FieldBoard_footprint:LED_WS2812B_PLCC4_5.0x5.0mm_P3.2mm" (id 2) (at 75.565 74.295 0)
       (effects (font (size 1.27 1.27)) (justify left top) hide)
     )
@@
       (effects (font (size 1.27 1.27)) hide)
     )
-    (property "Footprint" "LED_SMD:LED_WS2812B_PLCC4_5.0x5.0mm_P3.2mm" (id 2) (at 136.525 74.295 0)
+    (property "Footprint" "FieldBoard_footprint:LED_WS2812B_PLCC4_5.0x5.0mm_P3.2mm" (id 2) (at 136.525 74.295 0)
       (effects (font (size 1.27 1.27)) (justify left top) hide)
     )
@@
       (effects (font (size 1.27 1.27)) hide)
     )
-    (property "Footprint" "LED_SMD:LED_WS2812B_PLCC4_5.0x5.0mm_P3.2mm" (id 2) (at 177.165 105.41 0)
+    (property "Footprint" "FieldBoard_footprint:LED_WS2812B_PLCC4_5.0x5.0mm_P3.2mm" (id 2) (at 177.165 105.41 0)
       (effects (font (size 1.27 1.27)) (justify left top) hide)
     )
@@
       (effects (font (size 1.27 1.27)) hide)
     )
-    (property "Footprint" "LED_SMD:LED_WS2812B_PLCC4_5.0x5.0mm_P3.2mm" (id 2) (at 116.205 74.295 0)
+    (property "Footprint" "FieldBoard_footprint:LED_WS2812B_PLCC4_5.0x5.0mm_P3.2mm" (id 2) (at 116.205 74.295 0)
       (effects (font (size 1.27 1.27)) (justify left top) hide)
     )
@@
       (effects (font (size 1.27 1.27)) hide)
     )
-    (property "Footprint" "LED_SMD:LED_WS2812B_PLCC4_5.0x5.0mm_P3.2mm" (id 2) (at 177.165 74.295 0)
-      (effects (font (size 1.27 1.27)) (justify left top) hide)
-    )
+    (property "Footprint" "FieldBoard_footprint:LED_WS2812B_PLCC4_5.0x5.0mm_P3.2mm" (id 2) (at 177.165 74.295 0)
+      (effects (font (size 1.27 1.27)) (justify left top) hide)
+    )
