File: KiCad files/FieldBoard/Positions.kicad_sch (KiCad schematic)
At the start: 52 parts

Commit message: update
Parts:
- POS33, POS82, POS83, POS84: footprint (none) -> FieldBoard_footprint:WS2812-4020-dual-7mm_bezMaske
- POS34: renamed from POS38; footprint (none) -> FieldBoard_footprint:WS2812-4020-dual-7mm_bezMaske
- POS35: renamed from POS43; footprint (none) -> FieldBoard_footprint:WS2812-4020-dual-7mm_bezMaske
- POS36: renamed from POS48; footprint (none) -> FieldBoard_footprint:WS2812-4020-dual-7mm_bezMaske
- POS37: renamed from POS53; footprint (none) -> FieldBoard_footprint:WS2812-4020-dual-7mm_bezMaske
- POS38: renamed from POS58; footprint (none) -> FieldBoard_footprint:WS2812-4020-dual-7mm_bezMaske
- POS39: renamed from POS63; footprint (none) -> FieldBoard_footprint:WS2812-4020-dual-7mm_bezMaske
- POS40: renamed from POS68; footprint (none) -> FieldBoard_footprint:WS2812-4020-dual-7mm_bezMaske
- POS41: renamed from POS73; footprint (none) -> FieldBoard_footprint:WS2812-4020-dual-7mm_bezMaske
- POS42: renamed from POS78; footprint (none) -> FieldBoard_footprint:WS2812-4020-dual-7mm_bezMaske
- POS43: renamed from POS34; footprint (none) -> FieldBoard_footprint:WS2812-4020-dual-7mm_bezMaske
- POS44: renamed from POS39; footprint (none) -> FieldBoard_footprint:WS2812-4020-dual-7mm_bezMaske
- POS45: renamed from POS44; footprint (none) -> FieldBoard_footprint:WS2812-4020-dual-7mm_bezMaske
- POS46: renamed from POS49; footprint (none) -> FieldBoard_footprint:WS2812-4020-dual-7mm_bezMaske
- POS47: renamed from POS54; footprint (none) -> FieldBoard_footprint:WS2812-4020-dual-7mm_bezMaske
- POS48: renamed from POS59; footprint (none) -> FieldBoard_footprint:WS2812-4020-dual-7mm_bezMaske
- POS49: renamed from POS64; footprint (none) -> FieldBoard_footprint:WS2812-4020-dual-7mm_bezMaske
- POS50: renamed from POS69; footprint (none) -> FieldBoard_footprint:WS2812-4020-dual-7mm_bezMaske
- POS51: renamed from POS74; footprint (none) -> FieldBoard_footprint:WS2812-4020-dual-7mm_bezMaske
- POS52: renamed from POS79; footprint (none) -> FieldBoard_footprint:WS2812-4020-dual-7mm_bezMaske
- POS53: renamed from POS35; footprint (none) -> FieldBoard_footprint:WS2812-4020-dual-7mm_bezMaske
- POS54: renamed from POS40; footprint (none) -> FieldBoard_footprint:WS2812-4020-dual-7mm_bezMaske
- POS55: renamed from POS45; footprint (none) -> FieldBoard_footprint:WS2812-4020-dual-7mm_bezMaske
- POS56: renamed from POS50; footprint (none) -> FieldBoard_footprint:WS2812-4020-dual-7mm_bezMaske
- POS57: renamed from POS55; footprint (none) -> FieldBoard_footprint:WS2812-4020-dual-7mm_bezMaske
- POS58: renamed from POS60; footprint (none) -> FieldBoard_footprint:WS2812-4020-dual-7mm_bezMaske
- POS59: renamed from POS65; footprint (none) -> FieldBoard_footprint:WS2812-4020-dual-7mm_bezMaske
- POS60: renamed from POS70; footprint (none) -> FieldBoard_footprint:WS2812-4020-dual-7mm_bezMaske
- POS61: renamed from POS75; footprint (none) -> FieldBoard_footprint:WS2812-4020-dual-7mm_bezMaske
- POS62: renamed from POS80; footprint (none) -> FieldBoard_footprint:WS2812-4020-dual-7mm_bezMaske
- POS63: renamed from POS36; footprint (none) -> FieldBoard_footprint:WS2812-4020-dual-7mm_bezMaske
- POS64: renamed from POS41; footprint (none) -> FieldBoard_footprint:WS2812-4020-dual-7mm_bezMaske
- POS65: renamed from POS46; footprint (none) -> FieldBoard_footprint:WS2812-4020-dual-7mm_bezMaske
- POS66: renamed from POS51; footprint (none) -> FieldBoard_footprint:WS2812-4020-dual-7mm_bezMaske
- POS67: renamed from POS56; footprint (none) -> FieldBoard_footprint:WS2812-4020-dual-7mm_bezMaske
- POS68: renamed from POS61; footprint (none) -> FieldBoard_footprint:WS2812-4020-dual-7mm_bezMaske
- POS69: renamed from POS66; footprint (none) -> FieldBoard_footprint:WS2812-4020-dual-7mm_bezMaske
- POS70: renamed from POS71; footprint (none) -> FieldBoard_footprint:WS2812-4020-dual-7mm_bezMaske
- POS71: renamed from POS76; footprint (none) -> FieldBoard_footprint:WS2812-4020-dual-7mm_bezMaske
- POS72: renamed from POS81; footprint (none) -> FieldBoard_footprint:WS2812-4020-dual-7mm_bezMaske
- POS73: renamed from POS37; footprint (none) -> FieldBoard_footprint:WS2812-4020-dual-7mm_bezMaske
- POS74: renamed from POS42; footprint (none) -> FieldBoard_footprint:WS2812-4020-dual-7mm_bezMaske
- POS75: renamed from POS47; footprint (none) -> FieldBoard_footprint:WS2812-4020-dual-7mm_bezMaske
- POS76: renamed from POS52; footprint (none) -> FieldBoard_footprint:WS2812-4020-dual-7mm_bezMaske
- POS77: renamed from POS57; footprint (none) -> FieldBoard_footprint:WS2812-4020-dual-7mm_bezMaske
- POS78: renamed from POS62; footprint (none) -> FieldBoard_footprint:WS2812-4020-dual-7mm_bezMaske
- POS79: renamed from POS67; footprint (none) -> FieldBoard_footprint:WS2812-4020-dual-7mm_bezMaske
- POS80: renamed from POS72; footprint (none) -> FieldBoard_footprint:WS2812-4020-dual-7mm_bezMaske
- POS81: renamed from POS77; footprint (none) -> FieldBoard_footprint:WS2812-4020-dual-7mm_bezMaske

Commit message: v2
Parts:
- POS33, POS34, POS35, POS36, POS37, POS38, POS39, POS40, POS41, POS42, POS43, POS44, POS45, POS46, POS47, POS48, POS49, POS50, POS51, POS52, POS53, POS54, POS55, POS56, POS57, POS58, POS59, POS60, POS61, POS62, POS63, POS64, POS65, POS66, POS67, POS68, POS69, POS70, POS71, POS72, POS73, POS74, POS75, POS76, POS77, POS78, POS79, POS80, POS81, POS82, POS83, POS84: footprint FieldBoard_footprint:WS2812-4020-dual-7mm_bezMaske -> LED_SMD:LED_WS2812B_PLCC4_5.0x5.0mm_P3.2mm; symbol FieldBoard_symbol:WS2812-4020_dual -> LED:WS2812B
Connections:
- net GND: now also POS33.3 (VSS), POS34.3 (VSS), POS35.3 (VSS), POS36.3 (VSS), POS37.3 (VSS), POS38.3 (VSS), POS39.3 (VSS), POS40.3 (VSS), POS41.3 (VSS), POS42.3 (VSS), POS43.3 (VSS), POS44.3 (VSS), POS45.3 (VSS), POS46.3 (VSS), POS47.3 (VSS), POS48.3 (VSS), POS49.3 (VSS), POS50.3 (VSS), POS51.3 (VSS), POS52.3 (VSS), POS53.3 (VSS), POS54.3 (VSS), POS55.3 (VSS), POS56.3 (VSS), POS57.3 (VSS), POS58.3 (VSS), POS59.3 (VSS), POS60.3 (VSS), POS61.3 (VSS), POS62.3 (VSS), POS63.3 (VSS), POS64.3 (VSS), POS65.3 (VSS), POS66.3 (VSS), POS67.3 (VSS), POS68.3 (VSS), POS69.3 (VSS), POS70.3 (VSS), POS71.3 (VSS), POS72.3 (VSS), POS73.3 (VSS), POS74.3 (VSS), POS75.3 (VSS), POS76.3 (VSS), POS77.3 (VSS), POS78.3 (VSS), POS79.3 (VSS), POS80.3 (VSS), POS81.3 (VSS), POS82.3 (VSS), POS83.3 (VSS), POS84.3 (VSS); no longer POS33.4 (VSS), POS34.4 (VSS), POS35.4 (VSS), POS36.4 (VSS), POS37.4 (VSS), POS38.4 (VSS), POS39.4 (VSS), POS40.4 (VSS), POS41.4 (VSS), POS42.4 (VSS), POS43.4 (VSS), POS44.4 (VSS), POS45.4 (VSS), POS46.4 (VSS), POS47.4 (VSS), POS48.4 (VSS), POS49.4 (VSS), POS50.4 (VSS), POS51.4 (VSS), POS52.4 (VSS), POS53.4 (VSS), POS54.4 (VSS), POS55.4 (VSS), POS56.4 (VSS), POS57.4 (VSS), POS58.4 (VSS), POS59.4 (VSS), POS60.4 (VSS), POS61.4 (VSS), POS62.4 (VSS), POS63.4 (VSS), POS64.4 (VSS), POS65.4 (VSS), POS66.4 (VSS), POS67.4 (VSS), POS68.4 (VSS), POS69.4 (VSS), POS70.4 (VSS), POS71.4 (VSS), POS72.4 (VSS), POS73.4 (VSS), POS74.4 (VSS), POS75.4 (VSS), POS76.4 (VSS), POS77.4 (VSS), POS78.4 (VSS), POS79.4 (VSS), POS80.4 (VSS), POS81.4 (VSS), POS82.4 (VSS), POS83.4 (VSS), POS84.4 (VSS)
- net Positions-LEDs: no longer POS33.1 (DIN)
- net VDD: now also POS33.1 (VDD), POS34.1 (VDD), POS35.1 (VDD), POS36.1 (VDD), POS37.1 (VDD), POS38.1 (VDD), POS39.1 (VDD), POS40.1 (VDD), POS41.1 (VDD), POS42.1 (VDD), POS43.1 (VDD), POS44.1 (VDD), POS45.1 (VDD), POS46.1 (VDD), POS47.1 (VDD), POS48.1 (VDD), POS49.1 (VDD), POS50.1 (VDD), POS51.1 (VDD), POS52.1 (VDD), POS53.1 (VDD), POS54.1 (VDD), POS55.1 (VDD), POS56.1 (VDD), POS57.1 (VDD), POS58.1 (VDD), POS59.1 (VDD), POS60.1 (VDD), POS61.1 (VDD), POS62.1 (VDD), POS63.1 (VDD), POS64.1 (VDD), POS65.1 (VDD), POS66.1 (VDD), POS67.1 (VDD), POS68.1 (VDD), POS69.1 (VDD), POS70.1 (VDD), POS71.1 (VDD), POS72.1 (VDD), POS73.1 (VDD), POS74.1 (VDD), POS75.1 (VDD), POS76.1 (VDD), POS77.1 (VDD), POS78.1 (VDD), POS79.1 (VDD), POS80.1 (VDD), POS81.1 (VDD), POS82.1 (VDD), POS83.1 (VDD), POS84.1 (VDD); no longer POS33.2 (VDD), POS34.2 (VDD), POS35.2 (VDD), POS36.2 (VDD), POS37.2 (VDD), POS38.2 (VDD), POS39.2 (VDD), POS40.2 (VDD), POS41.2 (VDD), POS42.2 (VDD), POS43.2 (VDD), POS44.2 (VDD), POS45.2 (VDD), POS46.2 (VDD), POS47.2 (VDD), POS48.2 (VDD), POS49.2 (VDD), POS50.2 (VDD), POS51.2 (VDD), POS52.2 (VDD), POS53.2 (VDD), POS54.2 (VDD), POS55.2 (VDD), POS56.2 (VDD), POS57.2 (VDD), POS58.2 (VDD), POS59.2 (VDD), POS60.2 (VDD), POS61.2 (VDD), POS62.2 (VDD), POS63.2 (VDD), POS64.2 (VDD), POS65.2 (VDD), POS66.2 (VDD), POS67.2 (VDD), POS68.2 (VDD), POS69.2 (VDD), POS70.2 (VDD), POS71.2 (VDD), POS72.2 (VDD), POS73.2 (VDD), POS74.2 (VDD), POS75.2 (VDD), POS76.2 (VDD), POS77.2 (VDD), POS78.2 (VDD), POS79.2 (VDD), POS80.2 (VDD), POS81.2 (VDD), POS82.2 (VDD), POS83.2 (VDD), POS84.2 (VDD)

Commit message: update
Connections:
- net Positions-LEDs: now also POS33.4 (DIN)
- net at POS67.2 (DOUT): now also POS68.4 (DIN)
- net at POS67.4 (DIN): now also POS66.2 (DOUT)
- net at POS47.2 (DOUT): now also POS48.4 (DIN)
- net at POS47.4 (DIN): now also POS46.2 (DOUT)
- net at POS68.2 (DOUT): now also POS69.4 (DIN)
- net at POS61.2 (DOUT): now also POS62.4 (DIN)
- net at POS61.4 (DIN): now also POS60.2 (DOUT)
- net at POS64.2 (DOUT): now also POS65.4 (DIN)
- net at POS64.4 (DIN): now also POS63.2 (DOUT)
- net at POS72.2 (DOUT): now also POS73.4 (DIN)
- net at POS72.4 (DIN): now also POS71.2 (DOUT)
- net at POS75.2 (DOUT): now also POS76.4 (DIN)
- net at POS75.4 (DIN): now also POS74.2 (DOUT)
- net at POS65.2 (DOUT): now also POS66.4 (DIN)
- net at POS43.2 (DOUT): now also POS44.4 (DIN)
- net at POS43.4 (DIN): now also POS42.2 (DOUT)
- net at POS38.2 (DOUT): now also POS39.4 (DIN)
- net at POS38.4 (DIN): now also POS37.2 (DOUT)
- net at POS57.2 (DOUT): now also POS58.4 (DIN)
- net at POS57.4 (DIN): now also POS56.2 (DOUT)
- net at POS84.4 (DIN): now also POS83.2 (DOUT)
- net at POS81.2 (DOUT): now also POS82.4 (DIN)
- net at POS81.4 (DIN): now also POS80.2 (DOUT)
- net at POS80.4 (DIN): now also POS79.2 (DOUT)
- net at POS76.2 (DOUT): now also POS77.4 (DIN)
- net at POS55.2 (DOUT): now also POS56.4 (DIN)
- net at POS55.4 (DIN): now also POS54.2 (DOUT)
- net at POS78.2 (DOUT): now also POS79.4 (DIN)
- net at POS78.4 (DIN): now also POS77.2 (DOUT)
- net at POS37.4 (DIN): now also POS36.2 (DOUT)
- net at POS34.2 (DOUT): now also POS35.4 (DIN)
- net at POS34.4 (DIN): now also POS33.2 (DOUT)
- net at POS39.2 (DOUT): now also POS40.4 (DIN)
- net at POS44.2 (DOUT): now also POS45.4 (DIN)
- net at POS51.2 (DOUT): now also POS52.4 (DIN)
- net at POS51.4 (DIN): now also POS50.2 (DOUT)
- net at POS73.2 (DOUT): now also POS74.4 (DIN)
- net at POS40.2 (DOUT): now also POS41.4 (DIN)
- net at POS58.2 (DOUT): now also POS59.4 (DIN)
- net at POS36.4 (DIN): now also POS35.2 (DOUT)
- net at POS49.2 (DOUT): now also POS50.4 (DIN)
- net at POS49.4 (DIN): now also POS48.2 (DOUT)
- net at POS52.2 (DOUT): now also POS53.4 (DIN)
- net at POS62.2 (DOUT): now also POS63.4 (DIN)
- net at POS41.2 (DOUT): now also POS42.4 (DIN)
- net at POS71.4 (DIN): now also POS70.2 (DOUT)
- net at POS60.4 (DIN): now also POS59.2 (DOUT)
- net at POS45.2 (DOUT): now also POS46.4 (DIN)
- net at POS70.4 (DIN): now also POS69.2 (DOUT)
- net at POS53.2 (DOUT): now also POS54.4 (DIN)
- net at POS83.4 (DIN): now also POS82.2 (DOUT)
Changed lines of the file:
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@@
 (kicad_sch (version 20211123) (generator eeschema)
   (paper "A4")
-  (no_connect (at 283.21 150.495))
+  (no_connect (at 280.67 150.495))
+  (wire (pts (xy 199.39 57.15) (xy 204.47 57.15))
+    (stroke (width 0) (type default) (color 0 0 0 0))
+  )
+  (wire (pts (xy 179.07 57.15) (xy 184.15 57.15))
+    (stroke (width 0) (type default) (color 0 0 0 0))
+  )
+  (wire (pts (xy 199.39 88.265) (xy 204.47 88.265))
+    (stroke (width 0) (type default) (color 0 0 0 0))
+  )
+  (wire (pts (xy 240.03 88.265) (xy 244.475 88.265))
+    (stroke (width 0) (type default) (color 0 0 0 0))
+  )
   (wire (pts (xy 36.83 73.025) (xy 36.83 88.265))
     (stroke (width 0) (type default) (color 0 0 0 0))
   )
+  (wire (pts (xy 179.07 150.495) (xy 184.15 150.495))
+    (stroke (width 0) (type default) (color 0 0 0 0))
+  )
+  (wire (pts (xy 97.79 150.495) (xy 102.87 150.495))
+    (stroke (width 0) (type default) (color 0 0 0 0))
+  )
   (wire (pts (xy 36.83 104.14) (xy 244.475 104.14))
     (stroke (width 0) (type default) (color 0 0 0 0))
   )
-  (wire (pts (xy 36.83 119.38) (xy 39.37 119.38))
+  (wire (pts (xy 36.83 119.38) (xy 41.91 119.38))
+    (stroke (width 0) (type default) (color 0 0 0 0))
+  )
+  (wire (pts (xy 260.35 150.495) (xy 265.43 150.495))
+    (stroke (width 0) (type default) (color 0 0 0 0))
+  )
+  (wire (pts (xy 219.71 57.15) (xy 224.79 57.15))
+    (stroke (width 0) (type default) (color 0 0 0 0))
+  )
+  (wire (pts (xy 97.79 57.15) (xy 102.87 57.15))
+    (stroke (width 0) (type default) (color 0 0 0 0))
+  )
+  (wire (pts (xy 219.71 119.38) (xy 224.79 119.38))
+    (stroke (width 0) (type default) (color 0 0 0 0))
+  )
+  (wire (pts (xy 179.07 119.38) (xy 184.15 119.38))
     (stroke (width 0) (type default) (color 0 0 0 0))
   )
@@
     (stroke (width 0) (type default) (color 0 0 0 0))
   )
-  (wire (pts (xy 242.57 26.035) (xy 244.475 26.035))
-    (stroke (width 0) (type default) (color 0 0 0 0))
-  )
-  (wire (pts (xy 242.57 57.15) (xy 244.475 57.15))
-    (stroke (width 0) (type default) (color 0 0 0 0))
-  )
-  (wire (pts (xy 29.845 26.035) (xy 39.37 26.035))
+  (wire (pts (xy 77.47 150.495) (xy 82.55 150.495))
+    (stroke (width 0) (type default) (color 0 0 0 0))
+  )
+  (wire (pts (xy 138.43 57.15) (xy 143.51 57.15))
+    (stroke (width 0) (type default) (color 0 0 0 0))
+  )
+  (wire (pts (xy 158.75 150.495) (xy 163.83 150.495))
+    (stroke (width 0) (type default) (color 0 0 0 0))
+  )
+  (wire (pts (xy 219.71 26.035) (xy 224.79 26.035))
+    (stroke (width 0) (type default) (color 0 0 0 0))
+  )
+  (wire (pts (xy 240.03 26.035) (xy 244.475 26.035))
+    (stroke (width 0) (type default) (color 0 0 0 0))
+  )
+  (wire (pts (xy 57.15 57.15) (xy 62.23 57.15))
+    (stroke (width 0) (type default) (color 0 0 0 0))
+  )
+  (wire (pts (xy 240.03 57.15) (xy 244.475 57.15))
+    (stroke (width 0) (type default) (color 0 0 0 0))
+  )
+  (wire (pts (xy 179.07 88.265) (xy 184.15 88.265))
+    (stroke (width 0) (type default) (color 0 0 0 0))
+  )
+  (wire (pts (xy 57.15 26.035) (xy 62.23 26.035))
+    (stroke (width 0) (type default) (color 0 0 0 0))
+  )
+  (wire (pts (xy 57.15 88.265) (xy 62.23 88.265))
+    (stroke (width 0) (type default) (color 0 0 0 0))
+  )
+  (wire (pts (xy 29.845 26.035) (xy 41.91 26.035))
     (stroke (width 0) (type default) (color 0 0 0 0))
   )
@@
     (stroke (width 0) (type default) (color 0 0 0 0))
   )
-  (wire (pts (xy 36.83 57.15) (xy 39.37 57.15))
-    (stroke (width 0) (type default) (color 0 0 0 0))
-  )
-  (wire (pts (xy 242.57 119.38) (xy 244.475 119.38))
+  (wire (pts (xy 77.47 57.15) (xy 82.55 57.15))
+    (stroke (width 0) (type default) (color 0 0 0 0))
+  )
+  (wire (pts (xy 138.43 88.265) (xy 143.51 88.265))
+    (stroke (width 0) (type default) (color 0 0 0 0))
+  )
+  (wire (pts (xy 138.43 150.495) (xy 143.51 150.495))
+    (stroke (width 0) (type default) (color 0 0 0 0))
+  )
+  (wire (pts (xy 118.11 26.035) (xy 123.19 26.035))
+    (stroke (width 0) (type default) (color 0 0 0 0))
+  )
+  (wire (pts (xy 36.83 57.15) (xy 41.91 57.15))
+    (stroke (width 0) (type default) (color 0 0 0 0))
+  )
+  (wire (pts (xy 158.75 26.035) (xy 163.83 26.035))
+    (stroke (width 0) (type default) (color 0 0 0 0))
+  )
+  (wire (pts (xy 240.03 119.38) (xy 244.475 119.38))
     (stroke (width 0) (type default) (color 0 0 0 0))
   )
@@
     (stroke (width 0) (type default) (color 0 0 0 0))
   )
+  (wire (pts (xy 118.11 150.495) (xy 123.19 150.495))
+    (stroke (width 0) (type default) (color 0 0 0 0))
+  )
   (wire (pts (xy 244.475 57.15) (xy 244.475 73.025))
     (stroke (width 0) (type default) (color 0 0 0 0))
   )
+  (wire (pts (xy 240.03 150.495) (xy 245.11 150.495))
+    (stroke (width 0) (type default) (color 0 0 0 0))
+  )
+  (wire (pts (xy 158.75 57.15) (xy 163.83 57.15))
+    (stroke (width 0) (type default) (color 0 0 0 0))
+  )
+  (wire (pts (xy 158.75 119.38) (xy 163.83 119.38))
+    (stroke (width 0) (type default) (color 0 0 0 0))
+  )
+  (wire (pts (xy 199.39 119.38) (xy 204.47 119.38))
+    (stroke (width 0) (type default) (color 0 0 0 0))
+  )
+  (wire (pts (xy 219.71 88.265) (xy 224.79 88.265))
+    (stroke (width 0) (type default) (color 0 0 0 0))
+  )
+  (wire (pts (xy 179.07 26.035) (xy 184.15 26.035))
+    (stroke (width 0) (type default) (color 0 0 0 0))
+  )
+  (wire (pts (xy 57.15 119.38) (xy 62.23 119.38))
+    (stroke (width 0) (type default) (color 0 0 0 0))
+  )
+  (wire (pts (xy 77.47 88.265) (xy 82.55 88.265))
+    (stroke (width 0) (type default) (color 0 0 0 0))
+  )
+  (wire (pts (xy 118.11 119.38) (xy 123.19 119.38))
+    (stroke (width 0) (type default) (color 0 0 0 0))
+  )
+  (wire (pts (xy 118.11 57.15) (xy 123.19 57.15))
+    (stroke (width 0) (type default) (color 0 0 0 0))
+  )
+  (wire (pts (xy 77.47 119.38) (xy 82.55 119.38))
+    (stroke (width 0) (type default) (color 0 0 0 0))
+  )
+  (wire (pts (xy 219.71 150.495) (xy 224.79 150.495))
+    (stroke (width 0) (type default) (color 0 0 0 0))
+  )
+  (wire (pts (xy 118.11 88.265) (xy 123.19 88.265))
+    (stroke (width 0) (type default) (color 0 0 0 0))
+  )
+  (wire (pts (xy 138.43 119.38) (xy 143.51 119.38))
+    (stroke (width 0) (type default) (color 0 0 0 0))
+  )
+  (wire (pts (xy 97.79 119.38) (xy 102.87 119.38))
+    (stroke (width 0) (type default) (color 0 0 0 0))
+  )
   (wire (pts (xy 36.83 41.91) (xy 36.83 57.15))
     (stroke (width 0) (type default) (color 0 0 0 0))
@@
     (stroke (width 0) (type default) (color 0 0 0 0))
   )
-  (wire (pts (xy 242.57 88.265) (xy 244.475 88.265))
+  (wire (pts (xy 97.79 88.265) (xy 102.87 88.265))
+    (stroke (width 0) (type default) (color 0 0 0 0))
+  )
+  (wire (pts (xy 57.15 150.495) (xy 62.23 150.495))
+    (stroke (width 0) (type default) (color 0 0 0 0))
+  )
+  (wire (pts (xy 199.39 150.495) (xy 204.47 150.495))
+    (stroke (width 0) (type default) (color 0 0 0 0))
+  )
+  (wire (pts (xy 77.47 26.035) (xy 82.55 26.035))
     (stroke (width 0) (type default) (color 0 0 0 0))
   )
@@
     (stroke (width 0) (type default) (color 0 0 0 0))
   )
+  (wire (pts (xy 97.79 26.035) (xy 102.87 26.035))
+    (stroke (width 0) (type default) (color 0 0 0 0))
+  )
   (wire (pts (xy 244.475 119.38) (xy 244.475 135.255))
     (stroke (width 0) (type default) (color 0 0 0 0))
   )
-  (wire (pts (xy 36.83 88.265) (xy 39.37 88.265))
-    (stroke (width 0) (type default) (color 0 0 0 0))
-  )
-  (wire (pts (xy 36.83 150.495) (xy 39.37 150.495))
+  (wire (pts (xy 199.39 26.035) (xy 204.47 26.035))
+    (stroke (width 0) (type default) (color 0 0 0 0))
+  )
+  (wire (pts (xy 158.75 88.265) (xy 163.83 88.265))
+    (stroke (width 0) (type default) (color 0 0 0 0))
+  )
+  (wire (pts (xy 36.83 88.265) (xy 41.91 88.265))
+    (stroke (width 0) (type default) (color 0 0 0 0))
+  )
+  (wire (pts (xy 36.83 150.495) (xy 41.91 150.495))
     (stroke (width 0) (type default) (color 0 0 0 0))
   )
@@
     (stroke (width 0) (type default) (color 0 0 0 0))
   )
+  (wire (pts (xy 138.43 26.035) (xy 143.51 26.035))
+    (stroke (width 0) (type default) (color 0 0 0 0))
+  )

Commit message: update
Parts:
- POS33, POS34, POS35, POS36, POS37, POS38, POS39, POS40, POS41, POS42, POS43, POS44, POS45, POS46, POS47, POS48, POS49, POS50, POS51, POS52, POS53, POS54, POS55, POS56, POS57, POS58, POS59, POS60, POS61, POS62, POS63, POS64, POS65, POS66, POS67, POS68, POS69, POS70, POS71, POS72, POS73, POS74, POS75, POS76, POS77, POS78, POS79, POS80, POS81, POS82, POS83, POS84: footprint LED_SMD:LED_WS2812B_PLCC4_5.0x5.0mm_P3.2mm -> FieldBoard_footprint:LED_WS2812B_PLCC4_5.0x5.0mm_P3.2mm
