File: KiCad files/FieldBoard/Start.kicad_sch (KiCad schematic)
At the start: 16 parts

Commit message: update
Parts:
- POS17, POS32: footprint (none) -> FieldBoard_footprint:WS2812-4020-dual-7mm_bezMaske
- POS18: renamed from POS19; footprint (none) -> FieldBoard_footprint:WS2812-4020-dual-7mm_bezMaske
- POS19: renamed from POS21; footprint (none) -> FieldBoard_footprint:WS2812-4020-dual-7mm_bezMaske
- POS20: renamed from POS23; footprint (none) -> FieldBoard_footprint:WS2812-4020-dual-7mm_bezMaske
- POS21: renamed from POS25; footprint (none) -> FieldBoard_footprint:WS2812-4020-dual-7mm_bezMaske
- POS22: renamed from POS27; footprint (none) -> FieldBoard_footprint:WS2812-4020-dual-7mm_bezMaske
- POS23: renamed from POS29; footprint (none) -> FieldBoard_footprint:WS2812-4020-dual-7mm_bezMaske
- POS24: renamed from POS31; footprint (none) -> FieldBoard_footprint:WS2812-4020-dual-7mm_bezMaske
- POS25: renamed from POS18; footprint (none) -> FieldBoard_footprint:WS2812-4020-dual-7mm_bezMaske
- POS26: renamed from POS20; footprint (none) -> FieldBoard_footprint:WS2812-4020-dual-7mm_bezMaske
- POS27: renamed from POS22; footprint (none) -> FieldBoard_footprint:WS2812-4020-dual-7mm_bezMaske
- POS28: renamed from POS24; footprint (none) -> FieldBoard_footprint:WS2812-4020-dual-7mm_bezMaske
- POS29: renamed from POS26; footprint (none) -> FieldBoard_footprint:WS2812-4020-dual-7mm_bezMaske
- POS30: renamed from POS28; footprint (none) -> FieldBoard_footprint:WS2812-4020-dual-7mm_bezMaske
- POS31: renamed from POS30; footprint (none) -> FieldBoard_footprint:WS2812-4020-dual-7mm_bezMaske

Commit message: v2
Parts:
- POS17, POS18, POS19, POS20, POS21, POS22, POS23, POS24, POS25, POS26, POS27, POS28, POS29, POS30, POS31, POS32: footprint FieldBoard_footprint:WS2812-4020-dual-7mm_bezMaske -> LED_SMD:LED_WS2812B_PLCC4_5.0x5.0mm_P3.2mm; symbol FieldBoard_symbol:WS2812-4020_dual -> LED:WS2812B
Connections:
- net GND: now also POS17.3 (VSS), POS18.3 (VSS), POS19.3 (VSS), POS20.3 (VSS), POS21.3 (VSS), POS22.3 (VSS), POS23.3 (VSS), POS24.3 (VSS), POS25.3 (VSS), POS26.3 (VSS), POS27.3 (VSS), POS28.3 (VSS), POS29.3 (VSS), POS30.3 (VSS), POS31.3 (VSS), POS32.3 (VSS); no longer POS17.4 (VSS), POS18.4 (VSS), POS19.4 (VSS), POS20.4 (VSS), POS21.4 (VSS), POS22.4 (VSS), POS23.4 (VSS), POS24.4 (VSS), POS25.4 (VSS), POS26.4 (VSS), POS27.4 (VSS), POS28.4 (VSS), POS29.4 (VSS), POS30.4 (VSS), POS31.4 (VSS), POS32.4 (VSS)
- net Start-LEDs: now also POS17.4 (DIN); no longer POS17.1 (DIN)
- net VDD: now also POS17.1 (VDD), POS18.1 (VDD), POS19.1 (VDD), POS20.1 (VDD), POS21.1 (VDD), POS22.1 (VDD), POS23.1 (VDD), POS24.1 (VDD), POS25.1 (VDD), POS26.1 (VDD), POS27.1 (VDD), POS28.1 (VDD), POS29.1 (VDD), POS30.1 (VDD), POS31.1 (VDD), POS32.1 (VDD); no longer POS17.2 (VDD), POS18.2 (VDD), POS19.2 (VDD), POS20.2 (VDD), POS21.2 (VDD), POS22.2 (VDD), POS23.2 (VDD), POS24.2 (VDD), POS25.2 (VDD), POS26.2 (VDD), POS27.2 (VDD), POS28.2 (VDD), POS29.2 (VDD), POS30.2 (VDD), POS31.2 (VDD), POS32.2 (VDD)
- new net: POS20.2 (DOUT), POS21.4 (DIN)
- new net: POS19.2 (DOUT), POS20.4 (DIN)
- new net: POS21.2 (DOUT), POS22.4 (DIN)
- new net: POS23.2 (DOUT), POS24.4 (DIN)
- new net: POS18.2 (DOUT), POS19.4 (DIN)
- new net: POS17.2 (DOUT), POS18.4 (DIN)
- new net: POS22.2 (DOUT), POS23.4 (DIN)

Commit message: update
Connections:
- net at POS31.2 (DOUT): now also POS32.4 (DIN)
- net at POS31.4 (DIN): now also POS30.2 (DOUT)
- net at POS28.2 (DOUT): now also POS29.4 (DIN)
- net at POS28.4 (DIN): now also POS27.2 (DOUT)
- net at POS25.2 (DOUT): now also POS26.4 (DIN)
- net at POS25.4 (DIN): now also POS24.2 (DOUT)
- net at POS27.4 (DIN): now also POS26.2 (DOUT)
- net at POS30.4 (DIN): now also POS29.2 (DOUT)
Changed lines of the file:
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@@
 (kicad_sch (version 20211123) (generator eeschema)
   (paper "A4")
-  (no_connect (at 231.14 104.14))
+  (no_connect (at 228.6 104.14))
+  (wire (pts (xy 187.96 104.14) (xy 193.04 104.14))
+    (stroke (width 0) (type default) (color 0 0 0 0))
+  )
   (wire (pts (xy 127 73.025) (xy 132.08 73.025))
     (stroke (width 0) (type default) (color 0 0 0 0))
@@
     (stroke (width 0) (type default) (color 0 0 0 0))
   )
+  (wire (pts (xy 106.68 104.14) (xy 111.76 104.14))
+    (stroke (width 0) (type default) (color 0 0 0 0))
+  )
   (wire (pts (xy 233.045 73.025) (xy 233.045 88.9))
     (stroke (width 0) (type default) (color 0 0 0 0))
   )
-  (wire (pts (xy 66.04 104.14) (xy 68.58 104.14))
+  (wire (pts (xy 208.28 104.14) (xy 213.36 104.14))
+    (stroke (width 0) (type default) (color 0 0 0 0))
+  )
+  (wire (pts (xy 66.04 104.14) (xy 71.12 104.14))
     (stroke (width 0) (type default) (color 0 0 0 0))
   )
@@
     (stroke (width 0) (type default) (color 0 0 0 0))
   )
-  (wire (pts (xy 231.14 73.025) (xy 233.045 73.025))
+  (wire (pts (xy 228.6 73.025) (xy 233.045 73.025))
+    (stroke (width 0) (type default) (color 0 0 0 0))
+  )
+  (wire (pts (xy 86.36 104.14) (xy 91.44 104.14))
     (stroke (width 0) (type default) (color 0 0 0 0))
   )
   (wire (pts (xy 187.96 73.025) (xy 193.04 73.025))
+    (stroke (width 0) (type default) (color 0 0 0 0))
+  )
+  (wire (pts (xy 167.64 104.14) (xy 172.72 104.14))
+    (stroke (width 0) (type default) (color 0 0 0 0))
+  )
+  (wire (pts (xy 147.32 104.14) (xy 152.4 104.14))
     (stroke (width 0) (type default) (color 0 0 0 0))
   )
@@
     (stroke (width 0) (type default) (color 0 0 0 0))
   )
+  (wire (pts (xy 127 104.14) (xy 132.08 104.14))
+    (stroke (width 0) (type default) (color 0 0 0 0))
+  )

Commit message: update
Parts:
- POS17, POS18, POS19, POS20, POS21, POS22, POS23, POS24, POS25, POS26, POS27, POS28, POS29, POS30, POS31, POS32: footprint LED_SMD:LED_WS2812B_PLCC4_5.0x5.0mm_P3.2mm -> FieldBoard_footprint:LED_WS2812B_PLCC4_5.0x5.0mm_P3.2mm
Changed lines of the file:
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@@
       (effects (font (size 1.27 1.27)) hide)
     )
-    (property "Footprint" "LED_SMD:LED_WS2812B_PLCC4_5.0x5.0mm_P3.2mm" (id 2) (at 201.93 111.76 0)
+    (property "Footprint" "FieldBoard_footprint:LED_WS2812B_PLCC4_5.0x5.0mm_P3.2mm" (id 2) (at 201.93 111.76 0)
       (effects (font (size 1.27 1.27)) (justify left top) hide)
     )
@@
       (effects (font (size 1.27 1.27)) hide)
     )
-    (property "Footprint" "LED_SMD:LED_WS2812B_PLCC4_5.0x5.0mm_P3.2mm" (id 2) (at 222.25 111.76 0)
+    (property "Footprint" "FieldBoard_footprint:LED_WS2812B_PLCC4_5.0x5.0mm_P3.2mm" (id 2) (at 222.25 111.76 0)
       (effects (font (size 1.27 1.27)) (justify left top) hide)
     )
@@
       (effects (font (size 1.27 1.27)) hide)
     )
-    (property "Footprint" "LED_SMD:LED_WS2812B_PLCC4_5.0x5.0mm_P3.2mm" (id 2) (at 140.97 111.76 0)
+    (property "Footprint" "FieldBoard_footprint:LED_WS2812B_PLCC4_5.0x5.0mm_P3.2mm" (id 2) (at 140.97 111.76 0)
       (effects (font (size 1.27 1.27)) (justify left top) hide)
     )
@@
       (effects (font (size 1.27 1.27)) hide)
     )
-    (property "Footprint" "LED_SMD:LED_WS2812B_PLCC4_5.0x5.0mm_P3.2mm" (id 2) (at 140.97 80.645 0)
+    (property "Footprint" "FieldBoard_footprint:LED_WS2812B_PLCC4_5.0x5.0mm_P3.2mm" (id 2) (at 140.97 80.645 0)
       (effects (font (size 1.27 1.27)) (justify left top) hide)
     )
@@
       (effects (font (size 1.27 1.27)) hide)
     )
-    (property "Footprint" "LED_SMD:LED_WS2812B_PLCC4_5.0x5.0mm_P3.2mm" (id 2) (at 161.29 80.645 0)
+    (property "Footprint" "FieldBoard_footprint:LED_WS2812B_PLCC4_5.0x5.0mm_P3.2mm" (id 2) (at 161.29 80.645 0)
       (effects (font (size 1.27 1.27)) (justify left top) hide)
     )
@@
       (effects (font (size 1.27 1.27)) hide)
     )
-    (property "Footprint" "LED_SMD:LED_WS2812B_PLCC4_5.0x5.0mm_P3.2mm" (id 2) (at 80.01 111.76 0)
+    (property "Footprint" "FieldBoard_footprint:LED_WS2812B_PLCC4_5.0x5.0mm_P3.2mm" (id 2) (at 80.01 111.76 0)
       (effects (font (size 1.27 1.27)) (justify left top) hide)
     )
@@
       (effects (font (size 1.27 1.27)) hide)
     )
-    (property "Footprint" "LED_SMD:LED_WS2812B_PLCC4_5.0x5.0mm_P3.2mm" (id 2) (at 222.25 80.645 0)
+    (property "Footprint" "FieldBoard_footprint:LED_WS2812B_PLCC4_5.0x5.0mm_P3.2mm" (id 2) (at 222.25 80.645 0)
       (effects (font (size 1.27 1.27)) (justify left top) hide)
     )
@@
       (effects (font (size 1.27 1.27)) hide)
     )
-    (property "Footprint" "LED_SMD:LED_WS2812B_PLCC4_5.0x5.0mm_P3.2mm" (id 2) (at 120.65 111.76 0)
+    (property "Footprint" "FieldBoard_footprint:LED_WS2812B_PLCC4_5.0x5.0mm_P3.2mm" (id 2) (at 120.65 111.76 0)
       (effects (font (size 1.27 1.27)) (justify left top) hide)
     )
@@
       (effects (font (size 1.27 1.27)) hide)
     )
-    (property "Footprint" "LED_SMD:LED_WS2812B_PLCC4_5.0x5.0mm_P3.2mm" (id 2) (at 100.33 111.76 0)
+    (property "Footprint" "FieldBoard_footprint:LED_WS2812B_PLCC4_5.0x5.0mm_P3.2mm" (id 2) (at 100.33 111.76 0)
       (effects (font (size 1.27 1.27)) (justify left top) hide)
     )
@@
       (effects (font (size 1.27 1.27)) hide)
     )
-    (property "Footprint" "LED_SMD:LED_WS2812B_PLCC4_5.0x5.0mm_P3.2mm" (id 2) (at 100.33 80.645 0)
+    (property "Footprint" "FieldBoard_footprint:LED_WS2812B_PLCC4_5.0x5.0mm_P3.2mm" (id 2) (at 100.33 80.645 0)
       (effects (font (size 1.27 1.27)) (justify left top) hide)
     )
@@
       (effects (font (size 1.27 1.27)) hide)
     )
-    (property "Footprint" "LED_SMD:LED_WS2812B_PLCC4_5.0x5.0mm_P3.2mm" (id 2) (at 80.01 80.645 0)
+    (property "Footprint" "FieldBoard_footprint:LED_WS2812B_PLCC4_5.0x5.0mm_P3.2mm" (id 2) (at 80.01 80.645 0)
       (effects (font (size 1.27 1.27)) (justify left top) hide)
     )
@@
       (effects (font (size 1.27 1.27)) hide)
     )
-    (property "Footprint" "LED_SMD:LED_WS2812B_PLCC4_5.0x5.0mm_P3.2mm" (id 2) (at 181.61 111.76 0)
+    (property "Footprint" "FieldBoard_footprint:LED_WS2812B_PLCC4_5.0x5.0mm_P3.2mm" (id 2) (at 181.61 111.76 0)
       (effects (font (size 1.27 1.27)) (justify left top) hide)
     )
@@
       (effects (font (size 1.27 1.27)) hide)
     )
-    (property "Footprint" "LED_SMD:LED_WS2812B_PLCC4_5.0x5.0mm_P3.2mm" (id 2) (at 201.93 80.645 0)
+    (property "Footprint" "FieldBoard_footprint:LED_WS2812B_PLCC4_5.0x5.0mm_P3.2mm" (id 2) (at 201.93 80.645 0)
       (effects (font (size 1.27 1.27)) (justify left top) hide)
     )
@@
       (effects (font (size 1.27 1.27)) hide)
     )
-    (property "Footprint" "LED_SMD:LED_WS2812B_PLCC4_5.0x5.0mm_P3.2mm" (id 2) (at 181.61 80.645 0)
+    (property "Footprint" "FieldBoard_footprint:LED_WS2812B_PLCC4_5.0x5.0mm_P3.2mm" (id 2) (at 181.61 80.645 0)
       (effects (font (size 1.27 1.27)) (justify left top) hide)
     )
@@
       (effects (font (size 1.27 1.27)) hide)
     )
-    (property "Footprint" "LED_SMD:LED_WS2812B_PLCC4_5.0x5.0mm_P3.2mm" (id 2) (at 161.29 111.76 0)
+    (property "Footprint" "FieldBoard_footprint:LED_WS2812B_PLCC4_5.0x5.0mm_P3.2mm" (id 2) (at 161.29 111.76 0)
       (effects (font (size 1.27 1.27)) (justify left top) hide)
     )
@@
       (effects (font (size 1.27 1.27)) hide)
     )
-    (property "Footprint" "LED_SMD:LED_WS2812B_PLCC4_5.0x5.0mm_P3.2mm" (id 2) (at 120.65 80.645 0)
-      (effects (font (size 1.27 1.27)) (justify left top) hide)
-    )
+    (property "Footprint" "FieldBoard_footprint:LED_WS2812B_PLCC4_5.0x5.0mm_P3.2mm" (id 2) (at 120.65 80.645 0)
+      (effects (font (size 1.27 1.27)) (justify left top) hide)
+    )
