File: KiCad files/Test PCBs/Touchpad/_autosave-Touchpad.kicad_sch (KiCad schematic)
At the start: 45 parts, among them J1 Conn_01x08_Male, J2 Conn_01x03_Male, U2 TTP223-BA6, U3 TTP223-BA6, U5 TTP223-BA6

Commit message: update
Parts:
- removed D2, D3, D5: LED_Small, LED_SMD:LED_0603_1608Metric, symbol Device:LED_Small
- removed H1, H2, H3, H4: MountingHole, MountingHole:MountingHole_3.2mm_M3, symbol Mechanical:MountingHole
- removed R2, R3, R5: 470, Resistor_SMD:R_0603_1608Metric, symbol Device:R_Small
