File: KiCad files/Test PCBs/Touchpad/Touchpad.kicad_sch (KiCad schematic)
At the start: 45 parts, among them J1 Conn_01x08_Male, J2 Conn_01x03_Male, U2 TTP223-BA6, U3 TTP223-BA6, U5 TTP223-BA6

Commit message: update
Parts:
- removed C13, C14, C15, C16, C17, C18, C19, C20, C21, C22: 100n, Capacitor_SMD:C_0603_1608Metric, symbol Device:C_Small
- removed D10, D11, D12, D13, D14, D15, D16, D7, D8, D9: WS2812-4020, Touchpad:WS2812-4020, symbol ws2812-4020:WS2812-4020
- removed D2, D3, D5: LED_Small, LED_SMD:LED_0603_1608Metric, symbol Device:LED_Small
- removed H1, H2, H3, H4: MountingHole, MountingHole:MountingHole_3.2mm_M3, symbol Mechanical:MountingHole
- removed J1: Conn_01x08_Male, Connector_PinHeader_2.54mm:PinHeader_1x08_P2.54mm_Vertical, symbol Connector:Conn_01x08_Male
- removed J2: Conn_01x03_Male, Connector_PinHeader_2.54mm:PinHeader_1x03_P2.54mm_Vertical, symbol Connector:Conn_01x03_Male
- removed R2, R3, R5, R7: 470, Resistor_SMD:R_0603_1608Metric, symbol Device:R_Small
Connections:
- no-connect marks 10 -> 6

Commit message: update
Parts:
- added J1: Conn_02x03_Counter_Clockwise, Connector_PinHeader_1.27mm:PinHeader_2x03_P1.27mm_Vertical_SMD, symbol Connector_Generic:Conn_02x03_Counter_Clockwise
- renumbered C4 to C1, C7 to C2, C11 to C3, C2 to C4, C9 to C6, TP3 to TP1, TP4 to TP2, TP2 to TP3, U2 to U1, U3 to U2, U5 to U3
Connections:
- net +5V: now also J1.5 (Pin_5), J1.6 (Pin_6)
- net GND: now also J1.4 (Pin_4)
- net TP2: now also J1.3 (Pin_3)
- net TP3: now also J1.1 (Pin_1)
- net TP5: now also J1.2 (Pin_2)

Commit message: touchpad_v2
Parts:
- added D1, D2, D3: WS2812B, LED_SMD:LED_WS2812B_PLCC4_5.0x5.0mm_P3.2mm, symbol LED:WS2812B
- added J2: Conn_02x03_Counter_Clockwise, Connector_PinHeader_1.27mm:PinHeader_2x03_P1.27mm_Vertical, symbol Connector_Generic:Conn_02x03_Counter_Clockwise
- added J3: Conn_01x07_Male, Connector_PinHeader_2.54mm:PinHeader_1x07_P2.54mm_Vertical, symbol Connector:Conn_01x07_Male
- renumbered C5 to C1, C6 to C3, C3 to C4, C4 to C5, C1 to C6, TP3 to TP1, TP1 to TP2, TP2 to TP3, U2 to U1, U3 to U2, U1 to U3
Connections:
- net +5V: now also J1.3 (Pin_3), J1.4 (Pin_4), D1.1 (VDD), D2.1 (VDD), D3.1 (VDD), J2.3 (Pin_3), J2.4 (Pin_4), J3.1 (Pin_1); no longer J1.5 (Pin_5), J1.6 (Pin_6)
- net GND: now also J1.6 (Pin_6), D1.3 (VSS), D2.3 (VSS), D3.3 (VSS), J2.6 (Pin_6), J3.7 (Pin_7); no longer J1.4 (Pin_4)
- net TP2: now also J1.1 (Pin_1), U2.1 (Q), J2.1 (Pin_1), J3.4 (Pin_4); no longer J1.3 (Pin_3), U3.1 (Q)
- net TP3: now also J1.2 (Pin_2), U3.1 (Q), J2.2 (Pin_2), J3.5 (Pin_5); no longer J1.1 (Pin_1), U1.1 (Q)
- removed net TP5: J1.2 (Pin_2), U2.1 (Q)
- new net: D3.2 (DOUT), J3.6 (Pin_6)
- new net: D2.2 (DOUT), D3.4 (DIN)
- new net: D1.2 (DOUT), D2.4 (DIN)
- new net: D1.4 (DIN), J3.2 (Pin_2)
- new net TP1: J1.5 (Pin_5), J2.5 (Pin_5), J3.3 (Pin_3), U1.1 (Q)
