File: KiCad files/Test PCBs/Touchpad/Touchpad.kicad_pcb (KiCad board)
At the start: 2 copper layers, 100 x 51.2 mm, 63 parts, among them J1 Conn_01x08_Male, J2 Conn_01x03_Male, U1 TTP223-BA6, U2 TTP223-BA6, U3 TTP223-BA6, U4 TTP223-BA6, U5 TTP223-BA6, U6 TTP223-BA6

Commit message: update
Parts:
- removed C1, C10, C6: 0-50 pF, Capacitor_SMD:C_0603_1608Metric
- removed C12, C13, C14, C15, C16, C17, C18, C19, C20, C21, C22, C3, C8: 100n, Capacitor_SMD:C_0603_1608Metric
- removed D1, D2, D3, D4, D5, D6: LED_Small, LED_SMD:LED_0603_1608Metric
- removed D10, D11, D12, D13, D14, D15, D16, D7, D8, D9: WS2812-4020, Touchpad:WS2812-4020
- removed H1, H2, H3, H4: MountingHole, MountingHole:MountingHole_3.2mm_M3
- removed J1: Conn_01x08_Male, Connector_PinHeader_2.54mm:PinHeader_1x08_P2.54mm_Vertical
- removed J2: Conn_01x03_Male, Connector_PinHeader_2.54mm:PinHeader_1x03_P2.54mm_Vertical
- removed R1, R2, R3, R4, R5, R6, R7: 470, Resistor_SMD:R_0603_1608Metric
- removed TP1: TestPoint, Touchpad:TP_11mm_kocka
- removed TP5: TestPoint, Touchpad:TP_11mm_strelicaGore
- removed TP6: TestPoint, Touchpad:TP_11mm_strelicaDolje
- removed U1, U4, U6: TTP223-BA6, Package_TO_SOT_SMD:SOT-23-6
- C11, C2, C4, C5, C7, C9, U2, U3, U5: moved to B.Cu
- moved C4 88.5 mm to (209.9, 109.4), turned to 180 degrees
- moved TP4 87.5 mm to (217.6, 106.5)
- moved U2 85.1 mm to (209.9, 105.9), turned to -90 degrees
- moved C2 80.6 mm to (209.9, 102.4), turned to 180 degrees
- moved C7 59.0 mm to (191.4, 108.1), turned to 0 degrees
- moved U3 54.0 mm to (191.4, 104.6), turned to -90 degrees
- moved TP2 54.0 mm to (198.9, 106.5)
- moved C5 49.2 mm to (191.4, 101.1), turned to 180 degrees
- moved C11 39.9 mm to (187.7, 108.1), turned to 0 degrees
- moved U5 31.9 mm to (187.7, 104.6), turned to -90 degrees
- moved C9 27.6 mm to (187.7, 101.1), turned to 180 degrees
- moved TP3 17.5 mm to (180.2, 106.5)
Connections:
- U2 pad 4: Net-(U2-Pad4) -> unconnected-(U2-Pad4)
- U2 pad 6: Net-(U2-Pad6) -> unconnected-(U2-Pad6)
- U3 pad 4: Net-(U3-Pad4) -> unconnected-(U3-Pad4)
- U3 pad 6: Net-(U3-Pad6) -> unconnected-(U3-Pad6)
- U5 pad 4: Net-(U5-Pad4) -> unconnected-(U5-Pad4)
- U5 pad 6: Net-(U5-Pad6) -> unconnected-(U5-Pad6)
Routing:
- net VCC: track 218.0 -> 0.00 mm, vias 6 -> 0
- net +5V: track 174.4 -> 8.16 mm, vias 6 -> 0
- net Net-(D11-Pad1): track 118.7 -> 0.00 mm, vias 6 -> 0
- net TP1: track 55.9 -> 0.00 mm
- net TP2: track 42.1 -> 0.00 mm
- net TP6: track 39.2 -> 0.00 mm
- net TP5: track 28.6 -> 0.00 mm
- net TP3: track 28.6 -> 0.00 mm
- net Net-(D14-Pad3): track 24.5 -> 0.00 mm
- net TP4: track 20.3 -> 0.00 mm
- net Net-(D12-Pad3): track 18.0 -> 0.00 mm
- net Net-(D11-Pad3): track 16.7 -> 0.00 mm
- net Net-(D8-Pad3): track 14.0 -> 0.00 mm
- net Net-(D7-Pad3): track 12.8 -> 0.00 mm
- net Net-(D10-Pad1): track 11.7 -> 0.00 mm
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- removed copper zone on F.Cu, net GND
Other:
- board size 100 x 51.2 mm -> 78.2 x 33.2 mm
- board text removed: "gnd"
- board text removed: "in"
- board text removed: "vcc"
- board text removed: "vdd"

Commit message: update
Routing:
- net Net-(C5-Pad1): track 11.0 -> 9.86 mm
- net Net-(C2-Pad1): track 11.8 -> 10.6 mm
- net Net-(C9-Pad1): track 12.6 -> 12.0 mm
Changed lines of the file:
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@@
   (segment (start 209.125 102.4) (end 209.125 103.125) (width 0.3556) (layer "B.Cu") (net 1))
   (segment (start 191.45 103.5) (end 191.45 102.5) (width 0.3556) (layer "B.Cu") (net 1))
-  (segment (start 217.55 99.85) (end 217.55 100.55) (width 0.3556) (layer "F.Cu") (net 2))
-  (via (at 217.55 99.85) (size 0.8) (drill 0.4) (layers "F.Cu" "B.Cu") (net 2))
-  (segment (start 210.675 101.225) (end 210.675 102.4) (width 0.3556) (layer "B.Cu") (net 2))
+  (segment (start 217.55 100.25) (end 217.55 100.55) (width 0.3556) (layer "F.Cu") (net 2))
+  (via (at 217.55 100) (size 0.8) (drill 0.4) (layers "F.Cu" "B.Cu") (net 2))
+  (segment (start 211.9 102.4) (end 210.675 102.4) (width 0.3556) (layer "B.Cu") (net 2))
+  (segment (start 217.55 100) (end 214.3 100) (width 0.3556) (layer "B.Cu") (net 2))
+  (segment (start 214.3 100) (end 211.9 102.4) (width 0.3556) (layer "B.Cu") (net 2))
   (segment (start 210.675 103.475) (end 210.675 102.4) (width 0.3556) (layer "B.Cu") (net 2))
-  (segment (start 217.55 99.85) (end 212.05 99.85) (width 0.3556) (layer "B.Cu") (net 2))
-  (segment (start 212.05 99.85) (end 210.675 101.225) (width 0.3556) (layer "B.Cu") (net 2))
   (segment (start 210.85 104.8) (end 210.85 103.65) (width 0.3556) (layer "B.Cu") (net 2))
   (segment (start 210.85 103.65) (end 210.675 103.475) (width 0.3556) (layer "B.Cu") (net 2))
-  (segment (start 198.9 99.8) (end 198.9 100.5) (width 0.3556) (layer "F.Cu") (net 3))
-  (via (at 198.9 99.8) (size 0.8) (drill 0.4) (layers "F.Cu" "B.Cu") (net 3))
-  (segment (start 198.9 99.8) (end 198.7 99.6) (width 0.3556) (layer "B.Cu") (net 3))
+  (segment (start 196.55 100.15) (end 196.2 100.5) (width 0.3556) (layer "F.Cu") (net 3))
+  (segment (start 198.65 100.15) (end 196.55 100.15) (width 0.3556) (layer "F.Cu") (net 3))
+  (segment (start 198.9 100.61316) (end 198.9 100.4) (width 0.3556) (layer "F.Cu") (net 3))
+  (segment (start 198.9 100.4) (end 198.65 100.15) (width 0.3556) (layer "F.Cu") (net 3))
+  (via (at 196.2 100.5) (size 0.8) (drill 0.4) (layers "F.Cu" "B.Cu") (net 3))
   (segment (start 192.225 101.1) (end 192.225 102.325) (width 0.3556) (layer "B.Cu") (net 3))
-  (segment (start 192.9 99.6) (end 192.225 100.275) (width 0.3556) (layer "B.Cu") (net 3))
   (segment (start 192.225 102.325) (end 192.4 102.5) (width 0.3556) (layer "B.Cu") (net 3))
-  (segment (start 192.225 100.275) (end 192.225 101.1) (width 0.3556) (layer "B.Cu") (net 3))
+  (segment (start 192.225 101.1) (end 195.6 101.1) (width 0.3556) (layer "B.Cu") (net 3))
   (segment (start 192.4 102.5) (end 192.4 103.5) (width 0.3556) (layer "B.Cu") (net 3))
-  (segment (start 198.7 99.6) (end 192.9 99.6) (width 0.3556) (layer "B.Cu") (net 3))
-  (segment (start 180.25 99.8) (end 180.25 100.5) (width 0.3556) (layer "F.Cu") (net 4))
-  (via (at 180.25 99.8) (size 0.8) (drill 0.4) (layers "F.Cu" "B.Cu") (net 4))
-  (segment (start 187.8 99.6) (end 180.5 99.6) (width 0.3556) (layer "B.Cu") (net 4))
+  (segment (start 195.6 101.1) (end 196.2 100.5) (width 0.3556) (layer "B.Cu") (net 3))
+  (segment (start 180.25 100.2) (end 180.25 100.5) (width 0.3556) (layer "F.Cu") (net 4))
+  (via (at 180.25 99.95) (size 0.8) (drill 0.4) (layers "F.Cu" "B.Cu") (net 4))
   (segment (start 188.65 102.45) (end 188.65 103.5) (width 0.3556) (layer "B.Cu") (net 4))
-  (segment (start 180.5 99.6) (end 180.3 99.8) (width 0.3556) (layer "B.Cu") (net 4))
+  (segment (start 180.35 99.85) (end 180.25 99.95) (width 0.3556) (layer "B.Cu") (net 4))
+  (segment (start 188.05 99.85) (end 180.35 99.85) (width 0.3556) (layer "B.Cu") (net 4))
+  (segment (start 188.475 101.1) (end 188.475 100.275) (width 0.3556) (layer "B.Cu") (net 4))
   (segment (start 188.475 102.275) (end 188.65 102.45) (width 0.3556) (layer "B.Cu") (net 4))
+  (segment (start 188.475 100.275) (end 188.05 99.85) (width 0.3556) (layer "B.Cu") (net 4))
   (segment (start 188.475 101.1) (end 188.475 102.275) (width 0.3556) (layer "B.Cu") (net 4))
-  (segment (start 188.475 100.275) (end 187.8 99.6) (width 0.3556) (layer "B.Cu") (net 4))
-  (segment (start 188.475 101.1) (end 188.475 100.275) (width 0.3556) (layer "B.Cu") (net 4))
-  (segment (start 180.3 99.8) (end 180.25 99.8) (width 0.3556) (layer "B.Cu") (net 4))
   (segment (start 187.7 106.7) (end 187.7 105.7) (width 0.3556) (layer "B.Cu") (net 14))
   (segment (start 186.925 107.475) (end 187.7 106.7) (width 0.3556) (layer "B.Cu") (net 14))

Commit message: update
Parts:
- removed TP4: TestPoint, Touchpad:TP_11mm_strelicaDesno
- added J1: Conn_02x03_Counter_Clockwise, Connector_PinHeader_1.27mm:PinHeader_2x03_P1.27mm_Vertical_SMD, B.Cu at (207.3, 111.3)
- added TP2: TestPoint, Touchpad:TP_11mm_strelicaDesno, F.Cu at (217.6, 106.5)
- added mouse-bite-2mm-slot: VAL**, Touchpad:mouse-bite-2mm-slot, F.Cu at (208.2, 97.7)
- added mouse-bite-2mm-slot: VAL**, Touchpad:mouse-bite-2mm-slot, F.Cu at (189.6, 97.7)
- moved C2 1.34 mm to (210.2, 108.1)
- moved C5 1.34 mm to (210.2, 101.1)
- moved U2 1.34 mm to (210.2, 104.6)
- renumbered C11 to C1, C4 to C2, C7 to C3, C9 to C4, C2 to C5, C5 to C6, TP3 to TP1, TP2 to TP3, U5 to U1
Connections:
- C4 pad 1: Net-(C9-Pad1) -> Net-(C4-Pad1)
- C5 pad 1: Net-(C2-Pad1) -> Net-(C5-Pad1)
- C6 pad 1: Net-(C5-Pad1) -> Net-(C6-Pad1)
- TP1 pad 1: Net-(C9-Pad1) -> Net-(C6-Pad1)
- U1 pad 1: TP5 -> TP2
- U1 pad 3: Net-(C9-Pad1) -> Net-(C4-Pad1)
- U2 pad 1: TP2 -> TP3
- U2 pad 3: Net-(C2-Pad1) -> Net-(C5-Pad1)
- U3 pad 1: TP3 -> TP5
- U3 pad 3: Net-(C5-Pad1) -> Net-(C6-Pad1)
Routing:
- net Net-(C4-Pad1): track 0.00 -> 16.1 mm, vias 0 -> 2
- net Net-(C9-Pad1): track 12.0 -> 0.00 mm, vias 1 -> 0
- net +5V: track 8.16 -> 19.1 mm
- net Net-(C2-Pad1): track 10.6 -> 0.00 mm, vias 1 -> 0
- net Net-(C6-Pad1): track 0.00 -> 9.86 mm, vias 0 -> 1
- net TP3: track 0.00 -> 9.48 mm
- net Net-(C5-Pad1): track 9.86 -> 2.47 mm, vias 1 -> 0

Commit message: touchpad_v2
Parts:
- added C1: 0-50 pF, Capacitor_SMD:C_0603_1608Metric, B.Cu at (202.8, 65.2)
- added C2: 100n, Capacitor_SMD:C_0603_1608Metric, B.Cu at (206.8, 69.2)
- added C3: 0-50 pF, Capacitor_SMD:C_0603_1608Metric, B.Cu at (188.7, 66.8)
- added C4: 100n, Capacitor_SMD:C_0603_1608Metric, B.Cu at (188.7, 72.8)
- added C5: 0-50 pF, Capacitor_SMD:C_0603_1608Metric, B.Cu at (213.9, 65.2)
- added C6: 100n, Capacitor_SMD:C_0603_1608Metric, B.Cu at (209.9, 69.2)
- added D1: WS2812B, LED_SMD:LED_WS2812B_PLCC4_5.0x5.0mm_P3.2mm, F.Cu at (180.2, 89.0)
- added D2: WS2812B, LED_SMD:LED_WS2812B_PLCC4_5.0x5.0mm_P3.2mm, F.Cu at (198.9, 89.0)
- added D3: WS2812B, LED_SMD:LED_WS2812B_PLCC4_5.0x5.0mm_P3.2mm, F.Cu at (217.6, 89.0)
- added J1: Conn_02x03_Counter_Clockwise, Connector_PinHeader_1.27mm:PinHeader_2x03_P1.27mm_Vertical_SMD, B.Cu at (208.3, 76.2)
- added J2: Conn_02x03_Counter_Clockwise, Connector_PinHeader_1.27mm:PinHeader_2x03_P1.27mm_Vertical, F.Cu at (207.9, 92.4)
- added J3: Conn_01x07_Male, Connector_PinHeader_2.54mm:PinHeader_1x07_P2.54mm_Vertical, F.Cu at (191.3, 83.2)
- added TP1: TestPoint, Touchpad:TP_11mm_kvacica, F.Cu at (198.7, 71.5)
- added TP2: TestPoint, Touchpad:TP_11mm_strelicaLijevo, F.Cu at (180.1, 71.5)
- added TP3: TestPoint, Touchpad:TP_11mm_strelicaDesno, F.Cu at (217.3, 71.5)
- added U1: TTP223-BA6, Package_TO_SOT_SMD:SOT-23-6, B.Cu at (204.8, 67.2)
- added U2: TTP223-BA6, Package_TO_SOT_SMD:SOT-23-6, B.Cu at (188.7, 69.8)
- added U3: TTP223-BA6, Package_TO_SOT_SMD:SOT-23-6, B.Cu at (211.9, 67.2)
- added mouse-bite-2mm-slot: VAL**, Touchpad:mouse-bite-2mm-slot, F.Cu at (189.4, 80.2)
- added mouse-bite-2mm-slot: VAL**, Touchpad:mouse-bite-2mm-slot, F.Cu at (208.1, 80.2)
- C1, C3: value 100n -> 0-50 pF
- C4, C6: value 0-50 pF -> 100n
- moved U2 21.4 mm to (188.9, 104.8)
- moved U3 20.8 mm to (212.1, 102.2), turned to -135 degrees
- moved C6 18.9 mm to (210.1, 104.2), turned to 135 degrees
- moved U1 17.4 mm to (204.9, 102.2), turned to -45 degrees
- moved C1 17.2 mm to (202.9, 100.2), turned to -135 degrees
- moved C3 6.84 mm to (188.9, 101.8), turned to 180 degrees
- moved C4 6.77 mm to (188.9, 107.8)
- moved C2 5.09 mm to (206.9, 104.2), turned to 45 degrees
- moved C5 3.98 mm to (214.1, 100.2), turned to 135 degrees
- moved J1 1.22 mm to (208.5, 111.2), turned to 0 degrees
- renumbered TP3 to TP1, TP1 to TP2, TP2 to TP3
Connections:
- C1 pad 1: +5V -> Net-(C1-Pad1)
- C3 pad 1: +5V -> Net-(C3-Pad1)
- C4 pad 1: Net-(C4-Pad1) -> +5V
- C6 pad 1: Net-(C6-Pad1) -> +5V
- J1 pad 1: TP3 -> TP2
- J1 pad 2: TP5 -> TP3
- J1 pad 3: TP2 -> +5V
- J1 pad 4: GND -> +5V
- J1 pad 5: +5V -> TP1
- J1 pad 6: +5V -> GND
- TP1 pad 1: Net-(C5-Pad1) -> Net-(C1-Pad1)
- TP2 pad 1: Net-(C6-Pad1) -> Net-(C3-Pad1)
- TP3 pad 1: Net-(C4-Pad1) -> Net-(C5-Pad1)
- U1 pad 1: TP2 -> TP1
- U1 pad 3: Net-(C4-Pad1) -> Net-(C1-Pad1)
- U2 pad 1: TP3 -> TP2
- U2 pad 3: Net-(C5-Pad1) -> Net-(C3-Pad1)
- U3 pad 1: TP5 -> TP3
- U3 pad 3: Net-(C6-Pad1) -> Net-(C5-Pad1)
Routing:
- net +5V: track 19.1 -> 199.2 mm, vias 0 -> 6
- net TP2: track 0.00 -> 67.5 mm, vias 0 -> 4
- net TP1: track 0.00 -> 46.0 mm, vias 0 -> 4
- net TP3: track 9.48 -> 47.0 mm, vias 0 -> 4
- net Net-(C3-Pad1): track 0.00 -> 26.6 mm, vias 0 -> 2
- net Net-(D2-Pad2): track 0.00 -> 24.9 mm
- net Net-(D1-Pad2): track 0.00 -> 24.9 mm
- net GND: track 8.16 -> 30.8 mm
- net Net-(D3-Pad2): track 0.00 -> 20.9 mm, vias 0 -> 1
- net Net-(C4-Pad1): track 16.1 -> 0.00 mm, vias 2 -> 0
- net Net-(C1-Pad1): track 0.00 -> 14.2 mm, vias 0 -> 2
- net Net-(D1-Pad4): track 0.00 -> 13.8 mm
- net Net-(C6-Pad1): track 9.86 -> 0.00 mm, vias 1 -> 0
- net Net-(C5-Pad1): track 2.47 -> 10.8 mm, vias 0 -> 2
- added copper zone on F.Cu, net GND
Other:
- board size 78.2 x 33.2 mm -> 78.3 x 50.7 mm
- board text added: "5V"
- board text added: "GND"
- board text added: "IN"
- board text added: "JLCJLCJLCJLC"
- board text added: "OUT"
- board text added: "TP1"
- board text added: "TP2"
- board text added: "TP3"

Commit message: update
Parts:
- removed the C1 at (202.9, 100.2)
- removed the C2 at (206.9, 104.2)
- removed the C3 at (188.9, 101.8)
- removed the C4 at (188.9, 107.8)
- removed the C5 at (214.1, 100.2)
- removed the C6 at (210.1, 104.2)
- removed D1, D2, D3: WS2812B, LED_SMD:LED_WS2812B_PLCC4_5.0x5.0mm_P3.2mm
- removed the J1 at (208.5, 111.2)
- removed J2: Conn_02x03_Counter_Clockwise, Connector_PinHeader_1.27mm:PinHeader_2x03_P1.27mm_Vertical
- removed J3: Conn_01x07_Male, Connector_PinHeader_2.54mm:PinHeader_1x07_P2.54mm_Vertical
- removed the TP1 at (198.9, 106.5)
- removed the TP2 at (180.2, 106.5)
- removed the TP3 at (217.6, 106.5)
- removed the U1 at (204.9, 102.2)
- removed the U2 at (188.9, 104.8)
- removed the U3 at (212.1, 102.2)
- removed mouse-bite-2mm-slot (x4): VAL**, Touchpad:mouse-bite-2mm-slot
Routing:
- net +5V: track 199.2 -> 58.8 mm, vias 6 -> 2
- net TP2: track 67.5 -> 26.7 mm, vias 4 -> 2
- net TP1: track 46.0 -> 13.8 mm, vias 4 -> 2
- net TP3: track 47.0 -> 16.9 mm, vias 4 -> 2
- net Net-(D2-Pad2): track 24.9 -> 0.00 mm
- net Net-(D1-Pad2): track 24.9 -> 0.00 mm
- net Net-(D3-Pad2): track 20.9 -> 0.00 mm, vias 1 -> 0
- net GND: track 30.8 -> 15.4 mm
- net Net-(D1-Pad4): track 13.8 -> 0.00 mm
- net Net-(C3-Pad1): track 26.6 -> 13.3 mm, vias 2 -> 1
- net Net-(C1-Pad1): track 14.2 -> 7.10 mm, vias 2 -> 1
- net Net-(C5-Pad1): track 10.8 -> 5.40 mm, vias 2 -> 1
- removed copper zone on F.Cu, net GND
Other:
- board size 78.3 x 50.7 mm -> 78.1 x 15.5 mm
- board text removed: "5V"
- board text removed: "GND"
- board text removed: "IN"
- board text removed: "OUT"
- board text removed: "TP1"
- board text removed: "TP2"
- board text removed: "TP3"

Commit message: buzzer
Changed lines of the file:
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@@
   (segment (start 189.429045 72.775) (end 189.429045 72.125) (width 0.3556) (layer "B.Cu") (net 9))
   (segment (start 189.429045 72.125) (end 189.204045 71.9) (width 0.3556) (layer "B.Cu") (net 9))
-  (segment (start 210.448008 69.748008) (end 210.451992 69.748008) (width 0.254) (layer "B.Cu") (net 9))
-  (segment (start 210.448008 69.748008) (end 210.448008 69.701992) (width 0.254) (layer "B.Cu") (net 9))
   (segment (start 214.25 77.5) (end 212.55 75.8) (width 0.3556) (layer "B.Cu") (net 9))
   (segment (start 189.429045 72.775) (end 189.429045 74.679045) (width 0.3556) (layer "B.Cu") (net 9))
@@
   (segment (start 212.55 74.75) (end 211.3 73.5) (width 0.3556) (layer "B.Cu") (net 9))
   (segment (start 205.95 69.5) (end 205.95 68.4) (width 0.3556) (layer "B.Cu") (net 9))
-  (segment (start 210.25 69.946016) (end 210.448008 69.748008) (width 0.3556) (layer "B.Cu") (net 9))
   (segment (start 198.7 65.2) (end 198.7 65.5) (width 0.3556) (layer "F.Cu") (net 12))
   (segment (start 200.65 64.45) (end 199.45 64.45) (width 0.3556) (layer "F.Cu") (net 12))
@@
   (segment (start 203.298008 64.651992) (end 203.298008 64.648008) (width 0.254) (layer "B.Cu") (net 12))
   (segment (start 203.545495 64.651992) (end 204.643934 65.750431) (width 0.3556) (layer "B.Cu") (net 12))
-  (segment (start 188.775 64.85) (end 180.625 64.85) (width 0.3556) (layer "F.Cu") (net 13))
-  (segment (start 189.425 65.5) (end 188.775 64.85) (width 0.3556) (layer "F.Cu") (net 13))
+  (segment (start 180.625 64.85) (end 180.043597 65.431403) (width 0.3556) (layer "F.Cu") (net 13))
   (segment (start 180.043597 65.431403) (end 180.043597 65.613493) (width 0.3556) (layer "F.Cu") (net 13))
-  (segment (start 180.625 64.85) (end 180.043597 65.431403) (width 0.3556) (layer "F.Cu") (net 13))
+  (segment (start 189.45 65.5) (end 188.8 64.85) (width 0.3556) (layer "F.Cu") (net 13))
+  (segment (start 188.8 64.85) (end 180.625 64.85) (width 0.3556) (layer "F.Cu") (net 13))
   (via (at 189.45 65.5) (size 0.8) (drill 0.4) (layers "F.Cu" "B.Cu") (net 13))
   (segment (start 189.429045 65.504045) (end 189.425 65.5) (width 0.3556) (layer "B.Cu") (net 13))
+  (segment (start 189.429045 65.520955) (end 189.45 65.5) (width 0.3556) (layer "B.Cu") (net 13))
   (segment (start 189.604045 68.675) (end 189.604045 66.95) (width 0.3556) (layer "B.Cu") (net 13))
-  (segment (start 189.429045 66.775) (end 189.429045 65.504045) (width 0.3556) (layer "B.Cu") (net 13))
+  (segment (start 189.429045 66.775) (end 189.429045 65.520955) (width 0.3556) (layer "B.Cu") (net 13))
   (segment (start 189.604045 66.95) (end 189.429045 66.775) (width 0.3556) (layer "B.Cu") (net 13))
   (segment (start 206.35 73.35) (end 206.35 66.85) (width 0.254) (layer "F.Cu") (net 14))

Commit message: update
Other:
- board size 78.1 x 15.5 mm -> 56 x 16 mm
Changed lines of the file:
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@@
   (gr_line (start 179.65 75.3) (end 176.05 71.7) (layer "Edge.Cuts") (width 0.05))
   (gr_line (start 183.7 72.85) (end 180.55 72.85) (layer "Edge.Cuts") (width 0.05))
-  (gr_line (start 237.7 79.15) (end 217.3 63.65) (layer "Edge.Cuts") (width 0.05))
+  (gr_line (start 170.7 79.15) (end 170.7 73.15) (layer "Edge.Cuts") (width 0.18))
   (gr_line (start 194.7 72.1) (end 195.2 71.6) (layer "Edge.Cuts") (width 0.05))
-  (gr_line (start 191.45 79.15) (end 159.6 79.15) (layer "Edge.Cuts") (width 0.05))
   (gr_line (start 179.65 67.7) (end 176.05 71.3) (layer "Edge.Cuts") (width 0.05))
-  (gr_line (start 210.05 79.15) (end 191.45 79.15) (layer "Edge.Cuts") (width 0.05))
   (gr_arc (start 217.45 69.6) (mid 217.274264 70.024264) (end 216.85 70.2) (layer "Edge.Cuts") (width 0.05))
+  (gr_line (start 180.7 63.15) (end 216.7 63.15) (layer "Edge.Cuts") (width 0.18))
   (gr_arc (start 183.7 70.15) (mid 183.912132 70.237868) (end 184 70.45) (layer "Edge.Cuts") (width 0.05))
   (gr_line (start 184 70.45) (end 184 72.55) (layer "Edge.Cuts") (width 0.05))
+  (gr_arc (start 216.7 63.15) (mid 223.771068 66.078932) (end 226.7 73.15) (layer "Edge.Cuts") (width 0.18))
   (gr_line (start 213.7 70.2) (end 216.85 70.2) (layer "Edge.Cuts") (width 0.05))
   (gr_line (start 179.95 73.45) (end 179.95 75.2) (layer "Edge.Cuts") (width 0.05))
@@
   (gr_arc (start 180.55 70.15) (mid 180.125736 69.974264) (end 179.95 69.55) (layer "Edge.Cuts") (width 0.05))
   (gr_arc (start 213.7 72.9) (mid 213.487868 72.812132) (end 213.4 72.6) (layer "Edge.Cuts") (width 0.05))
+  (gr_line (start 170.7 79.15) (end 226.7 79.15) (layer "Edge.Cuts") (width 0.18))
   (gr_line (start 217.75 75.35) (end 221.35 71.75) (layer "Edge.Cuts") (width 0.05))
   (gr_arc (start 179.65 67.7) (mid 179.846353 67.682295) (end 179.95 67.85) (layer "Edge.Cuts") (width 0.05))
@@
   (gr_line (start 180.55 70.15) (end 183.7 70.15) (layer "Edge.Cuts") (width 0.05))
   (gr_arc (start 216.85 72.9) (mid 217.274264 73.075736) (end 217.45 73.5) (layer "Edge.Cuts") (width 0.05))
+  (gr_line (start 226.7 79.15) (end 226.7 73.15) (layer "Edge.Cuts") (width 0.18))
   (gr_line (start 197.15 74.4) (end 202.1 69.45) (layer "Edge.Cuts") (width 0.05))
   (gr_line (start 201.65 68.55) (end 202.15 69.05) (layer "Edge.Cuts") (width 0.05))
   (gr_line (start 217.45 69.6) (end 217.45 67.85) (layer "Edge.Cuts") (width 0.05))
-  (gr_line (start 217.3 63.65) (end 180 63.65) (layer "Edge.Cuts") (width 0.05))
   (gr_arc (start 195.200001 71.6) (mid 195.375 71.534793) (end 195.55 71.6) (layer "Edge.Cuts") (width 0.05))
   (gr_line (start 197.1 72.75) (end 201.25 68.6) (layer "Edge.Cuts") (width 0.05))
@@
   (gr_line (start 213.4 72.6) (end 213.4 70.5) (layer "Edge.Cuts") (width 0.05))
   (gr_arc (start 221.35 71.35) (mid 221.45 71.55) (end 221.35 71.75) (layer "Edge.Cuts") (width 0.05))
-  (gr_line (start 210.05 79.15) (end 237.7 79.15) (layer "Edge.Cuts") (width 0.05))
   (gr_arc (start 217.75 75.35) (mid 217.553647 75.367705) (end 217.45 75.2) (layer "Edge.Cuts") (width 0.05))
   (gr_arc (start 197.099999 72.75) (mid 196.9 72.82964) (end 196.700001 72.75) (layer "Edge.Cuts") (width 0.05))
@@
   (gr_arc (start 194.7 72.4) (mid 194.655832 72.25) (end 194.7 72.1) (layer "Edge.Cuts") (width 0.05))
   (gr_arc (start 217.45 67.85) (mid 217.575339 67.726017) (end 217.75 67.75) (layer "Edge.Cuts") (width 0.05))
-  (gr_line (start 180 63.65) (end 159.6 79.15) (layer "Edge.Cuts") (width 0.05))
   (gr_arc (start 179.95 73.45) (mid 180.125736 73.025736) (end 180.55 72.85) (layer "Edge.Cuts") (width 0.05))
+  (gr_arc (start 170.7 73.15) (mid 173.628932 66.078932) (end 180.7 63.15) (layer "Edge.Cuts") (width 0.18))
   (gr_arc (start 184 72.55) (mid 183.912132 72.762132) (end 183.7 72.85) (layer "Edge.Cuts") (width 0.05))
   (gr_arc (start 176.05 71.7) (mid 175.95 71.5) (end 176.05 71.3) (layer "Edge.Cuts") (width 0.05))
@@
     (polygon
       (pts
-        (xy 237.7 79.15)
-        (xy 159.6 79.15)
-        (xy 180 63.65)
-        (xy 217.3 63.65)
+        (xy 227.574158 80.440069)
+        (xy 170.3776 80.472287)
+        (xy 170.582991 62.700007)
+        (xy 227.37582 62.930341)
       )
     )
@@
     )
   )
+  (group "" (id 4561c42b-6cbc-48fe-84df-6b9b6f2860ab)
+    (members
+      18a894fc-dbaf-454b-80ba-18aa5e51605f
+      2e60753f-ee9b-4773-85d2-697a7064265e
+      47933637-597b-4f31-bf37-985673c5d0f7
+      6f7e9d9b-e5ce-495d-a78a-ddf07a127610
+      a1f8a5aa-4548-42aa-802d-f916ec5bce49
+      f52cf5a9-c64c-410b-99ca-6b347ff867c5
+    )
+  )
