File: KiCad files/Main Project/CNLJS.kicad_pcb (KiCad board)
At the start: 2 copper layers, 150 x 150 mm, 184 parts, among them J1 USBasp, J2 USB_C_Receptacle_USB2.0, Q1 Si2319CDS, SW2 SW_SPDT, U1 ATmega328P-AU, U18 TTP223-BA6, U19 TTP223-BA6, U2 MCP73871-2CC, U20 TTP223-BA6, U21 TTP223-BA6, U22 TTP223-BA6, U23 TTP223-BA6, U24 TTP223-BA6, U25 TTP223-BA6, U26 TTP223-BA6, U27 TTP223-BA6, U28 TTP223-BA6, U29 TTP223-BA6, U3 CH340C, U4 2108, Y1 16MHz

Commit message: Update CNLJS.kicad_pcb
Parts:
- removed C25, C26, C27, C28, C29, C35, C36, C37, C38, C39, C45, C46: 100n, Capacitor_SMD:C_0603_1608Metric
- removed C30, C31, C32, C33, C34, C40, C41, C42, C43, C44, C47, C48: 0-50 pF, Capacitor_SMD:C_0603_1608Metric
- removed U18, U19, U20, U21, U22, U23, U24, U25, U26, U27, U28, U29: TTP223-BA6, Package_TO_SOT_SMD:SOT-23-6

Commit message: update
Parts:
- added R20: 4k7, Resistor_SMD:R_0805_2012Metric, B.Cu at (326.1, 91.9)
- added R21: 4k7, Resistor_SMD:R_0805_2012Metric, B.Cu at (321.7, 91.9)
- BT1, C11, C12, C13, C14, C15, C16, C17, C18, C19, C20, C21, C22, C23, C24, D1, D13, D14, D15, D16, D2, F1, J1, L1, L2, Q1, R1, R10, R11, R12, R13, R14, R15, R18, R19, R3, R4, R5, R6, R7, R8, R9, SW2, U1, U2, U3, U4, Y1: moved to B.Cu
- moved C24 44.6 mm to (326.4, 105.3), turned to 180 degrees
- moved D2 40.3 mm to (358.2, 92.2), turned to 180 degrees
- moved C20 40.3 mm to (350.5, 96.2), turned to 180 degrees
- moved D1 40.3 mm to (350.2, 99.3), turned to 180 degrees
- moved D16 40.3 mm to (351.7, 92.2), turned to 180 degrees
- moved R1 40.3 mm to (349.8, 102.3), turned to 180 degrees
- moved U4 40.3 mm to (366.6, 86.3), turned to 180 degrees
- moved C21 40.3 mm to (352.6, 87.0), turned to 180 degrees
- moved L1 40.3 mm to (360.8, 87.4), turned to 180 degrees
- moved Q1 40.3 mm to (355.7, 96.8), turned to 180 degrees
- moved C13 14.8 mm to (285.8, 58.3), turned to 180 degrees
- moved R10 14.8 mm to (288.1, 66.6), turned to 180 degrees
- moved R11 14.8 mm to (292.6, 66.6), turned to 180 degrees
- moved R12 14.8 mm to (292.6, 69.5), turned to 180 degrees
- moved R13 14.8 mm to (283.7, 66.5), turned to 180 degrees
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Connections:
- U1 pad 32: unconnected-(U1-Pad32) -> INT

Commit message: update
Parts:
- removed U1: ATmega328P-AU, Package_QFP:TQFP-32_7x7mm_P0.8mm
- added J17: Conn_01x03_Male, Connector_PinHeader_2.54mm:PinHeader_1x03_P2.54mm_Vertical, B.Cu at (287.9, 130.7)
- added J18: Conn_01x03_Male, Connector_PinHeader_2.54mm:PinHeader_1x03_P2.54mm_Vertical, B.Cu at (283.2, 130.7)
- added J19: Conn_01x03_Male, Connector_PinHeader_2.54mm:PinHeader_1x03_P2.54mm_Vertical, B.Cu at (273.9, 130.7)
- added J20: Conn_01x03_Male, Connector_PinHeader_2.54mm:PinHeader_1x03_P2.54mm_Vertical, B.Cu at (278.6, 130.7)
- added R22: 470R, Resistor_SMD:R_0603_1608Metric, F.Cu at (295.7, 129.6)
- added SW1: SW_Push, Button_Switch_SMD:SW_SPST_TL3342, B.Cu at (275.1, 154.0)
- added TP_LED_1: WS2812-4020_dual, LED_SMD:LED_WS2812B_PLCC4_5.0x5.0mm_P3.2mm, F.Cu at (304.6, 160.4)
- added TP_LED_10: WS2812-4020_dual, LED_SMD:LED_WS2812B_PLCC4_5.0x5.0mm_P3.2mm, F.Cu at (329.9, 153.8)
- added TP_LED_11: WS2812-4020_dual, LED_SMD:LED_WS2812B_PLCC4_5.0x5.0mm_P3.2mm, F.Cu at (313.0, 147.2)
- added TP_LED_12: WS2812-4020_dual, LED_SMD:LED_WS2812B_PLCC4_5.0x5.0mm_P3.2mm, F.Cu at (329.9, 147.2)
- added TP_LED_2: WS2812-4020_dual, LED_SMD:LED_WS2812B_PLCC4_5.0x5.0mm_P3.2mm, F.Cu at (321.4, 153.8)
- added TP_LED_3: WS2812-4020_dual, LED_SMD:LED_WS2812B_PLCC4_5.0x5.0mm_P3.2mm, F.Cu at (304.6, 153.8)
- added TP_LED_4: WS2812-4020_dual, LED_SMD:LED_WS2812B_PLCC4_5.0x5.0mm_P3.2mm, F.Cu at (313.0, 153.8)
- added TP_LED_5: WS2812-4020_dual, LED_SMD:LED_WS2812B_PLCC4_5.0x5.0mm_P3.2mm, F.Cu at (321.4, 160.4)
- added TP_LED_6: WS2812-4020_dual, LED_SMD:LED_WS2812B_PLCC4_5.0x5.0mm_P3.2mm, F.Cu at (313.0, 160.4)
- added TP_LED_7: WS2812-4020_dual, LED_SMD:LED_WS2812B_PLCC4_5.0x5.0mm_P3.2mm, F.Cu at (329.9, 160.4)
- added TP_LED_8: WS2812-4020_dual, LED_SMD:LED_WS2812B_PLCC4_5.0x5.0mm_P3.2mm, F.Cu at (304.6, 147.2)
- added TP_LED_9: WS2812-4020_dual, LED_SMD:LED_WS2812B_PLCC4_5.0x5.0mm_P3.2mm, F.Cu at (321.4, 147.2)
- added U17: PCF8575, Package_SO:SOIC-24W_7.5x15.4mm_P1.27mm, B.Cu at (265.2, 136.8)
- added U18: ATmega328-A, Package_QFP:TQFP-32_7x7mm_P0.8mm, B.Cu at (264.5, 156.3)
- FIN1, FIN10, FIN11, FIN12, FIN13, FIN14, FIN15, FIN16, FIN2, FIN3, FIN4, FIN5, FIN6, FIN7, FIN8, FIN9, POS17, POS18, POS19, POS20, POS21, POS22, POS23, POS24, POS25, POS26, POS27, POS28, POS29, POS30, POS31, POS32, POS33, POS34, POS35, POS36, POS37, POS38, POS39, POS40, POS41, POS42, POS43, POS44, POS45, POS46, POS47, POS48, POS49, POS50, POS51, POS52, POS53, POS54, POS55, POS56, POS57, POS58, POS59, POS60, POS61, POS62, POS63, POS64, POS65, POS66, POS67, POS68, POS69, POS70, POS71, POS72, POS73, POS74, POS75, POS76, POS77, POS78, POS79, POS80, POS81, POS82, POS83, POS84: footprint FieldBoard_footprint:LED_WS2812B_PLCC4_5.0x5.0mm_P3.2mm -> LED_SMD:LED_WS2812B_PLCC4_5.0x5.0mm_P3.2mm
- J2, R16, R17: moved to B.Cu
- turned J2 to 180 degrees
- turned R16 to 180 degrees
- turned R17 to 180 degrees
Connections:
- R33 pad 1: unconnected-(R33-Pad1) -> NP_1
- R34 pad 1: unconnected-(R34-Pad1) -> NP_2
- R35 pad 1: unconnected-(R35-Pad1) -> NP_3
- R36 pad 1: unconnected-(R36-Pad1) -> NP_4

Commit message: Update CNLJS.kicad_pcb
Parts:
- moved TP_LED_7 179.7 mm to (153.8, 196.2)
- moved TP_LED_10 179.7 mm to (153.8, 189.5)
- moved TP_LED_12 179.7 mm to (153.8, 182.9)
- moved TP_LED_5 179.7 mm to (145.3, 196.2)
- moved TP_LED_6 179.7 mm to (136.9, 196.2)
- moved TP_LED_1 179.7 mm to (128.5, 196.2)
- moved TP_LED_11 179.7 mm to (136.9, 182.9)
- moved TP_LED_2 179.7 mm to (145.3, 189.5)
- moved TP_LED_4 179.7 mm to (136.9, 189.5)
- moved TP_LED_9 179.7 mm to (145.3, 182.9)
- moved TP_LED_3 179.7 mm to (128.5, 189.5)
- moved TP_LED_8 179.7 mm to (128.5, 182.9)
- moved C13 159.6 mm to (126.5, 48.2)
- moved C15 159.6 mm to (145.2, 47.3)
- moved C16 159.6 mm to (149.7, 47.3)
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
Commit message: Update CNLJS.kicad_pcb
Parts:
- moved TP_LED_6 169.7 mm to (127.3, 26.8)
- moved TP_LED_5 168.8 mm to (143.3, 27.4)
- moved TP_LED_4 163.7 mm to (157.3, 27.1)
- moved TP_LED_1 125.8 mm to (75.5, 82.1)
- moved TP_LED_2 118.2 mm to (75.5, 94.2)
- moved TP_LED_8 116.0 mm to (208.3, 98.8)
- moved TP_LED_9 114.0 mm to (207.9, 87.7)
- moved TP_LED_7 101.7 mm to (208.6, 110.5)
- moved TP_LED_3 96.3 mm to (75.7, 109.0)
- moved TP_LED_10 37.5 mm to (128.8, 161.6)
- moved TP_LED_11 22.5 mm to (144.4, 161.7)
- moved TP_LED_12 21.1 mm to (156.8, 162.1)
Changed lines of the file:
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@@
   )
   (footprint "LED_SMD:LED_WS2812B_PLCC4_5.0x5.0mm_P3.2mm" (layer "F.Cu")
-    (at 145.33 182.91)
+    (at 207.95 87.65)
     (descr "https://cdn-shop.adafruit.com/datasheets/WS2812B.pdf")
     (tags "LED RGB NeoPixel")
@@
   )
   (footprint "LED_SMD:LED_WS2812B_PLCC4_5.0x5.0mm_P3.2mm" (layer "F.Cu")
-    (at 145.33 189.53)
+    (at 75.45 94.25)
     (descr "https://cdn-shop.adafruit.com/datasheets/WS2812B.pdf")
     (tags "LED RGB NeoPixel")
@@
   )
   (footprint "LED_SMD:LED_WS2812B_PLCC4_5.0x5.0mm_P3.2mm" (layer "F.Cu")
-    (at 136.91 189.53)
+    (at 157.35 27.1)
     (descr "https://cdn-shop.adafruit.com/datasheets/WS2812B.pdf")
     (tags "LED RGB NeoPixel")
@@
   )
   (footprint "LED_SMD:LED_WS2812B_PLCC4_5.0x5.0mm_P3.2mm" (layer "F.Cu")
-    (at 153.75 182.91)
+    (at 156.75 162.05)
     (descr "https://cdn-shop.adafruit.com/datasheets/WS2812B.pdf")
     (tags "LED RGB NeoPixel")
@@
   )
   (footprint "LED_SMD:LED_WS2812B_PLCC4_5.0x5.0mm_P3.2mm" (layer "F.Cu")
-    (at 128.49 182.91)
+    (at 208.3 98.75)
     (descr "https://cdn-shop.adafruit.com/datasheets/WS2812B.pdf")
     (tags "LED RGB NeoPixel")
@@
   )
   (footprint "LED_SMD:LED_WS2812B_PLCC4_5.0x5.0mm_P3.2mm" (layer "F.Cu")
-    (at 136.91 182.91)
+    (at 144.4 161.7)
     (descr "https://cdn-shop.adafruit.com/datasheets/WS2812B.pdf")
     (tags "LED RGB NeoPixel")
@@
   )
   (footprint "LED_SMD:LED_WS2812B_PLCC4_5.0x5.0mm_P3.2mm" (layer "F.Cu")
-    (at 128.49 196.15)
+    (at 75.5 82.1)
     (descr "https://cdn-shop.adafruit.com/datasheets/WS2812B.pdf")
     (tags "LED RGB NeoPixel")
@@
   )
   (footprint "LED_SMD:LED_WS2812B_PLCC4_5.0x5.0mm_P3.2mm" (layer "F.Cu")
-    (at 145.33 196.15)
+    (at 143.3 27.35)
     (descr "https://cdn-shop.adafruit.com/datasheets/WS2812B.pdf")
     (tags "LED RGB NeoPixel")
@@
   )
   (footprint "LED_SMD:LED_WS2812B_PLCC4_5.0x5.0mm_P3.2mm" (layer "F.Cu")
-    (at 153.75 189.53)
+    (at 128.8 161.55)
     (descr "https://cdn-shop.adafruit.com/datasheets/WS2812B.pdf")
     (tags "LED RGB NeoPixel")
@@
   )
   (footprint "LED_SMD:LED_WS2812B_PLCC4_5.0x5.0mm_P3.2mm" (layer "F.Cu")
-    (at 128.49 189.53)
+    (at 75.7 109)
     (descr "https://cdn-shop.adafruit.com/datasheets/WS2812B.pdf")
     (tags "LED RGB NeoPixel")
@@
   )
   (footprint "LED_SMD:LED_WS2812B_PLCC4_5.0x5.0mm_P3.2mm" (layer "F.Cu")
-    (at 153.75 196.15)
+    (at 208.55 110.45)
     (descr "https://cdn-shop.adafruit.com/datasheets/WS2812B.pdf")
     (tags "LED RGB NeoPixel")
@@
   )
   (footprint "LED_SMD:LED_WS2812B_PLCC4_5.0x5.0mm_P3.2mm" (layer "F.Cu")
-    (at 136.91 196.15)
+    (at 127.3 26.75)
     (descr "https://cdn-shop.adafruit.com/datasheets/WS2812B.pdf")
     (tags "LED RGB NeoPixel")

Commit message: update
Parts:
- moved TP_LED_9 13.6 mm to (210.0, 74.2)
- moved TP_LED_1 7.85 mm to (75.4, 74.2)
- moved TP_LED_8 6.14 mm to (210.0, 92.8)
- moved TP_LED_10 5.05 mm to (123.9, 160.3)
- moved TP_LED_12 4.76 mm to (161.2, 160.3)
- moved TP_LED_4 4.25 mm to (161.4, 25.6)
- moved TP_LED_6 3.43 mm to (124.1, 25.6)
- moved TP_LED_3 2.57 mm to (75.4, 111.5)
- moved TP_LED_11 2.29 mm to (142.5, 160.3)
- moved TP_LED_5 1.80 mm to (142.7, 25.6)
- moved TP_LED_7 1.79 mm to (210.0, 111.5)
- moved TP_LED_2 1.35 mm to (75.4, 92.9)
Changed lines of the file:
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@@
   )
   (footprint "LED_SMD:LED_WS2812B_PLCC4_5.0x5.0mm_P3.2mm" (layer "F.Cu")
-    (at 207.95 87.65)
+    (at 210 74.196976)
     (descr "https://cdn-shop.adafruit.com/datasheets/WS2812B.pdf")
     (tags "LED RGB NeoPixel")
@@
   )
   (footprint "LED_SMD:LED_WS2812B_PLCC4_5.0x5.0mm_P3.2mm" (layer "F.Cu")
-    (at 75.45 94.25)
+    (at 75.4 92.9)
     (descr "https://cdn-shop.adafruit.com/datasheets/WS2812B.pdf")
     (tags "LED RGB NeoPixel")
@@
   )
   (footprint "LED_SMD:LED_WS2812B_PLCC4_5.0x5.0mm_P3.2mm" (layer "F.Cu")
-    (at 157.35 27.1)
+    (at 161.350004 25.65)
     (descr "https://cdn-shop.adafruit.com/datasheets/WS2812B.pdf")
     (tags "LED RGB NeoPixel")
@@
   )
   (footprint "LED_SMD:LED_WS2812B_PLCC4_5.0x5.0mm_P3.2mm" (layer "F.Cu")
-    (at 156.75 162.05)
+    (at 161.196969 160.35)
     (descr "https://cdn-shop.adafruit.com/datasheets/WS2812B.pdf")
     (tags "LED RGB NeoPixel")
@@
   )
   (footprint "LED_SMD:LED_WS2812B_PLCC4_5.0x5.0mm_P3.2mm" (layer "F.Cu")
-    (at 208.3 98.75)
+    (at 210 92.846976)
     (descr "https://cdn-shop.adafruit.com/datasheets/WS2812B.pdf")
     (tags "LED RGB NeoPixel")
@@
   )
   (footprint "LED_SMD:LED_WS2812B_PLCC4_5.0x5.0mm_P3.2mm" (layer "F.Cu")
-    (at 144.4 161.7)
+    (at 142.546969 160.35)
     (descr "https://cdn-shop.adafruit.com/datasheets/WS2812B.pdf")
     (tags "LED RGB NeoPixel")
@@
   )
   (footprint "LED_SMD:LED_WS2812B_PLCC4_5.0x5.0mm_P3.2mm" (layer "F.Cu")
-    (at 75.5 82.1)
+    (at 75.4 74.25)
     (descr "https://cdn-shop.adafruit.com/datasheets/WS2812B.pdf")
     (tags "LED RGB NeoPixel")
@@
   )
   (footprint "LED_SMD:LED_WS2812B_PLCC4_5.0x5.0mm_P3.2mm" (layer "F.Cu")
-    (at 143.3 27.35)
+    (at 142.7 25.65)
     (descr "https://cdn-shop.adafruit.com/datasheets/WS2812B.pdf")
     (tags "LED RGB NeoPixel")
@@
   )
   (footprint "LED_SMD:LED_WS2812B_PLCC4_5.0x5.0mm_P3.2mm" (layer "F.Cu")
-    (at 128.8 161.55)
+    (at 123.896969 160.35)
     (descr "https://cdn-shop.adafruit.com/datasheets/WS2812B.pdf")
     (tags "LED RGB NeoPixel")
@@
   )
   (footprint "LED_SMD:LED_WS2812B_PLCC4_5.0x5.0mm_P3.2mm" (layer "F.Cu")
-    (at 75.7 109)
+    (at 75.4 111.55)
     (descr "https://cdn-shop.adafruit.com/datasheets/WS2812B.pdf")
     (tags "LED RGB NeoPixel")
@@
   )
   (footprint "LED_SMD:LED_WS2812B_PLCC4_5.0x5.0mm_P3.2mm" (layer "F.Cu")
-    (at 208.55 110.45)
+    (at 210 111.496976)
     (descr "https://cdn-shop.adafruit.com/datasheets/WS2812B.pdf")
     (tags "LED RGB NeoPixel")
@@
   )
   (footprint "LED_SMD:LED_WS2812B_PLCC4_5.0x5.0mm_P3.2mm" (layer "F.Cu")
-    (at 127.3 26.75)
+    (at 124.050004 25.65)
     (descr "https://cdn-shop.adafruit.com/datasheets/WS2812B.pdf")
     (tags "LED RGB NeoPixel")
