File: KiCad files/Main Project/CNLJS.kicad_pcb (KiCad board)
At the start: 2 copper layers, 150 x 150 mm, 169 parts, among them J1 USBasp, J17 Conn_02x03_Odd_Even, J18 Conn_02x03_Odd_Even, J19 Conn_02x03_Odd_Even, J2 USB_C_Receptacle_USB2.0, J20 Conn_02x03_Odd_Even, Q1 Si2319CDS, SW1 SW_Push, SW2 SW_SPDT, U17 PCF8575, U18 ATmega328-A, U2 MCP73871-2CC, U3 CH340C, U4 2108, Y1 16MHz

Commit message: update
Parts:
- removed SW2: SW_SPDT, Button_Switch_SMD:SW_SPDT_PCM12
- added J21: Conn_01x01, CNLJS:Padovi_sklopke, B.Cu at (176.5, 152.6)
- added J22: Conn_01x01, CNLJS:Padovi_sklopke, B.Cu at (158.4, 142.8)
- moved C20 7.12 mm to (173.8, 144.9), turned to -90 degrees
- moved D2 6.74 mm to (173.4, 125.0)
- moved D1 6.03 mm to (176.3, 125.0), turned to -90 degrees
- moved Q1 5.51 mm to (173.4, 132.3)
- moved D16 2.20 mm to (169.3, 151.3)
- moved L1 2.17 mm to (178.9, 145.2)
- moved R1 1.10 mm to (177.2, 128.4)
- moved C15 0.89 mm to (158.0, 137.1), turned to 0 degrees
- moved C21 0.45 mm to (169.2, 138.5)
Routing:
- net VDD: track 137.4 -> 455.3 mm, vias 2 -> 6
- net RESET: track 21.8 -> 94.1 mm, vias 0 -> 4
- net INT: track 0.00 -> 41.5 mm, vias 0 -> 8
- net VBUS: track 62.5 -> 87.8 mm, vias 16 -> 0
- net TP_11: track 194.5 -> 207.2 mm
- net TP_10: track 204.2 -> 216.8 mm
- net TP_12: track 189.1 -> 201.0 mm
- net GND: track 38.9 -> 49.7 mm, vias 33 -> 77
- net /Power/CH_OUT: track 6.43 -> 0.00 mm
- net Net-(D2-Pad2): track 0.00 -> 5.11 mm
- net VCC: vias 9 -> 37
- added copper zone on B.Cu, net +BATT
- added copper zone on B.Cu, net /Power/CH_OUT
- added copper zone on B.Cu, net Net-(C20-Pad1)
- added copper zone on B.Cu, net Net-(C21-Pad1)
- added copper zone on B.Cu, net VCC

Commit message: Update CNLJS.kicad_pcb
Routing:
- net VDD: track 455.3 -> 584.9 mm, vias 6 -> 12
Changed lines of the file:
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@@
   (segment (start 150.15 142.6615) (end 150.15 143.8) (width 0.508) (layer "B.Cu") (net 2))
   (segment (start 150.1 130.7) (end 149.4 130) (width 0.2) (layer "B.Cu") (net 2))
+  (segment (start 132.6 81.7) (end 132.6 89.6) (width 0.508) (layer "F.Cu") (net 3))
+  (segment (start 175.45 108.25) (end 179.149635 104.550365) (width 0.508) (layer "F.Cu") (net 3))
   (segment (start 127.3 98.7) (end 127.3 94.7) (width 0.508) (layer "F.Cu") (net 3))
   (segment (start 76.1 102.5) (end 84.7 102.5) (width 0.508) (layer "F.Cu") (net 3))
+  (segment (start 133.1 28.1) (end 137.1 32.1) (width 0.508) (layer "F.Cu") (net 3))
+  (segment (start 137.1 32.1) (end 137.1 38) (width 0.508) (layer "F.Cu") (net 3))
   (segment (start 103.2 116.7) (end 97.6 116.7) (width 0.508) (layer "F.Cu") (net 3))
   (via (at 103.2 116.7) (size 0.8) (drill 0.4) (layers "F.Cu" "B.Cu") (net 3))
+  (via (at 133.1 28.1) (size 0.8) (drill 0.4) (layers "F.Cu" "B.Cu") (net 3))
   (via (at 97.6 116.7) (size 0.8) (drill 0.4) (layers "F.Cu" "B.Cu") (net 3))
+  (via (at 132.6 81.7) (size 0.8) (drill 0.4) (layers "F.Cu" "B.Cu") (net 3))
   (via (at 76.1 102.5) (size 0.8) (drill 0.4) (layers "F.Cu" "B.Cu") (net 3))
   (via (at 127.3 98.7) (size 0.8) (drill 0.4) (layers "F.Cu" "B.Cu") (net 3))
+  (via (at 179.149635 104.550365) (size 0.8) (drill 0.4) (layers "F.Cu" "B.Cu") (net 3))
+  (via (at 132.6 89.6) (size 0.8) (drill 0.4) (layers "F.Cu" "B.Cu") (net 3))
   (via (at 84.7 102.5) (size 0.8) (drill 0.4) (layers "F.Cu" "B.Cu") (net 3))
   (via (at 127.3 94.7) (size 0.8) (drill 0.4) (layers "F.Cu" "B.Cu") (net 3))
+  (via (at 175.45 108.25) (size 0.8) (drill 0.4) (layers "F.Cu" "B.Cu") (net 3))
+  (via (at 137.1 38) (size 0.8) (drill 0.4) (layers "F.Cu" "B.Cu") (net 3))
   (segment (start 111.3 98) (end 111.3 116.673) (width 0.508) (layer "B.Cu") (net 3))
   (segment (start 76.095 102.495) (end 76.1 102.5) (width 0.508) (layer "B.Cu") (net 3))
@@
   (segment (start 100.7 127.5) (end 101 127.5) (width 0.508) (layer "B.Cu") (net 3))
   (segment (start 146.4 102.9) (end 137 93.5) (width 0.508) (layer "B.Cu") (net 3))
-  (segment (start 181.4 121) (end 163.3 102.9) (width 0.508) (layer "B.Cu") (net 3))
   (segment (start 121.95 136.5) (end 121.595 136.855) (width 0.508) (layer "B.Cu") (net 3))
   (segment (start 173.4 123.75) (end 176.3 123.75) (width 0.508) (layer "B.Cu") (net 3))
@@
   (segment (start 191 157) (end 191 130.6) (width 0.508) (layer "B.Cu") (net 3))
   (segment (start 95.4 116.7) (end 95.25 116.85) (width 0.508) (layer "B.Cu") (net 3))
+  (segment (start 137.1 38) (end 137.1 77.2) (width 0.508) (layer "B.Cu") (net 3))
   (segment (start 127.349 106.95) (end 127.349 102.15) (width 0.508) (layer "B.Cu") (net 3))
   (segment (start 152.2 162) (end 151 162) (width 0.508) (layer "B.Cu") (net 3))
@@
   (segment (start 108.55 129.85) (end 108.55 128.35) (width 0.508) (layer "B.Cu") (net 3))
   (segment (start 108.6 131.6) (end 108.55 131.55) (width 0.508) (layer "B.Cu") (net 3))
+  (segment (start 133.105 28.095) (end 133.1 28.1) (width 0.508) (layer "B.Cu") (net 3))
+  (segment (start 137.1 77.2) (end 132.6 81.7) (width 0.508) (layer "B.Cu") (net 3))
+  (segment (start 172.05 111.65) (end 175.45 108.25) (width 0.508) (layer "B.Cu") (net 3))
   (segment (start 127.3 93.6) (end 127.2 93.5) (width 0.508) (layer "B.Cu") (net 3))
   (segment (start 100.2 127) (end 100.7 127.5) (width 0.508) (layer "B.Cu") (net 3))
@@
   (segment (start 100.15 121.485) (end 100.15 124.7) (width 0.508) (layer "B.Cu") (net 3))
   (segment (start 108.55 164.55) (end 111 167) (width 0.508) (layer "B.Cu") (net 3))
-  (segment (start 137 93.5) (end 127.2 93.5) (width 0.508) (layer "B.Cu") (net 3))
+  (segment (start 132.6 89.6) (end 132.6 93.5) (width 0.508) (layer "B.Cu") (net 3))
+  (segment (start 181.4 121) (end 172.05 111.65) (width 0.508) (layer "B.Cu") (net 3))
   (segment (start 121 131.6) (end 108.6 131.6) (width 0.508) (layer "B.Cu") (net 3))
   (segment (start 84.7 102.5) (end 88.6 102.5) (width 0.508) (layer "B.Cu") (net 3))
@@
   (segment (start 100.2 127.4) (end 100.1 127.5) (width 0.508) (layer "B.Cu") (net 3))
   (segment (start 152.095 164.555) (end 152.095 165.825) (width 0.508) (layer "B.Cu") (net 3))
+  (segment (start 137 93.5) (end 132.6 93.5) (width 0.508) (layer "B.Cu") (net 3))
   (segment (start 111.3 116.673) (end 111.3135 116.6865) (width 0.508) (layer "B.Cu") (net 3))
   (segment (start 133.105 20.125) (end 133.105 21.395) (width 0.508) (layer "B.Cu") (net 3))
@@
   (segment (start 130 110.3) (end 129.4 110.9) (width 0.508) (layer "B.Cu") (net 3))
   (segment (start 186 162) (end 191 157) (width 0.508) (layer "B.Cu") (net 3))
+  (segment (start 179.149635 104.550365) (end 200.445 83.255) (width 0.508) (layer "B.Cu") (net 3))
   (segment (start 108.55 131.55) (end 108.55 129.85) (width 0.508) (layer "B.Cu") (net 3))
   (segment (start 116.6135 116.6865) (end 111.3135 116.6865) (width 0.508) (layer "B.Cu") (net 3))
@@
   (segment (start 129.024 124.1) (end 108.6 124.1) (width 0.508) (layer "B.Cu") (net 3))
   (segment (start 100.15 127) (end 99.65 127.5) (width 0.508) (layer "B.Cu") (net 3))
+  (segment (start 172.05 111.65) (end 163.3 102.9) (width 0.508) (layer "B.Cu") (net 3))
   (segment (start 100.15 124.7) (end 100.2 124.75) (width 0.508) (layer "B.Cu") (net 3))
   (segment (start 108.55 122.5115) (end 108.55 124.15) (width 0.508) (layer "B.Cu") (net 3))
   (segment (start 69.875 102.495) (end 71.145 102.495) (width 0.508) (layer "B.Cu") (net 3))
   (segment (start 121.95 132.55) (end 121 131.6) (width 0.508) (layer "B.Cu") (net 3))
+  (segment (start 132.6 93.5) (end 127.2 93.5) (width 0.508) (layer "B.Cu") (net 3))
   (segment (start 127.349 110.149) (end 127.349 106.95) (width 0.508) (layer "B.Cu") (net 3))
   (segment (start 121.95 133.5) (end 121.95 132.55) (width 0.508) (layer "B.Cu") (net 3))
   (segment (start 152.2 162) (end 186 162) (width 0.508) (layer "B.Cu") (net 3))
+  (segment (start 200.445 83.255) (end 214.255 83.255) (width 0.508) (layer "B.Cu") (net 3))
   (segment (start 121.595 136.855) (end 120.425 136.855) (width 0.508) (layer "B.Cu") (net 3))
   (segment (start 108.55 124.15) (end 108.55 126.7) (width 0.508) (layer "B.Cu") (net 3))
   (segment (start 71.145 102.495) (end 76.095 102.495) (width 0.508) (layer "B.Cu") (net 3))
   (segment (start 191 130.6) (end 181.4 121) (width 0.508) (layer "B.Cu") (net 3))
+  (segment (start 133.105 21.395) (end 133.105 28.095) (width 0.508) (layer "B.Cu") (net 3))
   (segment (start 112.6 132.8) (end 112.6 130.5) (width 0.3556) (layer "F.Cu") (net 4))
   (segment (start 133.2 116.5) (end 129.9 113.2) (width 0.3556) (layer "F.Cu") (net 4))

Commit message: update
Routing:
- net VCC: track 25.2 -> 1150.0 mm, vias 37 -> 32
- net Net-(TP_LED_10-Pad2): track 0.00 -> 24.7 mm
- net Net-(POS17-Pad2): track 0.00 -> 20.2 mm
- net Net-(POS46-Pad2): track 0.00 -> 17.5 mm
- net Net-(POS29-Pad2): track 0.00 -> 17.1 mm
- net Net-(POS53-Pad2): track 0.00 -> 17.0 mm
- net Net-(POS26-Pad2): track 0.00 -> 15.5 mm
- net Net-(POS21-Pad2): track 0.00 -> 15.4 mm
- net Net-(POS56-Pad2): track 0.00 -> 15.4 mm
- net Net-(POS71-Pad2): track 0.00 -> 15.4 mm
- net Net-(POS45-Pad2): track 0.00 -> 15.2 mm
- net Net-(TP_LED_11-Pad2): track 0.00 -> 15.1 mm
- net Net-(TP_LED_4-Pad2): track 0.00 -> 15.1 mm
- net Net-(TP_LED_2-Pad2): track 0.00 -> 15.1 mm
- net Net-(TP_LED_1-Pad2): track 0.00 -> 15.1 mm
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
Commit message: Update CNLJS.kicad_pcb
Parts:
- moved R35 10.8 mm to (131.0, 93.0), turned to 90 degrees
Routing:
- net VCC: track 1150.0 -> 1482.2 mm, vias 32 -> 33
- net Net-(FIN12-Pad2): track 0.00 -> 109.7 mm
- net Net-(FIN4-Pad2): track 0.00 -> 104.1 mm
- net Net-(FIN8-Pad2): track 0.00 -> 103.8 mm
- net Net-(POS72-Pad2): track 0.00 -> 23.3 mm
- net NP_3: track 0.00 -> 15.7 mm, vias 0 -> 1
- net GND: track 53.6 -> 63.8 mm, vias 77 -> 80
- net /LEDs/Cube (9LEDs)/Cube-LEDs: track 0.00 -> 6.82 mm
- net Net-(LED4-Pad2): track 0.00 -> 6.68 mm
- net Net-(TP_LED_10-Pad2): track 24.7 -> 24.8 mm, vias 0 -> 2

Commit message: update v2
Routing:
- net Net-(TP_LED_10-Pad4): track 0.00 -> 197.9 mm, vias 0 -> 6
- net Net-(TP_LED_6-Pad2): track 0.00 -> 180.9 mm, vias 0 -> 6
- net Net-(TP_LED_3-Pad2): track 0.00 -> 169.3 mm, vias 0 -> 8
- net NP_5: track 0.00 -> 157.6 mm, vias 0 -> 5
- net VCC: track 1482.2 -> 1601.5 mm
- net Net-(POS20-Pad2): track 0.00 -> 72.3 mm, vias 0 -> 2
- net Net-(POS28-Pad2): track 0.00 -> 68.3 mm, vias 0 -> 6
- net Net-(POS24-Pad2): track 0.00 -> 64.9 mm, vias 0 -> 2
- net NP_4: track 0.00 -> 52.4 mm, vias 0 -> 3
- net NP_1: track 0.00 -> 49.6 mm, vias 0 -> 5
- net NP_2: track 0.00 -> 36.4 mm, vias 0 -> 3
- net GND: track 63.8 -> 82.0 mm, vias 80 -> 86
- net Net-(POS25-Pad2): track 0.00 -> 16.3 mm, vias 0 -> 2
- net Net-(POS58-Pad2): track 0.00 -> 11.4 mm, vias 0 -> 2
- net D+: track 23.1 -> 30.7 mm
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
Commit message: buzzer
Parts:
- added LS1: Buzzer, CNLJS:KLJ-1102, B.Cu at (89.5, 150.7)
Connections:
- U18 pad 14: unconnected-(U18-Pad14) -> Net-(U18-Pad14)
Routing:
- net Net-(U18-Pad14): track 0.00 -> 57.3 mm, vias 0 -> 6
- net GND: track 82.0 -> 84.2 mm, vias 86 -> 87
Changed lines of the file:
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@@
   (net 165 "unconnected-(U18-Pad12)")
   (net 166 "unconnected-(U18-Pad13)")
-  (net 167 "unconnected-(U18-Pad14)")
+  (net 167 "Net-(U18-Pad14)")
   (net 168 "unconnected-(U18-Pad19)")
   (net 169 "unconnected-(U18-Pad22)")
@@
       (net 166 "unconnected-(U18-Pad13)") (pinfunction "PB1") (pintype "bidirectional+no_connect"))
     (pad "14" smd rect (at 1.2 -4.25 180) (size 1.6 0.55) (layers "B.Cu" "B.Paste" "B.Mask")
-      (net 167 "unconnected-(U18-Pad14)") (pinfunction "PB2") (pintype "bidirectional+no_connect"))
+      (net 167 "Net-(U18-Pad14)") (pinfunction "PB2") (pintype "bidirectional"))
     (pad "15" smd rect (at 2 -4.25 180) (size 1.6 0.55) (layers "B.Cu" "B.Paste" "B.Mask")
       (net 36 "MOSI") (pinfunction "PB3") (pintype "bidirectional"))
@@
     )
   )
+  (footprint "CNLJS:KLJ-1102" (layer "B.Cu")
+    (at 89.5 150.65 90)
+    (property "Sheetfile" "Microcontroller.kicad_sch")
+    (property "Sheetname" "Microcontroller")
+    (attr smd)
+    (fp_text reference "LS1" (at 0 9 270 unlocked) (layer "B.Fab") hide
+      (effects (font (size 1 1) (thickness 0.15)) (justify mirror))
+    )
+    (fp_text value "Buzzer" (at 0 -1 270 unlocked) (layer "B.Fab")
+      (effects (font (size 1 1) (thickness 0.15)) (justify mirror))
+    )
+    (fp_line (start -1.75 5.25) (end -5.25 5.25) (layer "B.Fab") (width 0.12))
+    (fp_line (start -5.25 5.25) (end -5.25 -5.25) (layer "B.Fab") (width 0.12))
+    (fp_line (start 1.75 5.25) (end 5.25 5.25) (layer "B.Fab") (width 0.12))
+    (fp_line (start 5.25 5.25) (end 5.25 -5.25) (layer "B.Fab") (width 0.12))
+    (fp_line (start -5.25 -5.25) (end -1.75 -5.25) (layer "B.Fab") (width 0.12))
+    (fp_line (start 5.25 -5.25) (end 1.75 -5.25) (layer "B.Fab") (width 0.12))
+    (pad "1" smd rect (at 0 6.5 90) (size 3 3) (layers "B.Cu" "B.Paste" "B.Mask")
+      (net 167 "Net-(U18-Pad14)") (pinfunction "1") (pintype "input"))
+    (pad "2" smd rect (at 0 -6.5 90) (size 3 3) (layers "B.Cu" "B.Paste" "B.Mask")
+      (net 2 "GND") (pinfunction "2") (pintype "input"))
+    (model "${CNLJS}/KLJ-1102.STEP"
+      (offset (xyz 0 0 0))
+      (scale (xyz 1 1 1))
+      (rotate (xyz -90 0 0))
+    )
+  )
   (footprint "Resistor_SMD:R_0805_2012Metric" (layer "B.Cu")
     (at 145 134.849)
@@
   (via (at 167.7 138) (size 0.8) (drill 0.4) (layers "F.Cu" "B.Cu") (free) (net 2))
   (via (at 127.6 138) (size 0.8) (drill 0.4) (layers "F.Cu" "B.Cu") (net 2))
+  (via (at 80.8 150.65) (size 0.8) (drill 0.4) (layers "F.Cu" "B.Cu") (free) (net 2))
   (via (at 129.8 156) (size 0.8) (drill 0.4) (layers "F.Cu" "B.Cu") (net 2))
   (via (at 150.15 143.8) (size 0.8) (drill 0.4) (layers "F.Cu" "B.Cu") (net 2))
@@
   (segment (start 156 131.75) (end 156 130.65) (width 1.016) (layer "B.Cu") (net 2))
   (segment (start 146.699 123.051) (end 146.7 123.05) (width 0.508) (layer "B.Cu") (net 2))
+  (segment (start 83 150.65) (end 80.8 150.65) (width 0.762) (layer "B.Cu") (net 2))
   (segment (start 146.699 124.8365) (end 146.699 123.051) (width 0.508) (layer "B.Cu") (net 2))
   (segment (start 117.303 100.697) (end 119.6 100.697) (width 0.508) (layer "B.Cu") (net 2))
@@
   (segment (start 131.099 105.301) (end 131.099 102.1) (width 0.3556) (layer "B.Cu") (net 164))
   (segment (start 130.549 106.95) (end 130.549 105.851) (width 0.3556) (layer "B.Cu") (net 164))
+  (segment (start 130.05 111.65) (end 126.8 111.65) (width 0.3556) (layer "F.Cu") (net 167))
+  (segment (start 123.15 115.3) (end 124.05 114.4) (width 0.3556) (layer "F.Cu") (net 167))
+  (segment (start 109.75 130.6) (end 107.65 132.7) (width 0.3556) (layer "F.Cu") (net 167))
+  (segment (start 117.45 122.9) (end 115.15 125.2) (width 0.3556) (layer "F.Cu") (net 167))
+  (segment (start 123.15 116.3) (end 123.15 115.3) (width 0.3556) (layer "F.Cu") (net 167))
+  (segment (start 126.8 111.65) (end 124.05 114.4) (width 0.3556) (layer "F.Cu") (net 167))
+  (via (at 109.75 130.6) (size 0.8) (drill 0.4) (layers "F.Cu" "B.Cu") (net 167))
+  (via (at 130.05 111.65) (size 0.8) (drill 0.4) (layers "F.Cu" "B.Cu") (net 167))
+  (via (at 107.65 132.7) (size 0.8) (drill 0.4) (layers "F.Cu" "B.Cu") (net 167))
+  (via (at 115.15 125.2) (size 0.8) (drill 0.4) (layers "F.Cu" "B.Cu") (net 167))
+  (via (at 123.15 116.3) (size 0.8) (drill 0.4) (layers "F.Cu" "B.Cu") (net 167))
+  (via (at 117.45 122.9) (size 0.8) (drill 0.4) (layers "F.Cu" "B.Cu") (net 167))
+  (segment (start 130.8 112.4) (end 130.05 111.65) (width 0.3556) (layer "B.Cu") (net 167))
+  (segment (start 115.15 125.2) (end 109.75 130.6) (width 0.3556) (layer "B.Cu") (net 167))
+  (segment (start 96 144.35) (end 96 150.65) (width 0.3556) (layer "B.Cu") (net 167))
+  (segment (start 131.999 112.4) (end 130.8 112.4) (width 0.3556) (layer "B.Cu") (net 167))
+  (segment (start 107.65 132.7) (end 96 144.35) (width 0.3556) (layer "B.Cu") (net 167))
+  (segment (start 123.15 116.3) (end 123.15 117.2) (width 0.3556) (layer "B.Cu") (net 167))
+  (segment (start 122.425 117.925) (end 117.45 122.9) (width 0.3556) (layer "B.Cu") (net 167))
+  (segment (start 123.15 117.2) (end 122.425 117.925) (width 0.3556) (layer "B.Cu") (net 167))
   (segment (start 77 83) (end 77 76.7) (width 0.3556) (layer "F.Cu") (net 174))
   (segment (start 73.8 86.2) (end 77 83) (width 0.3556) (layer "F.Cu") (net 174))
