File: KiCad files/Main Project/CNLJS.kicad_sch (KiCad schematic)
At the start: 0 parts

Commit message: update
Other:
- note removed: "VCC (4.7V OR +BATT >>>>>>>>>>>>>>>>>"
Changed lines of the file:
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@@
     (effects (font (size 1.27 1.27)) (justify left bottom))
   )
-  (text "VCC (4.7V OR +BATT\n>>>>>>>>>>>>>>>>>" (at 128.905 59.055 0)
+  (text "VCC (4.7V OR +BATT)\n>>>>>>>>>>>>>>>>>" (at 128.905 59.055 0)
     (effects (font (size 1.27 1.27)) (justify left bottom))
   )
@@
       (reference "#PWR03") (unit 1) (value "VDD") (footprint "")
     )
-    (path "/00000000-0000-0000-0000-00006166ecfb/00000000-0000-0000-0000-000061c6ba58"
-      (reference "#PWR04") (unit 1) (value "+BATT") (footprint "")
-    )
-    (path "/00000000-0000-0000-0000-00006166ecfb/00000000-0000-0000-0000-000061673cfc"
-      (reference "#PWR05") (unit 1) (value "GND") (footprint "")
+    (path "/00000000-0000-0000-0000-00006166ecfb/b6871d13-0bc7-4b7b-a1db-b54d5790a4af"
+      (reference "#PWR04") (unit 1) (value "GND") (footprint "")
     )
     (path "/00000000-0000-0000-0000-00006165e463/00000000-0000-0000-0000-000061c74009"
@@
       (reference "#PWR0107") (unit 1) (value "GND") (footprint "")
     )
-    (path "/00000000-0000-0000-0000-00006166ecfb/af3bf9a4-bacc-4c97-80b2-8505239c4034"
-      (reference "#PWR0108") (unit 1) (value "+BATT") (footprint "")
-    )
-    (path "/00000000-0000-0000-0000-00006166ecfb/7366abd4-debc-456b-9c08-526324ee0172"
-      (reference "#PWR0109") (unit 1) (value "GND") (footprint "")
-    )
-    (path "/00000000-0000-0000-0000-00006166ecfb/f2f330dd-8962-4c15-8b02-b7407f2331e2"
-      (reference "#PWR0110") (unit 1) (value "GND") (footprint "")
-    )
-    (path "/00000000-0000-0000-0000-00006166ecfb/e8590814-34e6-485a-8470-d9c7becb8cd2"
-      (reference "#PWR0111") (unit 1) (value "+BATT") (footprint "")
-    )
-    (path "/00000000-0000-0000-0000-00006166ecfb/7a4edd8d-0d4c-4c43-a05c-7014fb66eabe"
-      (reference "#PWR0112") (unit 1) (value "+BATT") (footprint "")
-    )
-    (path "/00000000-0000-0000-0000-00006166ecfb/9dcdee11-51f3-4cf1-a0a1-d389be936601"
-      (reference "#PWR0113") (unit 1) (value "GND") (footprint "")
-    )
-    (path "/00000000-0000-0000-0000-00006166ecfb/41bc4358-778b-41af-a7fd-b643743fa4cd"
-      (reference "#PWR0114") (unit 1) (value "GND") (footprint "")
-    )
-    (path "/00000000-0000-0000-0000-00006166ecfb/2f3d163f-ec37-4f9f-bf29-45782bfeef0f"
-      (reference "#PWR0115") (unit 1) (value "+BATT") (footprint "")
-    )
-    (path "/00000000-0000-0000-0000-00006166ecfb/6c6a0548-87c7-4f7a-bb5b-ab5803f5e39b"
-      (reference "#PWR0116") (unit 1) (value "+BATT") (footprint "")
-    )
-    (path "/00000000-0000-0000-0000-00006166ecfb/23782083-0aa0-4e02-b8f9-d9eec5ddb2a8"
-      (reference "#PWR0117") (unit 1) (value "GND") (footprint "")
-    )
-    (path "/00000000-0000-0000-0000-00006166ecfb/a05a4346-0edf-416d-ad11-272f76e18098"
-      (reference "#PWR0118") (unit 1) (value "+BATT") (footprint "")
-    )
-    (path "/00000000-0000-0000-0000-00006166ecfb/5cb4a676-36cf-4997-bb65-cd3fd6a895e2"
-      (reference "#PWR0119") (unit 1) (value "GND") (footprint "")
-    )
-    (path "/00000000-0000-0000-0000-00006166ecfb/dfb0fffd-e8a5-405e-8004-b0b4f1649ef0"
-      (reference "#PWR0120") (unit 1) (value "GND") (footprint "")
-    )
-    (path "/00000000-0000-0000-0000-00006166ecfb/ca78b671-ccc8-4d72-b25a-7b1b5974f924"
-      (reference "#PWR0121") (unit 1) (value "+BATT") (footprint "")
-    )
-    (path "/00000000-0000-0000-0000-00006166ecfb/8f02fe52-7106-4eee-88d6-e8fc343bb5b0"
-      (reference "#PWR0122") (unit 1) (value "GND") (footprint "")
-    )
-    (path "/00000000-0000-0000-0000-00006166ecfb/9d0ac6b2-898b-44f0-a415-1933fa98df99"
-      (reference "#PWR0123") (unit 1) (value "+BATT") (footprint "")
-    )
-    (path "/00000000-0000-0000-0000-00006166ecfb/68103582-da79-4feb-9df4-63e37d9e5d66"
-      (reference "#PWR0124") (unit 1) (value "GND") (footprint "")
-    )
-    (path "/00000000-0000-0000-0000-00006166ecfb/fed1968d-af36-482b-b390-8d768aad6d5c"
-      (reference "#PWR0125") (unit 1) (value "+BATT") (footprint "")
-    )
-    (path "/00000000-0000-0000-0000-00006166ecfb/ee32ac0f-9123-4a85-9d2d-7a653f2debbb"
-      (reference "#PWR0126") (unit 1) (value "GND") (footprint "")
-    )
-    (path "/00000000-0000-0000-0000-00006166ecfb/0849840f-f7c7-4f31-9823-c20f9d86659c"
-      (reference "#PWR0127") (unit 1) (value "+BATT") (footprint "")
-    )
     (path "/00000000-0000-0000-0000-00006165e463/d045e7ba-b7a5-4eb8-ba31-1a87a3b8ae7d"
       (reference "#PWR0128") (unit 1) (value "VDD") (footprint "")
@@
       (reference "J2") (unit 1) (value "USB_C_Receptacle_USB2.0") (footprint "CNLJS:USB_C_Receptacle_HRO_TYPE-C-31-M-12")
     )
+    (path "/00000000-0000-0000-0000-00006166ecfb/4a123de1-4959-459b-8ea6-00ce0d5bb79a"
+      (reference "J3") (unit 1) (value "Conn_01x02_Male") (footprint "")
+    )
     (path "/00000000-0000-0000-0000-000061c555c0/2316558d-d6e5-4f42-a145-5ce18e9c2401"
       (reference "L1") (unit 1) (value "47uH") (footprint "CNLJS:L_Taiyo-Yuden_NR-50xx")
@@
       (reference "U4") (unit 1) (value "2108") (footprint "Package_TO_SOT_SMD:SOT-23")
     )
-    (path "/00000000-0000-0000-0000-00006166ecfb/c61728f6-a565-47bc-85a9-538460f05e63"
-      (reference "U5") (unit 1) (value "WS2812-4020_dual") (footprint "Josip_global:WS2812-4020-dual-6mm_bezMaske")
-    )
-    (path "/00000000-0000-0000-0000-00006166ecfb/b20d0817-6e1f-47f1-87be-06097301834d"
-      (reference "U6") (unit 1) (value "WS2812-4020_dual") (footprint "Josip_global:WS2812-4020-dual-6mm_bezMaske")
-    )
-    (path "/00000000-0000-0000-0000-00006166ecfb/e6988795-8bcf-4203-ab19-1f9170f960f3"
-      (reference "U7") (unit 1) (value "WS2812-4020_dual") (footprint "Josip_global:WS2812-4020-dual-6mm_bezMaske")
-    )
-    (path "/00000000-0000-0000-0000-00006166ecfb/377dc56f-67cf-4d58-a286-fd74b001963e"
-      (reference "U8") (unit 1) (value "WS2812-4020_dual") (footprint "Josip_global:WS2812-4020-dual-6mm_bezMaske")
-    )
-    (path "/00000000-0000-0000-0000-00006166ecfb/31a87c8a-4b46-4a45-a3a8-8766e92b52ee"
-      (reference "U9") (unit 1) (value "WS2812-4020_dual") (footprint "Josip_global:WS2812-4020-dual-6mm_bezMaske")
-    )
-    (path "/00000000-0000-0000-0000-00006166ecfb/b7d384ac-11c1-4580-9d0e-0f237463f608"
-      (reference "U10") (unit 1) (value "WS2812-4020_dual") (footprint "Josip_global:WS2812-4020-dual-6mm_bezMaske")
-    )
-    (path "/00000000-0000-0000-0000-00006166ecfb/2d6edfb4-f46d-48ef-9ae6-05cf2fb34a58"
-      (reference "U11") (unit 1) (value "WS2812-4020_dual") (footprint "Josip_global:WS2812-4020-dual-6mm_bezMaske")
-    )
-    (path "/00000000-0000-0000-0000-00006166ecfb/8d25d987-bf34-4cd4-a492-4bc0aa719ef1"
-      (reference "U12") (unit 1) (value "WS2812-4020_dual") (footprint "Josip_global:WS2812-4020-dual-6mm_bezMaske")
-    )
-    (path "/00000000-0000-0000-0000-00006166ecfb/c2bfd050-6cad-4791-96a0-3a01eaee2a12"
-      (reference "U13") (unit 1) (value "WS2812-4020_dual") (footprint "Josip_global:WS2812-4020-dual-6mm_bezMaske")
-    )
-    (path "/00000000-0000-0000-0000-00006166ecfb/d97a8b9d-d009-461d-8bc7-d5f28418e057"
-      (reference "U14") (unit 1) (value "WS2812-4020_dual") (footprint "Josip_global:WS2812-4020-dual-6mm_bezMaske")
-    )
-    (path "/00000000-0000-0000-0000-00006166ecfb/5a761b7e-c070-47bb-a4d0-734466d4119d"
-      (reference "U15") (unit 1) (value "WS2812-4020_dual") (footprint "Josip_global:WS2812-4020-dual-6mm_bezMaske")
-    )
     (path "/00000000-0000-0000-0000-00006165e463/00000000-0000-0000-0000-0000616779d1"

Commit message: update
Other:
- added sheet Touchpad (Touchpad.kicad_sch)
- note added: "TP"
- note removed: "touchpad"

Commit message: update
Other:
- sheet Touchpad renamed IO Expander
- note added: "I/O EXP"
- note removed: "TP"
Changed lines of the file:
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@@
     (effects (font (size 2.9972 2.9972) (thickness 0.5994) bold) (justify left bottom))
   )
-  (text "TP" (at 213.36 131.445 0)
+  (text "I/O EXP" (at 207.01 131.445 0)
     (effects (font (size 2.9972 2.9972) (thickness 0.5994) bold) (justify left bottom))
   )
@@
     (stroke (width 0.1524) (type solid) (color 0 0 0 0))
     (fill (color 0 0 0 0.0000))
-    (property "Sheet name" "Touchpad" (id 0) (at 205.105 122.4784 0)
+    (property "Sheet name" "IO Expander" (id 0) (at 205.105 122.4784 0)
       (effects (font (size 1.27 1.27)) (justify left bottom))
     )

Commit message: update
Other:
- note added: "TODO: - power sklopka koja može prekinuti 1A"
Changed lines of the file:
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@@
+    (effects (font (size 1.27 1.27)) (justify left bottom))
+  )
+  (text "TODO:\n\n- power sklopka koja može prekinuti 1A" (at 18.415 186.055 0)
     (effects (font (size 1.27 1.27)) (justify left bottom))
   )
@@
     )
     (path "/f9d26e2a-d901-40f9-932a-f51e34dd8264/e0d248f8-4d45-4c44-9cbe-ba124146b9fd"
-      (reference "R20") (unit 1) (value "4k7") (footprint "")
+      (reference "R20") (unit 1) (value "4k7") (footprint "Resistor_SMD:R_0805_2012Metric")
     )
     (path "/f9d26e2a-d901-40f9-932a-f51e34dd8264/da14fb81-16d7-4a73-ad65-9fc7097adf93"
-      (reference "R21") (unit 1) (value "4k7") (footprint "")
+      (reference "R21") (unit 1) (value "4k7") (footprint "Resistor_SMD:R_0805_2012Metric")
     )
     (path "/00000000-0000-0000-0000-00006166ecfb/ec148c32-c38a-49d8-bb9a-95d9b3c6258c"

Commit message: update
Other:
- note added: "TODO: - power sklopka koja može prekinuti 1A - rupe"
- note removed: "TODO: - power sklopka koja može prekinuti 1A"

Commit message: update
Other:
- note added: "TODO: - power sklopka koja može prekinuti 1A - rupe - ispraviti dvije pozicije koje su preblizu"
- note removed: "TODO: - power sklopka koja može prekinuti 1A - rupe"
Changed lines of the file:
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@@
     (effects (font (size 1.27 1.27)) (justify left bottom))
   )
-  (text "TODO:\n\n- power sklopka koja može prekinuti 1A\n- rupe"
+  (text "TODO:\n\n- power sklopka koja može prekinuti 1A\n- rupe\n- ispraviti dvije pozicije koje su preblizu"
     (at 18.415 186.055 0)
     (effects (font (size 1.27 1.27)) (justify left bottom))
@@
     (pin "1")
   )
-  (symbol (lib_id "power:GND") (at 269.875 153.67 0) (unit 1)
+  (symbol (lib_id "power:GND") (at 269.875 156.21 0) (unit 1)
     (in_bom yes) (on_board yes) (fields_autoplaced)
-    (property "Reference" "#PWR0256" (id 0) (at 269.875 160.02 0)
-      (effects (font (size 1.27 1.27)) hide)
-    )
-    (property "Value" "GND" (id 1) (at 269.875 158.1134 0))
-    (property "Footprint" "" (id 2) (at 269.875 153.67 0)
-      (effects (font (size 1.27 1.27)) hide)
-    )
-    (property "Datasheet" "" (id 3) (at 269.875 153.67 0)
+    (property "Reference" "#PWR0256" (id 0) (at 269.875 162.56 0)
+      (effects (font (size 1.27 1.27)) hide)
+    )
+    (property "Value" "GND" (id 1) (at 269.875 160.6534 0))
+    (property "Footprint" "" (id 2) (at 269.875 156.21 0)
+      (effects (font (size 1.27 1.27)) hide)
+    )
+    (property "Datasheet" "" (id 3) (at 269.875 156.21 0)
       (effects (font (size 1.27 1.27)) hide)
     )
@@
     (pin "1")
   )
-  (symbol (lib_id "power:PWR_FLAG") (at 269.875 153.67 0) (unit 1)
+  (symbol (lib_id "power:PWR_FLAG") (at 269.875 156.21 0) (unit 1)
     (in_bom yes) (on_board yes) (fields_autoplaced)
-    (property "Reference" "#FLG0101" (id 0) (at 269.875 151.765 0)
-      (effects (font (size 1.27 1.27)) hide)
-    )
-    (property "Value" "PWR_FLAG" (id 1) (at 269.875 150.0942 0))
-    (property "Footprint" "" (id 2) (at 269.875 153.67 0)
-      (effects (font (size 1.27 1.27)) hide)
-    )
-    (property "Datasheet" "~" (id 3) (at 269.875 153.67 0)
+    (property "Reference" "#FLG0101" (id 0) (at 269.875 154.305 0)
+      (effects (font (size 1.27 1.27)) hide)
+    )
+    (property "Value" "PWR_FLAG" (id 1) (at 269.875 152.6342 0))
+    (property "Footprint" "" (id 2) (at 269.875 156.21 0)
+      (effects (font (size 1.27 1.27)) hide)
+    )
+    (property "Datasheet" "~" (id 3) (at 269.875 156.21 0)
       (effects (font (size 1.27 1.27)) hide)
     )
@@
       (reference "#PWR0259") (unit 1) (value "+BATT") (footprint "")
     )
+    (path "/f9d26e2a-d901-40f9-932a-f51e34dd8264/224326e9-6721-42bd-923c-1d80b232d2d7"
+      (reference "#PWR?") (unit 1) (value "GND") (footprint "")
+    )
+    (path "/f9d26e2a-d901-40f9-932a-f51e34dd8264/4b9a06af-3889-4def-b72d-3db0778e8f70"
+      (reference "#PWR?") (unit 1) (value "GND") (footprint "")
+    )
+    (path "/f9d26e2a-d901-40f9-932a-f51e34dd8264/5ec035d5-980b-4bd6-9c7d-5f4aa6d059b4"
+      (reference "#PWR?") (unit 1) (value "GND") (footprint "")
+    )
+    (path "/f9d26e2a-d901-40f9-932a-f51e34dd8264/8239e60d-d898-47c8-912f-74ac7fedd9c6"
+      (reference "#PWR?") (unit 1) (value "VCC") (footprint "")
+    )
+    (path "/f9d26e2a-d901-40f9-932a-f51e34dd8264/8a060ca0-0b97-4550-b3d8-bbe0eec74aa8"
+      (reference "#PWR?") (unit 1) (value "VCC") (footprint "")
+    )
+    (path "/f9d26e2a-d901-40f9-932a-f51e34dd8264/a037445a-51f6-4c7c-9ab4-7237fcd97c9a"
+      (reference "#PWR?") (unit 1) (value "VCC") (footprint "")
+    )
+    (path "/f9d26e2a-d901-40f9-932a-f51e34dd8264/bd970e82-2a41-4aee-9244-6fd79951b48d"
+      (reference "#PWR?") (unit 1) (value "VCC") (footprint "")
+    )
+    (path "/f9d26e2a-d901-40f9-932a-f51e34dd8264/c58a8609-0659-42ba-84bc-36c9a5b1a304"
+      (reference "#PWR?") (unit 1) (value "GND") (footprint "")
+    )
     (path "/00000000-0000-0000-0000-00006165c380/00000000-0000-0000-0000-000061ca59bb"
       (reference "BT1") (unit 1) (value "Battery_Cell") (footprint "CNLJS:JST_PH_S2B-PH-SM4-TB_1x02-1MP_P2.00mm_Horizontal")
@@
       (reference "J2") (unit 1) (value "USB_C_Receptacle_USB2.0") (footprint "CNLJS:USB_C_Receptacle_HRO_TYPE-C-31-M-12")
     )
-    (path "/f9d26e2a-d901-40f9-932a-f51e34dd8264/ce1c4906-9993-48b6-803b-b85ec749e387"
-      (reference "J17") (unit 1) (value "Conn_01x03_Male") (footprint "Connector_PinHeader_2.54mm:PinHeader_1x03_P2.54mm_Vertical")
-    )
-    (path "/f9d26e2a-d901-40f9-932a-f51e34dd8264/a9696cbc-c331-44e1-a0a1-0ba85d32e607"
-      (reference "J18") (unit 1) (value "Conn_01x03_Male") (footprint "Connector_PinHeader_2.54mm:PinHeader_1x03_P2.54mm_Vertical")
-    )
-    (path "/f9d26e2a-d901-40f9-932a-f51e34dd8264/0c0e04c1-71d3-4ae9-ac89-b28fd17b95fe"
-      (reference "J19") (unit 1) (value "Conn_01x03_Male") (footprint "Connector_PinHeader_2.54mm:PinHeader_1x03_P2.54mm_Vertical")
-    )
-    (path "/f9d26e2a-d901-40f9-932a-f51e34dd8264/36ba6937-0893-4bfd-a918-18393dc34f97"
-      (reference "J20") (unit 1) (value "Conn_01x03_Male") (footprint "Connector_PinHeader_2.54mm:PinHeader_1x03_P2.54mm_Vertical")
+    (path "/f9d26e2a-d901-40f9-932a-f51e34dd8264/51b95aa3-e727-4d4c-a49c-fca270ad13c2"
+      (reference "J?") (unit 1) (value "Conn_01x06") (footprint "")
     )
     (path "/00000000-0000-0000-0000-000061c555c0/2316558d-d6e5-4f42-a145-5ce18e9c2401"
