File: KiCad files/Main Project/CNLJS.kicad_sch (KiCad schematic)
At the start: 0 parts

Commit message: update
Other:
- note added: "TODO: - simbol i footprint regulatora napona - power sklopka koja može prekinuti 1A - rupe - ispraviti dvije pozicije koje su preblizu"
- note removed: "TODO: - power sklopka koja može prekinuti 1A - rupe - ispraviti dvije pozicije koje su preblizu"
Changed lines of the file:
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@@
     (effects (font (size 1.27 1.27)) (justify left bottom))
   )
-  (text "TODO:\n\n- power sklopka koja može prekinuti 1A\n- rupe\n- ispraviti dvije pozicije koje su preblizu"
+  (text "TODO:\n\n- simbol i footprint regulatora napona\n- power sklopka koja može prekinuti 1A\n- rupe\n- ispraviti dvije pozicije koje su preblizu"
     (at 18.415 186.055 0)
     (effects (font (size 1.27 1.27)) (justify left bottom))
@@
       (reference "D16") (unit 1) (value "SS14") (footprint "Diode_SMD:D_SMA")
     )
-    (path "/00000000-0000-0000-0000-00006165c380/00000000-0000-0000-0000-000061c5d210"
-      (reference "F1") (unit 1) (value "1A") (footprint "Fuse:Fuse_1206_3216Metric_Pad1.42x1.75mm_HandSolder")
-    )
     (path "/00000000-0000-0000-0000-00006166ecfb/0fad21f5-d92d-48ee-888d-008cd1e4dd00/ae0b6982-f26e-4c7f-870c-208a6ca654b7"

Commit message: update
Other:
- note added: "TODO: - ako je spojen VBUS, onda ne dovoditi VCC na regulator napona - power sklopka koja može prekinuti 1A - rupe - ispraviti dvije pozicije koje su preblizu"
- note removed: "TODO: - simbol i footprint regulatora napona - power sklopka koja može prekinuti 1A - rupe - ispraviti dvije pozicije koje su preblizu"
Changed lines of the file:
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@@
     (effects (font (size 1.27 1.27)) (justify left bottom))
   )
-  (text "TODO:\n\n- simbol i footprint regulatora napona\n- power sklopka koja može prekinuti 1A\n- rupe\n- ispraviti dvije pozicije koje su preblizu"
+  (text "TODO:\n\n- ako je spojen VBUS, onda ne dovoditi VCC na regulator napona\n- power sklopka koja može prekinuti 1A\n- rupe\n- ispraviti dvije pozicije koje su preblizu"
     (at 18.415 186.055 0)
     (effects (font (size 1.27 1.27)) (justify left bottom))
@@
     (pin "1")
   )
-  (symbol (lib_id "power:PWR_FLAG") (at 223.52 156.21 180) (unit 1)
-    (in_bom yes) (on_board yes) (fields_autoplaced)
-    (property "Reference" "#FLG017" (id 0) (at 223.52 158.115 0)
-      (effects (font (size 1.27 1.27)) hide)
-    )
-    (property "Value" "PWR_FLAG" (id 1) (at 225.171 157.9138 0)
-      (effects (font (size 1.27 1.27)) (justify right))
-    )
-    (property "Footprint" "" (id 2) (at 223.52 156.21 0)
-      (effects (font (size 1.27 1.27)) hide)
-    )
-    (property "Datasheet" "~" (id 3) (at 223.52 156.21 0)
-      (effects (font (size 1.27 1.27)) hide)
-    )
-    (pin "1")
-  )
   (symbol (lib_id "power:VBUS") (at 254 156.21 0) (unit 1)
     (in_bom yes) (on_board yes) (fields_autoplaced)
@@
     )
     (property "Datasheet" "" (id 3) (at 254 156.21 0)
-      (effects (font (size 1.27 1.27)) hide)
-    )
-    (pin "1")
-  )
-  (symbol (lib_id "power:+BATT") (at 223.52 156.21 0) (unit 1)
-    (in_bom yes) (on_board yes) (fields_autoplaced)
-    (property "Reference" "#PWR0259" (id 0) (at 223.52 160.02 0)
-      (effects (font (size 1.27 1.27)) hide)
-    )
-    (property "Value" "+BATT" (id 1) (at 223.52 152.6342 0))
-    (property "Footprint" "" (id 2) (at 223.52 156.21 0)
-      (effects (font (size 1.27 1.27)) hide)
-    )
-    (property "Datasheet" "" (id 3) (at 223.52 156.21 0)
       (effects (font (size 1.27 1.27)) hide)
     )
@@
   )
   (symbol_instances
-    (path "/a365a5c3-a7f1-4e1e-a88d-d7ac72c8a5b4"
-      (reference "#FLG017") (unit 1) (value "PWR_FLAG") (footprint "")
-    )
     (path "/00000000-0000-0000-0000-00006165e463/19cdce5a-54ad-4d2a-bfdd-cc69216c4c9f"
       (reference "#FLG018") (unit 1) (value "PWR_FLAG") (footprint "")
@@
       (reference "#PWR0226") (unit 1) (value "GND") (footprint "")
     )
-    (path "/f9d26e2a-d901-40f9-932a-f51e34dd8264/1b936b10-bd0b-4cd2-a118-96aed6cc58d6"
-      (reference "#PWR0227") (unit 1) (value "VCC") (footprint "")
-    )
-    (path "/f9d26e2a-d901-40f9-932a-f51e34dd8264/fb71447b-1d46-4ddb-9bef-457de3e1fea9"
-      (reference "#PWR0228") (unit 1) (value "VCC") (footprint "")
+    (path "/f9d26e2a-d901-40f9-932a-f51e34dd8264/e62e149d-dc97-434c-8523-ab381540ffeb"
+      (reference "#PWR0227") (unit 1) (value "VDD") (footprint "")
+    )
+    (path "/f9d26e2a-d901-40f9-932a-f51e34dd8264/af277ab5-0337-440d-be85-051c8c2fab4c"
+      (reference "#PWR0228") (unit 1) (value "VDD") (footprint "")
     )
     (path "/f9d26e2a-d901-40f9-932a-f51e34dd8264/cc86950e-a532-483c-89b4-26a352c5501e"
       (reference "#PWR0229") (unit 1) (value "GND") (footprint "")
     )
-    (path "/f9d26e2a-d901-40f9-932a-f51e34dd8264/76ae9489-bb8e-4cf9-90d1-cbd64a055f9a"
-      (reference "#PWR0230") (unit 1) (value "VCC") (footprint "")
-    )
-    (path "/f9d26e2a-d901-40f9-932a-f51e34dd8264/a78735ab-40aa-4624-91c9-198c425b3e97"
-      (reference "#PWR0231") (unit 1) (value "VCC") (footprint "")
+    (path "/f9d26e2a-d901-40f9-932a-f51e34dd8264/7bb4082c-4708-4435-9495-4b0ab25b949c"
+      (reference "#PWR0230") (unit 1) (value "VDD") (footprint "")
+    )
+    (path "/f9d26e2a-d901-40f9-932a-f51e34dd8264/aafc586b-6d3d-4f57-aa92-2137355548f4"
+      (reference "#PWR0231") (unit 1) (value "VDD") (footprint "")
     )
     (path "/00000000-0000-0000-0000-00006166ecfb/a13ff330-ccbe-4157-b6cf-ffb97876cacd"
@@
       (reference "#PWR0258") (unit 1) (value "VCC") (footprint "")
     )
-    (path "/d15fae73-f2e2-41df-8bff-bf5121e77911"
-      (reference "#PWR0259") (unit 1) (value "+BATT") (footprint "")
-    )
-    (path "/f9d26e2a-d901-40f9-932a-f51e34dd8264/dbe6d465-f0c0-4d17-9b0b-89f1e30bbe0b"
-      (reference "#PWR0260") (unit 1) (value "VCC") (footprint "")
-    )
-    (path "/f9d26e2a-d901-40f9-932a-f51e34dd8264/0232ec8a-0781-48d3-91a3-712928f386cf"
-      (reference "#PWR0261") (unit 1) (value "VCC") (footprint "")
+    (path "/f9d26e2a-d901-40f9-932a-f51e34dd8264/ad866e92-da51-4123-b690-13a056a00cdf"
+      (reference "#PWR0259") (unit 1) (value "VDD") (footprint "")
+    )
+    (path "/f9d26e2a-d901-40f9-932a-f51e34dd8264/59fa2d8e-1ada-4920-8c01-f1ebdc9d5157"
+      (reference "#PWR0260") (unit 1) (value "VDD") (footprint "")
+    )
+    (path "/f9d26e2a-d901-40f9-932a-f51e34dd8264/615193ac-fb7d-46d4-9609-e5a91655a8a1"
+      (reference "#PWR0261") (unit 1) (value "VDD") (footprint "")
     )
     (path "/f9d26e2a-d901-40f9-932a-f51e34dd8264/05c1dbfd-1fdd-4b78-8b5c-11c9b323b91a"
       (reference "#PWR0262") (unit 1) (value "GND") (footprint "")
     )
-    (path "/f9d26e2a-d901-40f9-932a-f51e34dd8264/a5267b66-74d2-406c-98c0-cc2a751750b9"
-      (reference "#PWR0263") (unit 1) (value "VCC") (footprint "")
-    )
-    (path "/f9d26e2a-d901-40f9-932a-f51e34dd8264/f0491c0d-7706-4405-97e7-575ea56c9bdf"
-      (reference "#PWR0264") (unit 1) (value "VCC") (footprint "")
+    (path "/f9d26e2a-d901-40f9-932a-f51e34dd8264/bedb0b38-5d9d-4774-a03b-b03163ab2f1f"
+      (reference "#PWR0263") (unit 1) (value "VDD") (footprint "")
+    )
+    (path "/f9d26e2a-d901-40f9-932a-f51e34dd8264/90ea5f9f-fb78-4345-b300-6d1dfc62052e"
+      (reference "#PWR0264") (unit 1) (value "VDD") (footprint "")
     )
     (path "/f9d26e2a-d901-40f9-932a-f51e34dd8264/76ec0616-3436-4caa-a6e5-f92b07e4aa60"
       (reference "#PWR0265") (unit 1) (value "GND") (footprint "")
     )
-    (path "/f9d26e2a-d901-40f9-932a-f51e34dd8264/b517bf74-efef-4bde-a057-6d30e59ca24c"
-      (reference "#PWR0266") (unit 1) (value "VCC") (footprint "")
-    )
-    (path "/f9d26e2a-d901-40f9-932a-f51e34dd8264/b5ce72e8-fc7c-4d88-831b-4ea75cc659d8"
-      (reference "#PWR0267") (unit 1) (value "VCC") (footprint "")
+    (path "/f9d26e2a-d901-40f9-932a-f51e34dd8264/23ccb30f-82d7-44b5-9ee0-8106e1872971"
+      (reference "#PWR0266") (unit 1) (value "VDD") (footprint "")
+    )
+    (path "/f9d26e2a-d901-40f9-932a-f51e34dd8264/a86aa3e5-976f-4bf3-86ba-b60860c43415"
+      (reference "#PWR0267") (unit 1) (value "VDD") (footprint "")
     )
     (path "/f9d26e2a-d901-40f9-932a-f51e34dd8264/2925481e-08e4-479c-b152-d8651139facd"
       (reference "#PWR0268") (unit 1) (value "GND") (footprint "")
     )
-    (path "/f9d26e2a-d901-40f9-932a-f51e34dd8264/af984e30-7091-4a33-8f8a-928b314d5bf6"
-      (reference "#PWR0269") (unit 1) (value "VCC") (footprint "")
-    )
-    (path "/f9d26e2a-d901-40f9-932a-f51e34dd8264/59b9bc1c-c8b3-4840-9e74-079af1db52f4"
-      (reference "#PWR0270") (unit 1) (value "VCC") (footprint "")
+    (path "/f9d26e2a-d901-40f9-932a-f51e34dd8264/2ba41624-20cc-41a6-9c0d-1249b94007aa"
+      (reference "#PWR0269") (unit 1) (value "VDD") (footprint "")
     )
     (path "/f9d26e2a-d901-40f9-932a-f51e34dd8264/09f18de3-3583-4c3e-bbbf-26e9afd221eb"
       (reference "#PWR0271") (unit 1) (value "GND") (footprint "")
     )
+    (path "/00000000-0000-0000-0000-000061c3bc04/e895b2a7-400f-4f1f-979b-1deddd7fb9ef"
+      (reference "#PWR0272") (unit 1) (value "GND") (footprint "")
+    )
     (path "/00000000-0000-0000-0000-00006165c380/00000000-0000-0000-0000-000061ca59bb"
       (reference "BT1") (unit 1) (value "Battery_Cell") (footprint "CNLJS:JST_PH_S2B-PH-SM4-TB_1x02-1MP_P2.00mm_Horizontal")
@@
       (reference "R22") (unit 1) (value "470R") (footprint "Resistor_SMD:R_0603_1608Metric")
     )
+    (path "/00000000-0000-0000-0000-000061c3bc04/0591dc1a-2acd-487b-bc0c-1292f826b676"
+      (reference "R23") (unit 1) (value "1M") (footprint "Resistor_SMD:R_0805_2012Metric")
+    )
     (path "/00000000-0000-0000-0000-00006166ecfb/ec148c32-c38a-49d8-bb9a-95d9b3c6258c"
       (reference "R33") (unit 1) (value "470R") (footprint "Resistor_SMD:R_0603_1608Metric")
@@
     )
     (path "/00000000-0000-0000-0000-000061c555c0/457ced6b-c526-484b-8527-872cff7f6796"
-      (reference "U4") (unit 1) (value "2108") (footprint "Package_TO_SOT_SMD:SOT-23")
+      (reference "U4") (unit 1) (value "2108") (footprint "Package_TO_SOT_SMD:SOT-89-3_Handsoldering")
     )
     (path "/f9d26e2a-d901-40f9-932a-f51e34dd8264/78ff6519-41f4-4b2c-9518-f9ed158fb1f3"

Commit message: update
Other:
- note added: "TODO: - ako je spojen VBUS, onda ne dovoditi VCC na regulator napona - power sklopka koja može prekinuti 1A - rupe - ispraviti dvije pozicije koje su preblizu - kockica tipkalo"
- note removed: "TODO: - ako je spojen VBUS, onda ne dovoditi VCC na regulator napona - power sklopka koja može prekinuti 1A - rupe - ispraviti dvije pozicije koje su preblizu"
Changed lines of the file:
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@@
     (effects (font (size 1.27 1.27)) (justify left bottom))
   )
-  (text "TODO:\n\n- ako je spojen VBUS, onda ne dovoditi VCC na regulator napona\n- power sklopka koja može prekinuti 1A\n- rupe\n- ispraviti dvije pozicije koje su preblizu"
+  (text "TODO:\n\n- ako je spojen VBUS, onda ne dovoditi VCC na regulator napona\n- power sklopka koja može prekinuti 1A\n- rupe\n- ispraviti dvije pozicije koje su preblizu\n- kockica tipkalo"
     (at 18.415 186.055 0)
     (effects (font (size 1.27 1.27)) (justify left bottom))

Commit message: update
Other:
- note added: "TODO: - ako je spojen VBUS, onda ne dovoditi VCC na regulator napona - power sklopka koja može prekinuti 1A - rupe za montažu - ispraviti dvije pozicije koje su preblizu - kockica tipkalo - LEDice za punjenje baterije"
- note removed: "TODO: - ako je spojen VBUS, onda ne dovoditi VCC na regulator napona - power sklopka koja može prekinuti 1A - rupe - ispraviti dvije pozicije koje su preblizu - kockica tipkalo"
Changed lines of the file:
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@@
     (effects (font (size 1.27 1.27)) (justify left bottom))
   )
-  (text "TODO:\n\n- ako je spojen VBUS, onda ne dovoditi VCC na regulator napona\n- power sklopka koja može prekinuti 1A\n- rupe\n- ispraviti dvije pozicije koje su preblizu\n- kockica tipkalo"
+  (text "TODO:\n\n- ako je spojen VBUS, onda ne dovoditi VCC na regulator napona\n- power sklopka koja može prekinuti 1A\n- rupe za montažu\n- ispraviti dvije pozicije koje su preblizu\n- kockica tipkalo\n- LEDice za punjenje baterije"
     (at 18.415 186.055 0)
     (effects (font (size 1.27 1.27)) (justify left bottom))
