File: KiCad files/Main Project/Power.kicad_sch (KiCad schematic)
At the start: 23 parts, among them SW2 SW_SPDT, U2 MCP73871-2CC

Commit message: update
Parts:
- removed F1: 1A, Fuse:Fuse_1206_3216Metric_Pad1.42x1.75mm_HandSolder, symbol Device:Fuse_Small
Connections:
- net +BATT: now also C16.1, U2.14 (VBAT), U2.15 (VBAT), U2.16 (Vbat_SENSE)
Changed lines of the file:
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@@
     (stroke (width 0) (type default) (color 0 0 0 0))
   )
-  (wire (pts (xy 166.37 85.725) (xy 158.115 85.725))
+  (wire (pts (xy 158.115 85.725) (xy 175.895 85.725))
     (stroke (width 0) (type default) (color 0 0 0 0))
   )
@@
   )
   (wire (pts (xy 56.515 90.17) (xy 56.515 91.44))
-    (stroke (width 0) (type default) (color 0 0 0 0))
-  )
-  (wire (pts (xy 171.45 85.725) (xy 175.895 85.725))
     (stroke (width 0) (type default) (color 0 0 0 0))
   )
@@
     (pin "1")
   )
-  (symbol (lib_id "Device:Fuse_Small") (at 168.91 85.725 0) (unit 1)
-    (in_bom yes) (on_board yes)
-    (property "Reference" "F1" (id 0) (at 168.91 83.82 0))
-    (property "Value" "1A" (id 1) (at 168.91 87.63 0))
-    (property "Footprint" "Fuse:Fuse_1206_3216Metric_Pad1.42x1.75mm_HandSolder" (id 2) (at 168.91 85.725 0)
-      (effects (font (size 1.27 1.27)) hide)
-    )
-    (property "Datasheet" "~" (id 3) (at 168.91 85.725 0)
-      (effects (font (size 1.27 1.27)) hide)
-    )
-    (property "Basic/Extended" "Extended" (id 4) (at 168.91 85.725 0)
-      (effects (font (size 1.27 1.27)) hide)
-    )
-    (property "JLCPCB Part #" "C135338" (id 5) (at 168.91 85.725 0)
-      (effects (font (size 1.27 1.27)) hide)
-    )
-    (property "U labosu?" "Ne" (id 6) (at 168.91 85.725 0)
-      (effects (font (size 1.27 1.27)) hide)
-    )
-    (pin "1")
-    (pin "2")
-  )
   (symbol (lib_id "power:VBUS") (at 184.785 94.615 0) (unit 1)

Commit message: update
Connections:
- net CH_OUT: now reaches C15.1, SW2.2 (B), U2.1 (OUT), U2.20 (OUT)
Changed lines of the file:
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@@
+    (effects (font (size 1.27 1.27)) (justify left bottom))
+  )
+  (label "CH_OUT" (at 152.4 73.025 0)
     (effects (font (size 1.27 1.27)) (justify left bottom))
   )

Commit message: update
Parts:
- removed SW2: SW_SPDT, Button_Switch_SMD:SW_SPDT_PCM12, symbol Switch:SW_SPDT
- added J21, J22: Conn_01x01, CNLJS:Padovi_sklopke, symbol Connector_Generic:Conn_01x01
Connections:
- net CH_OUT: now also J22.1 (Pin_1)
- net VCC: now also J21.1 (Pin_1)
- no-connect marks 1 -> 0
Other:
- note added: "PADOVI SKLOPKE"
- note removed: "MAIN SWITCH"
Changed lines of the file:
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@@
   (junction (at 175.895 85.725) (diameter 0) (color 0 0 0 0)
   )
-  (no_connect (at 177.8 75.565))
   (wire (pts (xy 66.04 88.9) (xy 66.04 90.805))
     (stroke (width 0) (type default) (color 0 0 0 0))
@@
     (effects (font (size 0.9906 0.9906)) (justify left bottom))
   )
-  (text "MAIN SWITCH" (at 167.64 66.675 0)
+  (text "PADOVI\nSKLOPKE" (at 167.64 66.675 0)
     (effects (font (size 1.27 1.27)) (justify left bottom))
   )
@@
     (pin "1")
   )
-  (symbol (lib_id "Switch:SW_SPDT") (at 172.72 73.025 0) (unit 1)
+  (symbol (lib_id "Connector_Generic:Conn_01x01") (at 172.72 73.025 0) (unit 1)
     (in_bom yes) (on_board yes) (fields_autoplaced)
-    (property "Reference" "SW2" (id 0) (at 172.72 68.9125 0))
-    (property "Value" "SW_SPDT" (id 1) (at 172.72 68.9126 0)
-      (effects (font (size 1.27 1.27)) hide)
-    )
-    (property "Footprint" "Button_Switch_SMD:SW_SPDT_PCM12" (id 2) (at 172.72 73.025 0)
+    (property "Reference" "J22" (id 0) (at 174.752 73.4588 0)
+      (effects (font (size 1.27 1.27)) (justify left) hide)
+    )
+    (property "Value" "Conn_01x01" (id 1) (at 174.752 74.7272 0)
+      (effects (font (size 1.27 1.27)) (justify left) hide)
+    )
+    (property "Footprint" "CNLJS:Padovi_sklopke" (id 2) (at 172.72 73.025 0)
       (effects (font (size 1.27 1.27)) hide)
     )
@@
     )
     (pin "1")
-    (pin "2")
-    (pin "3")
+  )
+  (symbol (lib_id "Connector_Generic:Conn_01x01") (at 172.72 70.485 180) (unit 1)
+    (in_bom yes) (on_board yes) (fields_autoplaced)
+    (property "Reference" "J21" (id 0) (at 170.688 70.0512 0)
+      (effects (font (size 1.27 1.27)) (justify left) hide)
+    )
+    (property "Value" "Conn_01x01" (id 1) (at 170.688 68.7828 0)
+      (effects (font (size 1.27 1.27)) (justify left) hide)
+    )
+    (property "Footprint" "CNLJS:Padovi_sklopke" (id 2) (at 172.72 70.485 0)
+      (effects (font (size 1.27 1.27)) hide)
+    )
+    (property "Datasheet" "~" (id 3) (at 172.72 70.485 0)
+      (effects (font (size 1.27 1.27)) hide)
+    )
+    (pin "1")
   )
 )

Commit message: update
Parts:
- removed R10: 270k, Resistor_SMD:R_0805_2012Metric, symbol Device:R_Small
- removed R11: 100k, Resistor_SMD:R_0805_2012Metric, symbol Device:R_Small
Connections:
- net VBUS: now also U2.2 (VPCC)
Other:
- note added: "Preinake na modulu: 1. pin 3 (SEL) preko 10k otpornika spojen na GND (USB način rada) 2. pin 2 (VPCC) kratko spojen na pin 18 (VIN)"
- moved on the sheet: C13, C14
