File: KiCad files/Main Project/Cube.kicad_sch (KiCad schematic)
At the start: 9 parts

Commit message: shematic update
Parts:
- renumbered LED1 to LED17, LED2 to LED18, LED3 to LED19, LED4 to LED20, LED5 to LED21, LED6 to LED22, LED7 to LED23, LED8 to LED24, LED9 to LED25
Changed lines of the file:
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@@
   (symbol (lib_id "power:GND") (at 119.38 97.155 0) (unit 1)
     (in_bom yes) (on_board yes) (fields_autoplaced)
-    (property "Reference" "#PWR042" (id 0) (at 119.38 103.505 0)
+    (property "Reference" "#PWR0160" (id 0) (at 119.38 103.505 0)
       (effects (font (size 1.27 1.27)) hide)
     )
@@
   (symbol (lib_id "power:VCC") (at 220.98 81.915 0) (unit 1)
     (in_bom yes) (on_board yes) (fields_autoplaced)
-    (property "Reference" "#PWR0189" (id 0) (at 220.98 85.725 0)
+    (property "Reference" "#PWR0156" (id 0) (at 220.98 85.725 0)
       (effects (font (size 1.27 1.27)) hide)
     )
@@
   (symbol (lib_id "power:GND") (at 241.3 97.155 0) (unit 1)
     (in_bom yes) (on_board yes) (fields_autoplaced)
-    (property "Reference" "#PWR082" (id 0) (at 241.3 103.505 0)
+    (property "Reference" "#PWR0166" (id 0) (at 241.3 103.505 0)
       (effects (font (size 1.27 1.27)) hide)
     )
@@
   (symbol (lib_id "power:GND") (at 220.98 97.155 0) (unit 1)
     (in_bom yes) (on_board yes) (fields_autoplaced)
-    (property "Reference" "#PWR080" (id 0) (at 220.98 103.505 0)
+    (property "Reference" "#PWR0165" (id 0) (at 220.98 103.505 0)
       (effects (font (size 1.27 1.27)) hide)
     )
@@
   (symbol (lib_id "LED:WS2812B") (at 119.38 89.535 0) (unit 1)
     (in_bom yes) (on_board yes)
-    (property "Reference" "LED3" (id 0) (at 114.3 81.915 0))
+    (property "Reference" "LED19" (id 0) (at 114.3 81.915 0))
     (property "Value" "WS2812-4020_single" (id 1) (at 129.54 97.155 0)
       (effects (font (size 1.27 1.27)) hide)
@@
   (symbol (lib_id "power:VCC") (at 99.06 81.915 0) (unit 1)
     (in_bom yes) (on_board yes) (fields_autoplaced)
-    (property "Reference" "#PWR0177" (id 0) (at 99.06 85.725 0)
+    (property "Reference" "#PWR0150" (id 0) (at 99.06 85.725 0)
       (effects (font (size 1.27 1.27)) hide)
     )
@@
   (symbol (lib_id "LED:WS2812B") (at 241.3 89.535 0) (unit 1)
     (in_bom yes) (on_board yes)
-    (property "Reference" "LED9" (id 0) (at 236.22 81.915 0))
+    (property "Reference" "LED25" (id 0) (at 236.22 81.915 0))
     (property "Value" "WS2812-4020_single" (id 1) (at 251.46 97.155 0)
       (effects (font (size 1.27 1.27)) hide)
@@
   (symbol (lib_id "power:VCC") (at 119.38 81.915 0) (unit 1)
     (in_bom yes) (on_board yes) (fields_autoplaced)
-    (property "Reference" "#PWR0175" (id 0) (at 119.38 85.725 0)
+    (property "Reference" "#PWR0151" (id 0) (at 119.38 85.725 0)
       (effects (font (size 1.27 1.27)) hide)
     )
@@
   (symbol (lib_id "power:GND") (at 139.7 97.155 0) (unit 1)
     (in_bom yes) (on_board yes) (fields_autoplaced)
-    (property "Reference" "#PWR046" (id 0) (at 139.7 103.505 0)
+    (property "Reference" "#PWR0161" (id 0) (at 139.7 103.505 0)
       (effects (font (size 1.27 1.27)) hide)
     )
@@
   (symbol (lib_id "LED:WS2812B") (at 160.02 89.535 0) (unit 1)
     (in_bom yes) (on_board yes)
-    (property "Reference" "LED5" (id 0) (at 154.94 81.915 0))
+    (property "Reference" "LED21" (id 0) (at 154.94 81.915 0))
     (property "Value" "WS2812-4020_single" (id 1) (at 170.18 97.155 0)
       (effects (font (size 1.27 1.27)) hide)
@@
   (symbol (lib_id "power:GND") (at 200.66 97.155 0) (unit 1)
     (in_bom yes) (on_board yes) (fields_autoplaced)
-    (property "Reference" "#PWR078" (id 0) (at 200.66 103.505 0)
+    (property "Reference" "#PWR0164" (id 0) (at 200.66 103.505 0)
       (effects (font (size 1.27 1.27)) hide)
     )
@@
   (symbol (lib_id "power:GND") (at 99.06 97.155 0) (unit 1)
     (in_bom yes) (on_board yes) (fields_autoplaced)
-    (property "Reference" "#PWR040" (id 0) (at 99.06 103.505 0)
+    (property "Reference" "#PWR0159" (id 0) (at 99.06 103.505 0)
       (effects (font (size 1.27 1.27)) hide)
     )
@@
   (symbol (lib_id "LED:WS2812B") (at 200.66 89.535 0) (unit 1)
     (in_bom yes) (on_board yes)
-    (property "Reference" "LED7" (id 0) (at 195.58 81.915 0))
+    (property "Reference" "LED23" (id 0) (at 195.58 81.915 0))
     (property "Value" "WS2812-4020_single" (id 1) (at 210.82 97.155 0)
       (effects (font (size 1.27 1.27)) hide)
@@
   (symbol (lib_id "power:VCC") (at 160.02 81.915 0) (unit 1)
     (in_bom yes) (on_board yes) (fields_autoplaced)
-    (property "Reference" "#PWR0185" (id 0) (at 160.02 85.725 0)
+    (property "Reference" "#PWR0153" (id 0) (at 160.02 85.725 0)
       (effects (font (size 1.27 1.27)) hide)
     )
@@
   (symbol (lib_id "power:VCC") (at 241.3 81.915 0) (unit 1)
     (in_bom yes) (on_board yes) (fields_autoplaced)
-    (property "Reference" "#PWR0173" (id 0) (at 241.3 85.725 0)
+    (property "Reference" "#PWR0157" (id 0) (at 241.3 85.725 0)
       (effects (font (size 1.27 1.27)) hide)
     )
@@
   (symbol (lib_id "power:GND") (at 180.34 97.155 0) (unit 1)
     (in_bom yes) (on_board yes) (fields_autoplaced)
-    (property "Reference" "#PWR071" (id 0) (at 180.34 103.505 0)
+    (property "Reference" "#PWR0163" (id 0) (at 180.34 103.505 0)
       (effects (font (size 1.27 1.27)) hide)
     )
@@
   (symbol (lib_id "power:VCC") (at 180.34 81.915 0) (unit 1)
     (in_bom yes) (on_board yes) (fields_autoplaced)
-    (property "Reference" "#PWR0181" (id 0) (at 180.34 85.725 0)
+    (property "Reference" "#PWR0154" (id 0) (at 180.34 85.725 0)
       (effects (font (size 1.27 1.27)) hide)
     )
@@
   (symbol (lib_id "LED:WS2812B") (at 99.06 89.535 0) (unit 1)
     (in_bom yes) (on_board yes)
-    (property "Reference" "LED2" (id 0) (at 93.98 81.915 0))
+    (property "Reference" "LED18" (id 0) (at 93.98 81.915 0))
     (property "Value" "WS2812-4020_single" (id 1) (at 109.22 97.155 0)
       (effects (font (size 1.27 1.27)) hide)
@@
   (symbol (lib_id "LED:WS2812B") (at 139.7 89.535 0) (unit 1)
     (in_bom yes) (on_board yes)
-    (property "Reference" "LED4" (id 0) (at 134.62 81.915 0))
+    (property "Reference" "LED20" (id 0) (at 134.62 81.915 0))
     (property "Value" "WS2812-4020_single" (id 1) (at 149.86 97.155 0)
       (effects (font (size 1.27 1.27)) hide)
@@
   (symbol (lib_id "power:VCC") (at 78.74 81.915 0) (unit 1)
     (in_bom yes) (on_board yes) (fields_autoplaced)
-    (property "Reference" "#PWR0179" (id 0) (at 78.74 85.725 0)
+    (property "Reference" "#PWR0149" (id 0) (at 78.74 85.725 0)
       (effects (font (size 1.27 1.27)) hide)
     )
@@
   (symbol (lib_id "LED:WS2812B") (at 180.34 89.535 0) (unit 1)
     (in_bom yes) (on_board yes)
-    (property "Reference" "LED6" (id 0) (at 175.26 81.915 0))
+    (property "Reference" "LED22" (id 0) (at 175.26 81.915 0))
     (property "Value" "WS2812-4020_single" (id 1) (at 190.5 97.155 0)
       (effects (font (size 1.27 1.27)) hide)
@@
   (symbol (lib_id "power:VCC") (at 200.66 81.915 0) (unit 1)
     (in_bom yes) (on_board yes) (fields_autoplaced)
-    (property "Reference" "#PWR0187" (id 0) (at 200.66 85.725 0)
+    (property "Reference" "#PWR0155" (id 0) (at 200.66 85.725 0)
       (effects (font (size 1.27 1.27)) hide)
     )
@@
   (symbol (lib_id "LED:WS2812B") (at 220.98 89.535 0) (unit 1)
     (in_bom yes) (on_board yes)
-    (property "Reference" "LED8" (id 0) (at 215.9 81.915 0))
+    (property "Reference" "LED24" (id 0) (at 215.9 81.915 0))
     (property "Value" "WS2812-4020_single" (id 1) (at 231.14 97.155 0)
       (effects (font (size 1.27 1.27)) hide)
@@
   (symbol (lib_id "power:VCC") (at 139.7 81.915 0) (unit 1)
     (in_bom yes) (on_board yes) (fields_autoplaced)
-    (property "Reference" "#PWR0183" (id 0) (at 139.7 85.725 0)
+    (property "Reference" "#PWR0152" (id 0) (at 139.7 85.725 0)
       (effects (font (size 1.27 1.27)) hide)
     )
@@
   (symbol (lib_id "LED:WS2812B") (at 78.74 89.535 0) (unit 1)
     (in_bom yes) (on_board yes)
-    (property "Reference" "LED1" (id 0) (at 73.66 81.915 0))
+    (property "Reference" "LED17" (id 0) (at 73.66 81.915 0))
     (property "Value" "WS2812-4020_single" (id 1) (at 88.9 97.155 0)
       (effects (font (size 1.27 1.27)) hide)
@@
   (symbol (lib_id "power:GND") (at 78.74 97.155 0) (unit 1)
     (in_bom yes) (on_board yes) (fields_autoplaced)
-    (property "Reference" "#PWR038" (id 0) (at 78.74 103.505 0)
+    (property "Reference" "#PWR0158" (id 0) (at 78.74 103.505 0)
       (effects (font (size 1.27 1.27)) hide)
     )
@@
   (symbol (lib_id "power:GND") (at 160.02 97.155 0) (unit 1)
     (in_bom yes) (on_board yes) (fields_autoplaced)
-    (property "Reference" "#PWR058" (id 0) (at 160.02 103.505 0)
-      (effects (font (size 1.27 1.27)) hide)
-    )
+    (property "Reference" "#PWR0162" (id 0) (at 160.02 103.505 0)
+      (effects (font (size 1.27 1.27)) hide)
+    )

Commit message: update
Parts:
- renumbered LED17 to LED1, LED18 to LED2, LED19 to LED3, LED20 to LED4, LED21 to LED5, LED22 to LED6, LED23 to LED7, LED24 to LED8, LED25 to LED9
Changed lines of the file:
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@@
   (symbol (lib_id "power:GND") (at 119.38 97.155 0) (unit 1)
     (in_bom yes) (on_board yes) (fields_autoplaced)
-    (property "Reference" "#PWR0160" (id 0) (at 119.38 103.505 0)
+    (property "Reference" "#PWR0144" (id 0) (at 119.38 103.505 0)
       (effects (font (size 1.27 1.27)) hide)
     )
@@
   (symbol (lib_id "power:VCC") (at 220.98 81.915 0) (unit 1)
     (in_bom yes) (on_board yes) (fields_autoplaced)
-    (property "Reference" "#PWR0156" (id 0) (at 220.98 85.725 0)
+    (property "Reference" "#PWR0140" (id 0) (at 220.98 85.725 0)
       (effects (font (size 1.27 1.27)) hide)
     )
@@
   (symbol (lib_id "power:GND") (at 241.3 97.155 0) (unit 1)
     (in_bom yes) (on_board yes) (fields_autoplaced)
-    (property "Reference" "#PWR0166" (id 0) (at 241.3 103.505 0)
+    (property "Reference" "#PWR0150" (id 0) (at 241.3 103.505 0)
       (effects (font (size 1.27 1.27)) hide)
     )
@@
   (symbol (lib_id "power:GND") (at 220.98 97.155 0) (unit 1)
     (in_bom yes) (on_board yes) (fields_autoplaced)
-    (property "Reference" "#PWR0165" (id 0) (at 220.98 103.505 0)
+    (property "Reference" "#PWR0149" (id 0) (at 220.98 103.505 0)
       (effects (font (size 1.27 1.27)) hide)
     )
@@
   (symbol (lib_id "LED:WS2812B") (at 119.38 89.535 0) (unit 1)
     (in_bom yes) (on_board yes)
-    (property "Reference" "LED19" (id 0) (at 114.3 81.915 0))
+    (property "Reference" "LED3" (id 0) (at 114.3 81.915 0))
     (property "Value" "WS2812-4020_single" (id 1) (at 129.54 97.155 0)
       (effects (font (size 1.27 1.27)) hide)
@@
   (symbol (lib_id "power:VCC") (at 99.06 81.915 0) (unit 1)
     (in_bom yes) (on_board yes) (fields_autoplaced)
-    (property "Reference" "#PWR0150" (id 0) (at 99.06 85.725 0)
+    (property "Reference" "#PWR0134" (id 0) (at 99.06 85.725 0)
       (effects (font (size 1.27 1.27)) hide)
     )
@@
   (symbol (lib_id "LED:WS2812B") (at 241.3 89.535 0) (unit 1)
     (in_bom yes) (on_board yes)
-    (property "Reference" "LED25" (id 0) (at 236.22 81.915 0))
+    (property "Reference" "LED9" (id 0) (at 236.22 81.915 0))
     (property "Value" "WS2812-4020_single" (id 1) (at 251.46 97.155 0)
       (effects (font (size 1.27 1.27)) hide)
@@
   (symbol (lib_id "power:VCC") (at 119.38 81.915 0) (unit 1)
     (in_bom yes) (on_board yes) (fields_autoplaced)
-    (property "Reference" "#PWR0151" (id 0) (at 119.38 85.725 0)
+    (property "Reference" "#PWR0135" (id 0) (at 119.38 85.725 0)
       (effects (font (size 1.27 1.27)) hide)
     )
@@
   (symbol (lib_id "power:GND") (at 139.7 97.155 0) (unit 1)
     (in_bom yes) (on_board yes) (fields_autoplaced)
-    (property "Reference" "#PWR0161" (id 0) (at 139.7 103.505 0)
+    (property "Reference" "#PWR0145" (id 0) (at 139.7 103.505 0)
       (effects (font (size 1.27 1.27)) hide)
     )
@@
   (symbol (lib_id "LED:WS2812B") (at 160.02 89.535 0) (unit 1)
     (in_bom yes) (on_board yes)
-    (property "Reference" "LED21" (id 0) (at 154.94 81.915 0))
+    (property "Reference" "LED5" (id 0) (at 154.94 81.915 0))
     (property "Value" "WS2812-4020_single" (id 1) (at 170.18 97.155 0)
       (effects (font (size 1.27 1.27)) hide)
@@
   (symbol (lib_id "power:GND") (at 200.66 97.155 0) (unit 1)
     (in_bom yes) (on_board yes) (fields_autoplaced)
-    (property "Reference" "#PWR0164" (id 0) (at 200.66 103.505 0)
+    (property "Reference" "#PWR0148" (id 0) (at 200.66 103.505 0)
       (effects (font (size 1.27 1.27)) hide)
     )
@@
   (symbol (lib_id "power:GND") (at 99.06 97.155 0) (unit 1)
     (in_bom yes) (on_board yes) (fields_autoplaced)
-    (property "Reference" "#PWR0159" (id 0) (at 99.06 103.505 0)
+    (property "Reference" "#PWR0143" (id 0) (at 99.06 103.505 0)
       (effects (font (size 1.27 1.27)) hide)
     )
@@
   (symbol (lib_id "LED:WS2812B") (at 200.66 89.535 0) (unit 1)
     (in_bom yes) (on_board yes)
-    (property "Reference" "LED23" (id 0) (at 195.58 81.915 0))
+    (property "Reference" "LED7" (id 0) (at 195.58 81.915 0))
     (property "Value" "WS2812-4020_single" (id 1) (at 210.82 97.155 0)
       (effects (font (size 1.27 1.27)) hide)
@@
   (symbol (lib_id "power:VCC") (at 160.02 81.915 0) (unit 1)
     (in_bom yes) (on_board yes) (fields_autoplaced)
-    (property "Reference" "#PWR0153" (id 0) (at 160.02 85.725 0)
+    (property "Reference" "#PWR0137" (id 0) (at 160.02 85.725 0)
       (effects (font (size 1.27 1.27)) hide)
     )
@@
   (symbol (lib_id "power:VCC") (at 241.3 81.915 0) (unit 1)
     (in_bom yes) (on_board yes) (fields_autoplaced)
-    (property "Reference" "#PWR0157" (id 0) (at 241.3 85.725 0)
+    (property "Reference" "#PWR0141" (id 0) (at 241.3 85.725 0)
       (effects (font (size 1.27 1.27)) hide)
     )
@@
   (symbol (lib_id "power:GND") (at 180.34 97.155 0) (unit 1)
     (in_bom yes) (on_board yes) (fields_autoplaced)
-    (property "Reference" "#PWR0163" (id 0) (at 180.34 103.505 0)
+    (property "Reference" "#PWR0147" (id 0) (at 180.34 103.505 0)
       (effects (font (size 1.27 1.27)) hide)
     )
@@
   (symbol (lib_id "power:VCC") (at 180.34 81.915 0) (unit 1)
     (in_bom yes) (on_board yes) (fields_autoplaced)
-    (property "Reference" "#PWR0154" (id 0) (at 180.34 85.725 0)
+    (property "Reference" "#PWR0138" (id 0) (at 180.34 85.725 0)
       (effects (font (size 1.27 1.27)) hide)
     )
@@
   (symbol (lib_id "LED:WS2812B") (at 99.06 89.535 0) (unit 1)
     (in_bom yes) (on_board yes)
-    (property "Reference" "LED18" (id 0) (at 93.98 81.915 0))
+    (property "Reference" "LED2" (id 0) (at 93.98 81.915 0))
     (property "Value" "WS2812-4020_single" (id 1) (at 109.22 97.155 0)
       (effects (font (size 1.27 1.27)) hide)
@@
   (symbol (lib_id "LED:WS2812B") (at 139.7 89.535 0) (unit 1)
     (in_bom yes) (on_board yes)
-    (property "Reference" "LED20" (id 0) (at 134.62 81.915 0))
+    (property "Reference" "LED4" (id 0) (at 134.62 81.915 0))
     (property "Value" "WS2812-4020_single" (id 1) (at 149.86 97.155 0)
       (effects (font (size 1.27 1.27)) hide)
@@
   (symbol (lib_id "power:VCC") (at 78.74 81.915 0) (unit 1)
     (in_bom yes) (on_board yes) (fields_autoplaced)
-    (property "Reference" "#PWR0149" (id 0) (at 78.74 85.725 0)
+    (property "Reference" "#PWR0133" (id 0) (at 78.74 85.725 0)
       (effects (font (size 1.27 1.27)) hide)
     )
@@
   (symbol (lib_id "LED:WS2812B") (at 180.34 89.535 0) (unit 1)
     (in_bom yes) (on_board yes)
-    (property "Reference" "LED22" (id 0) (at 175.26 81.915 0))
+    (property "Reference" "LED6" (id 0) (at 175.26 81.915 0))
     (property "Value" "WS2812-4020_single" (id 1) (at 190.5 97.155 0)
       (effects (font (size 1.27 1.27)) hide)
@@
   (symbol (lib_id "power:VCC") (at 200.66 81.915 0) (unit 1)
     (in_bom yes) (on_board yes) (fields_autoplaced)
-    (property "Reference" "#PWR0155" (id 0) (at 200.66 85.725 0)
+    (property "Reference" "#PWR0139" (id 0) (at 200.66 85.725 0)
       (effects (font (size 1.27 1.27)) hide)
     )
@@
   (symbol (lib_id "LED:WS2812B") (at 220.98 89.535 0) (unit 1)
     (in_bom yes) (on_board yes)
-    (property "Reference" "LED24" (id 0) (at 215.9 81.915 0))
+    (property "Reference" "LED8" (id 0) (at 215.9 81.915 0))
     (property "Value" "WS2812-4020_single" (id 1) (at 231.14 97.155 0)
       (effects (font (size 1.27 1.27)) hide)
@@
   (symbol (lib_id "power:VCC") (at 139.7 81.915 0) (unit 1)
     (in_bom yes) (on_board yes) (fields_autoplaced)
-    (property "Reference" "#PWR0152" (id 0) (at 139.7 85.725 0)
+    (property "Reference" "#PWR0136" (id 0) (at 139.7 85.725 0)
       (effects (font (size 1.27 1.27)) hide)
     )
@@
   (symbol (lib_id "LED:WS2812B") (at 78.74 89.535 0) (unit 1)
     (in_bom yes) (on_board yes)
-    (property "Reference" "LED17" (id 0) (at 73.66 81.915 0))
+    (property "Reference" "LED1" (id 0) (at 73.66 81.915 0))
     (property "Value" "WS2812-4020_single" (id 1) (at 88.9 97.155 0)
       (effects (font (size 1.27 1.27)) hide)
@@
   (symbol (lib_id "power:GND") (at 78.74 97.155 0) (unit 1)
     (in_bom yes) (on_board yes) (fields_autoplaced)
-    (property "Reference" "#PWR0158" (id 0) (at 78.74 103.505 0)
+    (property "Reference" "#PWR0142" (id 0) (at 78.74 103.505 0)
       (effects (font (size 1.27 1.27)) hide)
     )
@@
   (symbol (lib_id "power:GND") (at 160.02 97.155 0) (unit 1)
     (in_bom yes) (on_board yes) (fields_autoplaced)
-    (property "Reference" "#PWR0162" (id 0) (at 160.02 103.505 0)
-      (effects (font (size 1.27 1.27)) hide)
-    )
+    (property "Reference" "#PWR0146" (id 0) (at 160.02 103.505 0)
+      (effects (font (size 1.27 1.27)) hide)
+    )
