File: KiCad files/Main Project/Finish.kicad_sch (KiCad schematic)
At the start: 16 parts

Commit message: update
Parts:
- FIN1, FIN10, FIN11, FIN12, FIN13, FIN14, FIN15, FIN16, FIN2, FIN3, FIN4, FIN5, FIN6, FIN7, FIN8, FIN9: footprint FieldBoard_footprint:LED_WS2812B_PLCC4_5.0x5.0mm_P3.2mm -> LED_SMD:LED_WS2812B_PLCC4_5.0x5.0mm_P3.2mm
Changed lines of the file:
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@@
       (effects (font (size 1.27 1.27)) hide)
     )
-    (property "Footprint" "FieldBoard_footprint:LED_WS2812B_PLCC4_5.0x5.0mm_P3.2mm" (id 2) (at 98.425 106.68 0)
+    (property "Footprint" "LED_SMD:LED_WS2812B_PLCC4_5.0x5.0mm_P3.2mm" (id 2) (at 98.425 106.68 0)
       (effects (font (size 1.27 1.27)) (justify left top) hide)
     )
@@
       (effects (font (size 1.27 1.27)) hide)
     )
-    (property "Footprint" "FieldBoard_footprint:LED_WS2812B_PLCC4_5.0x5.0mm_P3.2mm" (id 2) (at 118.745 75.565 0)
+    (property "Footprint" "LED_SMD:LED_WS2812B_PLCC4_5.0x5.0mm_P3.2mm" (id 2) (at 118.745 75.565 0)
       (effects (font (size 1.27 1.27)) (justify left top) hide)
     )
@@
       (effects (font (size 1.27 1.27)) hide)
     )
-    (property "Footprint" "FieldBoard_footprint:LED_WS2812B_PLCC4_5.0x5.0mm_P3.2mm" (id 2) (at 159.385 106.68 0)
+    (property "Footprint" "LED_SMD:LED_WS2812B_PLCC4_5.0x5.0mm_P3.2mm" (id 2) (at 159.385 106.68 0)
       (effects (font (size 1.27 1.27)) (justify left top) hide)
     )
@@
       (effects (font (size 1.27 1.27)) hide)
     )
-    (property "Footprint" "FieldBoard_footprint:LED_WS2812B_PLCC4_5.0x5.0mm_P3.2mm" (id 2) (at 220.345 75.565 0)
+    (property "Footprint" "LED_SMD:LED_WS2812B_PLCC4_5.0x5.0mm_P3.2mm" (id 2) (at 220.345 75.565 0)
       (effects (font (size 1.27 1.27)) (justify left top) hide)
     )
@@
       (effects (font (size 1.27 1.27)) hide)
     )
-    (property "Footprint" "FieldBoard_footprint:LED_WS2812B_PLCC4_5.0x5.0mm_P3.2mm" (id 2) (at 118.745 106.68 0)
+    (property "Footprint" "LED_SMD:LED_WS2812B_PLCC4_5.0x5.0mm_P3.2mm" (id 2) (at 118.745 106.68 0)
       (effects (font (size 1.27 1.27)) (justify left top) hide)
     )
@@
       (effects (font (size 1.27 1.27)) hide)
     )
-    (property "Footprint" "FieldBoard_footprint:LED_WS2812B_PLCC4_5.0x5.0mm_P3.2mm" (id 2) (at 220.345 106.68 0)
+    (property "Footprint" "LED_SMD:LED_WS2812B_PLCC4_5.0x5.0mm_P3.2mm" (id 2) (at 220.345 106.68 0)
       (effects (font (size 1.27 1.27)) (justify left top) hide)
     )
@@
       (effects (font (size 1.27 1.27)) hide)
     )
-    (property "Footprint" "FieldBoard_footprint:LED_WS2812B_PLCC4_5.0x5.0mm_P3.2mm" (id 2) (at 159.385 75.565 0)
+    (property "Footprint" "LED_SMD:LED_WS2812B_PLCC4_5.0x5.0mm_P3.2mm" (id 2) (at 159.385 75.565 0)
       (effects (font (size 1.27 1.27)) (justify left top) hide)
     )
@@
       (effects (font (size 1.27 1.27)) hide)
     )
-    (property "Footprint" "FieldBoard_footprint:LED_WS2812B_PLCC4_5.0x5.0mm_P3.2mm" (id 2) (at 78.105 106.68 0)
+    (property "Footprint" "LED_SMD:LED_WS2812B_PLCC4_5.0x5.0mm_P3.2mm" (id 2) (at 78.105 106.68 0)
       (effects (font (size 1.27 1.27)) (justify left top) hide)
     )
@@
       (effects (font (size 1.27 1.27)) hide)
     )
-    (property "Footprint" "FieldBoard_footprint:LED_WS2812B_PLCC4_5.0x5.0mm_P3.2mm" (id 2) (at 179.705 106.68 0)
+    (property "Footprint" "LED_SMD:LED_WS2812B_PLCC4_5.0x5.0mm_P3.2mm" (id 2) (at 179.705 106.68 0)
       (effects (font (size 1.27 1.27)) (justify left top) hide)
     )
@@
       (effects (font (size 1.27 1.27)) hide)
     )
-    (property "Footprint" "FieldBoard_footprint:LED_WS2812B_PLCC4_5.0x5.0mm_P3.2mm" (id 2) (at 139.065 106.68 0)
+    (property "Footprint" "LED_SMD:LED_WS2812B_PLCC4_5.0x5.0mm_P3.2mm" (id 2) (at 139.065 106.68 0)
       (effects (font (size 1.27 1.27)) (justify left top) hide)
     )
@@
       (effects (font (size 1.27 1.27)) hide)
     )
-    (property "Footprint" "FieldBoard_footprint:LED_WS2812B_PLCC4_5.0x5.0mm_P3.2mm" (id 2) (at 78.105 75.565 0)
+    (property "Footprint" "LED_SMD:LED_WS2812B_PLCC4_5.0x5.0mm_P3.2mm" (id 2) (at 78.105 75.565 0)
       (effects (font (size 1.27 1.27)) (justify left top) hide)
     )
@@
       (effects (font (size 1.27 1.27)) hide)
     )
-    (property "Footprint" "FieldBoard_footprint:LED_WS2812B_PLCC4_5.0x5.0mm_P3.2mm" (id 2) (at 139.065 75.565 0)
+    (property "Footprint" "LED_SMD:LED_WS2812B_PLCC4_5.0x5.0mm_P3.2mm" (id 2) (at 139.065 75.565 0)
       (effects (font (size 1.27 1.27)) (justify left top) hide)
     )
@@
       (effects (font (size 1.27 1.27)) hide)
     )
-    (property "Footprint" "FieldBoard_footprint:LED_WS2812B_PLCC4_5.0x5.0mm_P3.2mm" (id 2) (at 200.025 106.68 0)
+    (property "Footprint" "LED_SMD:LED_WS2812B_PLCC4_5.0x5.0mm_P3.2mm" (id 2) (at 200.025 106.68 0)
       (effects (font (size 1.27 1.27)) (justify left top) hide)
     )
@@
       (effects (font (size 1.27 1.27)) hide)
     )
-    (property "Footprint" "FieldBoard_footprint:LED_WS2812B_PLCC4_5.0x5.0mm_P3.2mm" (id 2) (at 200.025 75.565 0)
+    (property "Footprint" "LED_SMD:LED_WS2812B_PLCC4_5.0x5.0mm_P3.2mm" (id 2) (at 200.025 75.565 0)
       (effects (font (size 1.27 1.27)) (justify left top) hide)
     )
@@
       (effects (font (size 1.27 1.27)) hide)
     )
-    (property "Footprint" "FieldBoard_footprint:LED_WS2812B_PLCC4_5.0x5.0mm_P3.2mm" (id 2) (at 98.425 75.565 0)
+    (property "Footprint" "LED_SMD:LED_WS2812B_PLCC4_5.0x5.0mm_P3.2mm" (id 2) (at 98.425 75.565 0)
       (effects (font (size 1.27 1.27)) (justify left top) hide)
     )
@@
       (effects (font (size 1.27 1.27)) hide)
     )
-    (property "Footprint" "FieldBoard_footprint:LED_WS2812B_PLCC4_5.0x5.0mm_P3.2mm" (id 2) (at 179.705 75.565 0)
-      (effects (font (size 1.27 1.27)) (justify left top) hide)
-    )
+    (property "Footprint" "LED_SMD:LED_WS2812B_PLCC4_5.0x5.0mm_P3.2mm" (id 2) (at 179.705 75.565 0)
+      (effects (font (size 1.27 1.27)) (justify left top) hide)
+    )

Commit message: shematic update
Parts:
- renumbered FIN1 to FIN17, FIN2 to FIN18, FIN3 to FIN19, FIN4 to FIN20, FIN5 to FIN21, FIN6 to FIN22, FIN7 to FIN23, FIN8 to FIN24, FIN9 to FIN25, FIN10 to FIN26, FIN11 to FIN27, FIN12 to FIN28, FIN13 to FIN29, FIN14 to FIN30, FIN15 to FIN31, FIN16 to FIN32

Commit message: update
Parts:
- renumbered FIN17 to FIN1, FIN26 to FIN10, FIN27 to FIN11, FIN28 to FIN12, FIN29 to FIN13, FIN30 to FIN14, FIN31 to FIN15, FIN32 to FIN16, FIN18 to FIN2, FIN19 to FIN3, FIN20 to FIN4, FIN21 to FIN5, FIN22 to FIN6, FIN23 to FIN7, FIN24 to FIN8, FIN25 to FIN9
