File: KiCad files/Main Project/LEDs.kicad_sch (KiCad schematic)
At the start: 11 parts, among them U10 WS2812-4020_dual, U11 WS2812-4020_dual, U12 WS2812-4020_dual, U13 WS2812-4020_dual, U14 WS2812-4020_dual, U15 WS2812-4020_dual, U5 WS2812-4020_dual, U6 WS2812-4020_dual, U7 WS2812-4020_dual, U8 WS2812-4020_dual, U9 WS2812-4020_dual

Commit message: update
Parts:
- removed U10, U11, U12, U13, U14, U15, U5, U6, U7, U8, U9: WS2812-4020_dual, Josip_global:WS2812-4020-dual-6mm_bezMaske, symbol Josip_symbol_global:WS2812-4020_dual
- added J3: (no value), symbol Connector:Conn_01x02_Male
Connections:
- net GND: now also J3.1 (Pin_1)
- net NEOPIXEL: now also J3.2 (Pin_2)
- no-connect marks 1 -> 0

Commit message: update
Parts:
- removed J3: (no value), symbol Connector:Conn_01x02_Male
- added R33, R34, R35, R36: 470R, Resistor_SMD:R_0603_1608Metric, symbol Device:R_Small
Connections:
- new net Cube (9LEDs)/Cube-LEDs: R35.2
- new net Finish (16LEDs)/Finish-LEDs: R33.2
- new net Positions (52LEDs)/Positions-LEDs: R34.2
- new net Start (16LEDs)/Start-LEDs: R36.2
Other:
- added sheet Cube (9LEDs) (Cube.kicad_sch)
- added sheet Finish (16LEDs) (Finish.kicad_sch)
- added sheet Positions (52LEDs) (Positions.kicad_sch)
- added sheet Start (16LEDs) (Start.kicad_sch)
- note removed: "WS2812-4020 already include 100nF caps, no need to add them"
Changed lines of the file:
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@@
     (company "Josip&Zvonimir")
   )
-  (wire (pts (xy 42.545 100.965) (xy 42.545 99.06))
+  (wire (pts (xy 146.685 87.63) (xy 137.16 87.63))
     (stroke (width 0) (type default) (color 0 0 0 0))
   )
-  (wire (pts (xy 42.545 99.06) (xy 44.45 99.06))
+  (wire (pts (xy 130.175 80.01) (xy 130.175 78.74))
     (stroke (width 0) (type default) (color 0 0 0 0))
   )
-  (text "WS2812-4020 already include 100nF caps, no need to add them"
-    (at 42.545 123.19 0)
-    (effects (font (size 1.27 1.27)) (justify left bottom))
+  (wire (pts (xy 132.08 87.63) (xy 128.905 87.63))
+    (stroke (width 0) (type default) (color 0 0 0 0))
   )
-  (global_label "NEOPIXEL" (shape input) (at 44.45 96.52 180) (fields_autoplaced)
-    (effects (font (size 1.27 1.27)) (justify right))
-    (property "Intersheet References" "${INTERSHEET_REFS}" (id 0) (at -2.54 50.165 0)
+  (wire (pts (xy 128.905 87.63) (xy 128.905 85.09))
+    (stroke (width 0) (type default) (color 0 0 0 0))
+  )
+  (wire (pts (xy 163.83 72.39) (xy 154.94 72.39))
+    (stroke (width 0) (type default) (color 0 0 0 0))
+  )
+  (wire (pts (xy 137.16 74.295) (xy 146.685 74.295))
+    (stroke (width 0) (type default) (color 0 0 0 0))
+  )
+  (wire (pts (xy 146.685 53.975) (xy 163.83 53.975))
+    (stroke (width 0) (type default) (color 0 0 0 0))
+  )
+  (wire (pts (xy 137.16 83.185) (xy 154.94 83.185))
+    (stroke (width 0) (type default) (color 0 0 0 0))
+  )
+  (wire (pts (xy 124.46 77.47) (xy 128.905 77.47))
+    (stroke (width 0) (type default) (color 0 0 0 0))
+  )
+  (wire (pts (xy 146.685 74.295) (xy 146.685 53.975))
+    (stroke (width 0) (type default) (color 0 0 0 0))
+  )
+  (wire (pts (xy 146.685 109.22) (xy 146.685 87.63))
+    (stroke (width 0) (type default) (color 0 0 0 0))
+  )
+  (wire (pts (xy 128.905 77.47) (xy 128.905 74.295))
+    (stroke (width 0) (type default) (color 0 0 0 0))
+  )
+  (wire (pts (xy 163.83 109.22) (xy 146.685 109.22))
+    (stroke (width 0) (type default) (color 0 0 0 0))
+  )
+  (wire (pts (xy 124.46 82.55) (xy 130.175 82.55))
+    (stroke (width 0) (type default) (color 0 0 0 0))
+  )
+  (wire (pts (xy 124.46 80.01) (xy 130.175 80.01))
+    (stroke (width 0) (type default) (color 0 0 0 0))
+  )
+  (wire (pts (xy 128.905 74.295) (xy 132.08 74.295))
+    (stroke (width 0) (type default) (color 0 0 0 0))
+  )
+  (wire (pts (xy 154.94 83.185) (xy 154.94 91.44))
+    (stroke (width 0) (type default) (color 0 0 0 0))
+  )
+  (wire (pts (xy 154.94 78.74) (xy 137.16 78.74))
+    (stroke (width 0) (type default) (color 0 0 0 0))
+  )
+  (wire (pts (xy 154.94 72.39) (xy 154.94 78.74))
+    (stroke (width 0) (type default) (color 0 0 0 0))
+  )
+  (wire (pts (xy 130.175 78.74) (xy 132.08 78.74))
+    (stroke (width 0) (type default) (color 0 0 0 0))
+  )
+  (wire (pts (xy 154.94 91.44) (xy 163.83 91.44))
+    (stroke (width 0) (type default) (color 0 0 0 0))
+  )
+  (wire (pts (xy 130.175 82.55) (xy 130.175 83.185))
+    (stroke (width 0) (type default) (color 0 0 0 0))
+  )
+  (wire (pts (xy 130.175 83.185) (xy 132.08 83.185))
+    (stroke (width 0) (type default) (color 0 0 0 0))
+  )
+  (wire (pts (xy 128.905 85.09) (xy 124.46 85.09))
+    (stroke (width 0) (type default) (color 0 0 0 0))
+  )
+  (symbol (lib_id "Device:R_Small") (at 134.62 78.74 90) (unit 1)
+    (in_bom yes) (on_board yes)
+    (property "Reference" "R34" (id 0) (at 134.62 76.835 90))
+    (property "Value" "470R" (id 1) (at 134.62 78.74 90)
+      (effects (font (size 0.9 0.9)))
+    )
+    (property "Footprint" "Resistor_SMD:R_0603_1608Metric" (id 2) (at 134.62 78.74 0)
       (effects (font (size 1.27 1.27)) hide)
     )
-  )
-  (symbol (lib_id "Connector:Conn_01x02_Male") (at 49.53 99.06 180) (unit 1)
-    (in_bom yes) (on_board yes)
-    (property "Reference" "J3" (id 0) (at 46.355 92.71 0)
-      (effects (font (size 1.27 1.27)) (justify right))
-    )
-    (property "Value" "" (id 1) (at 50.2412 99.4922 0)
-      (effects (font (size 1.27 1.27)) (justify right) hide)
-    )
-    (property "Footprint" "" (id 2) (at 49.53 99.06 0)
-      (effects (font (size 1.27 1.27)) hide)
-    )
-    (property "Datasheet" "~" (id 3) (at 49.53 99.06 0)
+    (property "Datasheet" "~" (id 3) (at 134.62 78.74 0)
       (effects (font (size 1.27 1.27)) hide)
     )
@@
     (pin "2")
   )
-  (symbol (lib_id "power:GND") (at 42.545 100.965 0) (unit 1)
-    (in_bom yes) (on_board yes) (fields_autoplaced)
-    (property "Reference" "#PWR04" (id 0) (at 42.545 107.315 0)
+  (symbol (lib_id "Device:R_Small") (at 134.62 87.63 90) (unit 1)
+    (in_bom yes) (on_board yes)
+    (property "Reference" "R36" (id 0) (at 134.62 85.725 90))
+    (property "Value" "470R" (id 1) (at 134.62 87.63 90)
+      (effects (font (size 0.9 0.9)))
+    )
+    (property "Footprint" "Resistor_SMD:R_0603_1608Metric" (id 2) (at 134.62 87.63 0)
       (effects (font (size 1.27 1.27)) hide)
     )
-    (property "Value" "" (id 1) (at 42.545 105.4084 0))
-    (property "Footprint" "" (id 2) (at 42.545 100.965 0)
-      (effects (font (size 1.27 1.27)) hide)
-    )
-    (property "Datasheet" "" (id 3) (at 42.545 100.965 0)
+    (property "Datasheet" "~" (id 3) (at 134.62 87.63 0)
       (effects (font (size 1.27 1.27)) hide)
     )
     (pin "1")
+    (pin "2")
+  )
+  (symbol (lib_id "Device:R_Small") (at 134.62 74.295 90) (unit 1)
+    (in_bom yes) (on_board yes)
+    (property "Reference" "R33" (id 0) (at 134.62 72.39 90))
+    (property "Value" "470R" (id 1) (at 134.62 74.295 90)
+      (effects (font (size 0.9 0.9)))
+    )
+    (property "Footprint" "Resistor_SMD:R_0603_1608Metric" (id 2) (at 134.62 74.295 0)
+      (effects (font (size 1.27 1.27)) hide)
+    )
+    (property "Datasheet" "~" (id 3) (at 134.62 74.295 0)
+      (effects (font (size 1.27 1.27)) hide)
+    )
+    (pin "1")
+    (pin "2")
+  )
+  (symbol (lib_id "Device:R_Small") (at 134.62 83.185 90) (unit 1)
+    (in_bom yes) (on_board yes)
+    (property "Reference" "R35" (id 0) (at 134.62 81.28 90))
+    (property "Value" "470R" (id 1) (at 134.62 83.185 90)
+      (effects (font (size 0.9 0.9)))
+    )
+    (property "Footprint" "Resistor_SMD:R_0603_1608Metric" (id 2) (at 134.62 83.185 0)
+      (effects (font (size 1.27 1.27)) hide)
+    )
+    (property "Datasheet" "~" (id 3) (at 134.62 83.185 0)
+      (effects (font (size 1.27 1.27)) hide)
+    )
+    (pin "1")
+    (pin "2")
+  )
+  (sheet (at 163.83 45.085) (size 26.67 17.145)
+    (stroke (width 0.1524) (type solid) (color 0 0 0 0))
+    (fill (color 0 0 0 0.0000))
+    (property "Sheet name" "Finish (16LEDs)" (id 0) (at 164.465 47.625 0)
+      (effects (font (size 1.27 1.27)) (justify left bottom))
+    )
+    (property "Sheet file" "Finish.kicad_sch" (id 1) (at 164.465 59.69 0)
+      (effects (font (size 1.27 1.27)) (justify left top) hide)
+    )
+    (pin "Finish-LEDs" input (at 163.83 53.975 180)
+      (effects (font (size 1.27 1.27)) (justify left))
+    )
+  )
+  (sheet (at 163.83 63.5) (size 26.67 17.145)
+    (stroke (width 0.1524) (type solid) (color 0 0 0 0))
+    (fill (color 0 0 0 0.0000))
+    (property "Sheet name" "Positions (52LEDs)" (id 0) (at 164.465 66.04 0)
+      (effects (font (size 1.27 1.27)) (justify left bottom))
+    )
+    (property "Sheet file" "Positions.kicad_sch" (id 1) (at 164.465 74.93 0)
+      (effects (font (size 1.27 1.27)) (justify left top) hide)
+    )
+    (pin "Positions-LEDs" input (at 163.83 72.39 180)
+      (effects (font (size 1.27 1.27)) (justify left))
+    )
+  )
+  (sheet (at 163.83 100.33) (size 26.67 17.145)
+    (stroke (width 0.1524) (type solid) (color 0 0 0 0))
+    (fill (color 0 0 0 0.0000))
+    (property "Sheet name" "Start (16LEDs)" (id 0) (at 164.465 102.87 0)
+      (effects (font (size 1.27 1.27)) (justify left bottom))
+    )
+    (property "Sheet file" "Start.kicad_sch" (id 1) (at 164.465 114.935 0)
+      (effects (font (size 1.27 1.27)) (justify left top) hide)
+    )
+    (pin "Start-LEDs" input (at 163.83 109.22 180)
+      (effects (font (size 1.27 1.27)) (justify left))
+    )
+  )
+  (sheet (at 163.83 81.915) (size 26.67 17.145)
+    (stroke (width 0.1524) (type solid) (color 0 0 0 0))
+    (fill (color 0 0 0 0.0000))
+    (property "Sheet name" "Cube (9LEDs)" (id 0) (at 164.465 84.455 0)
+      (effects (font (size 1.27 1.27)) (justify left bottom))
+    )
+    (property "Sheet file" "Cube.kicad_sch" (id 1) (at 164.465 93.345 0)
+      (effects (font (size 1.27 1.27)) (justify left top) hide)
+    )
+    (pin "Cube-LEDs" input (at 163.83 91.44 180)
+      (effects (font (size 1.27 1.27)) (justify left))
+    )
   )
 )

Commit message: update
Parts:
- added R22: 470R, Resistor_SMD:R_0603_1608Metric, symbol Device:R_Small
- added TP_LED_1, TP_LED_10, TP_LED_11, TP_LED_12, TP_LED_2, TP_LED_3, TP_LED_4, TP_LED_5, TP_LED_6, TP_LED_7, TP_LED_8, TP_LED_9: WS2812-4020_dual, LED_SMD:LED_WS2812B_PLCC4_5.0x5.0mm_P3.2mm, symbol LED:WS2812B
Connections:
- net NP_2: now reaches R34.1
- net NP_4: now reaches R36.1
- net NP_1: now reaches R33.1
- net NP_3: now reaches R35.1
- new net: TP_LED_8.2 (DOUT), TP_LED_9.4 (DIN)
- new net: TP_LED_7.2 (DOUT), TP_LED_8.4 (DIN)
- new net: TP_LED_3.2 (DOUT), TP_LED_4.4 (DIN)
- new net: TP_LED_2.2 (DOUT), TP_LED_3.4 (DIN)
- new net: TP_LED_11.2 (DOUT), TP_LED_12.4 (DIN)
- new net: TP_LED_10.2 (DOUT), TP_LED_11.4 (DIN)
- new net: TP_LED_1.2 (DOUT), TP_LED_2.4 (DIN)
- new net: R22.2, TP_LED_1.4 (DIN)
- new net: TP_LED_4.2 (DOUT), TP_LED_5.4 (DIN)
- new net: TP_LED_10.4 (DIN), TP_LED_9.2 (DOUT)
- new net: TP_LED_6.2 (DOUT), TP_LED_7.4 (DIN)
- new net: TP_LED_5.2 (DOUT), TP_LED_6.4 (DIN)
- new net GND: TP_LED_1.3 (VSS), TP_LED_10.3 (VSS), TP_LED_11.3 (VSS), TP_LED_12.3 (VSS), TP_LED_2.3 (VSS), TP_LED_3.3 (VSS), TP_LED_4.3 (VSS), TP_LED_5.3 (VSS), TP_LED_6.3 (VSS), TP_LED_7.3 (VSS), TP_LED_8.3 (VSS), TP_LED_9.3 (VSS)
- new net NP_5: R22.1
- new net VCC: TP_LED_1.1 (VDD), TP_LED_10.1 (VDD), TP_LED_11.1 (VDD), TP_LED_12.1 (VDD), TP_LED_2.1 (VDD), TP_LED_3.1 (VDD), TP_LED_4.1 (VDD), TP_LED_5.1 (VDD), TP_LED_6.1 (VDD), TP_LED_7.1 (VDD), TP_LED_8.1 (VDD), TP_LED_9.1 (VDD)
- no-connect marks 0 -> 1
Other:
- moved on the sheet: R33, R34, R35, R36

Commit message: shematic update
Parts:
- renumbered R33 to R18, R34 to R19, R35 to R20, R36 to R21, TP_LED_1 to TP_LED_17, TP_LED_2 to TP_LED_18, TP_LED_3 to TP_LED_19, TP_LED_4 to TP_LED_20, TP_LED_5 to TP_LED_21, TP_LED_6 to TP_LED_22, TP_LED_7 to TP_LED_23, TP_LED_8 to TP_LED_24, TP_LED_9 to TP_LED_25, TP_LED_10 to TP_LED_26, TP_LED_11 to TP_LED_27, TP_LED_12 to TP_LED_28

Commit message: update
Parts:
- renumbered R18 to R2, R19 to R3, R20 to R4, R21 to R5, R22 to R6, TP_LED_17 to TP_LED_1, TP_LED_26 to TP_LED_10, TP_LED_27 to TP_LED_11, TP_LED_28 to TP_LED_12, TP_LED_18 to TP_LED_2, TP_LED_19 to TP_LED_3, TP_LED_20 to TP_LED_4, TP_LED_21 to TP_LED_5, TP_LED_22 to TP_LED_6, TP_LED_23 to TP_LED_7, TP_LED_24 to TP_LED_8, TP_LED_25 to TP_LED_9

Commit message: update
Parts:
- renumbered R6 to R22, R2 to R33, R3 to R34, R4 to R35, R5 to R36
Changed lines of the file:
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@@
   (symbol (lib_id "power:GND") (at 151.13 165.1 0) (unit 1)
     (in_bom yes) (on_board yes) (fields_autoplaced)
-    (property "Reference" "#PWR034" (id 0) (at 151.13 171.45 0)
+    (property "Reference" "#PWR0238" (id 0) (at 151.13 171.45 0)
       (effects (font (size 1.27 1.27)) hide)
     )
@@
   (symbol (lib_id "power:VCC") (at 232.41 118.745 0) (unit 1)
     (in_bom yes) (on_board yes) (fields_autoplaced)
-    (property "Reference" "#PWR018" (id 0) (at 232.41 122.555 0)
+    (property "Reference" "#PWR0255" (id 0) (at 232.41 122.555 0)
       (effects (font (size 1.27 1.27)) hide)
     )
@@
   (symbol (lib_id "power:GND") (at 130.81 133.985 0) (unit 1)
     (in_bom yes) (on_board yes) (fields_autoplaced)
-    (property "Reference" "#PWR021" (id 0) (at 130.81 140.335 0)
+    (property "Reference" "#PWR0252" (id 0) (at 130.81 140.335 0)
       (effects (font (size 1.27 1.27)) hide)
     )
@@
   (symbol (lib_id "power:GND") (at 151.13 133.985 0) (unit 1)
     (in_bom yes) (on_board yes) (fields_autoplaced)
-    (property "Reference" "#PWR022" (id 0) (at 151.13 140.335 0)
+    (property "Reference" "#PWR0248" (id 0) (at 151.13 140.335 0)
       (effects (font (size 1.27 1.27)) hide)
     )
@@
   (symbol (lib_id "power:GND") (at 90.17 133.985 0) (unit 1)
     (in_bom yes) (on_board yes) (fields_autoplaced)
-    (property "Reference" "#PWR019" (id 0) (at 90.17 140.335 0)
+    (property "Reference" "#PWR0234" (id 0) (at 90.17 140.335 0)
       (effects (font (size 1.27 1.27)) hide)
     )
@@
   (symbol (lib_id "Device:R_Small") (at 52.07 60.325 90) (unit 1)
     (in_bom yes) (on_board yes)
-    (property "Reference" "R3" (id 0) (at 52.07 58.42 90))
+    (property "Reference" "R34" (id 0) (at 52.07 58.42 90))
     (property "Value" "470R" (id 1) (at 52.07 60.325 90)
       (effects (font (size 0.9 0.9)))
@@
   (symbol (lib_id "power:GND") (at 110.49 165.1 0) (unit 1)
     (in_bom yes) (on_board yes) (fields_autoplaced)
-    (property "Reference" "#PWR032" (id 0) (at 110.49 171.45 0)
+    (property "Reference" "#PWR0240" (id 0) (at 110.49 171.45 0)
       (effects (font (size 1.27 1.27)) hide)
     )
@@
   (symbol (lib_id "power:VCC") (at 212.09 118.745 0) (unit 1)
     (in_bom yes) (on_board yes) (fields_autoplaced)
-    (property "Reference" "#PWR017" (id 0) (at 212.09 122.555 0)
+    (property "Reference" "#PWR0247" (id 0) (at 212.09 122.555 0)
       (effects (font (size 1.27 1.27)) hide)
     )
@@
   (symbol (lib_id "power:GND") (at 110.49 133.985 0) (unit 1)
     (in_bom yes) (on_board yes) (fields_autoplaced)
-    (property "Reference" "#PWR020" (id 0) (at 110.49 140.335 0)
+    (property "Reference" "#PWR0235" (id 0) (at 110.49 140.335 0)
       (effects (font (size 1.27 1.27)) hide)
     )
@@
   (symbol (lib_id "power:VCC") (at 151.13 149.86 0) (unit 1)
     (in_bom yes) (on_board yes) (fields_autoplaced)
-    (property "Reference" "#PWR030" (id 0) (at 151.13 153.67 0)
+    (property "Reference" "#PWR0236" (id 0) (at 151.13 153.67 0)
       (effects (font (size 1.27 1.27)) hide)
     )
@@
   (symbol (lib_id "power:VCC") (at 151.13 118.745 0) (unit 1)
     (in_bom yes) (on_board yes) (fields_autoplaced)
-    (property "Reference" "#PWR014" (id 0) (at 151.13 122.555 0)
+    (property "Reference" "#PWR0243" (id 0) (at 151.13 122.555 0)
       (effects (font (size 1.27 1.27)) hide)
     )
@@
   (symbol (lib_id "power:VCC") (at 171.45 118.745 0) (unit 1)
     (in_bom yes) (on_board yes) (fields_autoplaced)
-    (property "Reference" "#PWR015" (id 0) (at 171.45 122.555 0)
+    (property "Reference" "#PWR0249" (id 0) (at 171.45 122.555 0)
       (effects (font (size 1.27 1.27)) hide)
     )
@@
   (symbol (lib_id "power:VCC") (at 90.17 149.86 0) (unit 1)
     (in_bom yes) (on_board yes) (fields_autoplaced)
-    (property "Reference" "#PWR027" (id 0) (at 90.17 153.67 0)
+    (property "Reference" "#PWR0233" (id 0) (at 90.17 153.67 0)
       (effects (font (size 1.27 1.27)) hide)
     )
@@
   (symbol (lib_id "power:GND") (at 130.81 165.1 0) (unit 1)
     (in_bom yes) (on_board yes) (fields_autoplaced)
-    (property "Reference" "#PWR033" (id 0) (at 130.81 171.45 0)
+    (property "Reference" "#PWR0239" (id 0) (at 130.81 171.45 0)
       (effects (font (size 1.27 1.27)) hide)
     )
@@
   (symbol (lib_id "power:GND") (at 232.41 133.985 0) (unit 1)
     (in_bom yes) (on_board yes) (fields_autoplaced)
-    (property "Reference" "#PWR026" (id 0) (at 232.41 140.335 0)
+    (property "Reference" "#PWR0254" (id 0) (at 232.41 140.335 0)
       (effects (font (size 1.27 1.27)) hide)
     )
@@
   (symbol (lib_id "power:GND") (at 90.17 165.1 0) (unit 1)
     (in_bom yes) (on_board yes) (fields_autoplaced)
-    (property "Reference" "#PWR031" (id 0) (at 90.17 171.45 0)
+    (property "Reference" "#PWR0232" (id 0) (at 90.17 171.45 0)
       (effects (font (size 1.27 1.27)) hide)
     )
@@
   (symbol (lib_id "power:VCC") (at 130.81 118.745 0) (unit 1)
     (in_bom yes) (on_board yes) (fields_autoplaced)
-    (property "Reference" "#PWR013" (id 0) (at 130.81 122.555 0)
+    (property "Reference" "#PWR0242" (id 0) (at 130.81 122.555 0)
       (effects (font (size 1.27 1.27)) hide)
     )
@@
   (symbol (lib_id "power:VCC") (at 90.17 118.745 0) (unit 1)
     (in_bom yes) (on_board yes) (fields_autoplaced)
-    (property "Reference" "#PWR011" (id 0) (at 90.17 122.555 0)
+    (property "Reference" "#PWR0245" (id 0) (at 90.17 122.555 0)
       (effects (font (size 1.27 1.27)) hide)
     )
@@
   (symbol (lib_id "power:VCC") (at 110.49 149.86 0) (unit 1)
     (in_bom yes) (on_board yes) (fields_autoplaced)
-    (property "Reference" "#PWR028" (id 0) (at 110.49 153.67 0)
+    (property "Reference" "#PWR0241" (id 0) (at 110.49 153.67 0)
       (effects (font (size 1.27 1.27)) hide)
     )
@@
   (symbol (lib_id "power:VCC") (at 110.49 118.745 0) (unit 1)
     (in_bom yes) (on_board yes) (fields_autoplaced)
-    (property "Reference" "#PWR012" (id 0) (at 110.49 122.555 0)
+    (property "Reference" "#PWR0244" (id 0) (at 110.49 122.555 0)
       (effects (font (size 1.27 1.27)) hide)
     )
@@
   (symbol (lib_id "Device:R_Small") (at 52.07 73.66 90) (unit 1)
     (in_bom yes) (on_board yes)
-    (property "Reference" "R6" (id 0) (at 52.07 71.755 90))
+    (property "Reference" "R22" (id 0) (at 52.07 71.755 90))
     (property "Value" "470R" (id 1) (at 52.07 73.66 90)
       (effects (font (size 0.9 0.9)))
@@
   (symbol (lib_id "power:GND") (at 191.77 133.985 0) (unit 1)
     (in_bom yes) (on_board yes) (fields_autoplaced)
-    (property "Reference" "#PWR024" (id 0) (at 191.77 140.335 0)
+    (property "Reference" "#PWR0251" (id 0) (at 191.77 140.335 0)
       (effects (font (size 1.27 1.27)) hide)
     )
@@
   (symbol (lib_id "power:GND") (at 171.45 133.985 0) (unit 1)
     (in_bom yes) (on_board yes) (fields_autoplaced)
-    (property "Reference" "#PWR023" (id 0) (at 171.45 140.335 0)
+    (property "Reference" "#PWR0250" (id 0) (at 171.45 140.335 0)
       (effects (font (size 1.27 1.27)) hide)
     )
@@
   (symbol (lib_id "power:VCC") (at 191.77 118.745 0) (unit 1)
     (in_bom yes) (on_board yes) (fields_autoplaced)
-    (property "Reference" "#PWR016" (id 0) (at 191.77 122.555 0)
+    (property "Reference" "#PWR0253" (id 0) (at 191.77 122.555 0)
       (effects (font (size 1.27 1.27)) hide)
     )
@@
   (symbol (lib_id "power:GND") (at 212.09 133.985 0) (unit 1)
     (in_bom yes) (on_board yes) (fields_autoplaced)
-    (property "Reference" "#PWR025" (id 0) (at 212.09 140.335 0)
+    (property "Reference" "#PWR0246" (id 0) (at 212.09 140.335 0)
       (effects (font (size 1.27 1.27)) hide)
     )
@@
   (symbol (lib_id "Device:R_Small") (at 52.07 69.215 90) (unit 1)
     (in_bom yes) (on_board yes)
-    (property "Reference" "R5" (id 0) (at 52.07 67.31 90))
+    (property "Reference" "R36" (id 0) (at 52.07 67.31 90))
     (property "Value" "470R" (id 1) (at 52.07 69.215 90)
       (effects (font (size 0.9 0.9)))
@@
   (symbol (lib_id "Device:R_Small") (at 52.07 55.88 90) (unit 1)
     (in_bom yes) (on_board yes)
-    (property "Reference" "R2" (id 0) (at 52.07 53.975 90))
+    (property "Reference" "R33" (id 0) (at 52.07 53.975 90))
     (property "Value" "470R" (id 1) (at 52.07 55.88 90)
       (effects (font (size 0.9 0.9)))
@@
   (symbol (lib_id "power:VCC") (at 130.81 149.86 0) (unit 1)
     (in_bom yes) (on_board yes) (fields_autoplaced)
-    (property "Reference" "#PWR029" (id 0) (at 130.81 153.67 0)
+    (property "Reference" "#PWR0237" (id 0) (at 130.81 153.67 0)
       (effects (font (size 1.27 1.27)) hide)
     )
@@
   (symbol (lib_id "Device:R_Small") (at 52.07 64.77 90) (unit 1)
     (in_bom yes) (on_board yes)
-    (property "Reference" "R4" (id 0) (at 52.07 62.865 90))
+    (property "Reference" "R35" (id 0) (at 52.07 62.865 90))
     (property "Value" "470R" (id 1) (at 52.07 64.77 90)
       (effects (font (size 0.9 0.9)))
