File: KiCad files/Main Project/USB.kicad_sch (KiCad schematic)
At the start: 3 parts, among them J2 USB_C_Receptacle_USB2.0

Commit message: update
Parts:
- added R23: 1M, Resistor_SMD:R_0805_2012Metric, symbol Device:R_Small
Connections:
- net GND: now also R23.2; no longer J2.S1 (SHIELD)
- new net: J2.S1 (SHIELD), R23.1
Changed lines of the file:
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@@
   (junction (at 116.205 93.345) (diameter 0) (color 0 0 0 0)
-  )
-  (junction (at 92.71 120.015) (diameter 0) (color 0 0 0 0)
   )
   (junction (at 116.205 98.425) (diameter 0) (color 0 0 0 0)
@@
     (stroke (width 0) (type default) (color 0 0 0 0))
   )
-  (wire (pts (xy 88.9 120.015) (xy 92.71 120.015))
-    (stroke (width 0) (type default) (color 0 0 0 0))
-  )
   (wire (pts (xy 135.89 84.455) (xy 135.89 88.265))
     (stroke (width 0) (type default) (color 0 0 0 0))
@@
     (stroke (width 0) (type default) (color 0 0 0 0))
   )
-  (wire (pts (xy 92.71 120.015) (xy 96.52 120.015))
-    (stroke (width 0) (type default) (color 0 0 0 0))
-  )
   (wire (pts (xy 116.205 92.075) (xy 116.205 93.345))
     (stroke (width 0) (type default) (color 0 0 0 0))
@@
     (stroke (width 0) (type default) (color 0 0 0 0))
   )
-  (wire (pts (xy 88.9 117.475) (xy 88.9 120.015))
-    (stroke (width 0) (type default) (color 0 0 0 0))
-  )
   (wire (pts (xy 116.205 98.425) (xy 116.205 99.695))
     (stroke (width 0) (type default) (color 0 0 0 0))
@@
     (stroke (width 0) (type default) (color 0 0 0 0))
   )
-  (wire (pts (xy 92.71 120.015) (xy 92.71 121.285))
-    (stroke (width 0) (type default) (color 0 0 0 0))
-  )
   (wire (pts (xy 111.76 86.995) (xy 129.54 86.995))
     (stroke (width 0) (type default) (color 0 0 0 0))
@@
     (stroke (width 0) (type default) (color 0 0 0 0))
   )
-  (wire (pts (xy 96.52 117.475) (xy 96.52 120.015))
+  (wire (pts (xy 88.9 117.475) (xy 88.9 118.11))
+    (stroke (width 0) (type default) (color 0 0 0 0))
+  )
+  (wire (pts (xy 96.52 117.475) (xy 96.52 123.19))
     (stroke (width 0) (type default) (color 0 0 0 0))
   )
@@
     (pin "1")
   )
-  (symbol (lib_id "power:GND") (at 92.71 121.285 0) (unit 1)
-    (in_bom yes) (on_board yes)
-    (property "Reference" "#PWR069" (id 0) (at 92.71 127.635 0)
-      (effects (font (size 1.27 1.27)) hide)
-    )
-    (property "Value" "GND" (id 1) (at 92.837 125.6792 0))
-    (property "Footprint" "" (id 2) (at 92.71 121.285 0)
-      (effects (font (size 1.27 1.27)) hide)
-    )
-    (property "Datasheet" "" (id 3) (at 92.71 121.285 0)
+  (symbol (lib_id "power:GND") (at 96.52 123.19 0) (unit 1)
+    (in_bom yes) (on_board yes)
+    (property "Reference" "#PWR069" (id 0) (at 96.52 129.54 0)
+      (effects (font (size 1.27 1.27)) hide)
+    )
+    (property "Value" "GND" (id 1) (at 96.647 127.5842 0))
+    (property "Footprint" "" (id 2) (at 96.52 123.19 0)
+      (effects (font (size 1.27 1.27)) hide)
+    )
+    (property "Datasheet" "" (id 3) (at 96.52 123.19 0)
       (effects (font (size 1.27 1.27)) hide)
     )
@@
       (effects (font (size 1.27 1.27)) hide)
     )
+    (pin "1")
+  )
+  (symbol (lib_id "Device:R_Small") (at 88.9 120.65 0) (unit 1)
+    (in_bom yes) (on_board yes)
+    (property "Reference" "R23" (id 0) (at 90.17 120.65 0)
+      (effects (font (size 1.27 1.27)) (justify left))
+    )
+    (property "Value" "1M" (id 1) (at 88.9 121.92 90)
+      (effects (font (size 0.9906 0.9906)) (justify left))
+    )
+    (property "Footprint" "Resistor_SMD:R_0805_2012Metric" (id 2) (at 88.9 120.65 0)
+      (effects (font (size 1.27 1.27)) hide)
+    )
+    (property "Datasheet" "~" (id 3) (at 88.9 120.65 0)
+      (effects (font (size 1.27 1.27)) hide)
+    )
+    (pin "1")
+    (pin "2")
+  )
+  (symbol (lib_id "power:GND") (at 88.9 123.19 0) (unit 1)
+    (in_bom yes) (on_board yes)
+    (property "Reference" "#PWR0272" (id 0) (at 88.9 129.54 0)
+      (effects (font (size 1.27 1.27)) hide)
+    )
+    (property "Value" "GND" (id 1) (at 89.027 127.5842 0))
+    (property "Footprint" "" (id 2) (at 88.9 123.19 0)
+      (effects (font (size 1.27 1.27)) hide)
+    )
+    (property "Datasheet" "" (id 3) (at 88.9 123.19 0)
+      (effects (font (size 1.27 1.27)) hide)
+    )

Commit message: shematic update
Parts:
- renumbered J2 to J20, R16 to R36, R17 to R37, R23 to R38
Changed lines of the file:
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@@
   (symbol (lib_id "Connector:USB_C_Receptacle_USB2.0") (at 96.52 94.615 0) (unit 1)
     (in_bom yes) (on_board yes)
-    (property "Reference" "J2" (id 0) (at 87.63 75.438 0))
+    (property "Reference" "J20" (id 0) (at 87.63 75.438 0))
     (property "Value" "USB_C_Receptacle_USB2.0" (id 1) (at 99.2378 74.9046 0)
       (effects (font (size 1.27 1.27)) hide)
@@
   (symbol (lib_id "power:VBUS") (at 119.38 76.2 0) (unit 1)
     (in_bom yes) (on_board yes)
-    (property "Reference" "#PWR070" (id 0) (at 119.38 80.01 0)
+    (property "Reference" "#PWR077" (id 0) (at 119.38 80.01 0)
       (effects (font (size 1.27 1.27)) hide)
     )
@@
   (symbol (lib_id "power:GND") (at 96.52 123.19 0) (unit 1)
     (in_bom yes) (on_board yes)
-    (property "Reference" "#PWR069" (id 0) (at 96.52 129.54 0)
+    (property "Reference" "#PWR080" (id 0) (at 96.52 129.54 0)
       (effects (font (size 1.27 1.27)) hide)
     )
@@
   (symbol (lib_id "Device:R_Small") (at 129.54 90.805 0) (unit 1)
     (in_bom yes) (on_board yes)
-    (property "Reference" "R16" (id 0) (at 130.81 90.805 0)
+    (property "Reference" "R36" (id 0) (at 130.81 90.805 0)
       (effects (font (size 1.27 1.27)) (justify left))
     )
@@
   (symbol (lib_id "Device:R_Small") (at 135.89 90.805 0) (unit 1)
     (in_bom yes) (on_board yes)
-    (property "Reference" "R17" (id 0) (at 137.16 90.805 0)
+    (property "Reference" "R37" (id 0) (at 137.16 90.805 0)
       (effects (font (size 1.27 1.27)) (justify left))
     )
@@
   (symbol (lib_id "power:GND") (at 132.715 95.885 0) (unit 1)
     (in_bom yes) (on_board yes)
-    (property "Reference" "#PWR072" (id 0) (at 132.715 102.235 0)
+    (property "Reference" "#PWR078" (id 0) (at 132.715 102.235 0)
       (effects (font (size 1.27 1.27)) hide)
     )
@@
   (symbol (lib_id "Device:R_Small") (at 88.9 120.65 0) (unit 1)
     (in_bom yes) (on_board yes)
-    (property "Reference" "R23" (id 0) (at 90.17 120.65 0)
+    (property "Reference" "R38" (id 0) (at 90.17 120.65 0)
       (effects (font (size 1.27 1.27)) (justify left))
     )
@@
   (symbol (lib_id "power:GND") (at 88.9 123.19 0) (unit 1)
     (in_bom yes) (on_board yes)
-    (property "Reference" "#PWR0272" (id 0) (at 88.9 129.54 0)
+    (property "Reference" "#PWR079" (id 0) (at 88.9 129.54 0)
       (effects (font (size 1.27 1.27)) hide)
     )

Commit message: update
Parts:
- renumbered J20 to J4, R36 to R20, R37 to R21, R38 to R22
Changed lines of the file:
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@@
   (symbol (lib_id "Connector:USB_C_Receptacle_USB2.0") (at 96.52 94.615 0) (unit 1)
     (in_bom yes) (on_board yes)
-    (property "Reference" "J20" (id 0) (at 87.63 75.438 0))
+    (property "Reference" "J4" (id 0) (at 87.63 75.438 0))
     (property "Value" "USB_C_Receptacle_USB2.0" (id 1) (at 99.2378 74.9046 0)
       (effects (font (size 1.27 1.27)) hide)
@@
   (symbol (lib_id "power:VBUS") (at 119.38 76.2 0) (unit 1)
     (in_bom yes) (on_board yes)
-    (property "Reference" "#PWR077" (id 0) (at 119.38 80.01 0)
+    (property "Reference" "#PWR061" (id 0) (at 119.38 80.01 0)
       (effects (font (size 1.27 1.27)) hide)
     )
@@
   (symbol (lib_id "power:GND") (at 96.52 123.19 0) (unit 1)
     (in_bom yes) (on_board yes)
-    (property "Reference" "#PWR080" (id 0) (at 96.52 129.54 0)
+    (property "Reference" "#PWR064" (id 0) (at 96.52 129.54 0)
       (effects (font (size 1.27 1.27)) hide)
     )
@@
   (symbol (lib_id "Device:R_Small") (at 129.54 90.805 0) (unit 1)
     (in_bom yes) (on_board yes)
-    (property "Reference" "R36" (id 0) (at 130.81 90.805 0)
+    (property "Reference" "R20" (id 0) (at 130.81 90.805 0)
       (effects (font (size 1.27 1.27)) (justify left))
     )
@@
   (symbol (lib_id "Device:R_Small") (at 135.89 90.805 0) (unit 1)
     (in_bom yes) (on_board yes)
-    (property "Reference" "R37" (id 0) (at 137.16 90.805 0)
+    (property "Reference" "R21" (id 0) (at 137.16 90.805 0)
       (effects (font (size 1.27 1.27)) (justify left))
     )
@@
   (symbol (lib_id "power:GND") (at 132.715 95.885 0) (unit 1)
     (in_bom yes) (on_board yes)
-    (property "Reference" "#PWR078" (id 0) (at 132.715 102.235 0)
+    (property "Reference" "#PWR062" (id 0) (at 132.715 102.235 0)
       (effects (font (size 1.27 1.27)) hide)
     )
@@
   (symbol (lib_id "Device:R_Small") (at 88.9 120.65 0) (unit 1)
     (in_bom yes) (on_board yes)
-    (property "Reference" "R38" (id 0) (at 90.17 120.65 0)
+    (property "Reference" "R22" (id 0) (at 90.17 120.65 0)
       (effects (font (size 1.27 1.27)) (justify left))
     )
@@
   (symbol (lib_id "power:GND") (at 88.9 123.19 0) (unit 1)
     (in_bom yes) (on_board yes)
-    (property "Reference" "#PWR079" (id 0) (at 88.9 129.54 0)
+    (property "Reference" "#PWR063" (id 0) (at 88.9 129.54 0)
       (effects (font (size 1.27 1.27)) hide)
     )

Commit message: update
Parts:
- renumbered J4 to J2, R20 to R16, R21 to R17, R22 to R23
Changed lines of the file:
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@@
   (symbol (lib_id "Connector:USB_C_Receptacle_USB2.0") (at 96.52 94.615 0) (unit 1)
     (in_bom yes) (on_board yes)
-    (property "Reference" "J4" (id 0) (at 87.63 75.438 0))
+    (property "Reference" "J2" (id 0) (at 87.63 75.438 0))
     (property "Value" "USB_C_Receptacle_USB2.0" (id 1) (at 99.2378 74.9046 0)
       (effects (font (size 1.27 1.27)) hide)
@@
   (symbol (lib_id "power:VBUS") (at 119.38 76.2 0) (unit 1)
     (in_bom yes) (on_board yes)
-    (property "Reference" "#PWR061" (id 0) (at 119.38 80.01 0)
+    (property "Reference" "#PWR070" (id 0) (at 119.38 80.01 0)
       (effects (font (size 1.27 1.27)) hide)
     )
@@
   (symbol (lib_id "power:GND") (at 96.52 123.19 0) (unit 1)
     (in_bom yes) (on_board yes)
-    (property "Reference" "#PWR064" (id 0) (at 96.52 129.54 0)
+    (property "Reference" "#PWR069" (id 0) (at 96.52 129.54 0)
       (effects (font (size 1.27 1.27)) hide)
     )
@@
   (symbol (lib_id "Device:R_Small") (at 129.54 90.805 0) (unit 1)
     (in_bom yes) (on_board yes)
-    (property "Reference" "R20" (id 0) (at 130.81 90.805 0)
+    (property "Reference" "R16" (id 0) (at 130.81 90.805 0)
       (effects (font (size 1.27 1.27)) (justify left))
     )
@@
   (symbol (lib_id "Device:R_Small") (at 135.89 90.805 0) (unit 1)
     (in_bom yes) (on_board yes)
-    (property "Reference" "R21" (id 0) (at 137.16 90.805 0)
+    (property "Reference" "R17" (id 0) (at 137.16 90.805 0)
       (effects (font (size 1.27 1.27)) (justify left))
     )
@@
   (symbol (lib_id "power:GND") (at 132.715 95.885 0) (unit 1)
     (in_bom yes) (on_board yes)
-    (property "Reference" "#PWR062" (id 0) (at 132.715 102.235 0)
+    (property "Reference" "#PWR072" (id 0) (at 132.715 102.235 0)
       (effects (font (size 1.27 1.27)) hide)
     )
@@
   (symbol (lib_id "Device:R_Small") (at 88.9 120.65 0) (unit 1)
     (in_bom yes) (on_board yes)
-    (property "Reference" "R22" (id 0) (at 90.17 120.65 0)
+    (property "Reference" "R23" (id 0) (at 90.17 120.65 0)
       (effects (font (size 1.27 1.27)) (justify left))
     )
@@
   (symbol (lib_id "power:GND") (at 88.9 123.19 0) (unit 1)
     (in_bom yes) (on_board yes)
-    (property "Reference" "#PWR063" (id 0) (at 88.9 129.54 0)
+    (property "Reference" "#PWR0272" (id 0) (at 88.9 129.54 0)
       (effects (font (size 1.27 1.27)) hide)
     )
