File: KiCad files/Main Project/Microcontroller.kicad_sch (KiCad schematic)
At the start: 11 parts, among them J1 USBasp, SW1 SW_Push, U1 ATmega328P-AU, Y1 16MHz

Commit message: update
Parts:
- removed R2: 470, Resistor_SMD:R_0805_2012Metric, symbol Device:R_Small
Connections:
- net SDA: now reaches U1.27 (PC4)
- net SCL: now reaches U1.28 (PC5)
- no-connect marks 17 -> 16
Other:
- moved on the sheet: J1
Changed lines of the file:
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@@
   )
   (no_connect (at 153.67 116.84))
+  (no_connect (at 153.67 93.98))
   (no_connect (at 153.67 66.04))
   (no_connect (at 153.67 111.76))
@@
   (no_connect (at 153.67 68.58))
   (no_connect (at 153.67 124.46))
-  (no_connect (at 153.67 99.06))
   (no_connect (at 153.67 63.5))
   (no_connect (at 123.19 71.12))
-  (no_connect (at 238.125 55.245))
+  (no_connect (at 210.185 58.42))
   (no_connect (at 153.67 119.38))
   (no_connect (at 153.67 114.3))
   (no_connect (at 153.67 86.36))
-  (no_connect (at 153.67 96.52))
   (no_connect (at 153.67 88.9))
   (wire (pts (xy 189.23 113.03) (xy 189.23 111.76))
@@
     (stroke (width 0) (type default) (color 0 0 0 0))
   )
-  (wire (pts (xy 154.94 93.98) (xy 153.67 93.98))
-    (stroke (width 0) (type default) (color 0 0 0 0))
-  )
   (wire (pts (xy 172.72 81.28) (xy 172.72 83.185))
     (stroke (width 0) (type default) (color 0 0 0 0))
@@
     (stroke (width 0) (type default) (color 0 0 0 0))
   )
-  (wire (pts (xy 161.29 93.98) (xy 160.02 93.98))
-    (stroke (width 0) (type default) (color 0 0 0 0))
-  )
   (wire (pts (xy 180.34 116.84) (xy 176.53 116.84))
     (stroke (width 0) (type default) (color 0 0 0 0))
   )
-  (text "USBasp port" (at 226.695 50.165 0)
+  (text "USBasp port" (at 198.755 53.34 0)
     (effects (font (size 1.27 1.27)) (justify left bottom))
   )
-  (global_label "MISO" (shape input) (at 225.425 55.245 180) (fields_autoplaced)
+  (global_label "MISO" (shape input) (at 197.485 58.42 180) (fields_autoplaced)
     (effects (font (size 1.27 1.27)) (justify right))
-    (property "Intersheet References" "${INTERSHEET_REFS}" (id 0) (at 0 0 0)
+    (property "Intersheet References" "${INTERSHEET_REFS}" (id 0) (at -27.94 3.175 0)
       (effects (font (size 1.27 1.27)) hide)
     )
@@
     )
   )
+  (global_label "SCL" (shape input) (at 153.67 99.06 0) (fields_autoplaced)
+    (effects (font (size 1.27 1.27)) (justify left))
+    (property "Intersheet References" "${INTERSHEET_REFS}" (id 0) (at 159.5018 98.9806 0)
+      (effects (font (size 1.27 1.27)) (justify left) hide)
+    )
+  )
+  (global_label "SDA" (shape input) (at 153.67 96.52 0) (fields_autoplaced)
+    (effects (font (size 1.27 1.27)) (justify left))
+    (property "Intersheet References" "${INTERSHEET_REFS}" (id 0) (at 159.5623 96.4406 0)
+      (effects (font (size 1.27 1.27)) (justify left) hide)
+    )
+  )
   (global_label "MISO" (shape input) (at 153.67 73.66 0) (fields_autoplaced)
     (effects (font (size 1.27 1.27)) (justify left))
@@
     )
   )
-  (global_label "GND" (shape input) (at 238.125 60.325 0) (fields_autoplaced)
-    (effects (font (size 1.27 1.27)) (justify left))
-    (property "Intersheet References" "${INTERSHEET_REFS}" (id 0) (at 0 0 0)
-      (effects (font (size 1.27 1.27)) hide)
-    )
-  )
-  (global_label "NEOPIXEL" (shape input) (at 161.29 93.98 0) (fields_autoplaced)
-    (effects (font (size 1.27 1.27)) (justify left))
-    (property "Intersheet References" "${INTERSHEET_REFS}" (id 0) (at 0 0 0)
-      (effects (font (size 1.27 1.27)) hide)
-    )
-  )
-  (global_label "RESET" (shape input) (at 225.425 60.325 180) (fields_autoplaced)
+  (global_label "GND" (shape input) (at 210.185 63.5 0) (fields_autoplaced)
+    (effects (font (size 1.27 1.27)) (justify left))
+    (property "Intersheet References" "${INTERSHEET_REFS}" (id 0) (at -27.94 3.175 0)
+      (effects (font (size 1.27 1.27)) hide)
+    )
+  )
+  (global_label "RESET" (shape input) (at 197.485 63.5 180) (fields_autoplaced)
     (effects (font (size 1.27 1.27)) (justify right))
-    (property "Intersheet References" "${INTERSHEET_REFS}" (id 0) (at 0 0 0)
+    (property "Intersheet References" "${INTERSHEET_REFS}" (id 0) (at -27.94 3.175 0)
       (effects (font (size 1.27 1.27)) hide)
     )
@@
     )
   )
-  (global_label "MOSI" (shape input) (at 238.125 57.785 0) (fields_autoplaced)
-    (effects (font (size 1.27 1.27)) (justify left))
-    (property "Intersheet References" "${INTERSHEET_REFS}" (id 0) (at 0 0 0)
+  (global_label "MOSI" (shape input) (at 210.185 60.96 0) (fields_autoplaced)
+    (effects (font (size 1.27 1.27)) (justify left))
+    (property "Intersheet References" "${INTERSHEET_REFS}" (id 0) (at -27.94 3.175 0)
       (effects (font (size 1.27 1.27)) hide)
     )
@@
     )
   )
-  (global_label "SCK" (shape input) (at 225.425 57.785 180) (fields_autoplaced)
+  (global_label "SCK" (shape input) (at 197.485 60.96 180) (fields_autoplaced)
     (effects (font (size 1.27 1.27)) (justify right))
-    (property "Intersheet References" "${INTERSHEET_REFS}" (id 0) (at 0 0 0)
+    (property "Intersheet References" "${INTERSHEET_REFS}" (id 0) (at -27.94 3.175 0)
       (effects (font (size 1.27 1.27)) hide)
     )
@@
     (pin "1")
   )
-  (symbol (lib_id "Connector_Generic:Conn_02x03_Odd_Even") (at 230.505 57.785 0) (unit 1)
-    (in_bom yes) (on_board yes)
-    (property "Reference" "J1" (id 0) (at 231.775 52.705 0))
-    (property "Value" "USBasp" (id 1) (at 231.775 62.865 0))
-    (property "Footprint" "CNLJS:USBasp" (id 2) (at 230.505 57.785 0)
-      (effects (font (size 1.27 1.27)) hide)
-    )
-    (property "Datasheet" "~" (id 3) (at 230.505 57.785 0)
-      (effects (font (size 1.27 1.27)) hide)
-    )
-    (property "Basic/Extended" "-" (id 4) (at 230.505 57.785 0)
-      (effects (font (size 1.27 1.27)) hide)
-    )
-    (property "JLCPCB Part #" "-" (id 5) (at 230.505 57.785 0)
-      (effects (font (size 1.27 1.27)) hide)
-    )
-    (property "U labosu?" "Da" (id 6) (at 230.505 57.785 0)
+  (symbol (lib_id "Connector_Generic:Conn_02x03_Odd_Even") (at 202.565 60.96 0) (unit 1)
+    (in_bom yes) (on_board yes)
+    (property "Reference" "J1" (id 0) (at 203.835 55.88 0))
+    (property "Value" "USBasp" (id 1) (at 203.835 66.04 0))
+    (property "Footprint" "CNLJS:USBasp" (id 2) (at 202.565 60.96 0)
+      (effects (font (size 1.27 1.27)) hide)
+    )
+    (property "Datasheet" "~" (id 3) (at 202.565 60.96 0)
+      (effects (font (size 1.27 1.27)) hide)
+    )
+    (property "Basic/Extended" "-" (id 4) (at 202.565 60.96 0)
+      (effects (font (size 1.27 1.27)) hide)
+    )
+    (property "JLCPCB Part #" "-" (id 5) (at 202.565 60.96 0)
+      (effects (font (size 1.27 1.27)) hide)
+    )
+    (property "U labosu?" "Da" (id 6) (at 202.565 60.96 0)
       (effects (font (size 1.27 1.27)) hide)
     )
@@
     (pin "1")
   )
-  (symbol (lib_id "Device:R_Small") (at 157.48 93.98 270) (unit 1)
-    (in_bom yes) (on_board yes)
-    (property "Reference" "R2" (id 0) (at 157.48 92.075 90))
-    (property "Value" "470" (id 1) (at 157.48 93.98 90)
-      (effects (font (size 0.9906 0.9906)))
-    )
-    (property "Footprint" "Resistor_SMD:R_0805_2012Metric" (id 2) (at 157.48 93.98 0)
-      (effects (font (size 1.27 1.27)) hide)
-    )
-    (property "Datasheet" "~" (id 3) (at 157.48 93.98 0)
-      (effects (font (size 1.27 1.27)) hide)
-    )
-    (property "Basic/Extended" "Basic" (id 4) (at 157.48 93.98 0)
-      (effects (font (size 1.27 1.27)) hide)
-    )
-    (property "JLCPCB Part #" "C25804" (id 5) (at 157.48 93.98 0)
-      (effects (font (size 1.27 1.27)) hide)
-    )
-    (property "U labosu?" "Da" (id 6) (at 157.48 93.98 0)
-      (effects (font (size 1.27 1.27)) hide)
-    )
-    (pin "1")
-    (pin "2")
-  )
   (symbol (lib_id "power:VDD") (at 96.52 48.26 0) (unit 1)

Commit message: update
Connections:
- net INT: now reaches U1.32 (PD2)
- no-connect marks 16 -> 15
Changed lines of the file:
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@@
   (no_connect (at 153.67 93.98))
   (no_connect (at 153.67 66.04))
-  (no_connect (at 153.67 111.76))
   (no_connect (at 153.67 121.92))
   (no_connect (at 123.19 68.58))
@@
     (stroke (width 0) (type default) (color 0 0 0 0))
   )
-  (wire (pts (xy 154.94 109.22) (xy 153.67 109.22))
-    (stroke (width 0) (type default) (color 0 0 0 0))
-  )
   (wire (pts (xy 140.97 55.88) (xy 140.97 50.165))
-    (stroke (width 0) (type default) (color 0 0 0 0))
-  )
-  (wire (pts (xy 154.94 106.68) (xy 153.67 106.68))
     (stroke (width 0) (type default) (color 0 0 0 0))
   )
@@
     )
   )
-  (global_label "RX" (shape input) (at 154.94 106.68 0) (fields_autoplaced)
+  (global_label "RX" (shape input) (at 153.67 106.68 0) (fields_autoplaced)
     (effects (font (size 1.27 1.27)) (justify left))
-    (property "Intersheet References" "${INTERSHEET_REFS}" (id 0) (at 0 0 0)
+    (property "Intersheet References" "${INTERSHEET_REFS}" (id 0) (at -1.27 0 0)
       (effects (font (size 1.27 1.27)) hide)
     )
@@
     )
   )
-  (global_label "TX" (shape input) (at 154.94 109.22 0) (fields_autoplaced)
+  (global_label "TX" (shape input) (at 153.67 109.22 0) (fields_autoplaced)
     (effects (font (size 1.27 1.27)) (justify left))
-    (property "Intersheet References" "${INTERSHEET_REFS}" (id 0) (at 0 0 0)
+    (property "Intersheet References" "${INTERSHEET_REFS}" (id 0) (at -1.27 0 0)
       (effects (font (size 1.27 1.27)) hide)
     )
@@
     )
   )
+  (global_label "INT" (shape input) (at 153.67 111.76 0) (fields_autoplaced)
+    (effects (font (size 1.27 1.27)) (justify left))
+    (property "Intersheet References" "${INTERSHEET_REFS}" (id 0) (at 158.8971 111.6806 0)
+      (effects (font (size 1.27 1.27)) (justify left) hide)
+    )
+  )

Commit message: update
Parts:
- removed U1: ATmega328P-AU, Package_QFP:TQFP-32_7x7mm_P0.8mm, symbol MCU_Microchip_ATmega:ATmega328P-AU
- added U18: ATmega328-A, Package_QFP:TQFP-32_7x7mm_P0.8mm, symbol MCU_Microchip_ATmega:ATmega328-A
- SW1: footprint (none) -> Button_Switch_SMD:SW_SPST_TL3342
Connections:
- net GND: now also U18.21 (GND), U18.3 (GND), U18.5 (GND)
- net INT: now also U18.32 (PD2)
- net MISO: now also U18.16 (PB4)
- net MOSI: now also U18.15 (PB3)
- net RESET: now also U18.29 (~{RESET}/PC6)
- net RX: now also U18.30 (PD0)
- net SCK: now also U18.17 (PB5)
- net SCL: now also U18.28 (PC5)
- net SDA: now also U18.27 (PC4)
- net TX: now also U18.31 (PD1)
- net VDD: now also U18.20 (AREF), U18.4 (VCC), U18.6 (VCC)
- net at C23.1, L2.2: now also U18.18 (AVCC)
- net at Y1.3: now also U18.7 (XTAL1/PB6)
- net at Y1.1: now also U18.8 (XTAL2/PB7)
- new net NP_1: U18.1 (PD3)
- new net NP_2: U18.2 (PD4)
- new net NP_3: U18.9 (PD5)
- new net NP_4: U18.10 (PD6)
- new net NP_5: U18.11 (PD7)
- no-connect marks 15 -> 10

Commit message: update
Parts:
- J1: footprint CNLJS:USBasp -> Connector_PinSocket_1.27mm:PinSocket_2x03_P1.27mm_Vertical
Changed lines of the file:
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@@
     (property "Reference" "J1" (id 0) (at 203.835 55.88 0))
     (property "Value" "USBasp" (id 1) (at 203.835 66.04 0))
-    (property "Footprint" "CNLJS:USBasp" (id 2) (at 202.565 60.96 0)
+    (property "Footprint" "Connector_PinSocket_1.27mm:PinSocket_2x03_P1.27mm_Vertical" (id 2) (at 202.565 60.96 0)
       (effects (font (size 1.27 1.27)) hide)
     )

Commit message: shematic update
Parts:
- added LS17: Speaker, CNLJS:KLJ-1102, symbol Device:Speaker
- renumbered C11 to C19, C23 to C20, C22 to C21, C12 to C22, J1 to J17, L2 to L18, R3 to R23, SW1 to SW17, Y1 to Y17
Connections:
- net GND: now also LS17.2
- net BUZZER: now reaches U18.13 (PB1)
- net BUZZER: now also LS17.1
- no-connect marks 10 -> 9
Changed lines of the file:
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@@
   )
   (no_connect (at 153.67 93.98))
-  (no_connect (at 153.67 66.04))
   (no_connect (at 123.19 68.58))
   (no_connect (at 153.67 91.44))
@@
     (stroke (width 0) (type default) (color 0 0 0 0))
   )
+  (wire (pts (xy 215.265 89.535) (xy 215.265 88.265))
+    (stroke (width 0) (type default) (color 0 0 0 0))
+  )
+  (wire (pts (xy 215.265 88.265) (xy 216.535 88.265))
+    (stroke (width 0) (type default) (color 0 0 0 0))
+  )
   (wire (pts (xy 111.125 63.5) (xy 123.19 63.5))
     (stroke (width 0) (type default) (color 0 0 0 0))
@@
     )
   )
+  (global_label "BUZZER" (shape input) (at 153.67 66.04 0) (fields_autoplaced)
+    (effects (font (size 1.27 1.27)) (justify left))
+    (property "Intersheet References" "${INTERSHEET_REFS}" (id 0) (at 163.4328 65.9606 0)
+      (effects (font (size 1.27 1.27)) (justify left) hide)
+    )
+  )
   (global_label "NP_2" (shape input) (at 153.67 116.84 0) (fields_autoplaced)
     (effects (font (size 1.27 1.27)) (justify left))
@@
     )
   )
+  (global_label "BUZZER" (shape input) (at 216.535 85.725 180) (fields_autoplaced)
+    (effects (font (size 1.27 1.27)) (justify right))
+    (property "Intersheet References" "${INTERSHEET_REFS}" (id 0) (at 206.7722 85.8044 0)
+      (effects (font (size 1.27 1.27)) (justify right) hide)
+    )
+  )
   (global_label "SCK" (shape input) (at 153.67 76.2 0) (fields_autoplaced)
     (effects (font (size 1.27 1.27)) (justify left))
@@
   (symbol (lib_id "power:GND") (at 138.43 132.08 0) (unit 1)
     (in_bom yes) (on_board yes)
-    (property "Reference" "#PWR047" (id 0) (at 138.43 138.43 0)
+    (property "Reference" "#PWR061" (id 0) (at 138.43 138.43 0)
       (effects (font (size 1.27 1.27)) hide)
     )
@@
   (symbol (lib_id "Device:R_Small") (at 189.23 109.22 180) (unit 1)
     (in_bom yes) (on_board yes)
-    (property "Reference" "R3" (id 0) (at 191.135 109.22 90))
+    (property "Reference" "R23" (id 0) (at 191.135 109.22 90))
     (property "Value" "10k" (id 1) (at 189.23 109.22 90)
       (effects (font (size 0.9906 0.9906)))
@@
   (symbol (lib_id "Device:C_Small") (at 96.52 53.975 0) (unit 1)
     (in_bom yes) (on_board yes)
-    (property "Reference" "C11" (id 0) (at 98.8568 52.8066 0)
+    (property "Reference" "C19" (id 0) (at 98.8568 52.8066 0)
       (effects (font (size 1.27 1.27)) (justify left))
     )
@@
   (symbol (lib_id "power:GND") (at 96.52 56.515 0) (unit 1)
     (in_bom yes) (on_board yes)
-    (property "Reference" "#PWR045" (id 0) (at 96.52 62.865 0)
+    (property "Reference" "#PWR053" (id 0) (at 96.52 62.865 0)
       (effects (font (size 1.27 1.27)) hide)
     )
@@
   (symbol (lib_id "Device:Resonator_Small") (at 175.26 85.725 0) (unit 1)
     (in_bom yes) (on_board yes)
-    (property "Reference" "Y1" (id 0) (at 180.0352 85.8266 0)
+    (property "Reference" "Y17" (id 0) (at 180.0352 85.8266 0)
       (effects (font (size 1.27 1.27)) (justify left))
     )
@@
   (symbol (lib_id "power:GND") (at 175.26 90.805 0) (unit 1)
     (in_bom yes) (on_board yes)
-    (property "Reference" "#PWR049" (id 0) (at 175.26 97.155 0)
+    (property "Reference" "#PWR058" (id 0) (at 175.26 97.155 0)
       (effects (font (size 1.27 1.27)) hide)
     )
@@
   (symbol (lib_id "Connector_Generic:Conn_02x03_Odd_Even") (at 202.565 60.96 0) (unit 1)
     (in_bom yes) (on_board yes)
-    (property "Reference" "J1" (id 0) (at 203.835 55.88 0))
+    (property "Reference" "J17" (id 0) (at 203.835 55.88 0))
     (property "Value" "USBasp" (id 1) (at 203.835 66.04 0))
     (property "Footprint" "Connector_PinSocket_1.27mm:PinSocket_2x03_P1.27mm_Vertical" (id 2) (at 202.565 60.96 0)
@@
   (symbol (lib_id "Switch:SW_Push") (at 182.88 113.03 0) (unit 1)
     (in_bom yes) (on_board yes)
-    (property "Reference" "SW1" (id 0) (at 182.88 107.95 0))
+    (property "Reference" "SW17" (id 0) (at 182.88 107.95 0))
     (property "Value" "SW_Push" (id 1) (at 182.88 108.1024 0)
       (effects (font (size 1.27 1.27)) hide)
@@
   (symbol (lib_id "Device:C_Small") (at 182.88 116.84 270) (unit 1)
     (in_bom yes) (on_board yes)
-    (property "Reference" "C12" (id 0) (at 181.61 120.015 90)
+    (property "Reference" "C22" (id 0) (at 181.61 120.015 90)
       (effects (font (size 1.27 1.27)) (justify left))
     )
@@
   (symbol (lib_id "power:GND") (at 176.53 118.745 0) (unit 1)
     (in_bom yes) (on_board yes)
-    (property "Reference" "#PWR048" (id 0) (at 176.53 125.095 0)
+    (property "Reference" "#PWR060" (id 0) (at 176.53 125.095 0)
       (effects (font (size 1.27 1.27)) hide)
     )
@@
   (symbol (lib_id "power:VDD") (at 96.52 48.26 0) (unit 1)
     (in_bom yes) (on_board yes)
-    (property "Reference" "#PWR044" (id 0) (at 96.52 52.07 0)
+    (property "Reference" "#PWR052" (id 0) (at 96.52 52.07 0)
       (effects (font (size 1.27 1.27)) hide)
     )
@@
   (symbol (lib_id "power:VDD") (at 189.23 106.68 0) (unit 1)
     (in_bom yes) (on_board yes)
-    (property "Reference" "#PWR050" (id 0) (at 189.23 110.49 0)
+    (property "Reference" "#PWR059" (id 0) (at 189.23 110.49 0)
       (effects (font (size 1.27 1.27)) hide)
     )
@@
     (pin "1")
   )
+  (symbol (lib_id "Device:Speaker") (at 221.615 85.725 0) (unit 1)
+    (in_bom yes) (on_board yes) (fields_autoplaced)
+    (property "Reference" "LS17" (id 0) (at 225.933 86.1603 0)
+      (effects (font (size 1.27 1.27)) (justify left))
+    )
+    (property "Value" "Speaker" (id 1) (at 225.933 88.6972 0)
+      (effects (font (size 1.27 1.27)) (justify left))
+    )
+    (property "Footprint" "CNLJS:KLJ-1102" (id 2) (at 221.615 90.805 0)
+      (effects (font (size 1.27 1.27)) hide)
+    )
+    (property "Datasheet" "~" (id 3) (at 221.361 86.995 0)
+      (effects (font (size 1.27 1.27)) hide)
+    )
+    (pin "1")
+    (pin "2")
+  )
   (symbol (lib_id "power:VDD") (at 160.02 40.005 0) (unit 1)
     (in_bom yes) (on_board yes)
-    (property "Reference" "#PWR0106" (id 0) (at 160.02 43.815 0)
+    (property "Reference" "#PWR051" (id 0) (at 160.02 43.815 0)
       (effects (font (size 1.27 1.27)) hide)
     )
@@
   (symbol (lib_id "power:PWR_FLAG") (at 146.05 47.625 0) (unit 1)
     (in_bom yes) (on_board yes) (fields_autoplaced)
-    (property "Reference" "#FLG018" (id 0) (at 146.05 45.72 0)
+    (property "Reference" "#FLG021" (id 0) (at 146.05 45.72 0)
       (effects (font (size 1.27 1.27)) hide)
     )
@@
   (symbol (lib_id "Device:L_Small") (at 160.02 44.45 0) (unit 1)
     (in_bom yes) (on_board yes) (fields_autoplaced)
-    (property "Reference" "L2" (id 0) (at 161.163 43.5415 0)
+    (property "Reference" "L18" (id 0) (at 161.163 43.5415 0)
       (effects (font (size 1.27 1.27)) (justify left))
     )
@@
     (pin "1")
     (pin "2")
+  )
+  (symbol (lib_id "power:GND") (at 215.265 89.535 0) (unit 1)
+    (in_bom yes) (on_board yes) (fields_autoplaced)
+    (property "Reference" "#PWR057" (id 0) (at 215.265 95.885 0)
+      (effects (font (size 1.27 1.27)) hide)
+    )
+    (property "Value" "GND" (id 1) (at 215.265 93.9784 0))
+    (property "Footprint" "" (id 2) (at 215.265 89.535 0)
+      (effects (font (size 1.27 1.27)) hide)
+    )
+    (property "Datasheet" "" (id 3) (at 215.265 89.535 0)
+      (effects (font (size 1.27 1.27)) hide)
+    )
+    (pin "1")
   )
   (symbol (lib_id "power:PWR_FLAG") (at 128.905 47.625 0) (unit 1)
     (in_bom yes) (on_board yes) (fields_autoplaced)
-    (property "Reference" "#FLG0104" (id 0) (at 128.905 45.72 0)
+    (property "Reference" "#FLG020" (id 0) (at 128.905 45.72 0)
       (effects (font (size 1.27 1.27)) hide)
     )
@@
   (symbol (lib_id "power:GND") (at 111.125 73.025 0) (unit 1)
     (in_bom yes) (on_board yes)
-    (property "Reference" "#PWR0105" (id 0) (at 111.125 79.375 0)
+    (property "Reference" "#PWR056" (id 0) (at 111.125 79.375 0)
       (effects (font (size 1.27 1.27)) hide)
     )
@@
   (symbol (lib_id "Device:C_Small") (at 111.125 70.485 0) (unit 1)
     (in_bom yes) (on_board yes)
-    (property "Reference" "C22" (id 0) (at 113.4618 69.3166 0)
+    (property "Reference" "C21" (id 0) (at 113.4618 69.3166 0)
       (effects (font (size 1.27 1.27)) (justify left))
     )
@@
   (symbol (lib_id "Device:C_Small") (at 160.02 55.245 0) (unit 1)
     (in_bom yes) (on_board yes)
-    (property "Reference" "C23" (id 0) (at 162.3568 54.0766 0)
+    (property "Reference" "C20" (id 0) (at 162.3568 54.0766 0)
       (effects (font (size 1.27 1.27)) (justify left))
     )
@@
   (symbol (lib_id "power:VDD") (at 111.125 62.23 0) (unit 1)
     (in_bom yes) (on_board yes)
-    (property "Reference" "#PWR0128" (id 0) (at 111.125 66.04 0)
+    (property "Reference" "#PWR055" (id 0) (at 111.125 66.04 0)
       (effects (font (size 1.27 1.27)) hide)
     )
@@
   (symbol (lib_id "power:GND") (at 160.02 57.785 0) (unit 1)
     (in_bom yes) (on_board yes)
-    (property "Reference" "#PWR0107" (id 0) (at 160.02 64.135 0)
-      (effects (font (size 1.27 1.27)) hide)
-    )
+    (property "Reference" "#PWR054" (id 0) (at 160.02 64.135 0)
+      (effects (font (size 1.27 1.27)) hide)
+    )
