File: KiCad files/Main Project/Microcontroller.kicad_sch (KiCad schematic)
At the start: 11 parts, among them J17 USBasp, SW17 SW_Push, U18 ATmega328-A, Y17 16MHz

Commit message: update
Parts:
- renumbered C19 to C3, C20 to C4, C21 to C5, C22 to C6, J17 to J1, L18 to L2, LS17 to LS1, R23 to R7, SW17 to SW1, U18 to U2, Y17 to Y1
Changed lines of the file:
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@@
   (symbol (lib_id "power:GND") (at 138.43 132.08 0) (unit 1)
     (in_bom yes) (on_board yes)
-    (property "Reference" "#PWR061" (id 0) (at 138.43 138.43 0)
+    (property "Reference" "#PWR045" (id 0) (at 138.43 138.43 0)
       (effects (font (size 1.27 1.27)) hide)
     )
@@
   (symbol (lib_id "Device:R_Small") (at 189.23 109.22 180) (unit 1)
     (in_bom yes) (on_board yes)
-    (property "Reference" "R23" (id 0) (at 191.135 109.22 90))
+    (property "Reference" "R7" (id 0) (at 191.135 109.22 90))
     (property "Value" "10k" (id 1) (at 189.23 109.22 90)
       (effects (font (size 0.9906 0.9906)))
@@
   (symbol (lib_id "Device:C_Small") (at 96.52 53.975 0) (unit 1)
     (in_bom yes) (on_board yes)
-    (property "Reference" "C19" (id 0) (at 98.8568 52.8066 0)
+    (property "Reference" "C3" (id 0) (at 98.8568 52.8066 0)
       (effects (font (size 1.27 1.27)) (justify left))
     )
@@
   (symbol (lib_id "power:GND") (at 96.52 56.515 0) (unit 1)
     (in_bom yes) (on_board yes)
-    (property "Reference" "#PWR053" (id 0) (at 96.52 62.865 0)
+    (property "Reference" "#PWR037" (id 0) (at 96.52 62.865 0)
       (effects (font (size 1.27 1.27)) hide)
     )
@@
   (symbol (lib_id "Device:Resonator_Small") (at 175.26 85.725 0) (unit 1)
     (in_bom yes) (on_board yes)
-    (property "Reference" "Y17" (id 0) (at 180.0352 85.8266 0)
+    (property "Reference" "Y1" (id 0) (at 180.0352 85.8266 0)
       (effects (font (size 1.27 1.27)) (justify left))
     )
@@
   (symbol (lib_id "power:GND") (at 175.26 90.805 0) (unit 1)
     (in_bom yes) (on_board yes)
-    (property "Reference" "#PWR058" (id 0) (at 175.26 97.155 0)
+    (property "Reference" "#PWR042" (id 0) (at 175.26 97.155 0)
       (effects (font (size 1.27 1.27)) hide)
     )
@@
   (symbol (lib_id "Connector_Generic:Conn_02x03_Odd_Even") (at 202.565 60.96 0) (unit 1)
     (in_bom yes) (on_board yes)
-    (property "Reference" "J17" (id 0) (at 203.835 55.88 0))
+    (property "Reference" "J1" (id 0) (at 203.835 55.88 0))
     (property "Value" "USBasp" (id 1) (at 203.835 66.04 0))
     (property "Footprint" "Connector_PinSocket_1.27mm:PinSocket_2x03_P1.27mm_Vertical" (id 2) (at 202.565 60.96 0)
@@
   (symbol (lib_id "Switch:SW_Push") (at 182.88 113.03 0) (unit 1)
     (in_bom yes) (on_board yes)
-    (property "Reference" "SW17" (id 0) (at 182.88 107.95 0))
+    (property "Reference" "SW1" (id 0) (at 182.88 107.95 0))
     (property "Value" "SW_Push" (id 1) (at 182.88 108.1024 0)
       (effects (font (size 1.27 1.27)) hide)
@@
   (symbol (lib_id "Device:C_Small") (at 182.88 116.84 270) (unit 1)
     (in_bom yes) (on_board yes)
-    (property "Reference" "C22" (id 0) (at 181.61 120.015 90)
+    (property "Reference" "C6" (id 0) (at 181.61 120.015 90)
       (effects (font (size 1.27 1.27)) (justify left))
     )
@@
   (symbol (lib_id "power:GND") (at 176.53 118.745 0) (unit 1)
     (in_bom yes) (on_board yes)
-    (property "Reference" "#PWR060" (id 0) (at 176.53 125.095 0)
+    (property "Reference" "#PWR044" (id 0) (at 176.53 125.095 0)
       (effects (font (size 1.27 1.27)) hide)
     )
@@
   (symbol (lib_id "power:VDD") (at 96.52 48.26 0) (unit 1)
     (in_bom yes) (on_board yes)
-    (property "Reference" "#PWR052" (id 0) (at 96.52 52.07 0)
+    (property "Reference" "#PWR036" (id 0) (at 96.52 52.07 0)
       (effects (font (size 1.27 1.27)) hide)
     )
@@
   (symbol (lib_id "power:VDD") (at 189.23 106.68 0) (unit 1)
     (in_bom yes) (on_board yes)
-    (property "Reference" "#PWR059" (id 0) (at 189.23 110.49 0)
+    (property "Reference" "#PWR043" (id 0) (at 189.23 110.49 0)
       (effects (font (size 1.27 1.27)) hide)
     )
@@
   (symbol (lib_id "Device:Speaker") (at 221.615 85.725 0) (unit 1)
     (in_bom yes) (on_board yes) (fields_autoplaced)
-    (property "Reference" "LS17" (id 0) (at 225.933 86.1603 0)
+    (property "Reference" "LS1" (id 0) (at 225.933 86.1603 0)
       (effects (font (size 1.27 1.27)) (justify left))
     )
@@
   (symbol (lib_id "power:VDD") (at 160.02 40.005 0) (unit 1)
     (in_bom yes) (on_board yes)
-    (property "Reference" "#PWR051" (id 0) (at 160.02 43.815 0)
+    (property "Reference" "#PWR035" (id 0) (at 160.02 43.815 0)
       (effects (font (size 1.27 1.27)) hide)
     )
@@
   (symbol (lib_id "power:PWR_FLAG") (at 146.05 47.625 0) (unit 1)
     (in_bom yes) (on_board yes) (fields_autoplaced)
-    (property "Reference" "#FLG021" (id 0) (at 146.05 45.72 0)
+    (property "Reference" "#FLG05" (id 0) (at 146.05 45.72 0)
       (effects (font (size 1.27 1.27)) hide)
     )
@@
   (symbol (lib_id "Device:L_Small") (at 160.02 44.45 0) (unit 1)
     (in_bom yes) (on_board yes) (fields_autoplaced)
-    (property "Reference" "L18" (id 0) (at 161.163 43.5415 0)
+    (property "Reference" "L2" (id 0) (at 161.163 43.5415 0)
       (effects (font (size 1.27 1.27)) (justify left))
     )
@@
   (symbol (lib_id "power:GND") (at 215.265 89.535 0) (unit 1)
     (in_bom yes) (on_board yes) (fields_autoplaced)
-    (property "Reference" "#PWR057" (id 0) (at 215.265 95.885 0)
+    (property "Reference" "#PWR041" (id 0) (at 215.265 95.885 0)
       (effects (font (size 1.27 1.27)) hide)
     )
@@
   (symbol (lib_id "power:PWR_FLAG") (at 128.905 47.625 0) (unit 1)
     (in_bom yes) (on_board yes) (fields_autoplaced)
-    (property "Reference" "#FLG020" (id 0) (at 128.905 45.72 0)
+    (property "Reference" "#FLG04" (id 0) (at 128.905 45.72 0)
       (effects (font (size 1.27 1.27)) hide)
     )
@@
   (symbol (lib_id "power:GND") (at 111.125 73.025 0) (unit 1)
     (in_bom yes) (on_board yes)
-    (property "Reference" "#PWR056" (id 0) (at 111.125 79.375 0)
+    (property "Reference" "#PWR040" (id 0) (at 111.125 79.375 0)
       (effects (font (size 1.27 1.27)) hide)
     )
@@
   (symbol (lib_id "MCU_Microchip_ATmega:ATmega328-A") (at 138.43 93.98 0) (unit 1)
     (in_bom yes) (on_board yes) (fields_autoplaced)
-    (property "Reference" "U18" (id 0) (at 140.4494 131.5704 0)
+    (property "Reference" "U2" (id 0) (at 140.4494 131.5704 0)
       (effects (font (size 1.27 1.27)) (justify left))
     )
@@
   (symbol (lib_id "Device:C_Small") (at 111.125 70.485 0) (unit 1)
     (in_bom yes) (on_board yes)
-    (property "Reference" "C21" (id 0) (at 113.4618 69.3166 0)
+    (property "Reference" "C5" (id 0) (at 113.4618 69.3166 0)
       (effects (font (size 1.27 1.27)) (justify left))
     )
@@
   (symbol (lib_id "Device:C_Small") (at 160.02 55.245 0) (unit 1)
     (in_bom yes) (on_board yes)
-    (property "Reference" "C20" (id 0) (at 162.3568 54.0766 0)
+    (property "Reference" "C4" (id 0) (at 162.3568 54.0766 0)
       (effects (font (size 1.27 1.27)) (justify left))
     )
@@
   (symbol (lib_id "power:VDD") (at 111.125 62.23 0) (unit 1)
     (in_bom yes) (on_board yes)
-    (property "Reference" "#PWR055" (id 0) (at 111.125 66.04 0)
+    (property "Reference" "#PWR039" (id 0) (at 111.125 66.04 0)
       (effects (font (size 1.27 1.27)) hide)
     )
@@
   (symbol (lib_id "power:GND") (at 160.02 57.785 0) (unit 1)
     (in_bom yes) (on_board yes)
-    (property "Reference" "#PWR054" (id 0) (at 160.02 64.135 0)
-      (effects (font (size 1.27 1.27)) hide)
-    )
+    (property "Reference" "#PWR038" (id 0) (at 160.02 64.135 0)
+      (effects (font (size 1.27 1.27)) hide)
+    )

Commit message: update
Parts:
- removed LS1: Speaker, CNLJS:KLJ-1102, symbol Device:Speaker
- renumbered C3 to C11, C6 to C12, C5 to C22, C4 to C23, R7 to R3, U2 to U18
Connections:
- net BUZZER: no longer names the net of U18.13 (PB1)
- no-connect marks 9 -> 10
Changed lines of the file:
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@@
   )
   (no_connect (at 153.67 93.98))
+  (no_connect (at 153.67 66.04))
   (no_connect (at 123.19 68.58))
   (no_connect (at 153.67 91.44))
@@
     (stroke (width 0) (type default) (color 0 0 0 0))
   )
-  (wire (pts (xy 215.265 89.535) (xy 215.265 88.265))
-    (stroke (width 0) (type default) (color 0 0 0 0))
-  )
-  (wire (pts (xy 215.265 88.265) (xy 216.535 88.265))
-    (stroke (width 0) (type default) (color 0 0 0 0))
-  )
   (wire (pts (xy 111.125 63.5) (xy 123.19 63.5))
     (stroke (width 0) (type default) (color 0 0 0 0))
@@
     )
   )
-  (global_label "BUZZER" (shape input) (at 153.67 66.04 0) (fields_autoplaced)
-    (effects (font (size 1.27 1.27)) (justify left))
-    (property "Intersheet References" "${INTERSHEET_REFS}" (id 0) (at 163.4328 65.9606 0)
-      (effects (font (size 1.27 1.27)) (justify left) hide)
-    )
-  )
   (global_label "NP_2" (shape input) (at 153.67 116.84 0) (fields_autoplaced)
     (effects (font (size 1.27 1.27)) (justify left))
@@
     )
   )
-  (global_label "BUZZER" (shape input) (at 216.535 85.725 180) (fields_autoplaced)
-    (effects (font (size 1.27 1.27)) (justify right))
-    (property "Intersheet References" "${INTERSHEET_REFS}" (id 0) (at 206.7722 85.8044 0)
-      (effects (font (size 1.27 1.27)) (justify right) hide)
-    )
-  )
   (global_label "SCK" (shape input) (at 153.67 76.2 0) (fields_autoplaced)
     (effects (font (size 1.27 1.27)) (justify left))
@@
   (symbol (lib_id "power:GND") (at 138.43 132.08 0) (unit 1)
     (in_bom yes) (on_board yes)
-    (property "Reference" "#PWR045" (id 0) (at 138.43 138.43 0)
+    (property "Reference" "#PWR047" (id 0) (at 138.43 138.43 0)
       (effects (font (size 1.27 1.27)) hide)
     )
@@
   (symbol (lib_id "Device:R_Small") (at 189.23 109.22 180) (unit 1)
     (in_bom yes) (on_board yes)
-    (property "Reference" "R7" (id 0) (at 191.135 109.22 90))
+    (property "Reference" "R3" (id 0) (at 191.135 109.22 90))
     (property "Value" "10k" (id 1) (at 189.23 109.22 90)
       (effects (font (size 0.9906 0.9906)))
@@
   (symbol (lib_id "Device:C_Small") (at 96.52 53.975 0) (unit 1)
     (in_bom yes) (on_board yes)
-    (property "Reference" "C3" (id 0) (at 98.8568 52.8066 0)
+    (property "Reference" "C11" (id 0) (at 98.8568 52.8066 0)
       (effects (font (size 1.27 1.27)) (justify left))
     )
@@
   (symbol (lib_id "power:GND") (at 96.52 56.515 0) (unit 1)
     (in_bom yes) (on_board yes)
-    (property "Reference" "#PWR037" (id 0) (at 96.52 62.865 0)
+    (property "Reference" "#PWR045" (id 0) (at 96.52 62.865 0)
       (effects (font (size 1.27 1.27)) hide)
     )
@@
   (symbol (lib_id "power:GND") (at 175.26 90.805 0) (unit 1)
     (in_bom yes) (on_board yes)
-    (property "Reference" "#PWR042" (id 0) (at 175.26 97.155 0)
+    (property "Reference" "#PWR049" (id 0) (at 175.26 97.155 0)
       (effects (font (size 1.27 1.27)) hide)
     )
@@
   (symbol (lib_id "Device:C_Small") (at 182.88 116.84 270) (unit 1)
     (in_bom yes) (on_board yes)
-    (property "Reference" "C6" (id 0) (at 181.61 120.015 90)
+    (property "Reference" "C12" (id 0) (at 181.61 120.015 90)
       (effects (font (size 1.27 1.27)) (justify left))
     )
@@
   (symbol (lib_id "power:GND") (at 176.53 118.745 0) (unit 1)
     (in_bom yes) (on_board yes)
-    (property "Reference" "#PWR044" (id 0) (at 176.53 125.095 0)
+    (property "Reference" "#PWR048" (id 0) (at 176.53 125.095 0)
       (effects (font (size 1.27 1.27)) hide)
     )
@@
   (symbol (lib_id "power:VDD") (at 96.52 48.26 0) (unit 1)
     (in_bom yes) (on_board yes)
-    (property "Reference" "#PWR036" (id 0) (at 96.52 52.07 0)
+    (property "Reference" "#PWR044" (id 0) (at 96.52 52.07 0)
       (effects (font (size 1.27 1.27)) hide)
     )
@@
   (symbol (lib_id "power:VDD") (at 189.23 106.68 0) (unit 1)
     (in_bom yes) (on_board yes)
-    (property "Reference" "#PWR043" (id 0) (at 189.23 110.49 0)
+    (property "Reference" "#PWR050" (id 0) (at 189.23 110.49 0)
       (effects (font (size 1.27 1.27)) hide)
     )
@@
     (pin "1")
   )
-  (symbol (lib_id "Device:Speaker") (at 221.615 85.725 0) (unit 1)
-    (in_bom yes) (on_board yes) (fields_autoplaced)
-    (property "Reference" "LS1" (id 0) (at 225.933 86.1603 0)
-      (effects (font (size 1.27 1.27)) (justify left))
-    )
-    (property "Value" "Speaker" (id 1) (at 225.933 88.6972 0)
-      (effects (font (size 1.27 1.27)) (justify left))
-    )
-    (property "Footprint" "CNLJS:KLJ-1102" (id 2) (at 221.615 90.805 0)
-      (effects (font (size 1.27 1.27)) hide)
-    )
-    (property "Datasheet" "~" (id 3) (at 221.361 86.995 0)
-      (effects (font (size 1.27 1.27)) hide)
-    )
-    (pin "1")
-    (pin "2")
-  )
   (symbol (lib_id "power:VDD") (at 160.02 40.005 0) (unit 1)
     (in_bom yes) (on_board yes)
-    (property "Reference" "#PWR035" (id 0) (at 160.02 43.815 0)
+    (property "Reference" "#PWR0106" (id 0) (at 160.02 43.815 0)
       (effects (font (size 1.27 1.27)) hide)
     )
@@
   (symbol (lib_id "power:PWR_FLAG") (at 146.05 47.625 0) (unit 1)
     (in_bom yes) (on_board yes) (fields_autoplaced)
-    (property "Reference" "#FLG05" (id 0) (at 146.05 45.72 0)
+    (property "Reference" "#FLG018" (id 0) (at 146.05 45.72 0)
       (effects (font (size 1.27 1.27)) hide)
     )
@@
     (pin "2")
   )
-  (symbol (lib_id "power:GND") (at 215.265 89.535 0) (unit 1)
-    (in_bom yes) (on_board yes) (fields_autoplaced)
-    (property "Reference" "#PWR041" (id 0) (at 215.265 95.885 0)
-      (effects (font (size 1.27 1.27)) hide)
-    )
-    (property "Value" "GND" (id 1) (at 215.265 93.9784 0))
-    (property "Footprint" "" (id 2) (at 215.265 89.535 0)
-      (effects (font (size 1.27 1.27)) hide)
-    )
-    (property "Datasheet" "" (id 3) (at 215.265 89.535 0)
-      (effects (font (size 1.27 1.27)) hide)
-    )
-    (pin "1")
-  )
   (symbol (lib_id "power:PWR_FLAG") (at 128.905 47.625 0) (unit 1)
     (in_bom yes) (on_board yes) (fields_autoplaced)
-    (property "Reference" "#FLG04" (id 0) (at 128.905 45.72 0)
+    (property "Reference" "#FLG0104" (id 0) (at 128.905 45.72 0)
       (effects (font (size 1.27 1.27)) hide)
     )
@@
   (symbol (lib_id "power:GND") (at 111.125 73.025 0) (unit 1)
     (in_bom yes) (on_board yes)
-    (property "Reference" "#PWR040" (id 0) (at 111.125 79.375 0)
+    (property "Reference" "#PWR0105" (id 0) (at 111.125 79.375 0)
       (effects (font (size 1.27 1.27)) hide)
     )
@@
   (symbol (lib_id "MCU_Microchip_ATmega:ATmega328-A") (at 138.43 93.98 0) (unit 1)
     (in_bom yes) (on_board yes) (fields_autoplaced)
-    (property "Reference" "U2" (id 0) (at 140.4494 131.5704 0)
+    (property "Reference" "U18" (id 0) (at 140.4494 131.5704 0)
       (effects (font (size 1.27 1.27)) (justify left))
     )
@@
   (symbol (lib_id "Device:C_Small") (at 111.125 70.485 0) (unit 1)
     (in_bom yes) (on_board yes)
-    (property "Reference" "C5" (id 0) (at 113.4618 69.3166 0)
+    (property "Reference" "C22" (id 0) (at 113.4618 69.3166 0)
       (effects (font (size 1.27 1.27)) (justify left))
     )
@@
   (symbol (lib_id "Device:C_Small") (at 160.02 55.245 0) (unit 1)
     (in_bom yes) (on_board yes)
-    (property "Reference" "C4" (id 0) (at 162.3568 54.0766 0)
+    (property "Reference" "C23" (id 0) (at 162.3568 54.0766 0)
       (effects (font (size 1.27 1.27)) (justify left))
     )
@@
   (symbol (lib_id "power:VDD") (at 111.125 62.23 0) (unit 1)
     (in_bom yes) (on_board yes)
-    (property "Reference" "#PWR039" (id 0) (at 111.125 66.04 0)
+    (property "Reference" "#PWR0128" (id 0) (at 111.125 66.04 0)
       (effects (font (size 1.27 1.27)) hide)
     )
@@
   (symbol (lib_id "power:GND") (at 160.02 57.785 0) (unit 1)
     (in_bom yes) (on_board yes)
-    (property "Reference" "#PWR038" (id 0) (at 160.02 64.135 0)
-      (effects (font (size 1.27 1.27)) hide)
-    )
+    (property "Reference" "#PWR0107" (id 0) (at 160.02 64.135 0)
+      (effects (font (size 1.27 1.27)) hide)
+    )

Commit message: buzzer
Parts:
- added LS1: Buzzer, CNLJS:KLJ-1102, symbol Device:Speaker
Connections:
- net GND: now also LS1.2
- net at U18.14 (PB2): now also LS1.1
- no-connect marks 10 -> 9
Changed lines of the file:
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@@
   (no_connect (at 123.19 68.58))
   (no_connect (at 153.67 91.44))
-  (no_connect (at 153.67 68.58))
   (no_connect (at 153.67 63.5))
   (no_connect (at 123.19 71.12))
@@
     (stroke (width 0) (type default) (color 0 0 0 0))
   )
+  (wire (pts (xy 198.755 85.09) (xy 200.66 85.09))
+    (stroke (width 0) (type default) (color 0 0 0 0))
+  )
   (wire (pts (xy 111.125 63.5) (xy 123.19 63.5))
     (stroke (width 0) (type default) (color 0 0 0 0))
@@
     (stroke (width 0) (type default) (color 0 0 0 0))
   )
+  (wire (pts (xy 198.755 82.55) (xy 200.66 82.55))
+    (stroke (width 0) (type default) (color 0 0 0 0))
+  )
   (wire (pts (xy 177.8 78.74) (xy 177.8 83.185))
     (stroke (width 0) (type default) (color 0 0 0 0))
@@
     (stroke (width 0) (type default) (color 0 0 0 0))
   )
+  (wire (pts (xy 198.755 86.36) (xy 198.755 85.09))
+    (stroke (width 0) (type default) (color 0 0 0 0))
+  )
+  (wire (pts (xy 198.755 68.58) (xy 198.755 82.55))
+    (stroke (width 0) (type default) (color 0 0 0 0))
+  )
   (wire (pts (xy 180.34 116.84) (xy 176.53 116.84))
+    (stroke (width 0) (type default) (color 0 0 0 0))
+  )
+  (wire (pts (xy 153.67 68.58) (xy 198.755 68.58))
     (stroke (width 0) (type default) (color 0 0 0 0))
   )
@@
     (pin "1")
     (pin "2")
+  )
+  (symbol (lib_id "power:GND") (at 198.755 86.36 0) (unit 1)
+    (in_bom yes) (on_board yes) (fields_autoplaced)
+    (property "Reference" "#PWR0270" (id 0) (at 198.755 92.71 0)
+      (effects (font (size 1.27 1.27)) hide)
+    )
+    (property "Value" "GND" (id 1) (at 198.755 90.8034 0))
+    (property "Footprint" "" (id 2) (at 198.755 86.36 0)
+      (effects (font (size 1.27 1.27)) hide)
+    )
+    (property "Datasheet" "" (id 3) (at 198.755 86.36 0)
+      (effects (font (size 1.27 1.27)) hide)
+    )
+    (pin "1")
   )
   (symbol (lib_id "power:PWR_FLAG") (at 128.905 47.625 0) (unit 1)
@@
       (effects (font (size 1.27 1.27)) hide)
     )
+    (pin "1")
+    (pin "2")
+  )
+  (symbol (lib_id "Device:Speaker") (at 205.74 82.55 0) (unit 1)
+    (in_bom yes) (on_board yes) (fields_autoplaced)
+    (property "Reference" "LS1" (id 0) (at 210.058 82.9853 0)
+      (effects (font (size 1.27 1.27)) (justify left))
+    )
+    (property "Value" "Buzzer" (id 1) (at 210.058 85.5222 0)
+      (effects (font (size 1.27 1.27)) (justify left))
+    )
+    (property "Footprint" "CNLJS:KLJ-1102" (id 2) (at 205.74 87.63 0)
+      (effects (font (size 1.27 1.27)) hide)
+    )
+    (property "Datasheet" "~" (id 3) (at 205.486 83.82 0)
+      (effects (font (size 1.27 1.27)) hide)
+    )
