File: KiCad files/BoardGame/CNLJS.kicad_sch (KiCad schematic)
At the start: 0 parts

Commit message: update
Other:
- note added: "BoardGame"
- note removed: "ČOVJEČE NE LJUTI SE (CNLJS)"
Changed lines of the file:
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@@
     (effects (font (size 2.9972 2.9972) (thickness 0.5994) bold) (justify left bottom))
   )
-  (text "ČOVJEČE NE LJUTI SE (CNLJS)" (at 51.435 27.94 0)
+  (text "BoardGame\n" (at 111.76 25.4 0)
     (effects (font (size 8.001 8.001) (thickness 1.6002) bold) (justify left bottom))
   )
