File: KiCad files/BoardGame/Power.kicad_sch (KiCad schematic)
At the start: 21 parts

Commit message: update
Other:
- title: (none) -> BoardGame
Changed lines of the file:
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@@
 (kicad_sch (version 20211123) (generator eeschema)
   (paper "A4")
+  (title_block
+    (title "BoardGame")
+    (date "2022-09-21")
+    (rev "1")
+  )
   (junction (at 165.735 74.295) (diameter 0) (color 0 0 0 0)
   )

Commit message: update
Parts:
- removed C?: 10u, symbol Device:C_Small
- removed C?: 4.7u / 25V, symbol Device:C_Small
- removed D? (x2): LED_Small, symbol Device:LED_Small
- removed R? (x3): 1k, symbol Device:R_Small
- removed R? (x4): 10k, symbol Device:R_Small
- removed U?: MCP73871-2CC, symbol Battery_Management:MCP73871-2CC
- added C?: 10u, Capacitor_Tantalum_SMD:CP_EIA-3528-21_Kemet-B, symbol Device:C_Polarized_Small
- added C?: 10u, Capacitor_SMD:C_0603_1608Metric, symbol Device:C_Small
- added D? (x2): LED_Small, LED_SMD:LED_0603_1608Metric, symbol Device:LED_Small
- added R? (x4): 10k, Resistor_SMD:R_0603_1608Metric, symbol Device:R_Small
- added R? (x3): 1k, Resistor_SMD:R_0603_1608Metric, symbol Device:R_Small
- added U?: MCP73871-2CC, Package_DFN_QFN:QFN-20-1EP_4x4mm_P0.5mm_EP2.5x2.5mm, symbol Battery_Management:MCP73871-2CC
- BT?: Basic/Extended Extended -> (none); JLCPCB Part # C225233 -> (none); U labosu? Da -> (none)
- C? (x2): footprint (none) -> Capacitor_SMD:C_0603_1608Metric; Basic/Extended Basic -> (none); JLCPCB Part # C440198 -> (none); U labosu? Ne -> (none)
- D?: footprint (none) -> LED_SMD:LED_0603_1608Metric; Basic/Extended Extended -> (none); JLCPCB Part # C205442 -> (none); U labosu? Da -> (none)
- R?: footprint (none) -> Resistor_SMD:R_0603_1608Metric; Basic/Extended Basic -> (none); JLCPCB Part # C17414 -> (none); U labosu? Da -> (none)
- R? (x2): footprint (none) -> Resistor_SMD:R_0603_1608Metric
Connections:
- net +BATT: now also C?.1, U?.14 (VBAT), U?.15 (VBAT), U?.16 (Vbat_SENSE)
- net CH_OUT: now also U?.1 (OUT), U?.20 (OUT)
- net GND: now also C?.2, C?.2, R?.2, R?.2, R?.2, U?.10 (VSS), U?.11 (VSS), U?.21 (VSS)
- net VBUS: now also C?.1, D?.2 (A), D?.2 (A), R?.1, U?.18 (IN), U?.19 (IN), U?.2 (VPCC)
- net at D?.1 (K): now also R?.2
- net at R?.1: now also U?.4 (PROG2)
- net at R?.1: now also U?.12 (PROG3)
- net at R?.1: now also U?.13 (PROG1)
- new net: R?.1, U?.3 (SEL)
- new net: R?.1, U?.9 (~{TE})
- new net: R?.1, U?.8 (STAT1/~{LBO})
- new net: D?.1 (K), R?.2 (x2)
- new net: R?.1, U?.6 (~{PG})
- new net: R?.1, U?.5 (THERM)
- new net: R?.2, U?.17 (CE)
- new net: R?.1, U?.7 (STAT2)
Other:
- moved on the sheet: R?
