File: KiCad files/BoardGame/BoardGame.kicad_sch (KiCad schematic)
At the start: 5 parts

Commit message: update
Parts:
- removed D? (x5): WS2812B, LED_SMD:LED_WS2812B_PLCC4_5.0x5.0mm_P3.2mm, symbol LED:WS2812B
- added BT1: Battery_Cell, symbol Device:Battery_Cell
- added C1, C10, C11, C12, C13, C7: 100n, symbol Device:C_Small
- added C14: 1u, symbol Device:C_Small
- added C2: 4.7u / 25V, symbol Device:C_Small
- added C3, C4, C5: 10u, symbol Device:C_Small
- added C6: 10n, symbol Device:C_Small
- added D1, D2, D3: LED_Small, symbol Device:LED_Small
- added J1, J4, J6, J7: Conn_02x03_Odd_Even, symbol Connector_Generic:Conn_02x03_Odd_Even
- added J2, J3: Conn_01x01, symbol Connector_Generic:Conn_01x01
- added J5: USB_C_Receptacle_USB2.0, symbol Connector:USB_C_Receptacle_USB2.0
- added J8: USBasp, symbol Connector_Generic:Conn_02x03_Odd_Even
- added L1: 10u, symbol Device:L_Small
- added LS1: Buzzer, symbol Device:Speaker
- added R1, R11, R12, R15, R19, R7: 10k, symbol Device:R_Small
- added R10, R13, R16, R17, R8: 1k, symbol Device:R_Small
- added R14: 1M, symbol Device:R_Small
- added R2: 2k, symbol Device:R_Small
- added R20, R21, R22, R23, R24: 470R, symbol Device:R_Small
- added R3, R4: 4k7, symbol Device:R_Small
- added R5, R6: 5k1, symbol Device:R_Small
- added R9: 100k, symbol Device:R_Small
- added SW1: SW_Push, symbol Switch:SW_Push
- added U1: PCF8575, symbol CNLJS-symbols:PCF8575
- added U2: MCP73871-2CC, symbol Battery_Management:MCP73871-2CC
- added U4: CH340C, symbol Interface_USB:CH340C
- added U5: ATmega328-A, symbol MCU_Microchip_ATmega:ATmega328-A
- added Y1: 16MHz, symbol Device:Resonator_Small
Connections:
- new net: U5.8 (XTAL2/PB7), Y1.1
- new net: U5.7 (XTAL1/PB6), Y1.3
- new net: J5.A5 (CC1), R6.1
- new net: J5.B5 (CC2), R5.1
- new net: J5.S1 (SHIELD), R14.1
- new net: R9.1, U2.12 (PROG3)
- new net: C11.1, L1.2, U5.18 (AVCC)
- new net: R2.1, U2.13 (PROG1)
- new net: R15.1, U2.17 (CE)
- new net: R1.1, U2.3 (SEL)
- new net: R7.1, U2.4 (PROG2)
- new net: R11.1, U2.5 (THERM)
- new net: R8.2, U2.6 (~{PG})
- new net: R13.2, U2.7 (STAT2)
- new net: R10.2, U2.8 (STAT1/~{LBO})
- new net: R12.1, U2.9 (~{TE})
- new net: D1.1 (K), R8.1
- new net: LS1.1, U5.14 (PB2)
- new net: C12.2, U4.13 (~{DTR})
- new net: D3.1 (K), R13.1
- new net: R16.2, U4.2 (TXD)
- new net: R17.2, U4.3 (RXD)
- new net: C6.1, U4.4 (V3)
- new net: D2.1 (K), R10.1
- new net +BATT: BT1.1 (+), C5.1, U2.14 (VBAT), U2.15 (VBAT), U2.16 (Vbat_SENSE)
- new net CH_OUT: C4.1, J3.1 (Pin_1), U2.1 (OUT), U2.20 (OUT)
- new net D+: J5.A6 (D+), J5.B6 (D+), U4.5 (UD+)
- new net D-: J5.A7 (D-), J5.B7 (D-), U4.6 (UD-)
- new net GND: BT1.2 (-), C1.2, C10.2, C11.2, C13.2, C14.2, C2.2, C3.2, C4.2, C5.2, C6.2, C7.2, J1.1 (Pin_1), J4.1 (Pin_1), J5.A1 (GND), J5.A12 (GND), J5.B1 (GND), J5.B12 (GND), J6.1 (Pin_1), J7.1 (Pin_1), J8.6 (Pin_6), LS1.2, R1.2, R11.2, R12.2, R14.2, R2.2, R5.2, R6.2, R9.2, SW1.1, U1.12 (GND), U2.10 (VSS), U2.11 (VSS), U2.21 (VSS), U4.1 (GND), U5.21 (GND), U5.3 (GND), U5.5 (GND), Y1.2
- new net INT: U1.1 (~{INT}), U5.32 (PD2)
- new net MISO: J8.1 (Pin_1), U5.16 (PB4)
- new net MOSI: J8.4 (Pin_4), U5.15 (PB3)
- new net NP_1: R20.1, U5.1 (PD3)
- new net NP_2: R21.1, U5.2 (PD4)
- new net NP_3: R22.1, U5.9 (PD5)
- new net NP_4: R23.1, U5.10 (PD6)
- new net NP_5: R24.1, U5.11 (PD7)
- new net RESET: C12.1, C14.1, J8.5 (Pin_5), R19.1, SW1.2, U5.29 (~{RESET}/PC6)
- new net RX: R16.1, U5.30 (PD0)
- new net SCK: J8.3 (Pin_3), U5.17 (PB5)
- new net SCL: R3.2, U1.22 (SCL), U5.28 (PC5)
- new net SDA: R4.2, U1.23 (SDA), U5.27 (PC4)
- new net TP_1: J1.2 (Pin_2), U1.4 (P00)
- new net TP_10: J7.2 (Pin_2), U1.14 (P11)
- new net TP_11: J7.6 (Pin_6), U1.15 (P12)
- new net TP_12: J7.5 (Pin_5), U1.16 (P13)
- new net TP_2: J1.6 (Pin_6), U1.5 (P01)
- new net TP_3: J1.5 (Pin_5), U1.6 (P02)
- new net TP_4: J4.2 (Pin_2), U1.7 (P03)
- new net TP_5: J4.6 (Pin_6), U1.8 (P04)
- new net TP_6: J4.5 (Pin_5), U1.9 (P05)
- new net TP_7: J6.2 (Pin_2), U1.10 (P06)
- new net TP_8: J6.6 (Pin_6), U1.11 (P07)
- new net TP_9: J6.5 (Pin_5), U1.13 (P10)
- new net TX: R17.1, U5.31 (PD1)
- new net VBUS: C2.1, C3.1, D1.2 (A), D2.2 (A), D3.2 (A), J5.A4 (VBUS), J5.A9 (VBUS), J5.B4 (VBUS), J5.B9 (VBUS), R15.2, R7.2, U2.18 (IN), U2.19 (IN), U2.2 (VPCC)
- new net VCC: J2.1 (Pin_1)
- new net VDD: C1.1, C10.1, C13.1, C7.1, J1.3 (Pin_3), J1.4 (Pin_4), J4.3 (Pin_3), J4.4 (Pin_4), J6.3 (Pin_3), J6.4 (Pin_4), J7.3 (Pin_3), J7.4 (Pin_4), L1.1, R19.2, R3.1, R4.1, U1.24 (VCC), U4.16 (VCC), U5.20 (AREF), U5.4 (VCC), U5.6 (VCC)
- no-connect marks 0 -> 24
Other:
- note added: "CHARGE"
- note added: "DONE"
- note added: "For optimum voltage regulation, it is recommended to place the battery pack closest to the device's VBAT and VSS pins to minimize voltage drops along the high current-carrying PCB traces. If the PCB layout is used as a heat sink, adding many vias in the heat sink pad can help conduct more heat to the PCB backplane, thus reducing the maximum junction temperature."
- note added: "If temperature monitoring is not required, place a standard 10k resistor from THERM to VSS."
- note added: "MCP73871"
- note added: "PADOVI SKLOPKE"
- note added: "PG = POWER GOOD STATUS OUTPUT STAT1 = CHARGE STATUS UPDATE 1 STAT2 = CHARGE STATUS UPDATE 2"
- note added: "POWER"
- note added: "Preinake na modulu: 1. pin 3 (SEL) preko 10k otpornika spojen na GND (USB način rada) 2. pin 2 (VPCC) kratko spojen na pin 18 (VIN)"
- note added: "SBU1/SBU2: these are low-speed lines used only for Alternate Mode and accessory mode. For example, with DisplayPort, AUX+/AUX– transmit over the SBU lines. For audio adapter accessory mode, these lines are used for the microphone input and analog GND."
- note added: "TANTALUM KOND."
- note added: "TODO: - koristiti kompletnu englesku dokumentaciju - zamijeniti regulator napona i maknuti onaj dio gdje se vrši odabir naponskih razina, to nije dobro - mjeriti napon baterije i napraviti indikator (iskoristiti neopixele kao indikator?) - LEDice za punjenje baterije - da li treba LDR? - power sklopka koja može prekinuti 1A - rupe za montažu - ispraviti dvije pozicije koje su preblizu - kockica t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"
- note added: "The device must have 5.1k pull-down on the its port CC pin (on both pins). Once the C-C cable is connected between two link partners, the DFP (host) will sense the drag by 5.1k resistor (from device side). As result, it will turn the VBUS on. This is how a host recognizes that a connection has been made. The connect event is essentially controlled by sink side having 5.1k Rd."
- note added: "USB NAPAJANJE"
- note added: "USBasp port"
- note added: "ovdje idu WS2812B"

Commit message: update
Parts:
- removed BT1: Battery_Cell, symbol Device:Battery_Cell
- removed C1, C12, C7: 100n, symbol Device:C_Small
- removed C2: 4.7u / 25V, symbol Device:C_Small
- removed C3, C4, C5: 10u, symbol Device:C_Small
- removed C6: 10n, symbol Device:C_Small
- removed D1, D2, D3: LED_Small, symbol Device:LED_Small
- removed J1, J4, J6, J7: Conn_02x03_Odd_Even, symbol Connector_Generic:Conn_02x03_Odd_Even
- removed J2, J3: Conn_01x01, symbol Connector_Generic:Conn_01x01
- removed J5: USB_C_Receptacle_USB2.0, symbol Connector:USB_C_Receptacle_USB2.0
- removed R1, R11, R12, R15, R7: 10k, symbol Device:R_Small
- removed R10, R13, R16, R17, R8: 1k, symbol Device:R_Small
- removed R14: 1M, symbol Device:R_Small
- removed R2: 2k, symbol Device:R_Small
- removed R3, R4: 4k7, symbol Device:R_Small
- removed R5, R6: 5k1, symbol Device:R_Small
- removed R9: 100k, symbol Device:R_Small
- removed U1: PCF8575, symbol CNLJS-symbols:PCF8575
- removed U2: MCP73871-2CC, symbol Battery_Management:MCP73871-2CC
- removed U4: CH340C, symbol Interface_USB:CH340C
Connections:
- no-connect marks 24 -> 9
Other:
- added sheet IO Expander (IO Expander.kicad_sch)
- added sheet Power (Power.kicad_sch)
- added sheet USB (USB.kicad_sch)
- note removed: "CHARGE"
- note removed: "DONE"
- note removed: "For optimum voltage regulation, it is recommended to place the battery pack closest to the device's VBAT and VSS pins to minimize voltage drops along the high current-carrying PCB traces. If the PCB layout is used as a heat sink, adding many vias in the heat sink pad can help conduct more heat to the PCB backplane, thus reducing the maximum junction temperature."
- note removed: "If temperature monitoring is not required, place a standard 10k resistor from THERM to VSS."
- note removed: "MCP73871"
- note removed: "PADOVI SKLOPKE"
- note removed: "PG = POWER GOOD STATUS OUTPUT STAT1 = CHARGE STATUS UPDATE 1 STAT2 = CHARGE STATUS UPDATE 2"
- note removed: "POWER"
- note removed: "Preinake na modulu: 1. pin 3 (SEL) preko 10k otpornika spojen na GND (USB način rada) 2. pin 2 (VPCC) kratko spojen na pin 18 (VIN)"
- note removed: "SBU1/SBU2: these are low-speed lines used only for Alternate Mode and accessory mode. For example, with DisplayPort, AUX+/AUX– transmit over the SBU lines. For audio adapter accessory mode, these lines are used for the microphone input and analog GND."
- note removed: "TANTALUM KOND."
- note removed: "The device must have 5.1k pull-down on the its port CC pin (on both pins). Once the C-C cable is connected between two link partners, the DFP (host) will sense the drag by 5.1k resistor (from device side). As result, it will turn the VBUS on. This is how a host recognizes that a connection has been made. The connect event is essentially controlled by sink side having 5.1k Rd."
- note removed: "USB NAPAJANJE"
- moved on the sheet: C10, C11, C13, C14, J8, L1, LS1, R19, R20, R21, R22, R23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

Commit message: update
Parts:
- removed C10, C11, C13: 100n, symbol Device:C_Small
- removed C14: 1u, symbol Device:C_Small
- removed J8: USBasp, symbol Connector_Generic:Conn_02x03_Odd_Even
- removed L1: 10u, symbol Device:L_Small
- removed LS1: Buzzer, symbol Device:Speaker
- removed R19: 10k, symbol Device:R_Small
- removed SW1: SW_Push, symbol Switch:SW_Push
- removed U5: ATmega328-A, symbol MCU_Microchip_ATmega:ATmega328-A
- removed Y1: 16MHz, symbol Device:Resonator_Small
- renumbered R21 to R?, R22 to R?, R23 to R?, R24 to R?, R20 to R?
Connections:
- no-connect marks 9 -> 0
Other:
- added sheet Boost Converter (Boost Converter.kicad_sch)
- added sheet Microcontroller (Microcontroller.kicad_sch)
- note added: "TODO: - koristiti kompletnu englesku dokumentaciju - mjeriti napon baterije i napraviti indikator (iskoristiti neopixele kao indikator?) - LEDice za punjenje baterije - da li treba LDR? - power sklopka koja može prekinuti 1A - rupe za montažu - ispraviti dvije pozicije koje su preblizu - kockica touchpad - buzzer - provjeriti shemu - isprintati na papir i provjeriti footprinte"
- note removed: "TODO: - koristiti kompletnu englesku dokumentaciju - zamijeniti regulator napona i maknuti onaj dio gdje se vrši odabir naponskih razina, to nije dobro - mjeriti napon baterije i napraviti indikator (iskoristiti neopixele kao indikator?) - LEDice za punjenje baterije - da li treba LDR? - power sklopka koja može prekinuti 1A - rupe za montažu - ispraviti dvije pozicije koje su preblizu - kockica t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"
- note removed: "USBasp port"
- title: (none) -> BoardGame

Commit message: update
Other:
- note added: "ovdje idu WS2812B napajani sa VCC"
- note removed: "ovdje idu WS2812B"
- moved on the sheet: R?

Commit message: update
Other:
- sheet Power renamed Battery charger
- sheet Battery charger: file Power.kicad_sch -> Battery charger.kicad_sch
Changed lines of the file:
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@@
     (stroke (width 0.1524) (type solid) (color 0 0 0 1))
     (fill (color 255 229 191 1.0000))
-    (property "Sheet name" "Power" (id 0) (at 114.3 87.5534 0)
+    (property "Sheet name" "Battery charger" (id 0) (at 114.3 87.5534 0)
       (effects (font (size 1.27 1.27)) (justify left bottom))
     )
-    (property "Sheet file" "Power.kicad_sch" (id 1) (at 114.3 119.3296 0)
+    (property "Sheet file" "Battery charger.kicad_sch" (id 1) (at 114.3 119.3296 0)
       (effects (font (size 1.27 1.27)) (justify left top) hide)
     )

Commit message: update
Parts:
- removed R? (x5): 470R, symbol Device:R_Small
Other:
- added sheet Neopixel (Neopixel.kicad_sch)
- note removed: "ovdje idu WS2812B napajani sa VCC"

Commit message: update
Parts:
- added H1001, H1002, H1003, H1004, H1005, H1006, H1007, H1008: MountingHole, MountingHole:MountingHole_3.2mm_M3, symbol Mechanical:MountingHole
Other:
- note added: "TODO: - koristiti kompletnu englesku dokumentaciju - mjeriti napon baterije i napraviti indikator (iskoristiti neopixele kao indikator?) - LEDice za punjenje baterije - da li treba LDR? - power sklopka koja može prekinuti 1A - kockica touchpad - provjeriti shemu - isprintati na papir i provjeriti footprinte"
- note removed: "TODO: - koristiti kompletnu englesku dokumentaciju - mjeriti napon baterije i napraviti indikator (iskoristiti neopixele kao indikator?) - LEDice za punjenje baterije - da li treba LDR? - power sklopka koja može prekinuti 1A - rupe za montažu - ispraviti dvije pozicije koje su preblizu - kockica touchpad - buzzer - provjeriti shemu - isprintati na papir i provjeriti footprinte"
