File: KiCad files/BoardGame/BoardGame.kicad_sch (KiCad schematic)
At the start: 8 parts

Commit message: update
Other:
- note added: "TODO: - koristiti kompletnu englesku dokumentaciju - testirati da li STAT2 pin može biti očitan na mcu (high ili low) - mjeriti napon baterije i napraviti indikator (iskoristiti neopixele kao indikator?) - LEDice za punjenje baterije - power sklopka koja može prekinuti 1A - kockica touchpad - provjeriti shemu - isprintati na papir i provjeriti footprinte"
- note removed: "TODO: - koristiti kompletnu englesku dokumentaciju - mjeriti napon baterije i napraviti indikator (iskoristiti neopixele kao indikator?) - LEDice za punjenje baterije - da li treba LDR? - power sklopka koja može prekinuti 1A - kockica touchpad - provjeriti shemu - isprintati na papir i provjeriti footprinte"
Changed lines of the file:
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@@
     (rev "1")
   )
-  (text "TODO:\n- koristiti kompletnu englesku dokumentaciju\n- mjeriti napon baterije i napraviti indikator (iskoristiti neopixele kao indikator?)\n- LEDice za punjenje baterije\n- da li treba LDR?\n- power sklopka koja može prekinuti 1A\n- kockica touchpad\n- provjeriti shemu\n- isprintati na papir i provjeriti footprinte"
+  (text "TODO:\n- koristiti kompletnu englesku dokumentaciju\n- testirati da li STAT2 pin može biti očitan na mcu (high ili low)\n- mjeriti napon baterije i napraviti indikator (iskoristiti neopixele kao indikator?)\n- LEDice za punjenje baterije\n- power sklopka koja može prekinuti 1A\n- kockica touchpad\n- provjeriti shemu\n- isprintati na papir i provjeriti footprinte"
     (at 19.685 187.325 0)
     (effects (font (size 1.27 1.27)) (justify left bottom))
@@
     )
     (path "/137cdba1-cde3-4c49-b42e-e13f2be356c7/f39e5938-1d55-4ada-be42-3da5804b2a99"
-      (reference "BT301") (unit 1) (value "Battery_Cell") (footprint "Footprints:battery_906909_6000mah")
+      (reference "BT301") (unit 1) (value "Battery_Cell") (footprint "Footprints:battery_103565_3000mah")
     )
     (path "/ac94f7cf-c7fc-4258-a4c8-af0c3ef6d0a1/510a8aa0-9853-4d59-92da-cbd2cd9f9f7a"
@@
     )
     (path "/4ee94e79-8f79-4d3c-86ca-8e64aae4ab70/de15bc89-2244-45da-ba06-6a1603c41aa5"
-      (reference "J501") (unit 1) (value "USBasp") (footprint "Footprints:2x03_P2.54mm")
+      (reference "J501") (unit 1) (value "USBasp") (footprint "Connector_PinHeader_1.27mm:PinHeader_2x03_P1.27mm_Vertical_SMD")
     )
     (path "/4ee94e79-8f79-4d3c-86ca-8e64aae4ab70/d3f8e25f-4120-4ba2-9b66-04af3b9d8b2a"

Commit message: update
Other:
- note added: "TODO: - koristiti kompletnu englesku dokumentaciju - jedan neopixel koji je blizu punjača - power sklopka koja može prekinuti 1A - kockica touchpad - provjeriti shemu - isprintati na papir i provjeriti footprinte"
- note removed: "TODO: - koristiti kompletnu englesku dokumentaciju - testirati da li STAT2 pin može biti očitan na mcu (high ili low) - mjeriti napon baterije i napraviti indikator (iskoristiti neopixele kao indikator?) - LEDice za punjenje baterije - power sklopka koja može prekinuti 1A - kockica touchpad - provjeriti shemu - isprintati na papir i provjeriti footprinte"
Changed lines of the file:
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@@
     (rev "1")
   )
-  (text "TODO:\n- koristiti kompletnu englesku dokumentaciju\n- testirati da li STAT2 pin može biti očitan na mcu (high ili low)\n- mjeriti napon baterije i napraviti indikator (iskoristiti neopixele kao indikator?)\n- LEDice za punjenje baterije\n- power sklopka koja može prekinuti 1A\n- kockica touchpad\n- provjeriti shemu\n- isprintati na papir i provjeriti footprinte"
+  (text "TODO:\n- koristiti kompletnu englesku dokumentaciju\n- jedan neopixel koji je blizu punjača\n- power sklopka koja može prekinuti 1A\n- kockica touchpad\n- provjeriti shemu\n- isprintati na papir i provjeriti footprinte"
     (at 19.685 187.325 0)
     (effects (font (size 1.27 1.27)) (justify left bottom))
@@
       (reference "#PWR0309") (unit 1) (value "GND") (footprint "")
     )
-    (path "/137cdba1-cde3-4c49-b42e-e13f2be356c7/f9683d8e-8401-47e9-833d-ea3e456383bd"
-      (reference "#PWR0310") (unit 1) (value "VBUS") (footprint "")
-    )
     (path "/137cdba1-cde3-4c49-b42e-e13f2be356c7/299feb74-8e1d-42d5-a543-e61b0a810dd3"
       (reference "#PWR0311") (unit 1) (value "GND") (footprint "")
@@
       (reference "#PWR01168") (unit 1) (value "GND") (footprint "")
     )
+    (path "/4e78659c-21b0-4088-8876-cb944b9d811b/94f23a45-f80c-405a-953b-924a6f195d77"
+      (reference "#PWR01169") (unit 1) (value "VCC") (footprint "")
+    )
+    (path "/4e78659c-21b0-4088-8876-cb944b9d811b/ef8faf14-3c3f-4433-8ac7-7bb8c5995b5b"
+      (reference "#PWR01170") (unit 1) (value "GND") (footprint "")
+    )
+    (path "/137cdba1-cde3-4c49-b42e-e13f2be356c7/4fea6a02-2d17-430a-8782-08f7d6a7a885"
+      (reference "#PWR?") (unit 1) (value "VBUS") (footprint "")
+    )
+    (path "/137cdba1-cde3-4c49-b42e-e13f2be356c7/6ef946b1-68a2-4826-b9df-2ec18dd67d90"
+      (reference "#PWR?") (unit 1) (value "VBUS") (footprint "")
+    )
+    (path "/137cdba1-cde3-4c49-b42e-e13f2be356c7/b562b1ed-5661-41bb-aeb1-1c7c7d6b3a6d"
+      (reference "#PWR?") (unit 1) (value "VBUS") (footprint "")
+    )
     (path "/137cdba1-cde3-4c49-b42e-e13f2be356c7/f39e5938-1d55-4ada-be42-3da5804b2a99"
       (reference "BT301") (unit 1) (value "Battery_Cell") (footprint "Footprints:battery_103565_3000mah")
@@
       (reference "C1009") (unit 1) (value "100n") (footprint "Capacitor_SMD:C_0603_1608Metric")
     )
-    (path "/137cdba1-cde3-4c49-b42e-e13f2be356c7/f9b67d9d-4294-475a-84cb-9fe09914e36a"
-      (reference "D301") (unit 1) (value "LED_Small") (footprint "LED_SMD:LED_0603_1608Metric")
-    )
-    (path "/137cdba1-cde3-4c49-b42e-e13f2be356c7/7198921d-6f6d-40c9-b786-404a25255e97"
-      (reference "D302") (unit 1) (value "LED_Small") (footprint "LED_SMD:LED_0603_1608Metric")
-    )
-    (path "/137cdba1-cde3-4c49-b42e-e13f2be356c7/90aefc8a-c804-47eb-8919-82ead1a53bc0"
-      (reference "D303") (unit 1) (value "LED_Small") (footprint "LED_SMD:LED_0603_1608Metric")
-    )
     (path "/bfec7ff5-12b5-4af9-9131-b19e09596ace/8c1809b1-1a92-48e2-b214-386a6cd2fc28"
       (reference "D601") (unit 1) (value "SS12") (footprint "Diode_SMD:D_SMA")
@@
       (reference "D1105") (unit 1) (value "WS2812B") (footprint "Footprints:WS2812-mini")
     )
+    (path "/4e78659c-21b0-4088-8876-cb944b9d811b/13ee671d-2cc5-4735-b962-c0e37fa159a1"
+      (reference "D1106") (unit 1) (value "WS2812B") (footprint "LED_SMD:LED_WS2812B_PLCC4_5.0x5.0mm_P3.2mm")
+    )
     (path "/ac94f7cf-c7fc-4258-a4c8-af0c3ef6d0a1/c89382c0-bfaa-4808-a62d-d55c9ebe819b"
       (reference "FB201") (unit 1) (value "100 @ 100MHz") (footprint "Resistor_SMD:R_0603_1608Metric")
@@
       (reference "R303") (unit 1) (value "10k") (footprint "Resistor_SMD:R_0603_1608Metric")
     )
-    (path "/137cdba1-cde3-4c49-b42e-e13f2be356c7/63394e3b-e071-444b-936e-6b25139d4705"
-      (reference "R304") (unit 1) (value "1k") (footprint "Resistor_SMD:R_0603_1608Metric")
-    )
     (path "/137cdba1-cde3-4c49-b42e-e13f2be356c7/b603c655-745d-46e2-84d9-900527e7abda"
       (reference "R305") (unit 1) (value "100k") (footprint "Resistor_SMD:R_0603_1608Metric")
     )
-    (path "/137cdba1-cde3-4c49-b42e-e13f2be356c7/55587f14-1876-4a57-bb3d-fab89b0180b1"
-      (reference "R306") (unit 1) (value "1k") (footprint "Resistor_SMD:R_0603_1608Metric")
-    )
     (path "/137cdba1-cde3-4c49-b42e-e13f2be356c7/6d4ac1f5-54e1-49e0-b033-11329cfbf538"
       (reference "R307") (unit 1) (value "10k") (footprint "Resistor_SMD:R_0603_1608Metric")
@@
       (reference "R308") (unit 1) (value "10k") (footprint "Resistor_SMD:R_0603_1608Metric")
     )
-    (path "/137cdba1-cde3-4c49-b42e-e13f2be356c7/890c2240-239b-4afc-b060-9b9ca9249f7e"
-      (reference "R309") (unit 1) (value "1k") (footprint "Resistor_SMD:R_0603_1608Metric")
-    )
     (path "/137cdba1-cde3-4c49-b42e-e13f2be356c7/867a8dd9-b8e5-4c0d-9bd1-b51e3ff30de4"
       (reference "R310") (unit 1) (value "10k") (footprint "Resistor_SMD:R_0603_1608Metric")
@@
       (reference "R1001") (unit 1) (value "470R") (footprint "Resistor_SMD:R_0603_1608Metric")
     )
+    (path "/4e78659c-21b0-4088-8876-cb944b9d811b/fb7af6d0-c990-4b39-947e-e8f317bebc38"
+      (reference "R1002") (unit 1) (value "470R") (footprint "Resistor_SMD:R_0603_1608Metric")
+    )
     (path "/4e78659c-21b0-4088-8876-cb944b9d811b/75567645-26bd-43be-84de-f40c2e8d6559"
       (reference "R1003") (unit 1) (value "470R") (footprint "Resistor_SMD:R_0603_1608Metric")
     )
+    (path "/4e78659c-21b0-4088-8876-cb944b9d811b/11fa5df4-71ef-4ed9-8359-d3be4a6f88a0"
+      (reference "R1004") (unit 1) (value "470R") (footprint "Resistor_SMD:R_0603_1608Metric")
+    )
     (path "/4e78659c-21b0-4088-8876-cb944b9d811b/528ae980-7cc9-46ef-8dd6-ee722a68e949"
       (reference "R1005") (unit 1) (value "470R") (footprint "Resistor_SMD:R_0603_1608Metric")
     )
-    (path "/4e78659c-21b0-4088-8876-cb944b9d811b/fb7af6d0-c990-4b39-947e-e8f317bebc38"
-      (reference "R1085") (unit 1) (value "470R") (footprint "Resistor_SMD:R_0603_1608Metric")
-    )
-    (path "/4e78659c-21b0-4088-8876-cb944b9d811b/11fa5df4-71ef-4ed9-8359-d3be4a6f88a0"
-      (reference "R1086") (unit 1) (value "470R") (footprint "Resistor_SMD:R_0603_1608Metric")
+    (path "/4e78659c-21b0-4088-8876-cb944b9d811b/73df696c-05b6-4362-9683-d99e38498926"
+      (reference "R1006") (unit 1) (value "470R") (footprint "Resistor_SMD:R_0603_1608Metric")
+    )
+    (path "/137cdba1-cde3-4c49-b42e-e13f2be356c7/3c7cc35d-1ba6-4995-8d5a-d8587075b085"
+      (reference "R1007") (unit 1) (value "10k") (footprint "Resistor_SMD:R_0603_1608Metric")
+    )
+    (path "/137cdba1-cde3-4c49-b42e-e13f2be356c7/0450dcae-979c-4792-b7af-708781e9955d"
+      (reference "R1008") (unit 1) (value "10k") (footprint "Resistor_SMD:R_0603_1608Metric")
+    )
+    (path "/137cdba1-cde3-4c49-b42e-e13f2be356c7/32a3e460-cc61-4ff6-b885-d8b5f02c18af"
+      (reference "R1009") (unit 1) (value "10k") (footprint "Resistor_SMD:R_0603_1608Metric")
     )
     (path "/4ee94e79-8f79-4d3c-86ca-8e64aae4ab70/065793fe-edb2-4416-bdf1-8457eba820c6"

Commit message: layout_v2
Other:
- note added: "TODO: - koristiti kompletnu englesku dokumentaciju - programski implementirati da je prilikom punjenja svjetlina minimalna - jedan neopixel koji je blizu punjača - power sklopka koja može prekinuti 1A - kockica touchpad - provjeriti shemu - isprintati na papir i provjeriti footprinte"
- note removed: "TODO: - koristiti kompletnu englesku dokumentaciju - jedan neopixel koji je blizu punjača - power sklopka koja može prekinuti 1A - kockica touchpad - provjeriti shemu - isprintati na papir i provjeriti footprinte"
Changed lines of the file:
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@@
     (rev "1")
   )
-  (text "TODO:\n- koristiti kompletnu englesku dokumentaciju\n- jedan neopixel koji je blizu punjača\n- power sklopka koja može prekinuti 1A\n- kockica touchpad\n- provjeriti shemu\n- isprintati na papir i provjeriti footprinte"
+  (text "TODO:\n- koristiti kompletnu englesku dokumentaciju\n- programski implementirati da je prilikom punjenja svjetlina minimalna\n- jedan neopixel koji je blizu punjača\n- power sklopka koja može prekinuti 1A\n- kockica touchpad\n- provjeriti shemu\n- isprintati na papir i provjeriti footprinte"
     (at 19.685 187.325 0)
     (effects (font (size 1.27 1.27)) (justify left bottom))
@@
       (reference "#FLG0501") (unit 1) (value "PWR_FLAG") (footprint "")
     )
-    (path "/4ee94e79-8f79-4d3c-86ca-8e64aae4ab70/731f02f6-903a-4cf3-b60f-6f47d27141ce"
-      (reference "#FLG0502") (unit 1) (value "PWR_FLAG") (footprint "")
-    )
     (path "/734b1c6c-4834-4550-ac92-289626629bb9"
       (reference "#PWR0101") (unit 1) (value "VCC") (footprint "")
@@
       (reference "#PWR0163") (unit 1) (value "GND") (footprint "")
     )
-    (path "/137cdba1-cde3-4c49-b42e-e13f2be356c7/6ef946b1-68a2-4826-b9df-2ec18dd67d90"
-      (reference "#PWR0164") (unit 1) (value "VBUS") (footprint "")
-    )
-    (path "/137cdba1-cde3-4c49-b42e-e13f2be356c7/4fea6a02-2d17-430a-8782-08f7d6a7a885"
-      (reference "#PWR0165") (unit 1) (value "VBUS") (footprint "")
-    )
-    (path "/137cdba1-cde3-4c49-b42e-e13f2be356c7/b562b1ed-5661-41bb-aeb1-1c7c7d6b3a6d"
-      (reference "#PWR0166") (unit 1) (value "VBUS") (footprint "")
-    )
     (path "/ac94f7cf-c7fc-4258-a4c8-af0c3ef6d0a1/5e2b5f85-9000-493f-92f5-49f06d324b8b"
       (reference "#PWR0201") (unit 1) (value "VBUS") (footprint "")
@@
       (reference "#PWR0418") (unit 1) (value "GND") (footprint "")
     )
-    (path "/4ee94e79-8f79-4d3c-86ca-8e64aae4ab70/7c76a589-34d4-48a7-8f04-dc1c3247db60"
-      (reference "#PWR0501") (unit 1) (value "+5V") (footprint "")
-    )
     (path "/4ee94e79-8f79-4d3c-86ca-8e64aae4ab70/7cdf4a90-e8f9-47b4-9c46-5698e4fd1fbd"
       (reference "#PWR0502") (unit 1) (value "+5V") (footprint "")
@@
       (reference "#PWR0503") (unit 1) (value "GND") (footprint "")
     )
-    (path "/4ee94e79-8f79-4d3c-86ca-8e64aae4ab70/b17b5ae4-6a2b-4bbc-b6b7-3906ec89603d"
-      (reference "#PWR0504") (unit 1) (value "GND") (footprint "")
-    )
-    (path "/4ee94e79-8f79-4d3c-86ca-8e64aae4ab70/2543f27f-3b77-4a14-91e7-209236762b3d"
-      (reference "#PWR0505") (unit 1) (value "+5V") (footprint "")
-    )
-    (path "/4ee94e79-8f79-4d3c-86ca-8e64aae4ab70/d34e4f88-372a-4f42-9a4b-8203abd01ad8"
-      (reference "#PWR0506") (unit 1) (value "GND") (footprint "")
-    )
     (path "/4ee94e79-8f79-4d3c-86ca-8e64aae4ab70/1e528d40-7b6a-4327-ad03-b9ae3d3ed2ee"
       (reference "#PWR0507") (unit 1) (value "GND") (footprint "")
@@
       (reference "C501") (unit 1) (value "100n") (footprint "Capacitor_SMD:C_0603_1608Metric")
     )
-    (path "/4ee94e79-8f79-4d3c-86ca-8e64aae4ab70/5f66fb1d-6d17-43b1-b749-59a9e3970708"
-      (reference "C502") (unit 1) (value "100n") (footprint "Capacitor_SMD:C_0603_1608Metric")
-    )
-    (path "/4ee94e79-8f79-4d3c-86ca-8e64aae4ab70/dc037b4f-66ef-40cf-9af8-05c771cafd36"
-      (reference "C503") (unit 1) (value "100n") (footprint "Capacitor_SMD:C_0603_1608Metric")
-    )
     (path "/4ee94e79-8f79-4d3c-86ca-8e64aae4ab70/b9ee4bd4-f0be-4530-8a68-973b7c28f1c5"
       (reference "C504") (unit 1) (value "1u") (footprint "Capacitor_SMD:C_0603_1608Metric")
@@
       (reference "J501") (unit 1) (value "USBasp") (footprint "Connector_PinHeader_1.27mm:PinHeader_2x03_P1.27mm_Vertical_SMD")
     )
-    (path "/4ee94e79-8f79-4d3c-86ca-8e64aae4ab70/d3f8e25f-4120-4ba2-9b66-04af3b9d8b2a"
-      (reference "L501") (unit 1) (value "10u") (footprint "Inductor_SMD:L_1206_3216Metric")
-    )
     (path "/bfec7ff5-12b5-4af9-9131-b19e09596ace/a3653020-1727-4f10-819a-83fb9d6b7edc"
       (reference "L601") (unit 1) (value "4R7") (footprint "Footprints:Inductor_4mm(5x5mm pads)")
@@
       (reference "R1006") (unit 1) (value "470R") (footprint "Resistor_SMD:R_0603_1608Metric")
     )
-    (path "/137cdba1-cde3-4c49-b42e-e13f2be356c7/3c7cc35d-1ba6-4995-8d5a-d8587075b085"
-      (reference "R1007") (unit 1) (value "10k") (footprint "Resistor_SMD:R_0603_1608Metric")
-    )
-    (path "/137cdba1-cde3-4c49-b42e-e13f2be356c7/0450dcae-979c-4792-b7af-708781e9955d"
-      (reference "R1008") (unit 1) (value "10k") (footprint "Resistor_SMD:R_0603_1608Metric")
-    )
-    (path "/137cdba1-cde3-4c49-b42e-e13f2be356c7/32a3e460-cc61-4ff6-b885-d8b5f02c18af"
-      (reference "R1009") (unit 1) (value "10k") (footprint "Resistor_SMD:R_0603_1608Metric")
-    )
     (path "/4ee94e79-8f79-4d3c-86ca-8e64aae4ab70/065793fe-edb2-4416-bdf1-8457eba820c6"

Commit message: update
Other:
- note added: "TODO: - koristiti kompletnu englesku dokumentaciju - programski implementirati da je prilikom punjenja svjetlina minimalna - power sklopka koja može prekinuti 1A - kockica touchpad - provjeriti shemu - isprintati na papir i provjeriti footprinte"
- note removed: "TODO: - koristiti kompletnu englesku dokumentaciju - programski implementirati da je prilikom punjenja svjetlina minimalna - jedan neopixel koji je blizu punjača - power sklopka koja može prekinuti 1A - kockica touchpad - provjeriti shemu - isprintati na papir i provjeriti footprinte"
Changed lines of the file:
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@@
     (rev "1")
   )
-  (text "TODO:\n- koristiti kompletnu englesku dokumentaciju\n- programski implementirati da je prilikom punjenja svjetlina minimalna\n- jedan neopixel koji je blizu punjača\n- power sklopka koja može prekinuti 1A\n- kockica touchpad\n- provjeriti shemu\n- isprintati na papir i provjeriti footprinte"
+  (text "TODO:\n- koristiti kompletnu englesku dokumentaciju\n- programski implementirati da je prilikom punjenja svjetlina minimalna\n- power sklopka koja može prekinuti 1A\n- kockica touchpad\n- provjeriti shemu\n- isprintati na papir i provjeriti footprinte"
     (at 19.685 187.325 0)
     (effects (font (size 1.27 1.27)) (justify left bottom))
@@
     )
     (path "/4e78659c-21b0-4088-8876-cb944b9d811b/13ee671d-2cc5-4735-b962-c0e37fa159a1"
-      (reference "D1106") (unit 1) (value "WS2812B") (footprint "Footprints:LED_WS2812B_edited")
+      (reference "D1106") (unit 1) (value "WS2812B") (footprint "Footprints:WS2812-mini")
     )
     (path "/ac94f7cf-c7fc-4258-a4c8-af0c3ef6d0a1/c89382c0-bfaa-4808-a62d-d55c9ebe819b"

Commit message: update
Other:
- note added: "TODO: - koristiti kompletnu englesku dokumentaciju - tunel za zvučnik - spojiti kockicu (dodati još jedan ulaz na io expander) - programski implementirati da je prilikom punjenja svjetlina minimalna - power sklopka koja može prekinuti 1A (rupa na kućištu) - provjeriti shemu - isprintati na papir i provjeriti footprinte"
- note removed: "TODO: - koristiti kompletnu englesku dokumentaciju - programski implementirati da je prilikom punjenja svjetlina minimalna - power sklopka koja može prekinuti 1A - kockica touchpad - provjeriti shemu - isprintati na papir i provjeriti footprinte"
Changed lines of the file:
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@@
     (rev "1")
   )
-  (text "TODO:\n- koristiti kompletnu englesku dokumentaciju\n- programski implementirati da je prilikom punjenja svjetlina minimalna\n- power sklopka koja može prekinuti 1A\n- kockica touchpad\n- provjeriti shemu\n- isprintati na papir i provjeriti footprinte"
+  (text "TODO:\n- koristiti kompletnu englesku dokumentaciju\n- tunel za zvučnik\n- spojiti kockicu (dodati još jedan ulaz na io expander)\n- programski implementirati da je prilikom punjenja svjetlina minimalna\n- power sklopka koja može prekinuti 1A (rupa na kućištu)\n- provjeriti shemu\n- isprintati na papir i provjeriti footprinte"
     (at 19.685 187.325 0)
     (effects (font (size 1.27 1.27)) (justify left bottom))

Commit message: update
Other:
- note added: "TODO: - koristiti kompletnu englesku dokumentaciju - tunel za zvučnik - spojiti kockicu (dodati još jedan ulaz na io expander) - programski implementirati da je prilikom punjenja svjetlina minimalna - power sklopka koja može prekinuti 2A (rupa na kućištu) - provjeriti dimenzije usb-c konektora kabela, da li je rupa na kućištu dovoljno velika - izmjenjiva 18650 baterija - provjeriti shemu - isprin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"
- note removed: "TODO: - koristiti kompletnu englesku dokumentaciju - tunel za zvučnik - spojiti kockicu (dodati još jedan ulaz na io expander) - programski implementirati da je prilikom punjenja svjetlina minimalna - power sklopka koja može prekinuti 1A (rupa na kućištu) - provjeriti shemu - isprintati na papir i provjeriti footprinte"
Changed lines of the file:
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@@
     (rev "1")
   )
-  (text "TODO:\n- koristiti kompletnu englesku dokumentaciju\n- tunel za zvučnik\n- spojiti kockicu (dodati još jedan ulaz na io expander)\n- programski implementirati da je prilikom punjenja svjetlina minimalna\n- power sklopka koja može prekinuti 1A (rupa na kućištu)\n- provjeriti shemu\n- isprintati na papir i provjeriti footprinte"
+  (text "TODO:\n- koristiti kompletnu englesku dokumentaciju\n- tunel za zvučnik\n- spojiti kockicu (dodati još jedan ulaz na io expander)\n- programski implementirati da je prilikom punjenja svjetlina minimalna\n- power sklopka koja može prekinuti 2A (rupa na kućištu)\n- provjeriti dimenzije usb-c konektora kabela, da li je rupa na kućištu dovoljno velika\n- izmjenjiva 18650 baterija\n- provjeriti shemu\n- isprintati na papir i provjeriti footprinte"
     (at 19.685 187.325 0)
     (effects (font (size 1.27 1.27)) (justify left bottom))
