File: KiCad files/BoardGame/Battery charger.kicad_sch (KiCad schematic)
At the start: 21 parts

Commit message: update
Parts:
- BT?: value (none) -> Battery_Cell
- C? (x3): value (none) -> 10u; footprint (none) -> Capacitor_SMD:C_0603_1608Metric
- C?: value (none) -> 10u; footprint (none) -> Capacitor_Tantalum_SMD:CP_EIA-3528-21_Kemet-B
- D? (x3): value (none) -> LED_Small; footprint (none) -> LED_SMD:LED_0603_1608Metric
- J? (x2): value (none) -> Conn_01x01
- R? (x5): value (none) -> 10k; footprint (none) -> Resistor_SMD:R_0603_1608Metric
- R? (x3): value (none) -> 1k; footprint (none) -> Resistor_SMD:R_0603_1608Metric
- R?: value (none) -> 100k; footprint (none) -> Resistor_SMD:R_0603_1608Metric
- R?: value (none) -> 2k; footprint (none) -> Resistor_SMD:R_0603_1608Metric
- U?: value (none) -> MCP73871-2CC; footprint (none) -> Package_DFN_QFN:QFN-20-1EP_4x4mm_P0.5mm_EP2.5x2.5mm

Commit message: update
Parts:
- BT1: renamed from BT?; footprint (none) -> Footprints:battery_906909_6000mah
- J2, J3: renamed from J?; footprint (none) -> Footprints:PinHeader_1x01
- gave numbers to parts that had none: 18

Commit message: update
Parts:
- renumbered BT1 to BT301, C5 to C301, C6 to C302, C7 to C303, C8 to C304, D1 to D301, D2 to D302, D3 to D303, J2 to J301, J3 to J302, R5 to R301, R6 to R302, R7 to R303, R8 to R304, R9 to R305, R10 to R306, R11 to R307, R12 to R308, R13 to R309, R14 to R310, U3 to U301

Commit message: update
Parts:
- BT301: JLCPCB Part # (none) -> -; Ostalo (none) -> 1005003744354475; U labosu? (none) -> ne
- C301: JLCPCB Part # (none) -> C2798040; U labosu? (none) -> ne
- C302, C303, C304: footprint Capacitor_SMD:C_0603_1608Metric -> Capacitor_SMD:C_0805_2012Metric; JLCPCB Part # (none) -> C237493; U labosu? (none) -> ne
- D301, D302, D303: JLCPCB Part # (none) -> -; U labosu? (none) -> da
- J301, J302: JLCPCB Part # (none) -> -; Ostalo (none) -> -; U labosu? (none) -> da
- R301, R303, R304, R305, R306, R307, R308, R309, R310, U301: U labosu? (none) -> da
- R302: JLCPCB Part # (none) -> C25590; U labosu? (none) -> ne
Other:
- moved on the sheet: R301
Changed lines of the file:
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@@
-    (stroke (width 0) (type default) (color 0 0 0 0))
-  )
-  (wire (pts (xy 60.96 69.215) (xy 117.475 69.215))
     (stroke (width 0) (type default) (color 0 0 0 0))
   )
@@
     (stroke (width 0) (type default) (color 0 0 0 0))
   )
-  (wire (pts (xy 60.96 76.835) (xy 60.96 78.74))
+  (wire (pts (xy 58.42 76.835) (xy 58.42 78.74))
     (stroke (width 0) (type default) (color 0 0 0 0))
   )
@@
     (stroke (width 0) (type default) (color 0 0 0 0))
   )
-  (wire (pts (xy 60.96 78.74) (xy 64.135 78.74))
+  (wire (pts (xy 58.42 78.74) (xy 64.135 78.74))
     (stroke (width 0) (type default) (color 0 0 0 0))
   )
@@
     (stroke (width 0) (type default) (color 0 0 0 0))
   )
-  (wire (pts (xy 60.96 69.215) (xy 60.96 71.755))
+  (wire (pts (xy 58.42 69.215) (xy 58.42 71.755))
     (stroke (width 0) (type default) (color 0 0 0 0))
   )
@@
   )
   (wire (pts (xy 156.21 94.615) (xy 166.37 94.615))
+    (stroke (width 0) (type default) (color 0 0 0 0))
+  )
+  (wire (pts (xy 58.42 69.215) (xy 117.475 69.215))
     (stroke (width 0) (type default) (color 0 0 0 0))
   )
@@
       (effects (font (size 1.27 1.27)) (justify left))
     )
-    (property "Footprint" "Capacitor_SMD:C_0603_1608Metric" (id 2) (at 93.98 57.785 0)
+    (property "Footprint" "Capacitor_SMD:C_0805_2012Metric" (id 2) (at 93.98 57.785 0)
       (effects (font (size 1.27 1.27)) hide)
     )
     (property "Datasheet" "~" (id 3) (at 93.98 57.785 0)
+      (effects (font (size 1.27 1.27)) hide)
+    )
+    (property "JLCPCB Part #" "C237493" (id 4) (at 93.98 57.785 0)
+      (effects (font (size 1.27 1.27)) hide)
+    )
+    (property "U labosu?" "ne" (id 5) (at 93.98 57.785 0)
       (effects (font (size 1.27 1.27)) hide)
     )
@@
       (effects (font (size 1.27 1.27)) hide)
     )
+    (property "JLCPCB Part #" "-" (id 4) (at 180.34 59.055 0)
+      (effects (font (size 1.27 1.27)) hide)
+    )
+    (property "Ostalo" "-" (id 5) (at 180.34 59.055 0)
+      (effects (font (size 1.27 1.27)) hide)
+    )
+    (property "U labosu?" "da" (id 6) (at 180.34 59.055 0)
+      (effects (font (size 1.27 1.27)) hide)
+    )
     (pin "1")
   )
@@
       (effects (font (size 1.27 1.27)) hide)
     )
-    (pin "1")
-    (pin "2")
-  )
-  (symbol (lib_id "Device:R_Small") (at 60.96 74.295 0) (unit 1)
-    (in_bom yes) (on_board yes)
-    (property "Reference" "R301" (id 0) (at 63.5 73.025 0))
-    (property "Value" "10k" (id 1) (at 63.5 74.93 0))
-    (property "Footprint" "Resistor_SMD:R_0603_1608Metric" (id 2) (at 60.96 74.295 0)
-      (effects (font (size 1.27 1.27)) hide)
-    )
-    (property "Datasheet" "~" (id 3) (at 60.96 74.295 0)
+    (property "JLCPCB Part #" "C2798040" (id 4) (at 76.835 57.785 0)
+      (effects (font (size 1.27 1.27)) hide)
+    )
+    (property "U labosu?" "ne" (id 5) (at 76.835 57.785 0)
+      (effects (font (size 1.27 1.27)) hide)
+    )
+    (pin "1")
+    (pin "2")
+  )
+  (symbol (lib_id "Device:R_Small") (at 58.42 74.295 0) (unit 1)
+    (in_bom yes) (on_board yes)
+    (property "Reference" "R301" (id 0) (at 62.23 73.025 0))
+    (property "Value" "10k" (id 1) (at 61.595 74.93 0))
+    (property "Footprint" "Resistor_SMD:R_0603_1608Metric" (id 2) (at 58.42 74.295 0)
+      (effects (font (size 1.27 1.27)) hide)
+    )
+    (property "Datasheet" "~" (id 3) (at 58.42 74.295 0)
+      (effects (font (size 1.27 1.27)) hide)
+    )
+    (property "U labosu?" "da" (id 4) (at 58.42 74.295 0)
       (effects (font (size 1.27 1.27)) hide)
     )
@@
       (effects (font (size 1.27 1.27)) (justify left))
     )
-    (property "Footprint" "Capacitor_SMD:C_0603_1608Metric" (id 2) (at 165.735 65.405 0)
+    (property "Footprint" "Capacitor_SMD:C_0805_2012Metric" (id 2) (at 165.735 65.405 0)
       (effects (font (size 1.27 1.27)) hide)
     )
     (property "Datasheet" "~" (id 3) (at 165.735 65.405 0)
+      (effects (font (size 1.27 1.27)) hide)
+    )
+    (property "JLCPCB Part #" "C237493" (id 4) (at 165.735 65.405 0)
+      (effects (font (size 1.27 1.27)) hide)
+    )
+    (property "U labosu?" "ne" (id 5) (at 165.735 65.405 0)
       (effects (font (size 1.27 1.27)) hide)
     )
@@
       (effects (font (size 1.27 1.27)) hide)
     )
+    (property "U labosu?" "da" (id 4) (at 109.855 95.885 0)
+      (effects (font (size 1.27 1.27)) hide)
+    )
     (pin "1")
     (pin "2")
@@
       (effects (font (size 1.27 1.27)) hide)
     )
+    (property "U labosu?" "da" (id 4) (at 178.435 92.71 0)
+      (effects (font (size 1.27 1.27)) hide)
+    )
     (pin "1")
     (pin "2")
@@
       (effects (font (size 1.27 1.27)) (justify left))
     )
-    (property "Footprint" "Capacitor_SMD:C_0603_1608Metric" (id 2) (at 165.735 78.105 0)
+    (property "Footprint" "Capacitor_SMD:C_0805_2012Metric" (id 2) (at 165.735 78.105 0)
       (effects (font (size 1.27 1.27)) hide)
     )
     (property "Datasheet" "~" (id 3) (at 165.735 78.105 0)
+      (effects (font (size 1.27 1.27)) hide)
+    )
+    (property "JLCPCB Part #" "C237493" (id 4) (at 165.735 78.105 0)
+      (effects (font (size 1.27 1.27)) hide)
+    )
+    (property "U labosu?" "ne" (id 5) (at 165.735 78.105 0)
       (effects (font (size 1.27 1.27)) hide)
     )
@@
       (effects (font (size 1.27 1.27)) hide)
     )
+    (property "U labosu?" "da" (id 4) (at 178.435 86.995 0)
+      (effects (font (size 1.27 1.27)) hide)
+    )
     (pin "1")
     (pin "2")
@@
       (effects (font (size 1.27 1.27)) hide)
     )
+    (property "U labosu?" "da" (id 4) (at 100.965 95.885 0)
+      (effects (font (size 1.27 1.27)) hide)
+    )
     (pin "1")
     (pin "2")
@@
     )
     (property "Datasheet" "~" (id 3) (at 187.96 92.71 90)
+      (effects (font (size 1.27 1.27)) hide)
+    )
+    (property "U labosu?" "da" (id 4) (at 187.96 92.71 0)
+      (effects (font (size 1.27 1.27)) hide)
+    )
+    (property "JLCPCB Part #" "-" (id 5) (at 187.96 92.71 0)
       (effects (font (size 1.27 1.27)) hide)
     )
@@
       (effects (font (size 1.27 1.27)) hide)
     )
+    (property "U labosu?" "da" (id 4) (at 83.185 110.49 0)
+      (effects (font (size 1.27 1.27)) hide)
+    )
     (pin "1")
     (pin "2")
@@
       (effects (font (size 1.27 1.27)) hide)
     )
+    (property "U labosu?" "da" (id 4) (at 178.435 98.425 0)
+      (effects (font (size 1.27 1.27)) hide)
+    )
     (pin "1")
     (pin "2")
@@
     )
     (property "Datasheet" "~" (id 3) (at 187.96 98.425 90)
+      (effects (font (size 1.27 1.27)) hide)
+    )
+    (property "U labosu?" "da" (id 4) (at 187.96 98.425 0)
+      (effects (font (size 1.27 1.27)) hide)
+    )
+    (property "JLCPCB Part #" "-" (id 5) (at 187.96 98.425 0)
       (effects (font (size 1.27 1.27)) hide)
     )
@@
       (effects (font (size 1.27 1.27)) hide)
     )
+    (property "U labosu?" "da" (id 4) (at 83.185 79.375 0)
+      (effects (font (size 1.27 1.27)) hide)
+    )
     (pin "1")
     (pin "2")
@@
   (symbol (lib_id "Device:R_Small") (at 87.63 91.44 0) (unit 1)
     (in_bom yes) (on_board yes)
-    (property "Reference" "R305" (id 0) (at 90.17 90.17 0))
+    (property "Reference" "R305" (id 0) (at 91.44 90.17 0))
     (property "Value" "100k" (id 1) (at 91.44 92.075 0))
     (property "Footprint" "Resistor_SMD:R_0603_1608Metric" (id 2) (at 87.63 91.44 0)
@@
     )
     (property "Datasheet" "~" (id 3) (at 87.63 91.44 0)
+      (effects (font (size 1.27 1.27)) hide)
+    )
+    (property "U labosu?" "da" (id 4) (at 87.63 91.44 0)
       (effects (font (size 1.27 1.27)) hide)
     )
@@
       (effects (font (size 1.27 1.27)) hide)
     )
+    (property "JLCPCB Part #" "-" (id 4) (at 180.34 61.595 0)
+      (effects (font (size 1.27 1.27)) hide)
+    )
+    (property "Ostalo" "-" (id 5) (at 180.34 61.595 0)
+      (effects (font (size 1.27 1.27)) hide)
+    )
+    (property "U labosu?" "da" (id 6) (at 180.34 61.595 0)
+      (effects (font (size 1.27 1.27)) hide)
+    )
     (pin "1")
   )
@@
     )
     (property "Datasheet" "http://www.mouser.com/ds/2/268/22090a-52174.pdf" (id 3) (at 134.62 67.945 0)
+      (effects (font (size 1.27 1.27)) hide)
+    )
+    (property "U labosu?" "da" (id 4) (at 138.43 81.915 0)
       (effects (font (size 1.27 1.27)) hide)
     )
@@
   (symbol (lib_id "Device:R_Small") (at 67.31 74.295 0) (unit 1)
     (in_bom yes) (on_board yes)
-    (property "Reference" "R302" (id 0) (at 69.85 73.025 0))
+    (property "Reference" "R302" (id 0) (at 71.12 73.025 0))
     (property "Value" "2k" (id 1) (at 69.85 74.93 0))
     (property "Footprint" "Resistor_SMD:R_0603_1608Metric" (id 2) (at 67.31 74.295 0)
@@
       (effects (font (size 1.27 1.27)) hide)
     )
+    (property "JLCPCB Part #" "C25590" (id 4) (at 67.31 74.295 0)
+      (effects (font (size 1.27 1.27)) hide)
+    )
+    (property "U labosu?" "ne" (id 5) (at 67.31 74.295 0)
+      (effects (font (size 1.27 1.27)) hide)
+    )
     (pin "1")
     (pin "2")
@@
       (effects (font (size 1.27 1.27)) hide)
     )
+    (property "U labosu?" "ne" (id 4) (at 201.93 81.28 0)
+      (effects (font (size 1.27 1.27)) hide)
+    )
+    (property "Aliexpress" "" (id 5) (at 201.93 81.28 0)
+      (effects (font (size 1.27 1.27)) hide)
+    )
+    (property "JLCPCB Part #" "-" (id 6) (at 201.93 81.28 0)
+      (effects (font (size 1.27 1.27)) hide)
+    )
+    (property "Ostalo" "1005003744354475" (id 7) (at 201.93 81.28 0)
+      (effects (font (size 1.27 1.27)) hide)
+    )
     (pin "1")
     (pin "2")
@@
       (effects (font (size 1.27 1.27)) hide)
     )
+    (property "U labosu?" "da" (id 4) (at 187.96 86.995 0)
+      (effects (font (size 1.27 1.27)) hide)
+    )
+    (property "JLCPCB Part #" "-" (id 5) (at 187.96 86.995 0)
+      (effects (font (size 1.27 1.27)) hide)
+    )

Commit message: update
Parts:
- BT301: footprint Footprints:battery_906909_6000mah -> Footprints:battery_103565_3000mah
Changed lines of the file:
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@@
       (effects (font (size 1.27 1.27)) (justify left))
     )
-    (property "Footprint" "Footprints:battery_906909_6000mah" (id 2) (at 201.93 79.756 90)
+    (property "Footprint" "Footprints:battery_103565_3000mah" (id 2) (at 201.93 79.756 90)
       (effects (font (size 1.27 1.27)) hide)
     )

Commit message: update
Parts:
- removed D301, D302, D303: LED_Small, LED_SMD:LED_0603_1608Metric, symbol Device:LED_Small
- removed R304, R306, R309: 1k, Resistor_SMD:R_0603_1608Metric, symbol Device:R_Small
- added R1007, R1008, R1009: 10k, Resistor_SMD:R_0603_1608Metric, symbol Device:R_Small
Connections:
- net VBUS: now also R1007.1, R1008.1, R1009.1
- net STAT1: now reaches U301.8 (STAT1/~{LBO})
- net STAT1: now also R1008.2
- net PG: now reaches U301.6 (~{PG})
- net PG: now also R1007.2
- net STAT2: now reaches U301.7 (STAT2)
- net STAT2: now also R1009.2
Other:
- note removed: "CHARGE"
- note removed: "DONE"
- note removed: "POWER"

Commit message: layout_v2
Parts:
- removed R1007, R1008, R1009: 10k, Resistor_SMD:R_0603_1608Metric, symbol Device:R_Small
Changed lines of the file:
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@@
     (effects (font (size 1.27 1.27)) (justify left bottom))
-  )
-  (global_label "PG" (shape input) (at 236.855 107.95 270) (fields_autoplaced)
-    (effects (font (size 1.27 1.27)) (justify right))
-    (property "Intersheet References" "${INTERSHEET_REFS}" (id 0) (at 236.9344 112.9031 90)
-      (effects (font (size 1.27 1.27)) (justify right) hide)
-    )
-  )
-  (global_label "STAT1" (shape input) (at 245.745 107.95 270) (fields_autoplaced)
-    (effects (font (size 1.27 1.27)) (justify right))
-    (property "Intersheet References" "${INTERSHEET_REFS}" (id 0) (at 245.8244 115.806 90)
-      (effects (font (size 1.27 1.27)) (justify right) hide)
-    )
   )
   (global_label "PG" (shape input) (at 156.21 86.995 0) (fields_autoplaced)
@@
     )
   )
-  (global_label "STAT2" (shape input) (at 255.27 107.95 270) (fields_autoplaced)
-    (effects (font (size 1.27 1.27)) (justify right))
-    (property "Intersheet References" "${INTERSHEET_REFS}" (id 0) (at 255.3494 115.806 90)
-      (effects (font (size 1.27 1.27)) (justify right) hide)
-    )
-  )
-  (symbol (lib_id "Device:R_Small") (at 245.745 105.41 0) (unit 1)
-    (in_bom yes) (on_board yes)
-    (property "Reference" "R1008" (id 0) (at 250.19 104.14 0))
-    (property "Value" "10k" (id 1) (at 248.92 106.045 0))
-    (property "Footprint" "Resistor_SMD:R_0603_1608Metric" (id 2) (at 245.745 105.41 0)
-      (effects (font (size 1.27 1.27)) hide)
-    )
-    (property "Datasheet" "~" (id 3) (at 245.745 105.41 0)
-      (effects (font (size 1.27 1.27)) hide)
-    )
-    (property "U labosu?" "da" (id 4) (at 245.745 105.41 0)
-      (effects (font (size 1.27 1.27)) hide)
-    )
-    (pin "1")
-    (pin "2")
-  )
   (symbol (lib_id "power:GND") (at 76.835 62.865 0) (unit 1)
     (in_bom yes) (on_board yes)
@@
     (pin "2")
   )
-  (symbol (lib_id "Device:R_Small") (at 255.27 105.41 0) (unit 1)
-    (in_bom yes) (on_board yes)
-    (property "Reference" "R1009" (id 0) (at 259.715 104.14 0))
-    (property "Value" "10k" (id 1) (at 258.445 106.045 0))
-    (property "Footprint" "Resistor_SMD:R_0603_1608Metric" (id 2) (at 255.27 105.41 0)
-      (effects (font (size 1.27 1.27)) hide)
-    )
-    (property "Datasheet" "~" (id 3) (at 255.27 105.41 0)
-      (effects (font (size 1.27 1.27)) hide)
-    )
-    (property "U labosu?" "da" (id 4) (at 255.27 105.41 0)
-      (effects (font (size 1.27 1.27)) hide)
-    )
-    (pin "1")
-    (pin "2")
-  )
-  (symbol (lib_id "Device:R_Small") (at 236.855 105.41 0) (unit 1)
-    (in_bom yes) (on_board yes)
-    (property "Reference" "R1007" (id 0) (at 241.3 104.14 0))
-    (property "Value" "10k" (id 1) (at 240.03 106.045 0))
-    (property "Footprint" "Resistor_SMD:R_0603_1608Metric" (id 2) (at 236.855 105.41 0)
-      (effects (font (size 1.27 1.27)) hide)
-    )
-    (property "Datasheet" "~" (id 3) (at 236.855 105.41 0)
-      (effects (font (size 1.27 1.27)) hide)
-    )
-    (property "U labosu?" "da" (id 4) (at 236.855 105.41 0)
-      (effects (font (size 1.27 1.27)) hide)
-    )
-    (pin "1")
-    (pin "2")
-  )
   (symbol (lib_id "Device:R_Small") (at 109.855 95.885 0) (unit 1)
     (in_bom yes) (on_board yes)
-    (property "Reference" "R308" (id 0) (at 112.395 94.615 0))
+    (property "Reference" "R308" (id 0) (at 113.665 94.615 0))
     (property "Value" "10k" (id 1) (at 113.03 96.52 0))
     (property "Footprint" "Resistor_SMD:R_0603_1608Metric" (id 2) (at 109.855 95.885 0)
@@
     (pin "1")
   )
-  (symbol (lib_id "power:VBUS") (at 236.855 102.87 0) (unit 1)
-    (in_bom yes) (on_board yes)
-    (property "Reference" "#PWR0165" (id 0) (at 236.855 106.68 0)
-      (effects (font (size 1.27 1.27)) hide)
-    )
-    (property "Value" "VBUS" (id 1) (at 237.236 98.4758 0))
-    (property "Footprint" "" (id 2) (at 236.855 102.87 0)
-      (effects (font (size 1.27 1.27)) hide)
-    )
-    (property "Datasheet" "" (id 3) (at 236.855 102.87 0)
-      (effects (font (size 1.27 1.27)) hide)
-    )
-    (pin "1")
-  )
   (symbol (lib_id "Device:C_Small") (at 165.735 78.105 0) (unit 1)
     (in_bom yes) (on_board yes)
@@
   (symbol (lib_id "Device:R_Small") (at 100.965 95.885 0) (unit 1)
     (in_bom yes) (on_board yes)
-    (property "Reference" "R307" (id 0) (at 103.505 94.615 0))
+    (property "Reference" "R307" (id 0) (at 104.775 94.615 0))
     (property "Value" "10k" (id 1) (at 104.14 96.52 0))
     (property "Footprint" "Resistor_SMD:R_0603_1608Metric" (id 2) (at 100.965 95.885 0)
@@
     (pin "1")
     (pin "2")
-  )
-  (symbol (lib_id "power:VBUS") (at 245.745 102.87 0) (unit 1)
-    (in_bom yes) (on_board yes)
-    (property "Reference" "#PWR0164" (id 0) (at 245.745 106.68 0)
-      (effects (font (size 1.27 1.27)) hide)
-    )
-    (property "Value" "VBUS" (id 1) (at 246.126 98.4758 0))
-    (property "Footprint" "" (id 2) (at 245.745 102.87 0)
-      (effects (font (size 1.27 1.27)) hide)
-    )
-    (property "Datasheet" "" (id 3) (at 245.745 102.87 0)
-      (effects (font (size 1.27 1.27)) hide)
-    )
-    (pin "1")
   )
   (symbol (lib_id "power:GND") (at 93.98 62.865 0) (unit 1)
@@
     (pin "2")
   )
-  (symbol (lib_id "power:VBUS") (at 255.27 102.87 0) (unit 1)
-    (in_bom yes) (on_board yes)
-    (property "Reference" "#PWR0166" (id 0) (at 255.27 106.68 0)
-      (effects (font (size 1.27 1.27)) hide)
-    )
-    (property "Value" "VBUS" (id 1) (at 255.651 98.4758 0))
-    (property "Footprint" "" (id 2) (at 255.27 102.87 0)
-      (effects (font (size 1.27 1.27)) hide)
-    )
-    (property "Datasheet" "" (id 3) (at 255.27 102.87 0)
-      (effects (font (size 1.27 1.27)) hide)
-    )
-    (pin "1")
-  )
   (symbol (lib_id "Device:R_Small") (at 87.63 91.44 0) (unit 1)
