File: KiCad files/BoardGame/Battery charger.kicad_sch (KiCad schematic)
At the start: 15 parts, among them J301 Conn_01x01, J302 Conn_01x01, U301 MCP73871-2CC

Commit message: update
Other:
- note added: "POWER SKLOPKA"
- note removed: "PADOVI SKLOPKE"
Changed lines of the file:
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@@
     (effects (font (size 0.9906 0.9906)) (justify left bottom))
   )
-  (text "PADOVI\nSKLOPKE" (at 175.26 55.245 0)
+  (text "POWER\nSKLOPKA" (at 175.26 55.245 0)
     (effects (font (size 1.27 1.27)) (justify left bottom))
   )

Commit message: Documentation
Other:
- note added: "POWER SWITCH"
- note removed: "POWER SKLOPKA"
Changed lines of the file:
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@@
     (effects (font (size 0.9906 0.9906)) (justify left bottom))
   )
-  (text "POWER\nSKLOPKA" (at 175.26 55.245 0)
+  (text "POWER\nSWITCH" (at 175.26 55.245 0)
     (effects (font (size 1.27 1.27)) (justify left bottom))
   )

Commit message: Schematic update
Changed lines of the file:
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@@
     (effects (font (size 1.27 1.27)) (justify left bottom))
   )
-  (global_label "PG" (shape input) (at 156.21 86.995 0) (fields_autoplaced)
+  (hierarchical_label "STAT2" (shape output) (at 156.21 94.615 0)
     (effects (font (size 1.27 1.27)) (justify left))
-    (property "Intersheet References" "${INTERSHEET_REFS}" (id 0) (at 161.1631 86.9156 0)
-      (effects (font (size 1.27 1.27)) (justify left) hide)
-    )
   )
-  (global_label "STAT1" (shape input) (at 156.21 92.075 0) (fields_autoplaced)
+  (hierarchical_label "PG" (shape output) (at 156.21 86.995 0)
     (effects (font (size 1.27 1.27)) (justify left))
-    (property "Intersheet References" "${INTERSHEET_REFS}" (id 0) (at 164.066 91.9956 0)
-      (effects (font (size 1.27 1.27)) (justify left) hide)
-    )
   )
-  (global_label "STAT2" (shape input) (at 156.21 94.615 0) (fields_autoplaced)
+  (hierarchical_label "STAT1" (shape output) (at 156.21 92.075 0)
     (effects (font (size 1.27 1.27)) (justify left))
-    (property "Intersheet References" "${INTERSHEET_REFS}" (id 0) (at 164.066 94.5356 0)
-      (effects (font (size 1.27 1.27)) (justify left) hide)
-    )
   )
   (symbol (lib_id "power:GND") (at 76.835 62.865 0) (unit 1)

Commit message: update
Parts:
- C301: value 10u -> 4u7/25V
Changed lines of the file:
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@@
       (effects (font (size 1.27 1.27)) (justify left))
     )
-    (property "Value" "10u" (id 1) (at 78.994 58.9411 0)
+    (property "Value" "4u7/25V" (id 1) (at 78.994 58.9411 0)
       (effects (font (size 1.27 1.27)) (justify left))
     )
