File: KiCad files/BoardGame/BoardGame.kicad_pcb (KiCad board)
At the start: 2 copper layers, 116 parts, among them J201 USB_C_Receptacle_USB2.0, J301 Conn_01x01, J302 Conn_01x01, J401 Conn_02x03_Odd_Even, J402 Conn_02x03_Odd_Even, J403 Conn_02x03_Odd_Even, J404 Conn_02x03_Odd_Even, J501 USBasp, SW501 SW_Push, U201 USBLC6-2SC6, U202 CH340C, U301 MCP73871-2CC, U401 PCF8575, U501 ATmega328P-A, U601 MT3608, Y501 16MHz

Commit message: Update BoardGame.kicad_pcb
Parts:
- moved BT301 3.04 mm to (345.5, 58.0)
Changed lines of the file:
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@@
   )
   (footprint "Footprints:battery_906909_6000mah" (layer "F.Cu")
-    (at 346 61)
+    (at 345.5335 58)
     (property "Sheetfile" "Battery charger.kicad_sch")
     (property "Sheetname" "Battery charger")

Commit message: Update BoardGame.kicad_pcb
Parts:
- moved BT301 3.93 mm to (343.0, 55.0)
Changed lines of the file:
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@@
   )
   (footprint "Footprints:battery_906909_6000mah" (layer "F.Cu")
-    (at 345.5335 58)
+    (at 343 55)
     (property "Sheetfile" "Battery charger.kicad_sch")
     (property "Sheetname" "Battery charger")

Commit message: update
Parts:
- removed D701, D702, D703, D704, D705, D706, D707, D708, D709, D710, D711, D712, D713, D714, D715, D716, D717, D718, D719, D720, D721, D722, D723, D724, D725, D726, D727, D728, D729, D730, D731, D732, D733, D734, D735, D736, D737, D738, D739, D740, D741, D742, D743, D744, D745, D746, D747, D748, D749, D750, D751, D752: WS2812B, LED_SMD:LED_WS2812B_PLCC4_5.0x5.0mm_P3.2mm
- removed R701, R702, R703, R704, R705: 470R, Resistor_SMD:R_0603_1608Metric
- added C1001: 100n, Capacitor_SMD:C_0603_1608Metric, B.Cu at (148.0, 87.0)
- added C1002: 100n, Capacitor_SMD:C_0603_1608Metric, B.Cu at (140.0, 89.5)
- added C1003: 100n, Capacitor_SMD:C_0603_1608Metric, B.Cu at (144.0, 87.0)
- added C1004: 100n, Capacitor_SMD:C_0603_1608Metric, B.Cu at (148.0, 89.5)
- added C1005: 100n, Capacitor_SMD:C_0603_1608Metric, B.Cu at (144.0, 89.5)
- added C1006: 100n, Capacitor_SMD:C_0603_1608Metric, B.Cu at (140.0, 87.0)
- added C1007: 100n, Capacitor_SMD:C_0603_1608Metric, B.Cu at (144.0, 84.5)
- added C1008: 100n, Capacitor_SMD:C_0603_1608Metric, B.Cu at (148.0, 84.5)
- added C1009: 100n, Capacitor_SMD:C_0603_1608Metric, B.Cu at (140.0, 84.5)
- added D1001: WS2812B, LED_SMD:LED_WS2812B_PLCC4_5.0x5.0mm_P3.2mm, F.Cu at (125.4, 87.0)
- added D1002: WS2812B, LED_SMD:LED_WS2812B_PLCC4_5.0x5.0mm_P3.2mm, F.Cu at (114.6, 81.3)
- added D1003: WS2812B, LED_SMD:LED_WS2812B_PLCC4_5.0x5.0mm_P3.2mm, F.Cu at (102.9, 73.7)
- added D1004: WS2812B, LED_SMD:LED_WS2812B_PLCC4_5.0x5.0mm_P3.2mm, F.Cu at (91.9, 64.2)
- added D1005: WS2812B, LED_SMD:LED_WS2812B_PLCC4_5.0x5.0mm_P3.2mm, F.Cu at (83.4, 53.1)
- added D1006: WS2812B, LED_SMD:LED_WS2812B_PLCC4_5.0x5.0mm_P3.2mm, F.Cu at (79.0, 41.4)
- added D1007: WS2812B, LED_SMD:LED_WS2812B_PLCC4_5.0x5.0mm_P3.2mm, F.Cu at (80.1, 30.6)
- added D1008: WS2812B, LED_SMD:LED_WS2812B_PLCC4_5.0x5.0mm_P3.2mm, F.Cu at (87.7, 23.1)
- added D1009: WS2812B, LED_SMD:LED_WS2812B_PLCC4_5.0x5.0mm_P3.2mm, F.Cu at (98.5, 22.0)
- added D1010: WS2812B, LED_SMD:LED_WS2812B_PLCC4_5.0x5.0mm_P3.2mm, F.Cu at (110.2, 26.4)
- added D1011: WS2812B, LED_SMD:LED_WS2812B_PLCC4_5.0x5.0mm_P3.2mm, F.Cu at (121.3, 35.0)
- added D1012: WS2812B, LED_SMD:LED_WS2812B_PLCC4_5.0x5.0mm_P3.2mm, F.Cu at (130.8, 46.0)
- added D1013: WS2812B, LED_SMD:LED_WS2812B_PLCC4_5.0x5.0mm_P3.2mm, F.Cu at (138.4, 57.8)
- added D1014: WS2812B, LED_SMD:LED_WS2812B_PLCC4_5.0x5.0mm_P3.2mm, F.Cu at (144.0, 68.4)
- added D1015: WS2812B, LED_SMD:LED_WS2812B_PLCC4_5.0x5.0mm_P3.2mm, F.Cu at (149.7, 57.6)
- added D1016: WS2812B, LED_SMD:LED_WS2812B_PLCC4_5.0x5.0mm_P3.2mm, F.Cu at (157.3, 45.9)
- added D1017: WS2812B, LED_SMD:LED_WS2812B_PLCC4_5.0x5.0mm_P3.2mm, F.Cu at (166.8, 34.9)
- added D1018: WS2812B, LED_SMD:LED_WS2812B_PLCC4_5.0x5.0mm_P3.2mm, F.Cu at (177.9, 26.4)
- added D1019: WS2812B, LED_SMD:LED_WS2812B_PLCC4_5.0x5.0mm_P3.2mm, F.Cu at (189.6, 22.0)
- added D1020: WS2812B, LED_SMD:LED_WS2812B_PLCC4_5.0x5.0mm_P3.2mm, F.Cu at (200.4, 23.1)
- added D1021: WS2812B, LED_SMD:LED_WS2812B_PLCC4_5.0x5.0mm_P3.2mm, F.Cu at (207.9, 30.7)
- added D1022: WS2812B, LED_SMD:LED_WS2812B_PLCC4_5.0x5.0mm_P3.2mm, F.Cu at (209.0, 41.5)
- added D1023: WS2812B, LED_SMD:LED_WS2812B_PLCC4_5.0x5.0mm_P3.2mm, F.Cu at (204.6, 53.2)
- added D1024: WS2812B, LED_SMD:LED_WS2812B_PLCC4_5.0x5.0mm_P3.2mm, F.Cu at (196.0, 64.3)
- added D1025: WS2812B, LED_SMD:LED_WS2812B_PLCC4_5.0x5.0mm_P3.2mm, F.Cu at (185.0, 73.8)
- added D1026: WS2812B, LED_SMD:LED_WS2812B_PLCC4_5.0x5.0mm_P3.2mm, F.Cu at (173.2, 81.4)
- added D1027: WS2812B, LED_SMD:LED_WS2812B_PLCC4_5.0x5.0mm_P3.2mm, F.Cu at (162.6, 87.0)
- added D1028: WS2812B, LED_SMD:LED_WS2812B_PLCC4_5.0x5.0mm_P3.2mm, F.Cu at (173.4, 92.7)
- added D1029: WS2812B, LED_SMD:LED_WS2812B_PLCC4_5.0x5.0mm_P3.2mm, F.Cu at (185.1, 100.3)
- added D1030: WS2812B, LED_SMD:LED_WS2812B_PLCC4_5.0x5.0mm_P3.2mm, F.Cu at (196.1, 109.8)
- added D1031: WS2812B, LED_SMD:LED_WS2812B_PLCC4_5.0x5.0mm_P3.2mm, F.Cu at (204.6, 120.9)
- added D1032: WS2812B, LED_SMD:LED_WS2812B_PLCC4_5.0x5.0mm_P3.2mm, F.Cu at (209.0, 132.6)
- added D1033: WS2812B, LED_SMD:LED_WS2812B_PLCC4_5.0x5.0mm_P3.2mm, F.Cu at (207.9, 143.4)
- added D1034: WS2812B, LED_SMD:LED_WS2812B_PLCC4_5.0x5.0mm_P3.2mm, F.Cu at (200.3, 150.9)
- added D1035: WS2812B, LED_SMD:LED_WS2812B_PLCC4_5.0x5.0mm_P3.2mm, F.Cu at (189.5, 152.0)
- added D1036: WS2812B, LED_SMD:LED_WS2812B_PLCC4_5.0x5.0mm_P3.2mm, F.Cu at (177.8, 147.6)
- added D1037: WS2812B, LED_SMD:LED_WS2812B_PLCC4_5.0x5.0mm_P3.2mm, F.Cu at (166.7, 139.0)
- added D1038: WS2812B, LED_SMD:LED_WS2812B_PLCC4_5.0x5.0mm_P3.2mm, F.Cu at (157.2, 128.0)
- added D1039: WS2812B, LED_SMD:LED_WS2812B_PLCC4_5.0x5.0mm_P3.2mm, F.Cu at (149.6, 116.2)
- added D1040: WS2812B, LED_SMD:LED_WS2812B_PLCC4_5.0x5.0mm_P3.2mm, F.Cu at (144.0, 105.6)
- added D1041: WS2812B, LED_SMD:LED_WS2812B_PLCC4_5.0x5.0mm_P3.2mm, F.Cu at (138.3, 116.4)
- added D1042: WS2812B, LED_SMD:LED_WS2812B_PLCC4_5.0x5.0mm_P3.2mm, F.Cu at (130.7, 128.1)
- added D1043: WS2812B, LED_SMD:LED_WS2812B_PLCC4_5.0x5.0mm_P3.2mm, F.Cu at (121.2, 139.1)
- added D1044: WS2812B, LED_SMD:LED_WS2812B_PLCC4_5.0x5.0mm_P3.2mm, F.Cu at (110.1, 147.6)
- added D1045: WS2812B, LED_SMD:LED_WS2812B_PLCC4_5.0x5.0mm_P3.2mm, F.Cu at (98.4, 152.0)
- added D1046: WS2812B, LED_SMD:LED_WS2812B_PLCC4_5.0x5.0mm_P3.2mm, F.Cu at (87.6, 150.9)
- added D1047: WS2812B, LED_SMD:LED_WS2812B_PLCC4_5.0x5.0mm_P3.2mm, F.Cu at (80.1, 143.3)
- added D1048: WS2812B, LED_SMD:LED_WS2812B_PLCC4_5.0x5.0mm_P3.2mm, F.Cu at (79.0, 132.5)
- added D1049: WS2812B, LED_SMD:LED_WS2812B_PLCC4_5.0x5.0mm_P3.2mm, F.Cu at (83.4, 120.8)
- added D1050: WS2812B, LED_SMD:LED_WS2812B_PLCC4_5.0x5.0mm_P3.2mm, F.Cu at (92.0, 109.7)
- added D1051: WS2812B, LED_SMD:LED_WS2812B_PLCC4_5.0x5.0mm_P3.2mm, F.Cu at (103.0, 100.2)
- added D1052: WS2812B, LED_SMD:LED_WS2812B_PLCC4_5.0x5.0mm_P3.2mm, F.Cu at (114.8, 92.6)
- added D1053: WS2812B, LED_SMD:LED_WS2812B_PLCC4_5.0x5.0mm_P3.2mm, F.Cu at (102.9, 87.0)
- added D1054: WS2812B, LED_SMD:LED_WS2812B_PLCC4_5.0x5.0mm_P3.2mm, F.Cu at (93.0, 77.1)
- added D1055: WS2812B, LED_SMD:LED_WS2812B_PLCC4_5.0x5.0mm_P3.2mm, F.Cu at (93.0, 87.0)
- added D1056: WS2812B, LED_SMD:LED_WS2812B_PLCC4_5.0x5.0mm_P3.2mm, F.Cu at (93.0, 96.9)
- added D1057: WS2812B, LED_SMD:LED_WS2812B_PLCC4_5.0x5.0mm_P3.2mm, F.Cu at (144.0, 45.9)
- added D1058: WS2812B, LED_SMD:LED_WS2812B_PLCC4_5.0x5.0mm_P3.2mm, F.Cu at (153.9, 36.0)
- added D1059: WS2812B, LED_SMD:LED_WS2812B_PLCC4_5.0x5.0mm_P3.2mm, F.Cu at (144.0, 36.0)
- added D1060: WS2812B, LED_SMD:LED_WS2812B_PLCC4_5.0x5.0mm_P3.2mm, F.Cu at (134.1, 36.0)
- added D1061: WS2812B, LED_SMD:LED_WS2812B_PLCC4_5.0x5.0mm_P3.2mm, F.Cu at (185.1, 87.0)
- added D1062: WS2812B, LED_SMD:LED_WS2812B_PLCC4_5.0x5.0mm_P3.2mm, F.Cu at (195.0, 96.9)
- added D1063: WS2812B, LED_SMD:LED_WS2812B_PLCC4_5.0x5.0mm_P3.2mm, F.Cu at (195.0, 87.0)
- added D1064: WS2812B, LED_SMD:LED_WS2812B_PLCC4_5.0x5.0mm_P3.2mm, F.Cu at (195.0, 77.1)
- added D1065: WS2812B, LED_SMD:LED_WS2812B_PLCC4_5.0x5.0mm_P3.2mm, F.Cu at (144.0, 128.1)
- added D1066: WS2812B, LED_SMD:LED_WS2812B_PLCC4_5.0x5.0mm_P3.2mm, F.Cu at (134.1, 138.0)
- added D1067: WS2812B, LED_SMD:LED_WS2812B_PLCC4_5.0x5.0mm_P3.2mm, F.Cu at (144.0, 138.0)
- added D1068: WS2812B, LED_SMD:LED_WS2812B_PLCC4_5.0x5.0mm_P3.2mm, F.Cu at (153.9, 138.0)
- added D1069: WS2812B, LED_SMD:LED_WS2812B_PLCC4_5.0x5.0mm_P3.2mm, F.Cu at (119.2, 62.2)
- added D1070: WS2812B, LED_SMD:LED_WS2812B_PLCC4_5.0x5.0mm_P3.2mm, F.Cu at (111.8, 54.8)
- added D1071: WS2812B, LED_SMD:LED_WS2812B_PLCC4_5.0x5.0mm_P3.2mm, F.Cu at (104.4, 47.4)
- added D1072: WS2812B, LED_SMD:LED_WS2812B_PLCC4_5.0x5.0mm_P3.2mm, F.Cu at (96.9, 39.9)
- added D1073: WS2812B, LED_SMD:LED_WS2812B_PLCC4_5.0x5.0mm_P3.2mm, F.Cu at (168.8, 62.2)
- added D1074: WS2812B, LED_SMD:LED_WS2812B_PLCC4_5.0x5.0mm_P3.2mm, F.Cu at (176.2, 54.8)
- added D1075: WS2812B, LED_SMD:LED_WS2812B_PLCC4_5.0x5.0mm_P3.2mm, F.Cu at (183.6, 47.4)
- added D1076: WS2812B, LED_SMD:LED_WS2812B_PLCC4_5.0x5.0mm_P3.2mm, F.Cu at (191.1, 39.9)
- added D1077: WS2812B, LED_SMD:LED_WS2812B_PLCC4_5.0x5.0mm_P3.2mm, F.Cu at (168.8, 111.8)
- added D1078: WS2812B, LED_SMD:LED_WS2812B_PLCC4_5.0x5.0mm_P3.2mm, F.Cu at (176.2, 119.2)
- added D1079: WS2812B, LED_SMD:LED_WS2812B_PLCC4_5.0x5.0mm_P3.2mm, F.Cu at (183.6, 126.6)
- added D1080: WS2812B, LED_SMD:LED_WS2812B_PLCC4_5.0x5.0mm_P3.2mm, F.Cu at (191.1, 134.1)
- added D1081: WS2812B, LED_SMD:LED_WS2812B_PLCC4_5.0x5.0mm_P3.2mm, F.Cu at (119.2, 111.8)
- added D1082: WS2812B, LED_SMD:LED_WS2812B_PLCC4_5.0x5.0mm_P3.2mm, F.Cu at (111.8, 119.2)
- added D1083: WS2812B, LED_SMD:LED_WS2812B_PLCC4_5.0x5.0mm_P3.2mm, F.Cu at (104.4, 126.6)
- added D1084: WS2812B, LED_SMD:LED_WS2812B_PLCC4_5.0x5.0mm_P3.2mm, F.Cu at (96.9, 134.1)
- added D1085: WS2812B, LED_SMD:LED_WS2812B_PLCC4_5.0x5.0mm_P3.2mm, F.Cu at (79.6, 74.6)
- added D1086: WS2812B, LED_SMD:LED_WS2812B_PLCC4_5.0x5.0mm_P3.2mm, F.Cu at (79.6, 99.4)
- added D1087: WS2812B, LED_SMD:LED_WS2812B_PLCC4_5.0x5.0mm_P3.2mm, F.Cu at (79.6, 87.0)
- added D1088: WS2812B, LED_SMD:LED_WS2812B_PLCC4_5.0x5.0mm_P3.2mm, F.Cu at (156.4, 22.6)
- added D1089: WS2812B, LED_SMD:LED_WS2812B_PLCC4_5.0x5.0mm_P3.2mm, F.Cu at (131.6, 22.6)
- added D1090: WS2812B, LED_SMD:LED_WS2812B_PLCC4_5.0x5.0mm_P3.2mm, F.Cu at (144.0, 22.6)
- added D1091: WS2812B, LED_SMD:LED_WS2812B_PLCC4_5.0x5.0mm_P3.2mm, F.Cu at (208.4, 74.6)
- added D1092: WS2812B, LED_SMD:LED_WS2812B_PLCC4_5.0x5.0mm_P3.2mm, F.Cu at (208.4, 99.4)
- added D1093: WS2812B, LED_SMD:LED_WS2812B_PLCC4_5.0x5.0mm_P3.2mm, F.Cu at (208.4, 87.0)
- added D1094: WS2812B, LED_SMD:LED_WS2812B_PLCC4_5.0x5.0mm_P3.2mm, F.Cu at (156.4, 151.4)
- added D1095: WS2812B, LED_SMD:LED_WS2812B_PLCC4_5.0x5.0mm_P3.2mm, F.Cu at (131.6, 151.4)
- added D1096: WS2812B, LED_SMD:LED_WS2812B_PLCC4_5.0x5.0mm_P3.2mm, F.Cu at (144.0, 151.4)
- added D1097: WS2812B, Footprints:WS2812-mini, F.Cu at (137.8, 80.8)
- added D1098: WS2812B, Footprints:WS2812-mini, F.Cu at (144.0, 80.8)
- added D1099: WS2812B, Footprints:WS2812-mini, F.Cu at (150.2, 80.8)
- added D1100: WS2812B, Footprints:WS2812-mini, F.Cu at (150.2, 87.0)
- added D1101: WS2812B, Footprints:WS2812-mini, F.Cu at (150.2, 93.2)
- added D1102: WS2812B, Footprints:WS2812-mini, F.Cu at (144.0, 93.2)
- added D1103: WS2812B, Footprints:WS2812-mini, F.Cu at (137.8, 93.2)
- added D1104: WS2812B, Footprints:WS2812-mini, F.Cu at (137.8, 87.0)
- added D1105: WS2812B, Footprints:WS2812-mini, F.Cu at (144.0, 87.0)
- added H1001: MountingHole, MountingHole:MountingHole_3.2mm_M3, F.Cu at (198.0, 141.0)
- added H1002: MountingHole, MountingHole:MountingHole_3.2mm_M3, F.Cu at (90.0, 33.0)
- added H1003: MountingHole, MountingHole:MountingHole_3.2mm_M3, F.Cu at (90.0, 141.0)
- added H1004: MountingHole, MountingHole:MountingHole_3.2mm_M3, F.Cu at (198.0, 33.0)
- added H1005: MountingHole, MountingHole:MountingHole_3.2mm_M3, F.Cu at (127.0, 104.0)
- added H1006: MountingHole, MountingHole:MountingHole_3.2mm_M3, F.Cu at (161.0, 104.0)
- added H1007: MountingHole, MountingHole:MountingHole_3.2mm_M3, F.Cu at (161.0, 70.0)
- added H1008: MountingHole, MountingHole:MountingHole_3.2mm_M3, F.Cu at (127.0, 70.0)
- added R1001: 470R, Resistor_SMD:R_0603_1608Metric, B.Cu at (112.5, 75.5)
- added R1003: 470R, Resistor_SMD:R_0603_1608Metric, B.Cu at (104.5, 78.5)
- added R1005: 470R, Resistor_SMD:R_0603_1608Metric, B.Cu at (105.5, 71.0)
- added R1085: 470R, Resistor_SMD:R_0603_1608Metric, B.Cu at (117.5, 79.5)
- added R1086: 470R, Resistor_SMD:R_0603_1608Metric, B.Cu at (117.5, 75.5)
- BT301, C201, C202, C203, C204, C301, C401, C501, C502, C503, C504, C601, C602, D301, D302, D303, D601, FB201, J201, J401, J501, L501, L601, LS501, R201, R202, R203, R204, R301, R302, R303, R304, R305, R306, R307, R308, R309, R310, R401, R402, R501, R601, R602, SW501, U201, U202, U301, U401, U501, U601, Y501: moved to B.Cu
- C302, C303, C304: footprint Capacitor_SMD:C_0603_1608Metric -> Capacitor_SMD:C_0805_2012Metric; moved to B.Cu
- moved J401 400.5 mm to (79.5, 66.5), turned to 180 degrees
- moved C401 378.3 mm to (94.0, 104.0)
- moved R401 372.1 mm to (100.0, 106.0), turned to 180 degrees
- moved C601 370.5 mm to (172.3, 125.8), turned to 180 degrees
- moved D601 370.5 mm to (165.4, 126.0), turned to 180 degrees
- moved L601 370.5 mm to (164.9, 131.3), turned to 180 degrees
- moved R601 370.5 mm to (163.4, 139.8), turned to 180 degrees
- moved C602 370.5 mm to (164.2, 136.4), turned to 180 degrees
- moved R602 370.5 mm to (177.1, 125.0), turned to 180 degrees
- moved U601 370.5 mm to (171.0, 130.5), turned to 180 degrees
- moved U401 364.5 mm to (100.0, 95.5), turned to -90 degrees
- moved R402 360.7 mm to (103.5, 106.0), turned to 180 degrees
- moved J402 354.1 mm to (124.5, 21.5)
- moved C502 346.4 mm to (134.5, 113.0), turned to 180 degrees
- moved L501 344.8 mm to (132.5, 118.0), turned to 90 degrees
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Other:
- board outline added: 150 x 150 mm

Commit message: update
Parts:
- BT301: footprint Footprints:battery_906909_6000mah -> Footprints:battery_103565_3000mah
- J401: moved to F.Cu
- J501: footprint Footprints:2x03_P2.54mm -> Connector_PinHeader_1.27mm:PinHeader_2x03_P1.27mm_Vertical_SMD
- moved J401 31.4 mm to (73.2, 97.2), turned to -90 degrees
- moved J403 29.8 mm to (214.8, 76.8), turned to 90 degrees
- moved BT301 14.2 mm to (144.5, 44.2)
- moved J404 13.0 mm to (153.6, 157.7)
- moved J402 10.6 mm to (133.7, 16.2), turned to 180 degrees
- moved J201 9.50 mm to (134.5, 158.0)
- moved J301 7.90 mm to (163.1, 95.3)
- moved J302 7.79 mm to (163.0, 98.2)
- moved D1085 6.95 mm to (76.6, 68.3)
- moved D1086 6.95 mm to (76.6, 105.7)
- moved D1088 6.95 mm to (162.7, 19.6)
- moved D1089 6.95 mm to (125.3, 19.6)
- moved D1091 6.95 mm to (211.4, 68.3)
- moved D1092 6.95 mm to (211.4, 105.7)
- moved D1094 6.95 mm to (162.7, 154.4)
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
Commit message: update
Parts:
- removed D301, D302, D303: LED_Small, LED_SMD:LED_0603_1608Metric
- removed R1085, R1086: 470R, Resistor_SMD:R_0603_1608Metric
- removed R304, R306, R309: 1k, Resistor_SMD:R_0603_1608Metric
- added D1106: WS2812B, LED_SMD:LED_WS2812B_PLCC4_5.0x5.0mm_P3.2mm, F.Cu at (112.0, 157.0)
- added R1002: 470R, Resistor_SMD:R_0603_1608Metric, B.Cu at (97.6, 145.0)
- added R1004: 470R, Resistor_SMD:R_0603_1608Metric, B.Cu at (97.6, 140.0)
- added R1006: 470R, Resistor_SMD:R_0603_1608Metric, B.Cu at (97.6, 142.5)
- added R1007: 10k, Resistor_SMD:R_0603_1608Metric, B.Cu at (111.0, 140.0)
- added R1008: 10k, Resistor_SMD:R_0603_1608Metric, B.Cu at (107.0, 140.0)
- added R1009: 10k, Resistor_SMD:R_0603_1608Metric, B.Cu at (107.0, 142.5)
- moved J201 22.5 mm to (112.0, 158.0)
Connections:
- U301 pad 6: Net-(R304-Pad1) -> PG
- U301 pad 7: Net-(R309-Pad1) -> STAT2
- U301 pad 8: Net-(R306-Pad1) -> STAT1
- U501 pad 23: unconnected-(U501-Pad23) -> STAT1
- U501 pad 24: unconnected-(U501-Pad24) -> STAT2
- U501 pad 25: unconnected-(U501-Pad25) -> PG
- U501 pad 26: unconnected-(U501-Pad26) -> NP_6

Commit message: update
Parts:
- R1001, R1002, R1003, R1004, R1005, R1006: moved to F.Cu
- moved R1002 80.1 mm to (82.0, 66.5), turned to 0 degrees
- moved R1004 68.1 mm to (165.0, 149.5), turned to -90 degrees
- moved LS501 57.8 mm to (80.0, 137.0)
- moved FB201 31.5 mm to (115.0, 150.0)
- moved R202 31.5 mm to (107.5, 150.5)
- moved R203 31.5 mm to (112.0, 150.0)
- moved U201 31.5 mm to (112.5, 145.0)
- moved R1005 30.7 mm to (127.1, 92.8), turned to 90 degrees
- moved C201 27.2 mm to (123.0, 126.0)
- moved C203 27.2 mm to (110.0, 130.0)
- moved R201 27.2 mm to (123.0, 124.0)
- moved R204 27.2 mm to (123.0, 129.0)
- moved U202 27.2 mm to (117.0, 127.5)
- moved C202 27.2 mm to (110.5, 124.5)
- moved R1006 19.4 mm to (114.5, 152.0), turned to 0 degrees
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Routing:
- net Net-(D1051-Pad2): track 0.00 -> 15.3 mm
- net Net-(D1061-Pad2): track 0.00 -> 14.5 mm
- net Net-(D1057-Pad2): track 0.00 -> 14.2 mm
- net Net-(D1013-Pad2): track 0.00 -> 14.0 mm
- net Net-(D1053-Pad2): track 0.00 -> 13.9 mm
- net Net-(D1065-Pad2): track 0.00 -> 13.8 mm
- net Net-(D1039-Pad2): track 0.00 -> 13.3 mm
- net Net-(D1026-Pad2): track 0.00 -> 12.6 mm
- net Net-(D1015-Pad2): track 0.00 -> 11.6 mm
- net Net-(D1016-Pad2): track 0.00 -> 11.1 mm
- net Net-(D1024-Pad2): track 0.00 -> 10.9 mm
- net Net-(D1003-Pad2): track 0.00 -> 10.8 mm
- net Net-(D1029-Pad2): track 0.00 -> 10.8 mm
- net Net-(D1011-Pad2): track 0.00 -> 10.6 mm
- net Net-(D1022-Pad2): track 0.00 -> 10.5 mm
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
Commit message: update
Parts:
- moved R1004 78.4 mm to (137.8, 76.0), turned to 0 degrees
- moved R1002 8.36 mm to (75.0, 62.0), turned to -90 degrees
- turned D1073 to 180 degrees
- turned D1074 to 180 degrees
- turned D1075 to 180 degrees
- turned D1076 to 180 degrees
- turned D1077 to 90 degrees
- turned D1078 to 90 degrees
- turned D1079 to 90 degrees
- turned D1080 to 90 degrees
- turned D1085 to 90 degrees
- turned D1086 to -90 degrees
- turned D1087 to -90 degrees
- turned D1089 to 180 degrees
- turned D1090 to 180 degrees
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Connections:
- D1093 pad 2: unconnected-(D1093-Pad2) -> Net-(D1093-Pad2)
- D1094 pad 4: Net-(D1094-Pad4) -> Net-(D1093-Pad2)
- D1096 pad 2: Net-(D1096-Pad2) -> unconnected-(D1096-Pad2)
- D1097 pad 4: Net-(D1096-Pad2) -> Net-(R1004-Pad2)
- R1004 pad 2: Net-(D1094-Pad4) -> Net-(R1004-Pad2)
Routing:
- net VCC: track 0.00 -> 1063.0 mm
- net Net-(D1088-Pad2): track 0.00 -> 49.2 mm
- net Net-(D1085-Pad2): track 0.00 -> 43.2 mm
- net Net-(D1094-Pad2): track 0.00 -> 42.3 mm
- net Net-(D1091-Pad2): track 0.00 -> 40.7 mm
- net Net-(D1095-Pad2): track 0.00 -> 15.1 mm
- net Net-(D1089-Pad2): track 0.00 -> 15.1 mm
- net Net-(D1092-Pad2): track 0.00 -> 15.1 mm
- net Net-(D1086-Pad2): track 0.00 -> 15.1 mm
- net Net-(D1101-Pad2): track 0.00 -> 13.8 mm
- net Net-(D1103-Pad2): track 0.00 -> 9.83 mm
- net Net-(D1082-Pad2): track 0.00 -> 6.17 mm
- net Net-(D1081-Pad2): track 0.00 -> 6.17 mm
- net Net-(D1075-Pad2): track 0.00 -> 6.17 mm
- net Net-(D1074-Pad2): track 0.00 -> 6.17 mm
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
Commit message: layout_v2
Parts:
- removed C502, C503: 100n, Capacitor_SMD:C_0603_1608Metric
- removed L501: 10u, Inductor_SMD:L_1206_3216Metric
- removed R1007, R1008, R1009: 10k, Resistor_SMD:R_0603_1608Metric
- R1001, R1002, R1003, R1004, R1005, R1006: moved to B.Cu
- moved LS501 126.9 mm to (205.8, 120.0)
- moved R1002 99.0 mm to (155.5, 119.5), turned to 0 degrees
- moved C204 57.1 mm to (90.0, 128.5), turned to 0 degrees
- moved R1003 56.7 mm to (155.5, 117.8), turned to 0 degrees
- moved R1001 47.1 mm to (139.0, 111.5)
- moved J501 44.3 mm to (177.4, 122.8)
- moved R1004 43.7 mm to (155.5, 116.0)
- moved R303 41.9 mm to (172.0, 146.8)
- moved R301 39.2 mm to (172.0, 148.8)
- moved R307 38.6 mm to (172.0, 144.8)
- moved C401 38.6 mm to (124.1, 124.3), turned to -90 degrees
- moved C302 37.1 mm to (182.7, 140.6), turned to -90 degrees
- moved C301 36.1 mm to (185.5, 140.3), turned to -90 degrees
- moved C601 35.2 mm to (140.8, 141.6)
- moved L601 35.2 mm to (133.5, 147.0)
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- renumbered D1086 to D1085, D1087 to D1086, D1085 to D1087, D1089 to D1088, D1090 to D1089, D1088 to D1090, D1093 to D1092, D1092 to D1093, D1096 to D1095, D1095 to D1096
Connections:
- net Net-(FB201-Pad1) renamed /USB/USB
- D1085 pad 4: Net-(D1085-Pad2) (its old number) -> Net-(D1085-Pad4)
- D1086 pad 2: Net-(D1087-Pad2) -> Net-(D1086-Pad2)
- D1087 pad 2: Net-(D1085-Pad2) (its old number) -> Net-(D1087-Pad2)
- D1087 pad 4: Net-(D1085-Pad4) -> Net-(D1086-Pad2)
- D1088 pad 4: Net-(D1088-Pad2) (its old number) -> Net-(D1087-Pad2)
- D1089 pad 2: Net-(D1090-Pad2) -> Net-(D1089-Pad2)
- D1090 pad 2: Net-(D1088-Pad2) (its old number) -> Net-(D1090-Pad2)
- D1090 pad 4: Net-(D1087-Pad2) -> Net-(D1089-Pad2)
- D1092 pad 2: Net-(D1093-Pad2) -> Net-(D1092-Pad2)
- D1092 pad 4: Net-(D1092-Pad2) -> Net-(D1091-Pad2)
- D1093 pad 2: Net-(D1092-Pad2) -> Net-(D1093-Pad2)
- D1093 pad 4: Net-(D1091-Pad2) -> Net-(D1092-Pad2)
- D1095 pad 2: unconnected-(D1096-Pad2) -> Net-(D1095-Pad2)
- D1095 pad 4: Net-(D1095-Pad2) -> Net-(D1094-Pad2)
- D1096 pad 2: Net-(D1095-Pad2) -> unconnected-(D1096-Pad2)
- D1096 pad 4: Net-(D1094-Pad2) -> Net-(D1095-Pad2)
- U501 pad 18: Net-(C502-Pad1) -> unconnected-(U501-Pad18)
- U501 pad 20: +5V -> unconnected-(U501-Pad20)
Routing:
- net VCC: track 1063.0 -> 1517.9 mm, vias 0 -> 9
- net Net-(LS501-Pad1): track 0.00 -> 60.0 mm
- net GND: track 0.00 -> 56.6 mm, vias 0 -> 33
- net Net-(D1088-Pad2) (its old number): track 49.2 -> 0.00 mm
- net PG: track 0.00 -> 45.5 mm
- net SCK: track 0.00 -> 43.6 mm
- net Net-(D1085-Pad2) (its old number): track 43.2 -> 0.00 mm
- net TX: track 0.00 -> 42.7 mm
- net STAT2: track 0.00 -> 41.6 mm
- net STAT1: track 0.00 -> 39.0 mm
- net MISO: track 0.00 -> 34.5 mm
- net Net-(D1094-Pad2): track 42.3 -> 15.1 mm
- net USB_D+: track 0.00 -> 26.5 mm
- net MOSI: track 0.00 -> 26.2 mm
- net Net-(D1091-Pad2): track 40.7 -> 15.1 mm
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- added copper zone on B.Cu, net /USB/USB
- added copper zone on B.Cu, net GND
- added copper zone on F.Cu, net GND
