File: KiCad files/BoardGame/Microcontroller.kicad_sch (KiCad schematic)
At the start: 11 parts

Commit message: update
Parts:
- removed C? (x2): 100n, symbol Device:C_Small
- removed C?: 1u, symbol Device:C_Small
- added C? (x2): 100n, Capacitor_SMD:C_0603_1608Metric, symbol Device:C_Small
- added C?: 1u, Capacitor_SMD:C_0603_1608Metric, symbol Device:C_Small
- C?: footprint (none) -> Capacitor_SMD:C_0603_1608Metric; Basic/Extended Basic -> (none); JLCPCB Part # C49678 -> (none); U labosu? Da -> (none)
- L?: Basic/Extended Extended -> (none); JLCPCB Part # C279941 -> (none); U labosu? Ne -> (none)
- R?: footprint (none) -> Resistor_SMD:R_0603_1608Metric; Basic/Extended Basic -> (none); JLCPCB Part # C17414 -> (none); U labosu? Da -> (none)
Connections:
- net +5V: now also C?.1
- net GND: now also C?.1, C?.2, C?.2
- net RESET: now also C?.2
- net at L?.2, U?.18 (AVCC): now also C?.1
Changed lines of the file:
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@@
   (junction (at 154.305 62.23) (diameter 0) (color 0 0 0 0)
   )
-  (junction (at 170.815 128.905) (diameter 0) (color 0 0 0 0)
+  (junction (at 170.815 130.81) (diameter 0) (color 0 0 0 0)
   )
   (junction (at 123.19 62.23) (diameter 0) (color 0 0 0 0)
@@
     (stroke (width 0) (type default) (color 0 0 0 0))
   )
-  (wire (pts (xy 174.625 128.905) (xy 170.815 128.905))
-    (stroke (width 0) (type default) (color 0 0 0 0))
-  )
   (wire (pts (xy 135.255 67.945) (xy 135.255 62.23))
     (stroke (width 0) (type default) (color 0 0 0 0))
@@
     (stroke (width 0) (type default) (color 0 0 0 0))
   )
-  (wire (pts (xy 170.815 130.81) (xy 170.815 128.905))
+  (wire (pts (xy 179.705 130.81) (xy 183.515 130.81))
+    (stroke (width 0) (type default) (color 0 0 0 0))
+  )
+  (wire (pts (xy 170.815 132.715) (xy 170.815 130.81))
     (stroke (width 0) (type default) (color 0 0 0 0))
   )
@@
     (stroke (width 0) (type default) (color 0 0 0 0))
   )
-  (wire (pts (xy 179.705 128.905) (xy 183.515 128.905))
-    (stroke (width 0) (type default) (color 0 0 0 0))
-  )
   (wire (pts (xy 132.715 62.23) (xy 132.715 67.945))
     (stroke (width 0) (type default) (color 0 0 0 0))
@@
     (stroke (width 0) (type default) (color 0 0 0 0))
   )
-  (wire (pts (xy 183.515 128.905) (xy 183.515 125.095))
-    (stroke (width 0) (type default) (color 0 0 0 0))
-  )
   (wire (pts (xy 135.255 62.23) (xy 140.335 62.23))
     (stroke (width 0) (type default) (color 0 0 0 0))
@@
     (stroke (width 0) (type default) (color 0 0 0 0))
   )
-  (wire (pts (xy 170.815 128.905) (xy 170.815 125.095))
+  (wire (pts (xy 183.515 125.095) (xy 183.515 130.81))
+    (stroke (width 0) (type default) (color 0 0 0 0))
+  )
+  (wire (pts (xy 170.815 130.81) (xy 174.625 130.81))
+    (stroke (width 0) (type default) (color 0 0 0 0))
+  )
+  (wire (pts (xy 170.815 125.095) (xy 170.815 130.81))
     (stroke (width 0) (type default) (color 0 0 0 0))
   )
@@
   (symbol (lib_id "Device:R_Small") (at 183.515 121.285 180) (unit 1)
     (in_bom yes) (on_board yes)
-    (property "Reference" "R?" (id 0) (at 185.42 121.285 90))
-    (property "Value" "10k" (id 1) (at 183.515 121.285 90)
-      (effects (font (size 0.9906 0.9906)))
-    )
-    (property "Footprint" "" (id 2) (at 183.515 121.285 0)
+    (property "Reference" "R?" (id 0) (at 186.055 120.015 0))
+    (property "Value" "10k" (id 1) (at 186.69 121.92 0))
+    (property "Footprint" "Resistor_SMD:R_0603_1608Metric" (id 2) (at 183.515 121.285 0)
       (effects (font (size 1.27 1.27)) hide)
     )
     (property "Datasheet" "~" (id 3) (at 183.515 121.285 0)
-      (effects (font (size 1.27 1.27)) hide)
-    )
-    (property "Basic/Extended" "Basic" (id 4) (at 183.515 121.285 0)
-      (effects (font (size 1.27 1.27)) hide)
-    )
-    (property "JLCPCB Part #" "C17414" (id 5) (at 183.515 121.285 0)
-      (effects (font (size 1.27 1.27)) hide)
-    )
-    (property "U labosu?" "Da" (id 6) (at 183.515 121.285 0)
       (effects (font (size 1.27 1.27)) hide)
     )
@@
       (effects (font (size 1.27 1.27)) (justify left))
     )
-    (property "Footprint" "" (id 2) (at 90.805 66.04 0)
+    (property "Footprint" "Capacitor_SMD:C_0603_1608Metric" (id 2) (at 90.805 66.04 0)
       (effects (font (size 1.27 1.27)) hide)
     )
@@
       (effects (font (size 1.27 1.27)) hide)
     )
-    (property "Basic/Extended" "Basic" (id 4) (at 90.805 66.04 0)
-      (effects (font (size 1.27 1.27)) hide)
-    )
-    (property "JLCPCB Part #" "C49678" (id 5) (at 90.805 66.04 0)
-      (effects (font (size 1.27 1.27)) hide)
-    )
-    (property "U labosu?" "Da" (id 6) (at 90.805 66.04 0)
-      (effects (font (size 1.27 1.27)) hide)
-    )
-    (pin "1")
-    (pin "2")
-  )
-  (symbol (lib_id "power:GND") (at 170.815 130.81 0) (unit 1)
-    (in_bom yes) (on_board yes)
-    (property "Reference" "#PWR?" (id 0) (at 170.815 137.16 0)
-      (effects (font (size 1.27 1.27)) hide)
-    )
-    (property "Value" "GND" (id 1) (at 170.942 135.2042 0))
-    (property "Footprint" "" (id 2) (at 170.815 130.81 0)
-      (effects (font (size 1.27 1.27)) hide)
-    )
-    (property "Datasheet" "" (id 3) (at 170.815 130.81 0)
+    (pin "1")
+    (pin "2")
+  )
+  (symbol (lib_id "power:GND") (at 170.815 132.715 0) (unit 1)
+    (in_bom yes) (on_board yes)
+    (property "Reference" "#PWR?" (id 0) (at 170.815 139.065 0)
+      (effects (font (size 1.27 1.27)) hide)
+    )
+    (property "Value" "GND" (id 1) (at 170.942 137.1092 0))
+    (property "Footprint" "" (id 2) (at 170.815 132.715 0)
+      (effects (font (size 1.27 1.27)) hide)
+    )
+    (property "Datasheet" "" (id 3) (at 170.815 132.715 0)
       (effects (font (size 1.27 1.27)) hide)
     )
@@
       (effects (font (size 1.27 1.27)) (justify left))
     )
-    (property "Footprint" "" (id 2) (at 154.305 67.31 0)
+    (property "Footprint" "Capacitor_SMD:C_0603_1608Metric" (id 2) (at 154.305 67.31 0)
       (effects (font (size 1.27 1.27)) hide)
     )
     (property "Datasheet" "~" (id 3) (at 154.305 67.31 0)
-      (effects (font (size 1.27 1.27)) hide)
-    )
-    (property "Basic/Extended" "Basic" (id 4) (at 154.305 67.31 0)
-      (effects (font (size 1.27 1.27)) hide)
-    )
-    (property "JLCPCB Part #" "C49678" (id 5) (at 154.305 67.31 0)
-      (effects (font (size 1.27 1.27)) hide)
-    )
-    (property "U labosu?" "Da" (id 6) (at 154.305 67.31 0)
-      (effects (font (size 1.27 1.27)) hide)
-    )
-    (pin "1")
-    (pin "2")
-  )
-  (symbol (lib_id "Device:C_Small") (at 177.165 128.905 270) (unit 1)
-    (in_bom yes) (on_board yes)
-    (property "Reference" "C?" (id 0) (at 175.895 132.08 90)
-      (effects (font (size 1.27 1.27)) (justify left))
-    )
-    (property "Value" "1u" (id 1) (at 175.895 133.985 90)
-      (effects (font (size 1.27 1.27)) (justify left))
-    )
-    (property "Footprint" "" (id 2) (at 177.165 128.905 0)
-      (effects (font (size 1.27 1.27)) hide)
-    )
-    (property "Datasheet" "~" (id 3) (at 177.165 128.905 0)
-      (effects (font (size 1.27 1.27)) hide)
-    )
-    (property "Basic/Extended" "Basic" (id 4) (at 177.165 128.905 0)
-      (effects (font (size 1.27 1.27)) hide)
-    )
-    (property "JLCPCB Part #" "C28323" (id 5) (at 177.165 128.905 0)
-      (effects (font (size 1.27 1.27)) hide)
-    )
-    (property "U labosu?" "Da" (id 6) (at 177.165 128.905 0)
       (effects (font (size 1.27 1.27)) hide)
     )
@@
     (pin "1")
   )
-  (symbol (lib_id "Device:C_Small") (at 105.41 82.55 0) (unit 1)
-    (in_bom yes) (on_board yes)
-    (property "Reference" "C?" (id 0) (at 107.7468 81.3816 0)
-      (effects (font (size 1.27 1.27)) (justify left))
-    )
-    (property "Value" "100n" (id 1) (at 107.7468 83.693 0)
-      (effects (font (size 1.27 1.27)) (justify left))
-    )
-    (property "Footprint" "" (id 2) (at 105.41 82.55 0)
-      (effects (font (size 1.27 1.27)) hide)
-    )
-    (property "Datasheet" "~" (id 3) (at 105.41 82.55 0)
-      (effects (font (size 1.27 1.27)) hide)
-    )
-    (property "Basic/Extended" "Basic" (id 4) (at 105.41 82.55 0)
-      (effects (font (size 1.27 1.27)) hide)
-    )
-    (property "JLCPCB Part #" "C49678" (id 5) (at 105.41 82.55 0)
-      (effects (font (size 1.27 1.27)) hide)
-    )
-    (property "U labosu?" "Da" (id 6) (at 105.41 82.55 0)
-      (effects (font (size 1.27 1.27)) hide)
-    )
-    (pin "1")
-    (pin "2")
-  )
   (symbol (lib_id "power:+5V") (at 154.305 52.07 0) (unit 1)
     (in_bom yes) (on_board yes) (fields_autoplaced)
@@
     (pin "1")
   )
+  (symbol (lib_id "Device:C_Small") (at 177.165 130.81 90) (unit 1)
+    (in_bom yes) (on_board yes)
+    (property "Reference" "C?" (id 0) (at 178.435 127.635 90)
+      (effects (font (size 1.27 1.27)) (justify left))
+    )
+    (property "Value" "1u" (id 1) (at 178.435 133.985 90)
+      (effects (font (size 1.27 1.27)) (justify left))
+    )
+    (property "Footprint" "Capacitor_SMD:C_0603_1608Metric" (id 2) (at 177.165 130.81 0)
+      (effects (font (size 1.27 1.27)) hide)
+    )
+    (property "Datasheet" "~" (id 3) (at 177.165 130.81 0)
+      (effects (font (size 1.27 1.27)) hide)
+    )
+    (pin "1")
+    (pin "2")
+  )
   (symbol (lib_id "power:+5V") (at 183.515 118.745 0) (unit 1)
     (in_bom yes) (on_board yes) (fields_autoplaced)
@@
       (effects (font (size 1.27 1.27)) hide)
     )
-    (property "Basic/Extended" "Extended" (id 4) (at 154.305 56.515 0)
-      (effects (font (size 1.27 1.27)) hide)
-    )
-    (property "JLCPCB Part #" "C279941" (id 5) (at 154.305 56.515 0)
-      (effects (font (size 1.27 1.27)) hide)
-    )
-    (property "U labosu?" "Ne" (id 6) (at 154.305 56.515 0)
-      (effects (font (size 1.27 1.27)) hide)
-    )
     (pin "1")
     (pin "2")
@@
     (pin "1")
   )
+  (symbol (lib_id "Device:C_Small") (at 105.41 82.55 0) (unit 1)
+    (in_bom yes) (on_board yes)
+    (property "Reference" "C?" (id 0) (at 107.7468 81.3816 0)
+      (effects (font (size 1.27 1.27)) (justify left))
+    )
+    (property "Value" "100n" (id 1) (at 107.7468 83.693 0)
+      (effects (font (size 1.27 1.27)) (justify left))
+    )
+    (property "Footprint" "Capacitor_SMD:C_0603_1608Metric" (id 2) (at 105.41 82.55 0)
+      (effects (font (size 1.27 1.27)) hide)
+    )
+    (property "Datasheet" "~" (id 3) (at 105.41 82.55 0)
+      (effects (font (size 1.27 1.27)) hide)
+    )
+    (pin "1")
+    (pin "2")
+  )
   (symbol (lib_id "Connector_Generic:Conn_02x03_Odd_Even") (at 207.01 63.5 0) (unit 1)

Commit message: update
Parts:
- J8: renamed from J?; Basic/Extended - -> (none); JLCPCB Part # - -> (none); U labosu? Da -> (none)
- LS1: renamed from LS?; footprint (none) -> Footprints:KLJ-1102
- SW1: renamed from SW?; footprint (none) -> Button_Switch_SMD:SW_SPST_TL3342; Basic/Extended Basic -> (none); JLCPCB Part # C307331 -> (none); U labosu? Ne -> (none)
- Y1: renamed from Y?; footprint (none) -> Footprints:CSTCE16M0V53-R0; Basic/Extended Extended -> (none); JLCPCB Part # C32180 -> (none); U labosu? Da -> (none)
- gave numbers to parts that had none: 7
Changed lines of the file:
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@@
   (symbol (lib_id "Switch:SW_Push") (at 177.165 125.095 0) (unit 1)
     (in_bom yes) (on_board yes)
-    (property "Reference" "SW?" (id 0) (at 177.165 120.015 0))
+    (property "Reference" "SW1" (id 0) (at 177.165 120.015 0))
     (property "Value" "SW_Push" (id 1) (at 177.165 120.1674 0)
       (effects (font (size 1.27 1.27)) hide)
     )
-    (property "Footprint" "" (id 2) (at 177.165 120.015 0)
+    (property "Footprint" "Button_Switch_SMD:SW_SPST_TL3342" (id 2) (at 177.165 120.015 0)
       (effects (font (size 1.27 1.27)) hide)
     )
@@
       (effects (font (size 1.27 1.27)) hide)
     )
-    (property "Basic/Extended" "Basic" (id 4) (at 177.165 125.095 0)
-      (effects (font (size 1.27 1.27)) hide)
-    )
-    (property "JLCPCB Part #" "C307331" (id 5) (at 177.165 125.095 0)
-      (effects (font (size 1.27 1.27)) hide)
-    )
-    (property "U labosu?" "Ne" (id 6) (at 177.165 125.095 0)
-      (effects (font (size 1.27 1.27)) hide)
-    )
     (pin "1")
     (pin "2")
@@
   (symbol (lib_id "power:GND") (at 169.545 102.87 0) (unit 1)
     (in_bom yes) (on_board yes)
-    (property "Reference" "#PWR?" (id 0) (at 169.545 109.22 0)
+    (property "Reference" "#PWR053" (id 0) (at 169.545 109.22 0)
       (effects (font (size 1.27 1.27)) hide)
     )
@@
   (symbol (lib_id "power:GND") (at 193.04 98.425 0) (unit 1)
     (in_bom yes) (on_board yes) (fields_autoplaced)
-    (property "Reference" "#PWR?" (id 0) (at 193.04 104.775 0)
+    (property "Reference" "#PWR052" (id 0) (at 193.04 104.775 0)
       (effects (font (size 1.27 1.27)) hide)
     )
@@
   (symbol (lib_id "Device:R_Small") (at 183.515 121.285 180) (unit 1)
     (in_bom yes) (on_board yes)
-    (property "Reference" "R?" (id 0) (at 186.055 120.015 0))
+    (property "Reference" "R17" (id 0) (at 186.055 120.015 0))
     (property "Value" "10k" (id 1) (at 186.69 121.92 0))
     (property "Footprint" "Resistor_SMD:R_0603_1608Metric" (id 2) (at 183.515 121.285 0)
@@
   (symbol (lib_id "power:+5V") (at 105.41 74.295 0) (unit 1)
     (in_bom yes) (on_board yes) (fields_autoplaced)
-    (property "Reference" "#PWR?" (id 0) (at 105.41 78.105 0)
+    (property "Reference" "#PWR050" (id 0) (at 105.41 78.105 0)
       (effects (font (size 1.27 1.27)) hide)
     )
@@
   (symbol (lib_id "Device:Speaker") (at 200.025 94.615 0) (unit 1)
     (in_bom yes) (on_board yes) (fields_autoplaced)
-    (property "Reference" "LS?" (id 0) (at 204.343 95.0503 0)
+    (property "Reference" "LS1" (id 0) (at 204.343 95.0503 0)
       (effects (font (size 1.27 1.27)) (justify left))
     )
@@
       (effects (font (size 1.27 1.27)) (justify left))
     )
-    (property "Footprint" "" (id 2) (at 200.025 99.695 0)
+    (property "Footprint" "Footprints:KLJ-1102" (id 2) (at 200.025 99.695 0)
       (effects (font (size 1.27 1.27)) hide)
     )
@@
   (symbol (lib_id "power:PWR_FLAG") (at 123.19 59.69 0) (unit 1)
     (in_bom yes) (on_board yes) (fields_autoplaced)
-    (property "Reference" "#FLG?" (id 0) (at 123.19 57.785 0)
+    (property "Reference" "#FLG04" (id 0) (at 123.19 57.785 0)
       (effects (font (size 1.27 1.27)) hide)
     )
@@
   (symbol (lib_id "MCU_Microchip_ATmega:ATmega328P-A") (at 132.715 106.045 0) (unit 1)
     (in_bom yes) (on_board yes) (fields_autoplaced)
-    (property "Reference" "U?" (id 0) (at 134.7344 143.6354 0)
+    (property "Reference" "U5" (id 0) (at 134.7344 143.6354 0)
       (effects (font (size 1.27 1.27)) (justify left))
     )
@@
   (symbol (lib_id "Device:C_Small") (at 90.805 66.04 0) (unit 1)
     (in_bom yes) (on_board yes)
-    (property "Reference" "C?" (id 0) (at 93.1418 64.8716 0)
+    (property "Reference" "C10" (id 0) (at 93.1418 64.8716 0)
       (effects (font (size 1.27 1.27)) (justify left))
     )
@@
   (symbol (lib_id "power:GND") (at 170.815 132.715 0) (unit 1)
     (in_bom yes) (on_board yes)
-    (property "Reference" "#PWR?" (id 0) (at 170.815 139.065 0)
+    (property "Reference" "#PWR055" (id 0) (at 170.815 139.065 0)
       (effects (font (size 1.27 1.27)) hide)
     )
@@
   (symbol (lib_id "power:GND") (at 132.715 144.145 0) (unit 1)
     (in_bom yes) (on_board yes)
-    (property "Reference" "#PWR?" (id 0) (at 132.715 150.495 0)
+    (property "Reference" "#PWR056" (id 0) (at 132.715 150.495 0)
       (effects (font (size 1.27 1.27)) hide)
     )
@@
   (symbol (lib_id "Device:C_Small") (at 154.305 67.31 0) (unit 1)
     (in_bom yes) (on_board yes)
-    (property "Reference" "C?" (id 0) (at 156.6418 66.1416 0)
+    (property "Reference" "C11" (id 0) (at 156.6418 66.1416 0)
       (effects (font (size 1.27 1.27)) (justify left))
     )
@@
   (symbol (lib_id "power:PWR_FLAG") (at 140.335 59.69 0) (unit 1)
     (in_bom yes) (on_board yes) (fields_autoplaced)
-    (property "Reference" "#FLG?" (id 0) (at 140.335 57.785 0)
+    (property "Reference" "#FLG05" (id 0) (at 140.335 57.785 0)
       (effects (font (size 1.27 1.27)) hide)
     )
@@
   (symbol (lib_id "power:+5V") (at 154.305 52.07 0) (unit 1)
     (in_bom yes) (on_board yes) (fields_autoplaced)
-    (property "Reference" "#PWR?" (id 0) (at 154.305 55.88 0)
+    (property "Reference" "#PWR046" (id 0) (at 154.305 55.88 0)
       (effects (font (size 1.27 1.27)) hide)
     )
@@
   (symbol (lib_id "power:+5V") (at 90.805 60.325 0) (unit 1)
     (in_bom yes) (on_board yes) (fields_autoplaced)
-    (property "Reference" "#PWR?" (id 0) (at 90.805 64.135 0)
+    (property "Reference" "#PWR047" (id 0) (at 90.805 64.135 0)
       (effects (font (size 1.27 1.27)) hide)
     )
@@
   (symbol (lib_id "Device:Resonator_Small") (at 169.545 97.79 0) (unit 1)
     (in_bom yes) (on_board yes)
-    (property "Reference" "Y?" (id 0) (at 174.3202 97.8916 0)
+    (property "Reference" "Y1" (id 0) (at 174.3202 97.8916 0)
       (effects (font (size 1.27 1.27)) (justify left))
     )
@@
       (effects (font (size 1.27 1.27)) (justify left))
     )
-    (property "Footprint" "" (id 2) (at 168.91 97.79 0)
+    (property "Footprint" "Footprints:CSTCE16M0V53-R0" (id 2) (at 168.91 97.79 0)
       (effects (font (size 1.27 1.27)) hide)
     )
@@
       (effects (font (size 1.27 1.27)) hide)
     )
-    (property "JLCPCB Part #" "C32180" (id 4) (at 169.545 97.79 0)
-      (effects (font (size 1.27 1.27)) hide)
-    )
-    (property "Basic/Extended" "Extended" (id 5) (at 169.545 97.79 0)
-      (effects (font (size 1.27 1.27)) hide)
-    )
-    (property "U labosu?" "Da" (id 6) (at 169.545 97.79 0)
-      (effects (font (size 1.27 1.27)) hide)
-    )
     (pin "1")
     (pin "2")
@@
   (symbol (lib_id "power:GND") (at 154.305 69.85 0) (unit 1)
     (in_bom yes) (on_board yes)
-    (property "Reference" "#PWR?" (id 0) (at 154.305 76.2 0)
+    (property "Reference" "#PWR049" (id 0) (at 154.305 76.2 0)
       (effects (font (size 1.27 1.27)) hide)
     )
@@
   (symbol (lib_id "Device:C_Small") (at 177.165 130.81 90) (unit 1)
     (in_bom yes) (on_board yes)
-    (property "Reference" "C?" (id 0) (at 178.435 127.635 90)
+    (property "Reference" "C13" (id 0) (at 178.435 127.635 90)
       (effects (font (size 1.27 1.27)) (justify left))
     )
@@
   (symbol (lib_id "power:+5V") (at 183.515 118.745 0) (unit 1)
     (in_bom yes) (on_board yes) (fields_autoplaced)
-    (property "Reference" "#PWR?" (id 0) (at 183.515 122.555 0)
+    (property "Reference" "#PWR054" (id 0) (at 183.515 122.555 0)
       (effects (font (size 1.27 1.27)) hide)
     )
@@
   (symbol (lib_id "power:GND") (at 105.41 85.09 0) (unit 1)
     (in_bom yes) (on_board yes)
-    (property "Reference" "#PWR?" (id 0) (at 105.41 91.44 0)
+    (property "Reference" "#PWR051" (id 0) (at 105.41 91.44 0)
       (effects (font (size 1.27 1.27)) hide)
     )
@@
   (symbol (lib_id "Device:L_Small") (at 154.305 56.515 0) (unit 1)
     (in_bom yes) (on_board yes) (fields_autoplaced)
-    (property "Reference" "L?" (id 0) (at 155.448 55.6065 0)
+    (property "Reference" "L1" (id 0) (at 155.448 55.6065 0)
       (effects (font (size 1.27 1.27)) (justify left))
     )
@@
   (symbol (lib_id "power:GND") (at 90.805 68.58 0) (unit 1)
     (in_bom yes) (on_board yes)
-    (property "Reference" "#PWR?" (id 0) (at 90.805 74.93 0)
+    (property "Reference" "#PWR048" (id 0) (at 90.805 74.93 0)
       (effects (font (size 1.27 1.27)) hide)
     )
@@
   (symbol (lib_id "Device:C_Small") (at 105.41 82.55 0) (unit 1)
     (in_bom yes) (on_board yes)
-    (property "Reference" "C?" (id 0) (at 107.7468 81.3816 0)
+    (property "Reference" "C12" (id 0) (at 107.7468 81.3816 0)
       (effects (font (size 1.27 1.27)) (justify left))
     )
@@
   (symbol (lib_id "Connector_Generic:Conn_02x03_Odd_Even") (at 207.01 63.5 0) (unit 1)
     (in_bom yes) (on_board yes)
-    (property "Reference" "J?" (id 0) (at 208.28 58.42 0))
+    (property "Reference" "J8" (id 0) (at 208.28 58.42 0))
     (property "Value" "USBasp" (id 1) (at 208.28 68.58 0))
     (property "Footprint" "" (id 2) (at 207.01 63.5 0)
@@
       (effects (font (size 1.27 1.27)) hide)
     )
-    (property "Basic/Extended" "-" (id 4) (at 207.01 63.5 0)
-      (effects (font (size 1.27 1.27)) hide)
-    )
-    (property "JLCPCB Part #" "-" (id 5) (at 207.01 63.5 0)
-      (effects (font (size 1.27 1.27)) hide)
-    )
-    (property "U labosu?" "Da" (id 6) (at 207.01 63.5 0)
-      (effects (font (size 1.27 1.27)) hide)
-    )
