File: KiCad files/BoardGame/Microcontroller.kicad_sch (KiCad schematic)
At the start: 11 parts, among them J8 USBasp, SW1 SW_Push, U5 ATmega328P-A, Y1 16MHz

Commit message: update
Parts:
- J501: renamed from J8; footprint (none) -> Footprints:2x03_P2.54mm
- L501: renamed from L1; footprint (none) -> Inductor_SMD:L_1206_3216Metric
- renumbered C10 to C501, C11 to C502, C12 to C503, C13 to C504, LS1 to LS501, R17 to R501, SW1 to SW501, U5 to U501, Y1 to Y501
Changed lines of the file:
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@@
   (symbol (lib_id "Switch:SW_Push") (at 177.165 125.095 0) (unit 1)
     (in_bom yes) (on_board yes)
-    (property "Reference" "SW1" (id 0) (at 177.165 120.015 0))
+    (property "Reference" "SW501" (id 0) (at 177.165 120.015 0))
     (property "Value" "SW_Push" (id 1) (at 177.165 120.1674 0)
       (effects (font (size 1.27 1.27)) hide)
@@
   (symbol (lib_id "power:GND") (at 169.545 102.87 0) (unit 1)
     (in_bom yes) (on_board yes)
-    (property "Reference" "#PWR053" (id 0) (at 169.545 109.22 0)
+    (property "Reference" "#PWR0508" (id 0) (at 169.545 109.22 0)
       (effects (font (size 1.27 1.27)) hide)
     )
@@
   (symbol (lib_id "power:GND") (at 193.04 98.425 0) (unit 1)
     (in_bom yes) (on_board yes) (fields_autoplaced)
-    (property "Reference" "#PWR052" (id 0) (at 193.04 104.775 0)
+    (property "Reference" "#PWR0507" (id 0) (at 193.04 104.775 0)
       (effects (font (size 1.27 1.27)) hide)
     )
@@
   (symbol (lib_id "Device:R_Small") (at 183.515 121.285 180) (unit 1)
     (in_bom yes) (on_board yes)
-    (property "Reference" "R17" (id 0) (at 186.055 120.015 0))
+    (property "Reference" "R501" (id 0) (at 186.055 120.015 0))
     (property "Value" "10k" (id 1) (at 186.69 121.92 0))
     (property "Footprint" "Resistor_SMD:R_0603_1608Metric" (id 2) (at 183.515 121.285 0)
@@
   (symbol (lib_id "power:+5V") (at 105.41 74.295 0) (unit 1)
     (in_bom yes) (on_board yes) (fields_autoplaced)
-    (property "Reference" "#PWR050" (id 0) (at 105.41 78.105 0)
+    (property "Reference" "#PWR0505" (id 0) (at 105.41 78.105 0)
       (effects (font (size 1.27 1.27)) hide)
     )
@@
   (symbol (lib_id "Device:Speaker") (at 200.025 94.615 0) (unit 1)
     (in_bom yes) (on_board yes) (fields_autoplaced)
-    (property "Reference" "LS1" (id 0) (at 204.343 95.0503 0)
+    (property "Reference" "LS501" (id 0) (at 204.343 95.0503 0)
       (effects (font (size 1.27 1.27)) (justify left))
     )
@@
   (symbol (lib_id "power:PWR_FLAG") (at 123.19 59.69 0) (unit 1)
     (in_bom yes) (on_board yes) (fields_autoplaced)
-    (property "Reference" "#FLG04" (id 0) (at 123.19 57.785 0)
+    (property "Reference" "#FLG0501" (id 0) (at 123.19 57.785 0)
       (effects (font (size 1.27 1.27)) hide)
     )
@@
   (symbol (lib_id "MCU_Microchip_ATmega:ATmega328P-A") (at 132.715 106.045 0) (unit 1)
     (in_bom yes) (on_board yes) (fields_autoplaced)
-    (property "Reference" "U5" (id 0) (at 134.7344 143.6354 0)
+    (property "Reference" "U501" (id 0) (at 134.7344 143.6354 0)
       (effects (font (size 1.27 1.27)) (justify left))
     )
@@
   (symbol (lib_id "Device:C_Small") (at 90.805 66.04 0) (unit 1)
     (in_bom yes) (on_board yes)
-    (property "Reference" "C10" (id 0) (at 93.1418 64.8716 0)
+    (property "Reference" "C501" (id 0) (at 93.1418 64.8716 0)
       (effects (font (size 1.27 1.27)) (justify left))
     )
@@
   (symbol (lib_id "power:GND") (at 170.815 132.715 0) (unit 1)
     (in_bom yes) (on_board yes)
-    (property "Reference" "#PWR055" (id 0) (at 170.815 139.065 0)
+    (property "Reference" "#PWR0510" (id 0) (at 170.815 139.065 0)
       (effects (font (size 1.27 1.27)) hide)
     )
@@
   (symbol (lib_id "power:GND") (at 132.715 144.145 0) (unit 1)
     (in_bom yes) (on_board yes)
-    (property "Reference" "#PWR056" (id 0) (at 132.715 150.495 0)
+    (property "Reference" "#PWR0511" (id 0) (at 132.715 150.495 0)
       (effects (font (size 1.27 1.27)) hide)
     )
@@
   (symbol (lib_id "Device:C_Small") (at 154.305 67.31 0) (unit 1)
     (in_bom yes) (on_board yes)
-    (property "Reference" "C11" (id 0) (at 156.6418 66.1416 0)
+    (property "Reference" "C502" (id 0) (at 156.6418 66.1416 0)
       (effects (font (size 1.27 1.27)) (justify left))
     )
@@
   (symbol (lib_id "power:PWR_FLAG") (at 140.335 59.69 0) (unit 1)
     (in_bom yes) (on_board yes) (fields_autoplaced)
-    (property "Reference" "#FLG05" (id 0) (at 140.335 57.785 0)
+    (property "Reference" "#FLG0502" (id 0) (at 140.335 57.785 0)
       (effects (font (size 1.27 1.27)) hide)
     )
@@
   (symbol (lib_id "power:+5V") (at 154.305 52.07 0) (unit 1)
     (in_bom yes) (on_board yes) (fields_autoplaced)
-    (property "Reference" "#PWR046" (id 0) (at 154.305 55.88 0)
+    (property "Reference" "#PWR0501" (id 0) (at 154.305 55.88 0)
       (effects (font (size 1.27 1.27)) hide)
     )
@@
   (symbol (lib_id "power:+5V") (at 90.805 60.325 0) (unit 1)
     (in_bom yes) (on_board yes) (fields_autoplaced)
-    (property "Reference" "#PWR047" (id 0) (at 90.805 64.135 0)
+    (property "Reference" "#PWR0502" (id 0) (at 90.805 64.135 0)
       (effects (font (size 1.27 1.27)) hide)
     )
@@
   (symbol (lib_id "Device:Resonator_Small") (at 169.545 97.79 0) (unit 1)
     (in_bom yes) (on_board yes)
-    (property "Reference" "Y1" (id 0) (at 174.3202 97.8916 0)
+    (property "Reference" "Y501" (id 0) (at 174.3202 97.8916 0)
       (effects (font (size 1.27 1.27)) (justify left))
     )
@@
   (symbol (lib_id "power:GND") (at 154.305 69.85 0) (unit 1)
     (in_bom yes) (on_board yes)
-    (property "Reference" "#PWR049" (id 0) (at 154.305 76.2 0)
+    (property "Reference" "#PWR0504" (id 0) (at 154.305 76.2 0)
       (effects (font (size 1.27 1.27)) hide)
     )
@@
   (symbol (lib_id "Device:C_Small") (at 177.165 130.81 90) (unit 1)
     (in_bom yes) (on_board yes)
-    (property "Reference" "C13" (id 0) (at 178.435 127.635 90)
+    (property "Reference" "C504" (id 0) (at 178.435 127.635 90)
       (effects (font (size 1.27 1.27)) (justify left))
     )
@@
   (symbol (lib_id "power:+5V") (at 183.515 118.745 0) (unit 1)
     (in_bom yes) (on_board yes) (fields_autoplaced)
-    (property "Reference" "#PWR054" (id 0) (at 183.515 122.555 0)
+    (property "Reference" "#PWR0509" (id 0) (at 183.515 122.555 0)
       (effects (font (size 1.27 1.27)) hide)
     )
@@
   (symbol (lib_id "power:GND") (at 105.41 85.09 0) (unit 1)
     (in_bom yes) (on_board yes)
-    (property "Reference" "#PWR051" (id 0) (at 105.41 91.44 0)
+    (property "Reference" "#PWR0506" (id 0) (at 105.41 91.44 0)
       (effects (font (size 1.27 1.27)) hide)
     )
@@
   (symbol (lib_id "Device:L_Small") (at 154.305 56.515 0) (unit 1)
     (in_bom yes) (on_board yes) (fields_autoplaced)
-    (property "Reference" "L1" (id 0) (at 155.448 55.6065 0)
+    (property "Reference" "L501" (id 0) (at 155.448 55.6065 0)
       (effects (font (size 1.27 1.27)) (justify left))
     )
@@
       (effects (font (size 1.27 1.27)) (justify left))
     )
-    (property "Footprint" "" (id 2) (at 154.305 56.515 0)
+    (property "Footprint" "Inductor_SMD:L_1206_3216Metric" (id 2) (at 154.305 56.515 0)
       (effects (font (size 1.27 1.27)) hide)
     )
@@
   (symbol (lib_id "power:GND") (at 90.805 68.58 0) (unit 1)
     (in_bom yes) (on_board yes)
-    (property "Reference" "#PWR048" (id 0) (at 90.805 74.93 0)
+    (property "Reference" "#PWR0503" (id 0) (at 90.805 74.93 0)
       (effects (font (size 1.27 1.27)) hide)
     )
@@
   (symbol (lib_id "Device:C_Small") (at 105.41 82.55 0) (unit 1)
     (in_bom yes) (on_board yes)
-    (property "Reference" "C12" (id 0) (at 107.7468 81.3816 0)
+    (property "Reference" "C503" (id 0) (at 107.7468 81.3816 0)
       (effects (font (size 1.27 1.27)) (justify left))
     )
@@
   (symbol (lib_id "Connector_Generic:Conn_02x03_Odd_Even") (at 207.01 63.5 0) (unit 1)
     (in_bom yes) (on_board yes)
-    (property "Reference" "J8" (id 0) (at 208.28 58.42 0))
+    (property "Reference" "J501" (id 0) (at 208.28 58.42 0))
     (property "Value" "USBasp" (id 1) (at 208.28 68.58 0))
-    (property "Footprint" "" (id 2) (at 207.01 63.5 0)
-      (effects (font (size 1.27 1.27)) hide)
-    )
+    (property "Footprint" "Footprints:2x03_P2.54mm" (id 2) (at 207.01 63.5 0)
+      (effects (font (size 1.27 1.27)) hide)
+    )

Commit message: update
Parts:
- C501, C502, C503: JLCPCB Part # (none) -> C113803; U labosu? (none) -> ne
- C504: JLCPCB Part # (none) -> C559769; U labosu? (none) -> da
- J501: JLCPCB Part # (none) -> -; Ostalo (none) -> -; U labosu? (none) -> da
- L501: JLCPCB Part # (none) -> C281117; U labosu? (none) -> da
- LS501, R501, U501: U labosu? (none) -> da
- SW501: JLCPCB Part # (none) -> C2886894; U labosu? (none) -> ne
- Y501: JLCPCB Part # (none) -> C32180; U labosu? (none) -> da
Changed lines of the file:
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@@
+      (effects (font (size 1.27 1.27)) hide)
+    )
+    (property "JLCPCB Part #" "C2886894" (id 4) (at 177.165 125.095 0)
+      (effects (font (size 1.27 1.27)) hide)
+    )
+    (property "U labosu?" "ne" (id 5) (at 177.165 125.095 0)
       (effects (font (size 1.27 1.27)) hide)
     )
@@
   (symbol (lib_id "Device:R_Small") (at 183.515 121.285 180) (unit 1)
     (in_bom yes) (on_board yes)
-    (property "Reference" "R501" (id 0) (at 186.055 120.015 0))
+    (property "Reference" "R501" (id 0) (at 187.325 120.015 0))
     (property "Value" "10k" (id 1) (at 186.69 121.92 0))
     (property "Footprint" "Resistor_SMD:R_0603_1608Metric" (id 2) (at 183.515 121.285 0)
@@
       (effects (font (size 1.27 1.27)) hide)
     )
+    (property "U labosu?" "da" (id 4) (at 183.515 121.285 0)
+      (effects (font (size 1.27 1.27)) hide)
+    )
     (pin "1")
     (pin "2")
@@
       (effects (font (size 1.27 1.27)) hide)
     )
+    (property "U labosu?" "da" (id 4) (at 200.025 94.615 0)
+      (effects (font (size 1.27 1.27)) hide)
+    )
     (pin "1")
     (pin "2")
@@
     )
     (property "Datasheet" "http://ww1.microchip.com/downloads/en/DeviceDoc/ATmega328_P%20AVR%20MCU%20with%20picoPower%20Technology%20Data%20Sheet%2040001984A.pdf" (id 3) (at 132.715 106.045 0)
+      (effects (font (size 1.27 1.27)) hide)
+    )
+    (property "U labosu?" "da" (id 4) (at 132.715 106.045 0)
       (effects (font (size 1.27 1.27)) hide)
     )
@@
       (effects (font (size 1.27 1.27)) hide)
     )
+    (property "U labosu?" "ne" (id 4) (at 90.805 66.04 0)
+      (effects (font (size 1.27 1.27)) hide)
+    )
+    (property "JLCPCB Part #" "C113803" (id 5) (at 90.805 66.04 0)
+      (effects (font (size 1.27 1.27)) hide)
+    )
     (pin "1")
     (pin "2")
@@
       (effects (font (size 1.27 1.27)) hide)
     )
+    (property "U labosu?" "ne" (id 4) (at 154.305 67.31 0)
+      (effects (font (size 1.27 1.27)) hide)
+    )
+    (property "JLCPCB Part #" "C113803" (id 5) (at 154.305 67.31 0)
+      (effects (font (size 1.27 1.27)) hide)
+    )
     (pin "1")
     (pin "2")
@@
       (effects (font (size 1.27 1.27)) hide)
     )
+    (property "JLCPCB Part #" "C32180" (id 4) (at 169.545 97.79 0)
+      (effects (font (size 1.27 1.27)) hide)
+    )
+    (property "U labosu?" "da" (id 5) (at 169.545 97.79 0)
+      (effects (font (size 1.27 1.27)) hide)
+    )
     (pin "1")
     (pin "2")
@@
       (effects (font (size 1.27 1.27)) hide)
     )
+    (property "JLCPCB Part #" "C559769" (id 4) (at 177.165 130.81 0)
+      (effects (font (size 1.27 1.27)) hide)
+    )
+    (property "U labosu?" "da" (id 5) (at 177.165 130.81 0)
+      (effects (font (size 1.27 1.27)) hide)
+    )
     (pin "1")
     (pin "2")
@@
       (effects (font (size 1.27 1.27)) hide)
     )
+    (property "JLCPCB Part #" "C281117" (id 4) (at 154.305 56.515 0)
+      (effects (font (size 1.27 1.27)) hide)
+    )
+    (property "U labosu?" "da" (id 5) (at 154.305 56.515 0)
+      (effects (font (size 1.27 1.27)) hide)
+    )
     (pin "1")
     (pin "2")
@@
     )
     (property "Datasheet" "~" (id 3) (at 105.41 82.55 0)
+      (effects (font (size 1.27 1.27)) hide)
+    )
+    (property "U labosu?" "ne" (id 4) (at 105.41 82.55 0)
+      (effects (font (size 1.27 1.27)) hide)
+    )
+    (property "JLCPCB Part #" "C113803" (id 5) (at 105.41 82.55 0)
       (effects (font (size 1.27 1.27)) hide)
     )
@@
       (effects (font (size 1.27 1.27)) hide)
     )
+    (property "JLCPCB Part #" "-" (id 4) (at 207.01 63.5 0)
+      (effects (font (size 1.27 1.27)) hide)
+    )
+    (property "Ostalo" "-" (id 5) (at 207.01 63.5 0)
+      (effects (font (size 1.27 1.27)) hide)
+    )
+    (property "U labosu?" "da" (id 6) (at 207.01 63.5 0)
+      (effects (font (size 1.27 1.27)) hide)
+    )

Commit message: update
Parts:
- J501: footprint Footprints:2x03_P2.54mm -> Connector_PinHeader_1.27mm:PinHeader_2x03_P1.27mm_Vertical_SMD
Changed lines of the file:
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@@
     (property "Reference" "J501" (id 0) (at 208.28 58.42 0))
     (property "Value" "USBasp" (id 1) (at 208.28 68.58 0))
-    (property "Footprint" "Footprints:2x03_P2.54mm" (id 2) (at 207.01 63.5 0)
+    (property "Footprint" "Connector_PinHeader_1.27mm:PinHeader_2x03_P1.27mm_Vertical_SMD" (id 2) (at 207.01 63.5 0)
       (effects (font (size 1.27 1.27)) hide)
     )

Commit message: update
Connections:
- net STAT1: now reaches U501.23 (PC0)
- net STAT2: now reaches U501.24 (PC1)
- net PG: now reaches U501.25 (PC2)
- net NP_6: now reaches U501.26 (PC3)
- no-connect marks 9 -> 5
Changed lines of the file:
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@@
   )
   (no_connect (at 117.475 80.645))
-  (no_connect (at 147.955 100.965))
   (no_connect (at 117.475 83.185))
-  (no_connect (at 147.955 103.505))
   (no_connect (at 214.63 60.96))
-  (no_connect (at 147.955 98.425))
   (no_connect (at 147.955 78.105))
-  (no_connect (at 147.955 106.045))
   (no_connect (at 147.955 75.565))
   (wire (pts (xy 193.04 80.645) (xy 193.04 94.615))
@@
     (effects (font (size 1.27 1.27)) (justify left bottom))
   )
+  (global_label "STAT1" (shape input) (at 147.955 98.425 0) (fields_autoplaced)
+    (effects (font (size 1.27 1.27)) (justify left))
+    (property "Intersheet References" "${INTERSHEET_REFS}" (id 0) (at 155.811 98.3456 0)
+      (effects (font (size 1.27 1.27)) (justify left) hide)
+    )
+  )
   (global_label "MOSI" (shape input) (at 147.955 83.185 0) (fields_autoplaced)
     (effects (font (size 1.27 1.27)) (justify left))
@@
     )
   )
+  (global_label "PG" (shape input) (at 147.955 103.505 0) (fields_autoplaced)
+    (effects (font (size 1.27 1.27)) (justify left))
+    (property "Intersheet References" "${INTERSHEET_REFS}" (id 0) (at 152.9081 103.4256 0)
+      (effects (font (size 1.27 1.27)) (justify left) hide)
+    )
+  )
   (global_label "NP_1" (shape input) (at 147.955 126.365 0) (fields_autoplaced)
     (effects (font (size 1.27 1.27)) (justify left))
@@
     )
   )
+  (global_label "NP_6" (shape input) (at 147.955 106.045 0) (fields_autoplaced)
+    (effects (font (size 1.27 1.27)) (justify left))
+    (property "Intersheet References" "${INTERSHEET_REFS}" (id 0) (at 155.1457 105.9656 0)
+      (effects (font (size 1.27 1.27)) (justify left) hide)
+    )
+  )
   (global_label "NP_2" (shape input) (at 147.955 128.905 0) (fields_autoplaced)
     (effects (font (size 1.27 1.27)) (justify left))
@@
       (effects (font (size 1.27 1.27)) (justify left) hide)
     )
+  )
+  (global_label "STAT2" (shape input) (at 147.955 100.965 0) (fields_autoplaced)
+    (effects (font (size 1.27 1.27)) (justify left))
+    (property "Intersheet References" "${INTERSHEET_REFS}" (id 0) (at 155.811 100.8856 0)
+      (effects (font (size 1.27 1.27)) (justify left) hide)
+    )
