File: KiCad files/BoardGame/Microcontroller.kicad_sch (KiCad schematic)
At the start: 11 parts, among them J501 USBasp, SW501 SW_Push, U501 ATmega328P-A, Y501 16MHz

Commit message: layout_v2
Parts:
- removed C502, C503: 100n, Capacitor_SMD:C_0603_1608Metric, symbol Device:C_Small
- removed L501: 10u, Inductor_SMD:L_1206_3216Metric, symbol Device:L_Small
Connections:
- net +5V: no longer U501.20 (AREF)
- no-connect marks 5 -> 7
Changed lines of the file:
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@@
     (rev "1")
   )
-  (junction (at 154.305 62.23) (diameter 0) (color 0 0 0 0)
-  )
   (junction (at 170.815 130.81) (diameter 0) (color 0 0 0 0)
   )
@@
   (junction (at 183.515 125.095) (diameter 0) (color 0 0 0 0)
   )
-  (junction (at 105.41 75.565) (diameter 0) (color 0 0 0 0)
-  )
-  (junction (at 140.335 62.23) (diameter 0) (color 0 0 0 0)
-  )
   (junction (at 90.805 62.23) (diameter 0) (color 0 0 0 0)
   )
+  (no_connect (at 117.475 75.565))
+  (no_connect (at 135.255 67.945))
   (no_connect (at 117.475 80.645))
   (no_connect (at 117.475 83.185))
@@
     (stroke (width 0) (type default) (color 0 0 0 0))
   )
-  (wire (pts (xy 135.255 67.945) (xy 135.255 62.23))
-    (stroke (width 0) (type default) (color 0 0 0 0))
-  )
   (wire (pts (xy 170.815 125.095) (xy 172.085 125.095))
     (stroke (width 0) (type default) (color 0 0 0 0))
@@
     (stroke (width 0) (type default) (color 0 0 0 0))
   )
-  (wire (pts (xy 105.41 80.01) (xy 105.41 75.565))
-    (stroke (width 0) (type default) (color 0 0 0 0))
-  )
-  (wire (pts (xy 105.41 75.565) (xy 117.475 75.565))
-    (stroke (width 0) (type default) (color 0 0 0 0))
-  )
   (wire (pts (xy 90.805 60.325) (xy 90.805 62.23))
     (stroke (width 0) (type default) (color 0 0 0 0))
@@
     (stroke (width 0) (type default) (color 0 0 0 0))
   )
-  (wire (pts (xy 105.41 74.295) (xy 105.41 75.565))
-    (stroke (width 0) (type default) (color 0 0 0 0))
-  )
   (wire (pts (xy 182.245 125.095) (xy 183.515 125.095))
     (stroke (width 0) (type default) (color 0 0 0 0))
@@
     (stroke (width 0) (type default) (color 0 0 0 0))
   )
-  (wire (pts (xy 154.305 62.23) (xy 154.305 64.77))
-    (stroke (width 0) (type default) (color 0 0 0 0))
-  )
-  (wire (pts (xy 135.255 62.23) (xy 140.335 62.23))
-    (stroke (width 0) (type default) (color 0 0 0 0))
-  )
-  (wire (pts (xy 140.335 62.23) (xy 154.305 62.23))
-    (stroke (width 0) (type default) (color 0 0 0 0))
-  )
   (wire (pts (xy 183.515 125.095) (xy 183.515 130.81))
     (stroke (width 0) (type default) (color 0 0 0 0))
@@
   )
   (wire (pts (xy 90.805 62.23) (xy 123.19 62.23))
-    (stroke (width 0) (type default) (color 0 0 0 0))
-  )
-  (wire (pts (xy 154.305 52.07) (xy 154.305 53.975))
-    (stroke (width 0) (type default) (color 0 0 0 0))
-  )
-  (wire (pts (xy 140.335 59.69) (xy 140.335 62.23))
-    (stroke (width 0) (type default) (color 0 0 0 0))
-  )
-  (wire (pts (xy 154.305 59.055) (xy 154.305 62.23))
     (stroke (width 0) (type default) (color 0 0 0 0))
   )
@@
     (pin "1")
     (pin "2")
-  )
-  (symbol (lib_id "power:+5V") (at 105.41 74.295 0) (unit 1)
-    (in_bom yes) (on_board yes) (fields_autoplaced)
-    (property "Reference" "#PWR0505" (id 0) (at 105.41 78.105 0)
-      (effects (font (size 1.27 1.27)) hide)
-    )
-    (property "Value" "+5V" (id 1) (at 105.41 70.7192 0))
-    (property "Footprint" "" (id 2) (at 105.41 74.295 0)
-      (effects (font (size 1.27 1.27)) hide)
-    )
-    (property "Datasheet" "" (id 3) (at 105.41 74.295 0)
-      (effects (font (size 1.27 1.27)) hide)
-    )
-    (pin "1")
   )
   (symbol (lib_id "Device:Speaker") (at 200.025 94.615 0) (unit 1)
@@
     (pin "1")
   )
-  (symbol (lib_id "Device:C_Small") (at 154.305 67.31 0) (unit 1)
-    (in_bom yes) (on_board yes)
-    (property "Reference" "C502" (id 0) (at 156.6418 66.1416 0)
-      (effects (font (size 1.27 1.27)) (justify left))
-    )
-    (property "Value" "100n" (id 1) (at 156.6418 68.453 0)
-      (effects (font (size 1.27 1.27)) (justify left))
-    )
-    (property "Footprint" "Capacitor_SMD:C_0603_1608Metric" (id 2) (at 154.305 67.31 0)
-      (effects (font (size 1.27 1.27)) hide)
-    )
-    (property "Datasheet" "~" (id 3) (at 154.305 67.31 0)
-      (effects (font (size 1.27 1.27)) hide)
-    )
-    (property "U labosu?" "ne" (id 4) (at 154.305 67.31 0)
-      (effects (font (size 1.27 1.27)) hide)
-    )
-    (property "JLCPCB Part #" "C113803" (id 5) (at 154.305 67.31 0)
-      (effects (font (size 1.27 1.27)) hide)
-    )
-    (pin "1")
-    (pin "2")
-  )
-  (symbol (lib_id "power:PWR_FLAG") (at 140.335 59.69 0) (unit 1)
-    (in_bom yes) (on_board yes) (fields_autoplaced)
-    (property "Reference" "#FLG0502" (id 0) (at 140.335 57.785 0)
-      (effects (font (size 1.27 1.27)) hide)
-    )
-    (property "Value" "PWR_FLAG" (id 1) (at 140.335 56.1142 0))
-    (property "Footprint" "" (id 2) (at 140.335 59.69 0)
-      (effects (font (size 1.27 1.27)) hide)
-    )
-    (property "Datasheet" "~" (id 3) (at 140.335 59.69 0)
-      (effects (font (size 1.27 1.27)) hide)
-    )
-    (pin "1")
-  )
-  (symbol (lib_id "power:+5V") (at 154.305 52.07 0) (unit 1)
-    (in_bom yes) (on_board yes) (fields_autoplaced)
-    (property "Reference" "#PWR0501" (id 0) (at 154.305 55.88 0)
-      (effects (font (size 1.27 1.27)) hide)
-    )
-    (property "Value" "+5V" (id 1) (at 154.305 48.4942 0))
-    (property "Footprint" "" (id 2) (at 154.305 52.07 0)
-      (effects (font (size 1.27 1.27)) hide)
-    )
-    (property "Datasheet" "" (id 3) (at 154.305 52.07 0)
-      (effects (font (size 1.27 1.27)) hide)
-    )
-    (pin "1")
-  )
   (symbol (lib_id "power:+5V") (at 90.805 60.325 0) (unit 1)
     (in_bom yes) (on_board yes) (fields_autoplaced)
@@
     (pin "3")
   )
-  (symbol (lib_id "power:GND") (at 154.305 69.85 0) (unit 1)
-    (in_bom yes) (on_board yes)
-    (property "Reference" "#PWR0504" (id 0) (at 154.305 76.2 0)
-      (effects (font (size 1.27 1.27)) hide)
-    )
-    (property "Value" "GND" (id 1) (at 154.432 74.2442 0))
-    (property "Footprint" "" (id 2) (at 154.305 69.85 0)
-      (effects (font (size 1.27 1.27)) hide)
-    )
-    (property "Datasheet" "" (id 3) (at 154.305 69.85 0)
-      (effects (font (size 1.27 1.27)) hide)
-    )
-    (pin "1")
-  )
   (symbol (lib_id "Device:C_Small") (at 177.165 130.81 90) (unit 1)
     (in_bom yes) (on_board yes)
@@
     (pin "1")
   )
-  (symbol (lib_id "power:GND") (at 105.41 85.09 0) (unit 1)
-    (in_bom yes) (on_board yes)
-    (property "Reference" "#PWR0506" (id 0) (at 105.41 91.44 0)
-      (effects (font (size 1.27 1.27)) hide)
-    )
-    (property "Value" "GND" (id 1) (at 105.537 89.4842 0))
-    (property "Footprint" "" (id 2) (at 105.41 85.09 0)
-      (effects (font (size 1.27 1.27)) hide)
-    )
-    (property "Datasheet" "" (id 3) (at 105.41 85.09 0)
-      (effects (font (size 1.27 1.27)) hide)
-    )
-    (pin "1")
-  )
-  (symbol (lib_id "Device:L_Small") (at 154.305 56.515 0) (unit 1)
-    (in_bom yes) (on_board yes) (fields_autoplaced)
-    (property "Reference" "L501" (id 0) (at 155.448 55.6065 0)
-      (effects (font (size 1.27 1.27)) (justify left))
-    )
-    (property "Value" "10u" (id 1) (at 155.448 58.3816 0)
-      (effects (font (size 1.27 1.27)) (justify left))
-    )
-    (property "Footprint" "Inductor_SMD:L_1206_3216Metric" (id 2) (at 154.305 56.515 0)
-      (effects (font (size 1.27 1.27)) hide)
-    )
-    (property "Datasheet" "~" (id 3) (at 154.305 56.515 0)
-      (effects (font (size 1.27 1.27)) hide)
-    )
-    (property "JLCPCB Part #" "C281117" (id 4) (at 154.305 56.515 0)
-      (effects (font (size 1.27 1.27)) hide)
-    )
-    (property "U labosu?" "da" (id 5) (at 154.305 56.515 0)
-      (effects (font (size 1.27 1.27)) hide)
-    )
-    (pin "1")
-    (pin "2")
-  )
   (symbol (lib_id "power:GND") (at 90.805 68.58 0) (unit 1)
     (in_bom yes) (on_board yes)
@@
     (pin "1")
   )
-  (symbol (lib_id "Device:C_Small") (at 105.41 82.55 0) (unit 1)
-    (in_bom yes) (on_board yes)
-    (property "Reference" "C503" (id 0) (at 107.7468 81.3816 0)
-      (effects (font (size 1.27 1.27)) (justify left))
-    )
-    (property "Value" "100n" (id 1) (at 107.7468 83.693 0)
-      (effects (font (size 1.27 1.27)) (justify left))
-    )
-    (property "Footprint" "Capacitor_SMD:C_0603_1608Metric" (id 2) (at 105.41 82.55 0)
-      (effects (font (size 1.27 1.27)) hide)
-    )
-    (property "Datasheet" "~" (id 3) (at 105.41 82.55 0)
-      (effects (font (size 1.27 1.27)) hide)
-    )
-    (property "U labosu?" "ne" (id 4) (at 105.41 82.55 0)
-      (effects (font (size 1.27 1.27)) hide)
-    )
-    (property "JLCPCB Part #" "C113803" (id 5) (at 105.41 82.55 0)
-      (effects (font (size 1.27 1.27)) hide)
-    )
-    (pin "1")
-    (pin "2")
-  )
   (symbol (lib_id "Connector_Generic:Conn_02x03_Odd_Even") (at 207.01 63.5 0) (unit 1)
