File: KiCad files/BoardGame/IO Expander.kicad_sch (KiCad schematic)
At the start: 8 parts

Commit message: update
Parts:
- removed J? (x3): Conn_02x03_Odd_Even, symbol Connector_Generic:Conn_02x03_Odd_Even
- removed R?: 4k7, symbol Device:R_Small
- removed U?: PCF8575, symbol CNLJS-symbols:PCF8575
- added J? (x3): Conn_02x03_Odd_Even, Footprints:2x03_P1.27mm_conn, symbol Connector_Generic:Conn_02x03_Odd_Even
- added R?: 2k2, Resistor_SMD:R_0603_1608Metric, symbol Device:R_Small
- added U?: PCF8575, symbol Symbols:PCF8575
- C?: footprint (none) -> Capacitor_SMD:C_0603_1608Metric
- J?: footprint (none) -> Footprints:2x03_P1.27mm_conn
- R?: value 4k7 -> 2k2; footprint (none) -> Resistor_SMD:R_0603_1608Metric
Connections:
- net GND: now also J?.1 (Pin_1), J?.1 (Pin_1), J?.1 (Pin_1), U?.12 (GND)
- net INT: now also U?.1 (~{INT})
- net SCL: now also U?.22 (SCL)
- net SDA: now also R?.2, U?.23 (SDA)
- net TP_1: now also U?.4 (P00)
- net TP_10: now also J?.2 (Pin_2), U?.14 (P11)
- net TP_11: now also J?.6 (Pin_6), U?.15 (P12)
- net TP_12: now also J?.5 (Pin_5), U?.16 (P13)
- net TP_2: now also U?.5 (P01)
- net TP_3: now also U?.6 (P02)
- net TP_4: now also J?.2 (Pin_2), U?.7 (P03)
- net TP_5: now also J?.6 (Pin_6), U?.8 (P04)
- net TP_6: now also J?.5 (Pin_5), U?.9 (P05)
- net TP_7: now also J?.2 (Pin_2), U?.10 (P06)
- net TP_8: now also J?.6 (Pin_6), U?.11 (P07)
- net TP_9: now also J?.5 (Pin_5), U?.13 (P10)
- net VDD renamed +5V
- net +5V: now also J?.3 (Pin_3), J?.3 (Pin_3), J?.3 (Pin_3), J?.4 (Pin_4), J?.4 (Pin_4), J?.4 (Pin_4), R?.1, U?.24 (VCC)
Other:
- title: (none) -> BoardGame

Commit message: update
Parts:
- U4: renamed from U?; footprint (none) -> Package_SO:SOIC-24W_7.5x15.4mm_P1.27mm
- gave numbers to parts that had none: 7
Changed lines of the file:
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@@
   (symbol (lib_id "power:+5V") (at 165.1 127 0) (unit 1)
     (in_bom yes) (on_board yes) (fields_autoplaced)
-    (property "Reference" "#PWR?" (id 0) (at 165.1 130.81 0)
+    (property "Reference" "#PWR043" (id 0) (at 165.1 130.81 0)
       (effects (font (size 1.27 1.27)) hide)
     )
@@
   (symbol (lib_id "power:GND") (at 165.1 89.535 0) (unit 1)
     (in_bom yes) (on_board yes) (fields_autoplaced)
-    (property "Reference" "#PWR?" (id 0) (at 165.1 95.885 0)
+    (property "Reference" "#PWR036" (id 0) (at 165.1 95.885 0)
       (effects (font (size 1.27 1.27)) hide)
     )
@@
   (symbol (lib_id "power:+5V") (at 196.85 127.635 0) (unit 1)
     (in_bom yes) (on_board yes) (fields_autoplaced)
-    (property "Reference" "#PWR?" (id 0) (at 196.85 131.445 0)
+    (property "Reference" "#PWR044" (id 0) (at 196.85 131.445 0)
       (effects (font (size 1.27 1.27)) hide)
     )
@@
   (symbol (lib_id "Device:R_Small") (at 89.535 99.06 0) (unit 1)
     (in_bom yes) (on_board yes)
-    (property "Reference" "R?" (id 0) (at 90.805 97.79 0)
+    (property "Reference" "R15" (id 0) (at 90.805 97.79 0)
       (effects (font (size 1.27 1.27)) (justify left))
     )
@@
   (symbol (lib_id "Connector_Generic:Conn_02x03_Odd_Even") (at 179.07 83.82 0) (mirror x) (unit 1)
     (in_bom yes) (on_board yes) (fields_autoplaced)
-    (property "Reference" "J?" (id 0) (at 180.34 78.8472 0))
+    (property "Reference" "J5" (id 0) (at 180.34 78.8472 0))
     (property "Value" "Conn_02x03_Odd_Even" (id 1) (at 180.34 88.7929 0)
       (effects (font (size 1.27 1.27)) hide)
@@
   (symbol (lib_id "power:+5V") (at 196.85 104.775 0) (unit 1)
     (in_bom yes) (on_board yes) (fields_autoplaced)
-    (property "Reference" "#PWR?" (id 0) (at 196.85 108.585 0)
+    (property "Reference" "#PWR040" (id 0) (at 196.85 108.585 0)
       (effects (font (size 1.27 1.27)) hide)
     )
@@
   (symbol (lib_id "power:+5V") (at 97.155 96.52 0) (unit 1)
     (in_bom yes) (on_board yes) (fields_autoplaced)
-    (property "Reference" "#PWR?" (id 0) (at 97.155 100.33 0)
+    (property "Reference" "#PWR038" (id 0) (at 97.155 100.33 0)
       (effects (font (size 1.27 1.27)) hide)
     )
@@
   (symbol (lib_id "Connector_Generic:Conn_02x03_Odd_Even") (at 179.07 109.22 0) (mirror x) (unit 1)
     (in_bom yes) (on_board yes) (fields_autoplaced)
-    (property "Reference" "J?" (id 0) (at 180.34 104.2472 0))
+    (property "Reference" "J6" (id 0) (at 180.34 104.2472 0))
     (property "Value" "Conn_02x03_Odd_Even" (id 1) (at 180.34 114.1929 0)
       (effects (font (size 1.27 1.27)) hide)
@@
   (symbol (lib_id "power:+5V") (at 196.85 56.515 0) (unit 1)
     (in_bom yes) (on_board yes) (fields_autoplaced)
-    (property "Reference" "#PWR?" (id 0) (at 196.85 60.325 0)
+    (property "Reference" "#PWR029" (id 0) (at 196.85 60.325 0)
       (effects (font (size 1.27 1.27)) hide)
     )
@@
   (symbol (lib_id "power:GND") (at 165.1 137.795 0) (unit 1)
     (in_bom yes) (on_board yes) (fields_autoplaced)
-    (property "Reference" "#PWR?" (id 0) (at 165.1 144.145 0)
+    (property "Reference" "#PWR045" (id 0) (at 165.1 144.145 0)
       (effects (font (size 1.27 1.27)) hide)
     )
@@
   (symbol (lib_id "power:+5V") (at 86.995 69.85 0) (unit 1)
     (in_bom yes) (on_board yes) (fields_autoplaced)
-    (property "Reference" "#PWR?" (id 0) (at 86.995 73.66 0)
+    (property "Reference" "#PWR032" (id 0) (at 86.995 73.66 0)
       (effects (font (size 1.27 1.27)) hide)
     )
@@
   (symbol (lib_id "Device:R_Small") (at 97.155 99.06 0) (unit 1)
     (in_bom yes) (on_board yes)
-    (property "Reference" "R?" (id 0) (at 98.425 97.79 0)
+    (property "Reference" "R16" (id 0) (at 98.425 97.79 0)
       (effects (font (size 1.27 1.27)) (justify left))
     )
@@
   (symbol (lib_id "power:GND") (at 165.1 66.675 0) (unit 1)
     (in_bom yes) (on_board yes) (fields_autoplaced)
-    (property "Reference" "#PWR?" (id 0) (at 165.1 73.025 0)
+    (property "Reference" "#PWR031" (id 0) (at 165.1 73.025 0)
       (effects (font (size 1.27 1.27)) hide)
     )
@@
   (symbol (lib_id "power:+5V") (at 165.1 55.88 0) (unit 1)
     (in_bom yes) (on_board yes) (fields_autoplaced)
-    (property "Reference" "#PWR?" (id 0) (at 165.1 59.69 0)
+    (property "Reference" "#PWR028" (id 0) (at 165.1 59.69 0)
       (effects (font (size 1.27 1.27)) hide)
     )
@@
   (symbol (lib_id "power:+5V") (at 165.1 78.74 0) (unit 1)
     (in_bom yes) (on_board yes) (fields_autoplaced)
-    (property "Reference" "#PWR?" (id 0) (at 165.1 82.55 0)
+    (property "Reference" "#PWR034" (id 0) (at 165.1 82.55 0)
       (effects (font (size 1.27 1.27)) hide)
     )
@@
   (symbol (lib_id "Connector_Generic:Conn_02x03_Odd_Even") (at 179.07 132.08 0) (mirror x) (unit 1)
     (in_bom yes) (on_board yes) (fields_autoplaced)
-    (property "Reference" "J?" (id 0) (at 180.34 127.1072 0))
+    (property "Reference" "J7" (id 0) (at 180.34 127.1072 0))
     (property "Value" "Conn_02x03_Odd_Even" (id 1) (at 180.34 137.0529 0)
       (effects (font (size 1.27 1.27)) hide)
@@
   (symbol (lib_id "power:+5V") (at 196.85 79.375 0) (unit 1)
     (in_bom yes) (on_board yes) (fields_autoplaced)
-    (property "Reference" "#PWR?" (id 0) (at 196.85 83.185 0)
+    (property "Reference" "#PWR035" (id 0) (at 196.85 83.185 0)
       (effects (font (size 1.27 1.27)) hide)
     )
@@
   (symbol (lib_id "Symbols:PCF8575") (at 113.665 90.17 0) (unit 1)
     (in_bom yes) (on_board yes)
-    (property "Reference" "U?" (id 0) (at 106.045 63.5 0)
+    (property "Reference" "U4" (id 0) (at 106.045 63.5 0)
       (effects (font (size 1.27 1.27)) (justify left))
     )
@@
       (effects (font (size 1.27 1.27)) (justify left))
     )
-    (property "Footprint" "" (id 2) (at 113.665 115.57 0)
+    (property "Footprint" "Package_SO:SOIC-24W_7.5x15.4mm_P1.27mm" (id 2) (at 113.665 115.57 0)
       (effects (font (size 1.27 1.27)) hide)
     )
@@
   (symbol (lib_id "power:GND") (at 113.665 115.57 0) (unit 1)
     (in_bom yes) (on_board yes) (fields_autoplaced)
-    (property "Reference" "#PWR?" (id 0) (at 113.665 121.92 0)
+    (property "Reference" "#PWR042" (id 0) (at 113.665 121.92 0)
       (effects (font (size 1.27 1.27)) hide)
     )
@@
   (symbol (lib_id "power:GND") (at 86.995 74.93 0) (unit 1)
     (in_bom yes) (on_board yes) (fields_autoplaced)
-    (property "Reference" "#PWR?" (id 0) (at 86.995 81.28 0)
+    (property "Reference" "#PWR033" (id 0) (at 86.995 81.28 0)
       (effects (font (size 1.27 1.27)) hide)
     )
@@
   (symbol (lib_id "Connector_Generic:Conn_02x03_Odd_Even") (at 179.07 60.96 0) (mirror x) (unit 1)
     (in_bom yes) (on_board yes) (fields_autoplaced)
-    (property "Reference" "J?" (id 0) (at 180.34 55.9872 0))
+    (property "Reference" "J4" (id 0) (at 180.34 55.9872 0))
     (property "Value" "Conn_02x03_Odd_Even" (id 1) (at 180.34 65.9329 0)
       (effects (font (size 1.27 1.27)) hide)
@@
   (symbol (lib_id "power:+5V") (at 89.535 96.52 0) (unit 1)
     (in_bom yes) (on_board yes) (fields_autoplaced)
-    (property "Reference" "#PWR?" (id 0) (at 89.535 100.33 0)
+    (property "Reference" "#PWR037" (id 0) (at 89.535 100.33 0)
       (effects (font (size 1.27 1.27)) hide)
     )
@@
   (symbol (lib_id "power:+5V") (at 165.1 104.14 0) (unit 1)
     (in_bom yes) (on_board yes) (fields_autoplaced)
-    (property "Reference" "#PWR?" (id 0) (at 165.1 107.95 0)
+    (property "Reference" "#PWR039" (id 0) (at 165.1 107.95 0)
       (effects (font (size 1.27 1.27)) hide)
     )
@@
   (symbol (lib_id "power:GND") (at 165.1 114.935 0) (unit 1)
     (in_bom yes) (on_board yes) (fields_autoplaced)
-    (property "Reference" "#PWR?" (id 0) (at 165.1 121.285 0)
+    (property "Reference" "#PWR041" (id 0) (at 165.1 121.285 0)
       (effects (font (size 1.27 1.27)) hide)
     )
@@
   (symbol (lib_id "power:+5V") (at 113.665 62.23 0) (unit 1)
     (in_bom yes) (on_board yes) (fields_autoplaced)
-    (property "Reference" "#PWR?" (id 0) (at 113.665 66.04 0)
+    (property "Reference" "#PWR030" (id 0) (at 113.665 66.04 0)
       (effects (font (size 1.27 1.27)) hide)
     )
@@
   (symbol (lib_id "Device:C_Small") (at 86.995 72.39 0) (unit 1)
     (in_bom yes) (on_board yes) (fields_autoplaced)
-    (property "Reference" "C?" (id 0) (at 89.3191 71.5616 0)
-      (effects (font (size 1.27 1.27)) (justify left))
-    )
+    (property "Reference" "C9" (id 0) (at 89.3191 71.5616 0)
+      (effects (font (size 1.27 1.27)) (justify left))
+    )

Commit message: update
Parts:
- renumbered C9 to C401, J4 to J401, J5 to J402, J6 to J403, J7 to J404, R15 to R401, R16 to R402, U4 to U401
Changed lines of the file:
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@@
   (symbol (lib_id "power:+5V") (at 165.1 127 0) (unit 1)
     (in_bom yes) (on_board yes) (fields_autoplaced)
-    (property "Reference" "#PWR043" (id 0) (at 165.1 130.81 0)
+    (property "Reference" "#PWR0416" (id 0) (at 165.1 130.81 0)
       (effects (font (size 1.27 1.27)) hide)
     )
@@
   (symbol (lib_id "power:GND") (at 165.1 89.535 0) (unit 1)
     (in_bom yes) (on_board yes) (fields_autoplaced)
-    (property "Reference" "#PWR036" (id 0) (at 165.1 95.885 0)
+    (property "Reference" "#PWR0409" (id 0) (at 165.1 95.885 0)
       (effects (font (size 1.27 1.27)) hide)
     )
@@
   (symbol (lib_id "power:+5V") (at 196.85 127.635 0) (unit 1)
     (in_bom yes) (on_board yes) (fields_autoplaced)
-    (property "Reference" "#PWR044" (id 0) (at 196.85 131.445 0)
+    (property "Reference" "#PWR0417" (id 0) (at 196.85 131.445 0)
       (effects (font (size 1.27 1.27)) hide)
     )
@@
   (symbol (lib_id "Device:R_Small") (at 89.535 99.06 0) (unit 1)
     (in_bom yes) (on_board yes)
-    (property "Reference" "R15" (id 0) (at 90.805 97.79 0)
+    (property "Reference" "R401" (id 0) (at 90.805 97.79 0)
       (effects (font (size 1.27 1.27)) (justify left))
     )
@@
   (symbol (lib_id "Connector_Generic:Conn_02x03_Odd_Even") (at 179.07 83.82 0) (mirror x) (unit 1)
     (in_bom yes) (on_board yes) (fields_autoplaced)
-    (property "Reference" "J5" (id 0) (at 180.34 78.8472 0))
+    (property "Reference" "J402" (id 0) (at 180.34 78.8472 0))
     (property "Value" "Conn_02x03_Odd_Even" (id 1) (at 180.34 88.7929 0)
       (effects (font (size 1.27 1.27)) hide)
@@
   (symbol (lib_id "power:+5V") (at 196.85 104.775 0) (unit 1)
     (in_bom yes) (on_board yes) (fields_autoplaced)
-    (property "Reference" "#PWR040" (id 0) (at 196.85 108.585 0)
+    (property "Reference" "#PWR0413" (id 0) (at 196.85 108.585 0)
       (effects (font (size 1.27 1.27)) hide)
     )
@@
   (symbol (lib_id "power:+5V") (at 97.155 96.52 0) (unit 1)
     (in_bom yes) (on_board yes) (fields_autoplaced)
-    (property "Reference" "#PWR038" (id 0) (at 97.155 100.33 0)
+    (property "Reference" "#PWR0411" (id 0) (at 97.155 100.33 0)
       (effects (font (size 1.27 1.27)) hide)
     )
@@
   (symbol (lib_id "Connector_Generic:Conn_02x03_Odd_Even") (at 179.07 109.22 0) (mirror x) (unit 1)
     (in_bom yes) (on_board yes) (fields_autoplaced)
-    (property "Reference" "J6" (id 0) (at 180.34 104.2472 0))
+    (property "Reference" "J403" (id 0) (at 180.34 104.2472 0))
     (property "Value" "Conn_02x03_Odd_Even" (id 1) (at 180.34 114.1929 0)
       (effects (font (size 1.27 1.27)) hide)
@@
   (symbol (lib_id "power:+5V") (at 196.85 56.515 0) (unit 1)
     (in_bom yes) (on_board yes) (fields_autoplaced)
-    (property "Reference" "#PWR029" (id 0) (at 196.85 60.325 0)
+    (property "Reference" "#PWR0402" (id 0) (at 196.85 60.325 0)
       (effects (font (size 1.27 1.27)) hide)
     )
@@
   (symbol (lib_id "power:GND") (at 165.1 137.795 0) (unit 1)
     (in_bom yes) (on_board yes) (fields_autoplaced)
-    (property "Reference" "#PWR045" (id 0) (at 165.1 144.145 0)
+    (property "Reference" "#PWR0418" (id 0) (at 165.1 144.145 0)
       (effects (font (size 1.27 1.27)) hide)
     )
@@
   (symbol (lib_id "power:+5V") (at 86.995 69.85 0) (unit 1)
     (in_bom yes) (on_board yes) (fields_autoplaced)
-    (property "Reference" "#PWR032" (id 0) (at 86.995 73.66 0)
+    (property "Reference" "#PWR0405" (id 0) (at 86.995 73.66 0)
       (effects (font (size 1.27 1.27)) hide)
     )
@@
   (symbol (lib_id "Device:R_Small") (at 97.155 99.06 0) (unit 1)
     (in_bom yes) (on_board yes)
-    (property "Reference" "R16" (id 0) (at 98.425 97.79 0)
+    (property "Reference" "R402" (id 0) (at 98.425 97.79 0)
       (effects (font (size 1.27 1.27)) (justify left))
     )
@@
   (symbol (lib_id "power:GND") (at 165.1 66.675 0) (unit 1)
     (in_bom yes) (on_board yes) (fields_autoplaced)
-    (property "Reference" "#PWR031" (id 0) (at 165.1 73.025 0)
+    (property "Reference" "#PWR0404" (id 0) (at 165.1 73.025 0)
       (effects (font (size 1.27 1.27)) hide)
     )
@@
   (symbol (lib_id "power:+5V") (at 165.1 55.88 0) (unit 1)
     (in_bom yes) (on_board yes) (fields_autoplaced)
-    (property "Reference" "#PWR028" (id 0) (at 165.1 59.69 0)
+    (property "Reference" "#PWR0401" (id 0) (at 165.1 59.69 0)
       (effects (font (size 1.27 1.27)) hide)
     )
@@
   (symbol (lib_id "power:+5V") (at 165.1 78.74 0) (unit 1)
     (in_bom yes) (on_board yes) (fields_autoplaced)
-    (property "Reference" "#PWR034" (id 0) (at 165.1 82.55 0)
+    (property "Reference" "#PWR0407" (id 0) (at 165.1 82.55 0)
       (effects (font (size 1.27 1.27)) hide)
     )
@@
   (symbol (lib_id "Connector_Generic:Conn_02x03_Odd_Even") (at 179.07 132.08 0) (mirror x) (unit 1)
     (in_bom yes) (on_board yes) (fields_autoplaced)
-    (property "Reference" "J7" (id 0) (at 180.34 127.1072 0))
+    (property "Reference" "J404" (id 0) (at 180.34 127.1072 0))
     (property "Value" "Conn_02x03_Odd_Even" (id 1) (at 180.34 137.0529 0)
       (effects (font (size 1.27 1.27)) hide)
@@
   (symbol (lib_id "power:+5V") (at 196.85 79.375 0) (unit 1)
     (in_bom yes) (on_board yes) (fields_autoplaced)
-    (property "Reference" "#PWR035" (id 0) (at 196.85 83.185 0)
+    (property "Reference" "#PWR0408" (id 0) (at 196.85 83.185 0)
       (effects (font (size 1.27 1.27)) hide)
     )
@@
   (symbol (lib_id "Symbols:PCF8575") (at 113.665 90.17 0) (unit 1)
     (in_bom yes) (on_board yes)
-    (property "Reference" "U4" (id 0) (at 106.045 63.5 0)
+    (property "Reference" "U401" (id 0) (at 106.045 63.5 0)
       (effects (font (size 1.27 1.27)) (justify left))
     )
@@
   (symbol (lib_id "power:GND") (at 113.665 115.57 0) (unit 1)
     (in_bom yes) (on_board yes) (fields_autoplaced)
-    (property "Reference" "#PWR042" (id 0) (at 113.665 121.92 0)
+    (property "Reference" "#PWR0415" (id 0) (at 113.665 121.92 0)
       (effects (font (size 1.27 1.27)) hide)
     )
@@
   (symbol (lib_id "power:GND") (at 86.995 74.93 0) (unit 1)
     (in_bom yes) (on_board yes) (fields_autoplaced)
-    (property "Reference" "#PWR033" (id 0) (at 86.995 81.28 0)
+    (property "Reference" "#PWR0406" (id 0) (at 86.995 81.28 0)
       (effects (font (size 1.27 1.27)) hide)
     )
@@
   (symbol (lib_id "Connector_Generic:Conn_02x03_Odd_Even") (at 179.07 60.96 0) (mirror x) (unit 1)
     (in_bom yes) (on_board yes) (fields_autoplaced)
-    (property "Reference" "J4" (id 0) (at 180.34 55.9872 0))
+    (property "Reference" "J401" (id 0) (at 180.34 55.9872 0))
     (property "Value" "Conn_02x03_Odd_Even" (id 1) (at 180.34 65.9329 0)
       (effects (font (size 1.27 1.27)) hide)
@@
   (symbol (lib_id "power:+5V") (at 89.535 96.52 0) (unit 1)
     (in_bom yes) (on_board yes) (fields_autoplaced)
-    (property "Reference" "#PWR037" (id 0) (at 89.535 100.33 0)
+    (property "Reference" "#PWR0410" (id 0) (at 89.535 100.33 0)
       (effects (font (size 1.27 1.27)) hide)
     )
@@
   (symbol (lib_id "power:+5V") (at 165.1 104.14 0) (unit 1)
     (in_bom yes) (on_board yes) (fields_autoplaced)
-    (property "Reference" "#PWR039" (id 0) (at 165.1 107.95 0)
+    (property "Reference" "#PWR0412" (id 0) (at 165.1 107.95 0)
       (effects (font (size 1.27 1.27)) hide)
     )
@@
   (symbol (lib_id "power:GND") (at 165.1 114.935 0) (unit 1)
     (in_bom yes) (on_board yes) (fields_autoplaced)
-    (property "Reference" "#PWR041" (id 0) (at 165.1 121.285 0)
+    (property "Reference" "#PWR0414" (id 0) (at 165.1 121.285 0)
       (effects (font (size 1.27 1.27)) hide)
     )
@@
   (symbol (lib_id "power:+5V") (at 113.665 62.23 0) (unit 1)
     (in_bom yes) (on_board yes) (fields_autoplaced)
-    (property "Reference" "#PWR030" (id 0) (at 113.665 66.04 0)
+    (property "Reference" "#PWR0403" (id 0) (at 113.665 66.04 0)
       (effects (font (size 1.27 1.27)) hide)
     )
@@
   (symbol (lib_id "Device:C_Small") (at 86.995 72.39 0) (unit 1)
     (in_bom yes) (on_board yes) (fields_autoplaced)
-    (property "Reference" "C9" (id 0) (at 89.3191 71.5616 0)
-      (effects (font (size 1.27 1.27)) (justify left))
-    )
+    (property "Reference" "C401" (id 0) (at 89.3191 71.5616 0)
+      (effects (font (size 1.27 1.27)) (justify left))
+    )

Commit message: update
Parts:
- C401: JLCPCB Part # (none) -> C113803; U labosu? (none) -> ne
- J401, J402, J403, J404: JLCPCB Part # (none) -> -; Ostalo (none) -> -; U labosu? (none) -> da
- R401, R402: JLCPCB Part # (none) -> C114662; U labosu? (none) -> ne
- U401: U labosu? (none) -> da
Changed lines of the file:
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@@
+      (effects (font (size 1.27 1.27)) hide)
+    )
+    (property "JLCPCB Part #" "C114662" (id 4) (at 89.535 99.06 0)
+      (effects (font (size 1.27 1.27)) hide)
+    )
+    (property "U labosu?" "ne" (id 5) (at 89.535 99.06 0)
       (effects (font (size 1.27 1.27)) hide)
     )
@@
     )
     (property "Datasheet" "~" (id 3) (at 179.07 83.82 0)
+      (effects (font (size 1.27 1.27)) hide)
+    )
+    (property "JLCPCB Part #" "-" (id 4) (at 179.07 83.82 0)
+      (effects (font (size 1.27 1.27)) hide)
+    )
+    (property "Ostalo" "-" (id 5) (at 179.07 83.82 0)
+      (effects (font (size 1.27 1.27)) hide)
+    )
+    (property "U labosu?" "da" (id 6) (at 179.07 83.82 0)
       (effects (font (size 1.27 1.27)) hide)
     )
@@
       (effects (font (size 1.27 1.27)) hide)
     )
+    (property "JLCPCB Part #" "-" (id 4) (at 179.07 109.22 0)
+      (effects (font (size 1.27 1.27)) hide)
+    )
+    (property "Ostalo" "-" (id 5) (at 179.07 109.22 0)
+      (effects (font (size 1.27 1.27)) hide)
+    )
+    (property "U labosu?" "da" (id 6) (at 179.07 109.22 0)
+      (effects (font (size 1.27 1.27)) hide)
+    )
     (pin "1")
     (pin "2")
@@
       (effects (font (size 1.27 1.27)) hide)
     )
+    (property "JLCPCB Part #" "C114662" (id 4) (at 97.155 99.06 0)
+      (effects (font (size 1.27 1.27)) hide)
+    )
+    (property "U labosu?" "ne" (id 5) (at 97.155 99.06 0)
+      (effects (font (size 1.27 1.27)) hide)
+    )
     (pin "1")
     (pin "2")
@@
     )
     (property "Datasheet" "~" (id 3) (at 179.07 132.08 0)
+      (effects (font (size 1.27 1.27)) hide)
+    )
+    (property "JLCPCB Part #" "-" (id 4) (at 179.07 132.08 0)
+      (effects (font (size 1.27 1.27)) hide)
+    )
+    (property "Ostalo" "-" (id 5) (at 179.07 132.08 0)
+      (effects (font (size 1.27 1.27)) hide)
+    )
+    (property "U labosu?" "da" (id 6) (at 179.07 132.08 0)
       (effects (font (size 1.27 1.27)) hide)
     )
@@
     )
     (property "Datasheet" "" (id 3) (at 113.665 115.57 0)
+      (effects (font (size 1.27 1.27)) hide)
+    )
+    (property "U labosu?" "da" (id 4) (at 113.665 90.17 0)
       (effects (font (size 1.27 1.27)) hide)
     )
@@
       (effects (font (size 1.27 1.27)) hide)
     )
+    (property "JLCPCB Part #" "-" (id 4) (at 179.07 60.96 0)
+      (effects (font (size 1.27 1.27)) hide)
+    )
+    (property "Ostalo" "-" (id 5) (at 179.07 60.96 0)
+      (effects (font (size 1.27 1.27)) hide)
+    )
+    (property "U labosu?" "da" (id 6) (at 179.07 60.96 0)
+      (effects (font (size 1.27 1.27)) hide)
+    )
     (pin "1")
     (pin "2")
@@
       (effects (font (size 1.27 1.27)) hide)
     )
+    (property "U labosu?" "ne" (id 4) (at 86.995 72.39 0)
+      (effects (font (size 1.27 1.27)) hide)
+    )
+    (property "JLCPCB Part #" "C113803" (id 5) (at 86.995 72.39 0)
+      (effects (font (size 1.27 1.27)) hide)
+    )
