File: KiCad files/BoardGame/IO Expander.kicad_sch (KiCad schematic)
At the start: 8 parts, among them J401 Conn_02x03_Odd_Even, J402 Conn_02x03_Odd_Even, J403 Conn_02x03_Odd_Even, J404 Conn_02x03_Odd_Even, U401 PCF8575

Commit message: update
Parts:
- added J405, J406, J407, J408: Conn_01x02_Female, Connector_PinHeader_1.27mm:PinHeader_1x02_P1.27mm_Vertical, symbol Connector:Conn_01x02_Female
Connections:
- net +5V: now also J406.1 (Pin_1), J406.2 (Pin_2)
- net GND: now also J405.1 (Pin_1), J405.2 (Pin_2)
- net TP_13: now reaches U401.17 (P14)
- net TP_13: now also J408.1 (Pin_1), J408.2 (Pin_2)
- no-connect marks 7 -> 8
Changed lines of the file:
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@@
   (junction (at 97.155 110.49) (diameter 0) (color 0 0 0 0)
   )
+  (junction (at 217.805 60.325) (diameter 0) (color 0 0 0 0)
+  )
   (junction (at 89.535 107.95) (diameter 0) (color 0 0 0 0)
+  )
+  (junction (at 242.57 62.865) (diameter 0) (color 0 0 0 0)
+  )
+  (junction (at 219.71 67.945) (diameter 0) (color 0 0 0 0)
   )
   (no_connect (at 103.505 90.17))
   (no_connect (at 123.825 107.95))
+  (no_connect (at 258.445 62.865))
+  (no_connect (at 258.445 60.325))
   (no_connect (at 103.505 87.63))
   (no_connect (at 123.825 105.41))
   (no_connect (at 123.825 110.49))
-  (no_connect (at 123.825 102.87))
   (no_connect (at 103.505 92.71))
   (wire (pts (xy 86.36 107.95) (xy 89.535 107.95))
@@
     (stroke (width 0) (type default) (color 0 0 0 0))
   )
+  (wire (pts (xy 220.98 69.215) (xy 219.71 69.215))
+    (stroke (width 0) (type default) (color 0 0 0 0))
+  )
+  (wire (pts (xy 242.57 60.325) (xy 242.57 62.865))
+    (stroke (width 0) (type default) (color 0 0 0 0))
+  )
   (wire (pts (xy 165.1 86.36) (xy 165.1 89.535))
     (stroke (width 0) (type default) (color 0 0 0 0))
   )
+  (wire (pts (xy 242.57 62.865) (xy 242.57 64.77))
+    (stroke (width 0) (type default) (color 0 0 0 0))
+  )
+  (wire (pts (xy 217.805 60.325) (xy 217.805 62.865))
+    (stroke (width 0) (type default) (color 0 0 0 0))
+  )
   (wire (pts (xy 196.85 132.08) (xy 186.69 132.08))
     (stroke (width 0) (type default) (color 0 0 0 0))
@@
     (stroke (width 0) (type default) (color 0 0 0 0))
   )
+  (wire (pts (xy 217.805 57.785) (xy 217.805 60.325))
+    (stroke (width 0) (type default) (color 0 0 0 0))
+  )
   (wire (pts (xy 165.1 109.22) (xy 165.1 104.14))
     (stroke (width 0) (type default) (color 0 0 0 0))
   )
+  (wire (pts (xy 219.71 69.215) (xy 219.71 67.945))
+    (stroke (width 0) (type default) (color 0 0 0 0))
+  )
   (wire (pts (xy 97.155 101.6) (xy 97.155 110.49))
     (stroke (width 0) (type default) (color 0 0 0 0))
@@
     (stroke (width 0) (type default) (color 0 0 0 0))
   )
+  (wire (pts (xy 217.805 60.325) (xy 220.98 60.325))
+    (stroke (width 0) (type default) (color 0 0 0 0))
+  )
   (wire (pts (xy 173.99 86.36) (xy 165.1 86.36))
     (stroke (width 0) (type default) (color 0 0 0 0))
@@
     (stroke (width 0) (type default) (color 0 0 0 0))
   )
+  (wire (pts (xy 242.57 62.865) (xy 245.745 62.865))
+    (stroke (width 0) (type default) (color 0 0 0 0))
+  )
+  (wire (pts (xy 242.57 60.325) (xy 245.745 60.325))
+    (stroke (width 0) (type default) (color 0 0 0 0))
+  )
   (wire (pts (xy 97.155 110.49) (xy 103.505 110.49))
     (stroke (width 0) (type default) (color 0 0 0 0))
@@
     (stroke (width 0) (type default) (color 0 0 0 0))
   )
+  (wire (pts (xy 219.71 67.945) (xy 219.71 66.675))
+    (stroke (width 0) (type default) (color 0 0 0 0))
+  )
   (wire (pts (xy 173.99 111.76) (xy 165.1 111.76))
     (stroke (width 0) (type default) (color 0 0 0 0))
   )
+  (wire (pts (xy 217.805 67.945) (xy 219.71 67.945))
+    (stroke (width 0) (type default) (color 0 0 0 0))
+  )
+  (wire (pts (xy 219.71 66.675) (xy 220.98 66.675))
+    (stroke (width 0) (type default) (color 0 0 0 0))
+  )
   (wire (pts (xy 165.1 83.82) (xy 165.1 78.74))
     (stroke (width 0) (type default) (color 0 0 0 0))
   )
+  (wire (pts (xy 217.805 62.865) (xy 220.98 62.865))
+    (stroke (width 0) (type default) (color 0 0 0 0))
+  )
   (global_label "TP_8" (shape input) (at 123.825 85.09 0) (fields_autoplaced)
     (effects (font (size 1.27 1.27)) (justify left))
     (property "Intersheet References" "${INTERSHEET_REFS}" (id 0) (at 130.564 85.0106 0)
+      (effects (font (size 1.27 1.27)) (justify left) hide)
+    )
+  )
+  (global_label "TP_13" (shape input) (at 123.825 102.87 0) (fields_autoplaced)
+    (effects (font (size 1.27 1.27)) (justify left))
+    (property "Intersheet References" "${INTERSHEET_REFS}" (id 0) (at 131.8624 102.7906 0)
       (effects (font (size 1.27 1.27)) (justify left) hide)
     )
@@
     )
   )
+  (global_label "TP_13" (shape input) (at 217.805 67.945 180) (fields_autoplaced)
+    (effects (font (size 1.27 1.27)) (justify right))
+    (property "Intersheet References" "${INTERSHEET_REFS}" (id 0) (at 209.7676 68.0244 0)
+      (effects (font (size 1.27 1.27)) (justify right) hide)
+    )
+  )
   (global_label "TP_1" (shape input) (at 186.69 63.5 0) (fields_autoplaced)
     (effects (font (size 1.27 1.27)) (justify left))
@@
     (pin "1")
   )
+  (symbol (lib_id "Connector:Conn_01x02_Female") (at 263.525 60.325 0) (unit 1)
+    (in_bom yes) (on_board yes) (fields_autoplaced)
+    (property "Reference" "J407" (id 0) (at 264.2362 62.0288 0)
+      (effects (font (size 1.27 1.27)) (justify left))
+    )
+    (property "Value" "Conn_01x02_Female" (id 1) (at 264.2362 63.2972 0)
+      (effects (font (size 1.27 1.27)) (justify left) hide)
+    )
+    (property "Footprint" "Connector_PinHeader_1.27mm:PinHeader_1x02_P1.27mm_Vertical" (id 2) (at 263.525 60.325 0)
+      (effects (font (size 1.27 1.27)) hide)
+    )
+    (property "Datasheet" "~" (id 3) (at 263.525 60.325 0)
+      (effects (font (size 1.27 1.27)) hide)
+    )
+    (pin "1")
+    (pin "2")
+  )
   (symbol (lib_id "Device:R_Small") (at 89.535 99.06 0) (unit 1)
     (in_bom yes) (on_board yes)
@@
     (pin "6")
   )
+  (symbol (lib_id "power:+5V") (at 217.805 57.785 0) (unit 1)
+    (in_bom yes) (on_board yes) (fields_autoplaced)
+    (property "Reference" "#PWR0419" (id 0) (at 217.805 61.595 0)
+      (effects (font (size 1.27 1.27)) hide)
+    )
+    (property "Value" "+5V" (id 1) (at 217.805 54.2092 0))
+    (property "Footprint" "" (id 2) (at 217.805 57.785 0)
+      (effects (font (size 1.27 1.27)) hide)
+    )
+    (property "Datasheet" "" (id 3) (at 217.805 57.785 0)
+      (effects (font (size 1.27 1.27)) hide)
+    )
+    (pin "1")
+  )
+  (symbol (lib_id "Connector:Conn_01x02_Female") (at 250.825 60.325 0) (unit 1)
+    (in_bom yes) (on_board yes) (fields_autoplaced)
+    (property "Reference" "J405" (id 0) (at 251.5362 62.0288 0)
+      (effects (font (size 1.27 1.27)) (justify left))
+    )
+    (property "Value" "Conn_01x02_Female" (id 1) (at 251.5362 63.2972 0)
+      (effects (font (size 1.27 1.27)) (justify left) hide)
+    )
+    (property "Footprint" "Connector_PinHeader_1.27mm:PinHeader_1x02_P1.27mm_Vertical" (id 2) (at 250.825 60.325 0)
+      (effects (font (size 1.27 1.27)) hide)
+    )
+    (property "Datasheet" "~" (id 3) (at 250.825 60.325 0)
+      (effects (font (size 1.27 1.27)) hide)
+    )
+    (pin "1")
+    (pin "2")
+  )
   (symbol (lib_id "power:+5V") (at 196.85 56.515 0) (unit 1)
     (in_bom yes) (on_board yes) (fields_autoplaced)
@@
     (pin "5")
     (pin "6")
+  )
+  (symbol (lib_id "Connector:Conn_01x02_Female") (at 226.06 60.325 0) (unit 1)
+    (in_bom yes) (on_board yes) (fields_autoplaced)
+    (property "Reference" "J406" (id 0) (at 226.7712 62.0288 0)
+      (effects (font (size 1.27 1.27)) (justify left))
+    )
+    (property "Value" "Conn_01x02_Female" (id 1) (at 226.7712 63.2972 0)
+      (effects (font (size 1.27 1.27)) (justify left) hide)
+    )
+    (property "Footprint" "Connector_PinHeader_1.27mm:PinHeader_1x02_P1.27mm_Vertical" (id 2) (at 226.06 60.325 0)
+      (effects (font (size 1.27 1.27)) hide)
+    )
+    (property "Datasheet" "~" (id 3) (at 226.06 60.325 0)
+      (effects (font (size 1.27 1.27)) hide)
+    )
+    (pin "1")
+    (pin "2")
   )
   (symbol (lib_id "power:+5V") (at 196.85 79.375 0) (unit 1)
@@
       (effects (font (size 1.27 1.27)) hide)
     )
+    (pin "1")
+  )
+  (symbol (lib_id "Connector:Conn_01x02_Female") (at 226.06 66.675 0) (unit 1)
+    (in_bom yes) (on_board yes) (fields_autoplaced)
+    (property "Reference" "J408" (id 0) (at 226.7712 68.3788 0)
+      (effects (font (size 1.27 1.27)) (justify left))
+    )
+    (property "Value" "Conn_01x02_Female" (id 1) (at 226.7712 69.6472 0)
+      (effects (font (size 1.27 1.27)) (justify left) hide)
+    )
+    (property "Footprint" "Connector_PinHeader_1.27mm:PinHeader_1x02_P1.27mm_Vertical" (id 2) (at 226.06 66.675 0)
+      (effects (font (size 1.27 1.27)) hide)
+    )
+    (property "Datasheet" "~" (id 3) (at 226.06 66.675 0)
+      (effects (font (size 1.27 1.27)) hide)
+    )
+    (pin "1")
+    (pin "2")
+  )
+  (symbol (lib_id "power:GND") (at 242.57 64.77 0) (unit 1)
+    (in_bom yes) (on_board yes) (fields_autoplaced)
+    (property "Reference" "#PWR0420" (id 0) (at 242.57 71.12 0)
+      (effects (font (size 1.27 1.27)) hide)
+    )
+    (property "Value" "GND" (id 1) (at 242.57 69.2134 0))
+    (property "Footprint" "" (id 2) (at 242.57 64.77 0)
+      (effects (font (size 1.27 1.27)) hide)
+    )
+    (property "Datasheet" "" (id 3) (at 242.57 64.77 0)
+      (effects (font (size 1.27 1.27)) hide)
+    )

Commit message: Documentation
Parts:
- R401, R402: value 2k2 -> 4k7
Other:
- note added: "Dice touchpad connectors"
- note added: "PCF8575 I/O Expander"
- note added: "Touchpad connectors"
- moved on the sheet: C401, J401, J402, J403, J404, J405, J406, J407, J408, R401, R402, U401

Commit message: Schematic update
Parts:
- renumbered J406 to J405, J405 to J406
Changed lines of the file:
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@@
-    )
-  )
-  (global_label "SDA" (shape input) (at 59.055 107.95 180) (fields_autoplaced)
-    (effects (font (size 1.27 1.27)) (justify right))
-    (property "Intersheet References" "${INTERSHEET_REFS}" (id 0) (at 53.1627 107.8706 0)
-      (effects (font (size 1.27 1.27)) (justify right) hide)
     )
   )
@@
     (property "Intersheet References" "${INTERSHEET_REFS}" (id 0) (at 180.094 51.3556 0)
       (effects (font (size 1.27 1.27)) (justify left) hide)
-    )
-  )
-  (global_label "SCL" (shape input) (at 59.055 105.41 180) (fields_autoplaced)
-    (effects (font (size 1.27 1.27)) (justify right))
-    (property "Intersheet References" "${INTERSHEET_REFS}" (id 0) (at 53.2232 105.3306 0)
-      (effects (font (size 1.27 1.27)) (justify right) hide)
     )
   )
@@
     )
   )
-  (global_label "INT" (shape input) (at 76.2 64.77 180) (fields_autoplaced)
-    (effects (font (size 1.27 1.27)) (justify right))
-    (property "Intersheet References" "${INTERSHEET_REFS}" (id 0) (at 70.9729 64.6906 0)
-      (effects (font (size 1.27 1.27)) (justify right) hide)
-    )
-  )
   (global_label "TP_3" (shape input) (at 160.655 51.435 180) (fields_autoplaced)
     (effects (font (size 1.27 1.27)) (justify right))
@@
       (effects (font (size 1.27 1.27)) (justify right) hide)
     )
+  )
+  (hierarchical_label "SDA" (shape bidirectional) (at 59.055 107.95 180)
+    (effects (font (size 1.27 1.27)) (justify right))
+  )
+  (hierarchical_label "SCL" (shape input) (at 59.055 105.41 180)
+    (effects (font (size 1.27 1.27)) (justify right))
+  )
+  (hierarchical_label "INT" (shape output) (at 76.2 64.77 180)
+    (effects (font (size 1.27 1.27)) (justify right))
   )
   (symbol (lib_id "power:+5V") (at 151.765 120.015 0) (unit 1)
@@
   (symbol (lib_id "Connector:Conn_01x02_Female") (at 248.285 67.31 0) (unit 1)
     (in_bom yes) (on_board yes) (fields_autoplaced)
-    (property "Reference" "J405" (id 0) (at 248.9962 69.0138 0)
+    (property "Reference" "J406" (id 0) (at 248.9962 69.0138 0)
       (effects (font (size 1.27 1.27)) (justify left))
     )
@@
   (symbol (lib_id "Connector:Conn_01x02_Female") (at 248.285 86.36 0) (unit 1)
     (in_bom yes) (on_board yes) (fields_autoplaced)
-    (property "Reference" "J406" (id 0) (at 248.9962 88.0638 0)
-      (effects (font (size 1.27 1.27)) (justify left))
-    )
+    (property "Reference" "J405" (id 0) (at 248.9962 88.0638 0)
+      (effects (font (size 1.27 1.27)) (justify left))
+    )
