File: KiCad files/BoardGame/Neopixel.kicad_sch (KiCad schematic)
At the start: 5 parts

Commit message: update
Parts:
- added D701, D702, D703, D704, D705, D706, D707, D708, D709, D710, D711, D712, D713, D714, D715, D716, D717, D718, D719, D720, D721, D722, D723, D724, D725, D726, D727, D728, D729, D730, D731, D732, D733, D734, D735, D736, D737, D738, D739, D740, D741, D742, D743, D744, D745, D746, D747, D748, D749, D750, D751, D752: WS2812B, LED_SMD:LED_WS2812B_PLCC4_5.0x5.0mm_P3.2mm, symbol LED:WS2812B
- renumbered R20 to R701, R22 to R702, R23 to R703, R24 to R704, R21 to R705
Connections:
- net at R705.2: now also D701.4 (DIN)
- new net: D717.2 (DOUT), D718.4 (DIN)
- new net: D716.2 (DOUT), D717.4 (DIN)
- new net: D723.2 (DOUT), D724.4 (DIN)
- new net: D722.2 (DOUT), D723.4 (DIN)
- new net: D709.2 (DOUT), D710.4 (DIN)
- new net: D708.2 (DOUT), D709.4 (DIN)
- new net: D710.2 (DOUT), D711.4 (DIN)
- new net: D714.2 (DOUT), D715.4 (DIN)
- new net: D713.2 (DOUT), D714.4 (DIN)
- new net: D740.2 (DOUT), D741.4 (DIN)
- new net: D739.2 (DOUT), D740.4 (DIN)
- new net: D707.2 (DOUT), D708.4 (DIN)
- new net: D706.2 (DOUT), D707.4 (DIN)
- new net: D721.2 (DOUT), D722.4 (DIN)
- new net: D720.2 (DOUT), D721.4 (DIN)
- new net: D749.2 (DOUT), D750.4 (DIN)
- new net: D748.2 (DOUT), D749.4 (DIN)
- new net: D705.2 (DOUT), D706.4 (DIN)
- new net: D704.2 (DOUT), D705.4 (DIN)
- new net: D719.2 (DOUT), D720.4 (DIN)
- new net: D718.2 (DOUT), D719.4 (DIN)
- new net: D712.2 (DOUT), D713.4 (DIN)
- new net: D711.2 (DOUT), D712.4 (DIN)
- new net: D747.2 (DOUT), D748.4 (DIN)
- new net: D746.2 (DOUT), D747.4 (DIN)
- new net: D703.2 (DOUT), D704.4 (DIN)
- new net: D715.2 (DOUT), D716.4 (DIN)
- new net: D731.2 (DOUT), D732.4 (DIN)
- new net: D730.2 (DOUT), D731.4 (DIN)
- new net: D744.2 (DOUT), D745.4 (DIN)
- new net: D743.2 (DOUT), D744.4 (DIN)
- new net: D734.2 (DOUT), D735.4 (DIN)
- new net: D733.2 (DOUT), D734.4 (DIN)
- new net: D737.2 (DOUT), D738.4 (DIN)
- new net: D736.2 (DOUT), D737.4 (DIN)
- new net: D701.2 (DOUT), D702.4 (DIN)
- new net: D738.2 (DOUT), D739.4 (DIN)
- new net: D729.2 (DOUT), D730.4 (DIN)
- new net: D728.2 (DOUT), D729.4 (DIN)
- new net: D735.2 (DOUT), D736.4 (DIN)
- new net: D732.2 (DOUT), D733.4 (DIN)
- new net: D750.2 (DOUT), D751.4 (DIN)
- new net: D741.2 (DOUT), D742.4 (DIN)
- new net: D726.2 (DOUT), D727.4 (DIN)
- new net: D725.2 (DOUT), D726.4 (DIN)
- new net: D724.2 (DOUT), D725.4 (DIN)
- new net: D742.2 (DOUT), D743.4 (DIN)
- new net: D727.2 (DOUT), D728.4 (DIN)
- new net: D745.2 (DOUT), D746.4 (DIN)
- new net: D702.2 (DOUT), D703.4 (DIN)
- new net: D751.2 (DOUT), D752.4 (DIN)
- new net GND: D701.3 (VSS), D702.3 (VSS), D703.3 (VSS), D704.3 (VSS), D705.3 (VSS), D706.3 (VSS), D707.3 (VSS), D708.3 (VSS), D709.3 (VSS), D710.3 (VSS), D711.3 (VSS), D712.3 (VSS), D713.3 (VSS), D714.3 (VSS), D715.3 (VSS), D716.3 (VSS), D717.3 (VSS), D718.3 (VSS), D719.3 (VSS), D720.3 (VSS), D721.3 (VSS), D722.3 (VSS), D723.3 (VSS), D724.3 (VSS), D725.3 (VSS), D726.3 (VSS), D727.3 (VSS), D728.3 (VSS), D729.3 (VSS), D730.3 (VSS), D731.3 (VSS), D732.3 (VSS), D733.3 (VSS), D734.3 (VSS), D735.3 (VSS), D736.3 (VSS), D737.3 (VSS), D738.3 (VSS), D739.3 (VSS), D740.3 (VSS), D741.3 (VSS), D742.3 (VSS), D743.3 (VSS), D744.3 (VSS), D745.3 (VSS), D746.3 (VSS), D747.3 (VSS), D748.3 (VSS), D749.3 (VSS), D750.3 (VSS), D751.3 (VSS), D752.3 (VSS)
- new net VCC: D701.1 (VDD), D702.1 (VDD), D703.1 (VDD), D704.1 (VDD), D705.1 (VDD), D706.1 (VDD), D707.1 (VDD), D708.1 (VDD), D709.1 (VDD), D710.1 (VDD), D711.1 (VDD), D712.1 (VDD), D713.1 (VDD), D714.1 (VDD), D715.1 (VDD), D716.1 (VDD), D717.1 (VDD), D718.1 (VDD), D719.1 (VDD), D720.1 (VDD), D721.1 (VDD), D722.1 (VDD), D723.1 (VDD), D724.1 (VDD), D725.1 (VDD), D726.1 (VDD), D727.1 (VDD), D728.1 (VDD), D729.1 (VDD), D730.1 (VDD), D731.1 (VDD), D732.1 (VDD), D733.1 (VDD), D734.1 (VDD), D735.1 (VDD), D736.1 (VDD), D737.1 (VDD), D738.1 (VDD), D739.1 (VDD), D740.1 (VDD), D741.1 (VDD), D742.1 (VDD), D743.1 (VDD), D744.1 (VDD), D745.1 (VDD), D746.1 (VDD), D747.1 (VDD), D748.1 (VDD), D749.1 (VDD), D750.1 (VDD), D751.1 (VDD), D752.1 (VDD)
- no-connect marks 5 -> 9
Other:
- moved on the sheet: R701, R702, R703, R704, R705

Commit message: update
Parts:
- removed R702, R704: 470R, Resistor_SMD:R_0603_1608Metric, symbol Device:R_Small
- added C1001, C1002, C1003, C1004, C1005, C1006, C1007, C1008, C1009: 100n, Capacitor_SMD:C_0603_1608Metric, symbol Device:C_Small
- added D1053, D1054, D1055, D1056, D1057, D1058, D1059, D1060, D1061, D1062, D1063, D1064, D1065, D1066, D1067, D1068, D1069, D1070, D1071, D1072, D1073, D1074, D1075, D1076, D1077, D1078, D1079, D1080, D1081, D1082, D1083, D1084, D1085, D1086, D1087, D1088, D1089, D1090, D1091, D1092, D1093, D1094, D1095, D1096: WS2812B, LED_SMD:LED_WS2812B_PLCC4_5.0x5.0mm_P3.2mm, symbol LED:WS2812B
- added D1097, D1098, D1099, D1100, D1101, D1102, D1103, D1104, D1105: WS2812B, Footprints:WS2812-mini, symbol LED:WS2812B
- added R1085, R1086: 470R, Resistor_SMD:R_0603_1608Metric, symbol Device:R_Small
- D1001: renamed from D701; JLCPCB Part # (none) -> -; Ostalo (none) -> forma; U labosu? (none) -> ne
- D1002: renamed from D702; JLCPCB Part # (none) -> -; Ostalo (none) -> forma; U labosu? (none) -> ne
- D1003: renamed from D703; JLCPCB Part # (none) -> -; Ostalo (none) -> forma; U labosu? (none) -> ne
- D1004: renamed from D704; JLCPCB Part # (none) -> -; Ostalo (none) -> forma; U labosu? (none) -> ne
- D1005: renamed from D705; JLCPCB Part # (none) -> -; Ostalo (none) -> forma; U labosu? (none) -> ne
- D1006: renamed from D706; JLCPCB Part # (none) -> -; Ostalo (none) -> forma; U labosu? (none) -> ne
- D1007: renamed from D707; JLCPCB Part # (none) -> -; Ostalo (none) -> forma; U labosu? (none) -> ne
- D1008: renamed from D708; JLCPCB Part # (none) -> -; Ostalo (none) -> forma; U labosu? (none) -> ne
- D1009: renamed from D709; JLCPCB Part # (none) -> -; Ostalo (none) -> forma; U labosu? (none) -> ne
- D1010: renamed from D710; JLCPCB Part # (none) -> -; Ostalo (none) -> forma; U labosu? (none) -> ne
- D1011: renamed from D711; JLCPCB Part # (none) -> -; Ostalo (none) -> forma; U labosu? (none) -> ne
- D1012: renamed from D712; JLCPCB Part # (none) -> -; Ostalo (none) -> forma; U labosu? (none) -> ne
- D1013: renamed from D713; JLCPCB Part # (none) -> -; Ostalo (none) -> forma; U labosu? (none) -> ne
- D1014: renamed from D714; JLCPCB Part # (none) -> -; Ostalo (none) -> forma; U labosu? (none) -> ne
- D1015: renamed from D715; JLCPCB Part # (none) -> -; Ostalo (none) -> forma; U labosu? (none) -> ne
- D1016: renamed from D716; JLCPCB Part # (none) -> -; Ostalo (none) -> forma; U labosu? (none) -> ne
- D1017: renamed from D717; JLCPCB Part # (none) -> -; Ostalo (none) -> forma; U labosu? (none) -> ne
- D1018: renamed from D718; JLCPCB Part # (none) -> -; Ostalo (none) -> forma; U labosu? (none) -> ne
- D1019: renamed from D719; JLCPCB Part # (none) -> -; Ostalo (none) -> forma; U labosu? (none) -> ne
- D1020: renamed from D720; JLCPCB Part # (none) -> -; Ostalo (none) -> forma; U labosu? (none) -> ne
- D1021: renamed from D721; JLCPCB Part # (none) -> -; Ostalo (none) -> forma; U labosu? (none) -> ne
- D1022: renamed from D722; JLCPCB Part # (none) -> -; Ostalo (none) -> forma; U labosu? (none) -> ne
- D1023: renamed from D723; JLCPCB Part # (none) -> -; Ostalo (none) -> forma; U labosu? (none) -> ne
- D1024: renamed from D724; JLCPCB Part # (none) -> -; Ostalo (none) -> forma; U labosu? (none) -> ne
- D1025: renamed from D725; JLCPCB Part # (none) -> -; Ostalo (none) -> forma; U labosu? (none) -> ne
- D1026: renamed from D726; JLCPCB Part # (none) -> -; Ostalo (none) -> forma; U labosu? (none) -> ne
- D1027: renamed from D727; JLCPCB Part # (none) -> -; Ostalo (none) -> forma; U labosu? (none) -> ne
- D1028: renamed from D728; JLCPCB Part # (none) -> -; Ostalo (none) -> forma; U labosu? (none) -> ne
- D1029: renamed from D729; JLCPCB Part # (none) -> -; Ostalo (none) -> forma; U labosu? (none) -> ne
- D1030: renamed from D730; JLCPCB Part # (none) -> -; Ostalo (none) -> forma; U labosu? (none) -> ne
- D1031: renamed from D731; JLCPCB Part # (none) -> -; Ostalo (none) -> forma; U labosu? (none) -> ne
- D1032: renamed from D732; JLCPCB Part # (none) -> -; Ostalo (none) -> forma; U labosu? (none) -> ne
- D1033: renamed from D733; JLCPCB Part # (none) -> -; Ostalo (none) -> forma; U labosu? (none) -> ne
- D1034: renamed from D734; JLCPCB Part # (none) -> -; Ostalo (none) -> forma; U labosu? (none) -> ne
- D1035: renamed from D735; JLCPCB Part # (none) -> -; Ostalo (none) -> forma; U labosu? (none) -> ne
- D1036: renamed from D736; JLCPCB Part # (none) -> -; Ostalo (none) -> forma; U labosu? (none) -> ne
- D1037: renamed from D737; JLCPCB Part # (none) -> -; Ostalo (none) -> forma; U labosu? (none) -> ne
- D1038: renamed from D738; JLCPCB Part # (none) -> -; Ostalo (none) -> forma; U labosu? (none) -> ne
- D1039: renamed from D739; JLCPCB Part # (none) -> -; Ostalo (none) -> forma; U labosu? (none) -> ne
- D1040: renamed from D740; JLCPCB Part # (none) -> -; Ostalo (none) -> forma; U labosu? (none) -> ne
- D1041: renamed from D741; JLCPCB Part # (none) -> -; Ostalo (none) -> forma; U labosu? (none) -> ne
- D1042: renamed from D742; JLCPCB Part # (none) -> -; Ostalo (none) -> forma; U labosu? (none) -> ne
- D1043: renamed from D743; JLCPCB Part # (none) -> -; Ostalo (none) -> forma; U labosu? (none) -> ne
- D1044: renamed from D744; JLCPCB Part # (none) -> -; Ostalo (none) -> forma; U labosu? (none) -> ne
- D1045: renamed from D745; JLCPCB Part # (none) -> -; Ostalo (none) -> forma; U labosu? (none) -> ne
- D1046: renamed from D746; JLCPCB Part # (none) -> -; Ostalo (none) -> forma; U labosu? (none) -> ne
- D1047: renamed from D747; JLCPCB Part # (none) -> -; Ostalo (none) -> forma; U labosu? (none) -> ne
- D1048: renamed from D748; JLCPCB Part # (none) -> -; Ostalo (none) -> forma; U labosu? (none) -> ne
- D1049: renamed from D749; JLCPCB Part # (none) -> -; Ostalo (none) -> forma; U labosu? (none) -> ne
- D1050: renamed from D750; JLCPCB Part # (none) -> -; Ostalo (none) -> forma; U labosu? (none) -> ne
- D1051: renamed from D751; JLCPCB Part # (none) -> -; Ostalo (none) -> forma; U labosu? (none) -> ne
- D1052: renamed from D752; JLCPCB Part # (none) -> -; Ostalo (none) -> forma; U labosu? (none) -> ne
- R1001: renamed from R701; U labosu? (none) -> da
- R1003: renamed from R703; U labosu? (none) -> da
- R1005: renamed from R705; U labosu? (none) -> da
Connections:
- net GND: now also C1001.2, C1002.2, C1003.2, C1004.2, C1005.2, C1006.2, C1007.2, C1008.2, C1009.2, D1053.3 (VSS), D1054.3 (VSS), D1055.3 (VSS), D1056.3 (VSS), D1057.3 (VSS), D1058.3 (VSS), D1059.3 (VSS), D1060.3 (VSS), D1061.3 (VSS), D1062.3 (VSS), D1063.3 (VSS), D1064.3 (VSS), D1065.3 (VSS), D1066.3 (VSS), D1067.3 (VSS), D1068.3 (VSS), D1069.3 (VSS), D1070.3 (VSS), D1071.3 (VSS), D1072.3 (VSS), D1073.3 (VSS), D1074.3 (VSS), D1075.3 (VSS), D1076.3 (VSS), D1077.3 (VSS), D1078.3 (VSS), D1079.3 (VSS), D1080.3 (VSS), D1081.3 (VSS), D1082.3 (VSS), D1083.3 (VSS), D1084.3 (VSS), D1085.3 (VSS), D1086.3 (VSS), D1087.3 (VSS), D1088.3 (VSS), D1089.3 (VSS), D1090.3 (VSS), D1091.3 (VSS), D1092.3 (VSS), D1093.3 (VSS), D1094.3 (VSS), D1095.3 (VSS), D1096.3 (VSS), D1097.3 (VSS), D1098.3 (VSS), D1099.3 (VSS), D1100.3 (VSS), D1101.3 (VSS), D1102.3 (VSS), D1103.3 (VSS), D1104.3 (VSS), D1105.3 (VSS)
- net NP_3: now also R1086.1
- net NP_5: now also R1085.1
- net VCC: now also C1001.1, C1002.1, C1003.1, C1004.1, C1005.1, C1006.1, C1007.1, C1008.1, C1009.1, D1053.1 (VDD), D1054.1 (VDD), D1055.1 (VDD), D1056.1 (VDD), D1057.1 (VDD), D1058.1 (VDD), D1059.1 (VDD), D1060.1 (VDD), D1061.1 (VDD), D1062.1 (VDD), D1063.1 (VDD), D1064.1 (VDD), D1065.1 (VDD), D1066.1 (VDD), D1067.1 (VDD), D1068.1 (VDD), D1069.1 (VDD), D1070.1 (VDD), D1071.1 (VDD), D1072.1 (VDD), D1073.1 (VDD), D1074.1 (VDD), D1075.1 (VDD), D1076.1 (VDD), D1077.1 (VDD), D1078.1 (VDD), D1079.1 (VDD), D1080.1 (VDD), D1081.1 (VDD), D1082.1 (VDD), D1083.1 (VDD), D1084.1 (VDD), D1085.1 (VDD), D1086.1 (VDD), D1087.1 (VDD), D1088.1 (VDD), D1089.1 (VDD), D1090.1 (VDD), D1091.1 (VDD), D1092.1 (VDD), D1093.1 (VDD), D1094.1 (VDD), D1095.1 (VDD), D1096.1 (VDD), D1097.1 (VDD), D1098.1 (VDD), D1099.1 (VDD), D1100.1 (VDD), D1101.1 (VDD), D1102.1 (VDD), D1103.1 (VDD), D1104.1 (VDD), D1105.1 (VDD)
- net at R1001.2: now also D1069.4 (DIN)
- net at R1003.2: now also D1053.4 (DIN)
- new net: D1100.2 (DOUT), D1101.4 (DIN)
- new net: D1099.2 (DOUT), D1100.4 (DIN)
- new net: D1069.2 (DOUT), D1070.4 (DIN)
- new net: D1075.2 (DOUT), D1076.4 (DIN)
- new net: D1074.2 (DOUT), D1075.4 (DIN)
- new net: D1072.2 (DOUT), D1073.4 (DIN)
- new net: D1071.2 (DOUT), D1072.4 (DIN)
- new net: D1094.4 (DIN), R1086.2
- new net: D1080.2 (DOUT), D1081.4 (DIN)
- new net: D1079.2 (DOUT), D1080.4 (DIN)
- new net: D1092.2 (DOUT), D1093.4 (DIN)
- new net: D1091.2 (DOUT), D1092.4 (DIN)
- new net: D1094.2 (DOUT), D1095.4 (DIN)
- new net: D1060.2 (DOUT), D1061.4 (DIN)
- new net: D1059.2 (DOUT), D1060.4 (DIN)
- new net: D1067.2 (DOUT), D1068.4 (DIN)
- new net: D1066.2 (DOUT), D1067.4 (DIN)
- new net: D1065.2 (DOUT), D1066.4 (DIN)
- new net: D1064.2 (DOUT), D1065.4 (DIN)
- new net: D1085.2 (DOUT), D1086.4 (DIN)
- new net: D1085.4 (DIN), R1085.2
- new net: D1073.2 (DOUT), D1074.4 (DIN)
- new net: D1090.2 (DOUT), D1091.4 (DIN)
- new net: D1089.2 (DOUT), D1090.4 (DIN)
- new net: D1104.2 (DOUT), D1105.4 (DIN)
- new net: D1103.2 (DOUT), D1104.4 (DIN)
- new net: D1070.2 (DOUT), D1071.4 (DIN)
- new net: D1053.2 (DOUT), D1054.4 (DIN)
- new net: D1082.2 (DOUT), D1083.4 (DIN)
- new net: D1081.2 (DOUT), D1082.4 (DIN)
- new net: D1101.2 (DOUT), D1102.4 (DIN)
- new net: D1057.2 (DOUT), D1058.4 (DIN)
- new net: D1056.2 (DOUT), D1057.4 (DIN)
- new net: D1058.2 (DOUT), D1059.4 (DIN)
- new net: D1097.2 (DOUT), D1098.4 (DIN)
- new net: D1096.2 (DOUT), D1097.4 (DIN)
- new net: D1077.2 (DOUT), D1078.4 (DIN)
- new net: D1076.2 (DOUT), D1077.4 (DIN)
- new net: D1087.2 (DOUT), D1088.4 (DIN)
- new net: D1086.2 (DOUT), D1087.4 (DIN)
- new net: D1063.2 (DOUT), D1064.4 (DIN)
- new net: D1062.2 (DOUT), D1063.4 (DIN)
- new net: D1061.2 (DOUT), D1062.4 (DIN)
- new net: D1078.2 (DOUT), D1079.4 (DIN)
- new net: D1102.2 (DOUT), D1103.4 (DIN)
- new net: D1083.2 (DOUT), D1084.4 (DIN)
- new net: D1095.2 (DOUT), D1096.4 (DIN)
- new net: D1054.2 (DOUT), D1055.4 (DIN)
- new net: D1098.2 (DOUT), D1099.4 (DIN)
- new net: D1088.2 (DOUT), D1089.4 (DIN)
- new net: D1055.2 (DOUT), D1056.4 (DIN)
- no-connect marks 9 -> 5
Other:
- note removed: "ovdje idu WS2812B napajani sa VCC i mali neopixeli"
- moved on the sheet: R1001, R1003

Commit message: update
Parts:
- added D1106: WS2812B, LED_SMD:LED_WS2812B_PLCC4_5.0x5.0mm_P3.2mm, symbol LED:WS2812B
- added R1006: 470R, Resistor_SMD:R_0603_1608Metric, symbol Device:R_Small
- renumbered R1085 to R1002, R1086 to R1004
Connections:
- net GND: now also D1106.3 (VSS)
- net VCC: now also D1106.1 (VDD)
- new net: D1106.4 (DIN), R1006.2
- new net NP_6: R1006.1
- no-connect marks 5 -> 6
Changed lines of the file:
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@@
   (no_connect (at 520.7 186.69))
   (no_connect (at 471.17 156.845))
+  (no_connect (at 340.36 214.63))
   (wire (pts (xy 416.56 27.305) (xy 417.83 27.305))
     (stroke (width 0) (type default) (color 0 0 0 0))
@@
     (stroke (width 0) (type default) (color 0 0 0 0))
   )
+  (wire (pts (xy 318.135 214.63) (xy 320.04 214.63))
+    (stroke (width 0) (type default) (color 0 0 0 0))
+  )
   (wire (pts (xy 455.295 97.155) (xy 456.565 97.155))
     (stroke (width 0) (type default) (color 0 0 0 0))
@@
     )
   )
+  (global_label "NP_6" (shape input) (at 318.135 214.63 180) (fields_autoplaced)
+    (effects (font (size 1.27 1.27)) (justify right))
+    (property "Intersheet References" "${INTERSHEET_REFS}" (id 0) (at 310.9443 214.5506 0)
+      (effects (font (size 1.27 1.27)) (justify right) hide)
+    )
+  )
   (global_label "NP_5" (shape input) (at 316.865 156.845 180) (fields_autoplaced)
     (effects (font (size 1.27 1.27)) (justify right))
@@
   (symbol (lib_id "Device:R_Small") (at 322.58 186.69 90) (unit 1)
     (in_bom yes) (on_board yes)
-    (property "Reference" "R1086" (id 0) (at 322.58 184.785 90))
+    (property "Reference" "R1004" (id 0) (at 322.58 184.785 90))
     (property "Value" "470R" (id 1) (at 322.58 188.595 90)
       (effects (font (size 1.2 1.2)))
@@
     (pin "1")
   )
+  (symbol (lib_id "LED:WS2812B") (at 332.74 214.63 0) (unit 1)
+    (in_bom yes) (on_board yes)
+    (property "Reference" "D1106" (id 0) (at 328.295 208.28 0))
+    (property "Value" "WS2812B" (id 1) (at 338.455 220.98 0)
+      (effects (font (size 1.27 1.27)) hide)
+    )
+    (property "Footprint" "LED_SMD:LED_WS2812B_PLCC4_5.0x5.0mm_P3.2mm" (id 2) (at 334.01 222.25 0)
+      (effects (font (size 1.27 1.27)) (justify left top) hide)
+    )
+    (property "Datasheet" "https://cdn-shop.adafruit.com/datasheets/WS2812B.pdf" (id 3) (at 335.28 224.155 0)
+      (effects (font (size 1.27 1.27)) (justify left top) hide)
+    )
+    (property "Ostalo" "forma" (id 4) (at 332.74 214.63 0)
+      (effects (font (size 1.27 1.27)) hide)
+    )
+    (property "U labosu?" "ne" (id 5) (at 332.74 214.63 0)
+      (effects (font (size 1.27 1.27)) hide)
+    )
+    (property "JLCPCB Part #" "-" (id 6) (at 332.74 214.63 0)
+      (effects (font (size 1.27 1.27)) hide)
+    )
+    (pin "1")
+    (pin "2")
+    (pin "3")
+    (pin "4")
+  )
   (symbol (lib_id "LED:WS2812B") (at 97.155 60.325 0) (unit 1)
     (in_bom yes) (on_board yes)
@@
     (pin "1")
   )
+  (symbol (lib_id "Device:R_Small") (at 322.58 214.63 90) (unit 1)
+    (in_bom yes) (on_board yes)
+    (property "Reference" "R1006" (id 0) (at 322.58 212.725 90))
+    (property "Value" "470R" (id 1) (at 322.58 216.535 90)
+      (effects (font (size 1.2 1.2)))
+    )
+    (property "Footprint" "Resistor_SMD:R_0603_1608Metric" (id 2) (at 322.58 214.63 0)
+      (effects (font (size 1.27 1.27)) hide)
+    )
+    (property "Datasheet" "~" (id 3) (at 322.58 214.63 0)
+      (effects (font (size 1.27 1.27)) hide)
+    )
+    (property "U labosu?" "da" (id 4) (at 322.58 214.63 0)
+      (effects (font (size 1.27 1.27)) hide)
+    )
+    (pin "1")
+    (pin "2")
+  )
   (symbol (lib_id "LED:WS2812B") (at 47.625 33.02 0) (unit 1)
     (in_bom yes) (on_board yes)
@@
     (pin "1")
   )
+  (symbol (lib_id "power:VCC") (at 332.74 207.01 0) (unit 1)
+    (in_bom yes) (on_board yes) (fields_autoplaced)
+    (property "Reference" "#PWR01169" (id 0) (at 332.74 210.82 0)
+      (effects (font (size 1.27 1.27)) hide)
+    )
+    (property "Value" "VCC" (id 1) (at 332.74 203.4342 0))
+    (property "Footprint" "" (id 2) (at 332.74 207.01 0)
+      (effects (font (size 1.27 1.27)) hide)
+    )
+    (property "Datasheet" "" (id 3) (at 332.74 207.01 0)
+      (effects (font (size 1.27 1.27)) hide)
+    )
+    (pin "1")
+  )
   (symbol (lib_id "power:GND") (at 163.195 123.19 0) (unit 1)
     (in_bom yes) (on_board yes) (fields_autoplaced)
@@
     (pin "1")
   )
+  (symbol (lib_id "power:GND") (at 332.74 222.25 0) (unit 1)
+    (in_bom yes) (on_board yes) (fields_autoplaced)
+    (property "Reference" "#PWR01170" (id 0) (at 332.74 228.6 0)
+      (effects (font (size 1.27 1.27)) hide)
+    )
+    (property "Value" "GND" (id 1) (at 332.74 226.6934 0))
+    (property "Footprint" "" (id 2) (at 332.74 222.25 0)
+      (effects (font (size 1.27 1.27)) hide)
+    )
+    (property "Datasheet" "" (id 3) (at 332.74 222.25 0)
+      (effects (font (size 1.27 1.27)) hide)
+    )
+    (pin "1")
+  )
   (symbol (lib_id "power:VCC") (at 458.47 19.685 0) (unit 1)
     (in_bom yes) (on_board yes) (fields_autoplaced)
@@
   (symbol (lib_id "Device:R_Small") (at 321.31 156.845 90) (unit 1)
     (in_bom yes) (on_board yes)
-    (property "Reference" "R1085" (id 0) (at 321.31 154.94 90))
+    (property "Reference" "R1002" (id 0) (at 321.31 154.94 90))
     (property "Value" "470R" (id 1) (at 321.31 158.75 90)
       (effects (font (size 1.2 1.2)))

Commit message: update
Connections:
- net at R1004.2: now also D1097.4 (DIN); no longer D1094.4 (DIN)
- net at D1093.2 (DOUT): now also D1094.4 (DIN)
- net at D1096.2 (DOUT): no longer D1097.4 (DIN)
Other:
- note added: "BATERIJA"
- note added: "FINISH"
- note added: "GUMBI"
- note added: "KOCKICA"
- note added: "PATH"
- note added: "SAFEHOUSE"
- moved on the sheet: C1001, C1002, C1003, C1004, C1005, C1006, C1007, C1008, C1009, D1094, D1095, D1096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

Commit message: update
Parts:
- D1001, D1002, D1003, D1004, D1005, D1006, D1007, D1008, D1009, D1010, D1011, D1012, D1013, D1014, D1015, D1016, D1017, D1018, D1019, D1020, D1021, D1022, D1023, D1024, D1025, D1026, D1027, D1028, D1029, D1030, D1031, D1032, D1033, D1034, D1035, D1036, D1037, D1038, D1039, D1040, D1041, D1042, D1043, D1044, D1045, D1046, D1047, D1048, D1049, D1050, D1051, D1052, D1053, D1054, D1055, D1056, D1057, D1058, D1059, D1060, D1061, D1062, D1063, D1064, D1065, D1066, D1067, D1068, D1069, D1070, D1071, D1072, D1073, D1074, D1075, D1076, D1077, D1078, D1079, D1080, D1081, D1082, D1083, D1084, D1085, D1086, D1087, D1088, D1089, D1090, D1091, D1092, D1093, D1094, D1095, D1096, D1106: footprint LED_SMD:LED_WS2812B_PLCC4_5.0x5.0mm_P3.2mm -> Footprints:LED_WS2812B_edited

Commit message: update
Parts:
- D1106: footprint Footprints:LED_WS2812B_edited -> Footprints:WS2812-mini
Changed lines of the file:
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@@
       (effects (font (size 1.27 1.27)) hide)
     )
-    (property "Footprint" "Footprints:LED_WS2812B_edited" (id 2) (at 334.01 222.25 0)
+    (property "Footprint" "Footprints:WS2812-mini" (id 2) (at 334.01 222.25 0)
       (effects (font (size 1.27 1.27)) (justify left top) hide)
     )

Commit message: Documentation
Parts:
- removed C1001, C1002, C1003, C1004, C1005, C1006, C1007, C1008, C1009: 100n, Capacitor_SMD:C_0603_1608Metric, symbol Device:C_Small
- removed D1001, D1002, D1003, D1004, D1005, D1006, D1007, D1008, D1009, D1010, D1011, D1012, D1013, D1014, D1015, D1016, D1017, D1018, D1019, D1020, D1021, D1022, D1023, D1024, D1025, D1026, D1027, D1028, D1029, D1030, D1031, D1032, D1033, D1034, D1035, D1036, D1037, D1038, D1039, D1040, D1041, D1042, D1043, D1044, D1045, D1046, D1047, D1048, D1049, D1050, D1051, D1052, D1053, D1054, D1055, D1056, D1057, D1058, D1059, D1060, D1061, D1062, D1063, D1064, D1065, D1066, D1067, D1068, D1069, D1070, D1071, D1072, D1073, D1074, D1075, D1076, D1077, D1078, D1079, D1080, D1081, D1082, D1083, D1084, D1085, D1086, D1087, D1088, D1089, D1090, D1091, D1092, D1093, D1094, D1095, D1096: WS2812B, Footprints:LED_WS2812B_edited, symbol LED:WS2812B
- removed D1097, D1098, D1099, D1100, D1101, D1102, D1103, D1104, D1105, D1106: WS2812B, Footprints:WS2812-mini, symbol LED:WS2812B
- removed R1001, R1002, R1003, R1004, R1005, R1006: 470R, Resistor_SMD:R_0603_1608Metric, symbol Device:R_Small
Connections:
- no-connect marks 6 -> 0
Other:
- added sheet Battery indicator LED (Battery indicator LED.kicad_sch)
- added sheet Dice LEDs (Dice LEDs.kicad_sch)
- added sheet Finish LEDs (Finish LEDs.kicad_sch)
- added sheet Path LEDs (Path LEDs.kicad_sch)
- added sheet Safehouse LEDs (Safehouse LEDs.kicad_sch)
- added sheet Touchpad LEDs (Touchpad LEDs.kicad_sch)
- note removed: "BATERIJA"
- note removed: "FINISH"
- note removed: "GUMBI"
- note removed: "KOCKICA"
- note removed: "PATH"
- note removed: "SAFEHOUSE"

Commit message: Schematic update
Other:
- removed sheet Battery indicator LED
- removed sheet Dice LEDs
- removed sheet Finish LEDs
- removed sheet Path LEDs
- removed sheet Safehouse LEDs
- removed sheet Touchpad LEDs
Changed lines of the file:
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@@
 (kicad_sch (version 20211123) (generator eeschema)
   (paper "A4")
-  (sheet (at 160.02 77.47) (size 30.48 30.48) (fields_autoplaced)
-    (stroke (width 0.1524) (type solid) (color 0 0 0 0))
-    (fill (color 255 229 191 1.0000))
-    (property "Sheet name" "Touchpad LEDs" (id 0) (at 160.02 76.7584 0)
-      (effects (font (size 1.27 1.27)) (justify left bottom))
-    )
-    (property "Sheet file" "Touchpad LEDs.kicad_sch" (id 1) (at 160.02 108.5346 0)
-      (effects (font (size 1.27 1.27)) (justify left top) hide)
-    )
-  )
-  (sheet (at 193.04 77.47) (size 30.48 30.48) (fields_autoplaced)
-    (stroke (width 0.1524) (type solid) (color 0 0 0 0))
-    (fill (color 255 229 191 1.0000))
-    (property "Sheet name" "Dice LEDs" (id 0) (at 193.04 76.7584 0)
-      (effects (font (size 1.27 1.27)) (justify left bottom))
-    )
-    (property "Sheet file" "Dice LEDs.kicad_sch" (id 1) (at 193.04 108.5346 0)
-      (effects (font (size 1.27 1.27)) (justify left top) hide)
-    )
-  )
-  (sheet (at 93.98 77.47) (size 30.48 30.48) (fields_autoplaced)
-    (stroke (width 0.1524) (type solid) (color 0 0 0 0))
-    (fill (color 255 229 191 1.0000))
-    (property "Sheet name" "Safehouse LEDs" (id 0) (at 93.98 76.7584 0)
-      (effects (font (size 1.27 1.27)) (justify left bottom))
-    )
-    (property "Sheet file" "Safehouse LEDs.kicad_sch" (id 1) (at 93.98 108.5346 0)
-      (effects (font (size 1.27 1.27)) (justify left top) hide)
-    )
-  )
-  (sheet (at 127 77.47) (size 30.48 30.48) (fields_autoplaced)
-    (stroke (width 0.1524) (type solid) (color 0 0 0 0))
-    (fill (color 255 229 191 1.0000))
-    (property "Sheet name" "Finish LEDs" (id 0) (at 127 76.7584 0)
-      (effects (font (size 1.27 1.27)) (justify left bottom))
-    )
-    (property "Sheet file" "Finish LEDs.kicad_sch" (id 1) (at 127 108.5346 0)
-      (effects (font (size 1.27 1.27)) (justify left top) hide)
-    )
-  )
-  (sheet (at 60.325 77.47) (size 30.48 30.48) (fields_autoplaced)
-    (stroke (width 0.1524) (type solid) (color 0 0 0 0))
-    (fill (color 255 229 191 1.0000))
-    (property "Sheet name" "Path LEDs" (id 0) (at 60.325 76.7584 0)
-      (effects (font (size 1.27 1.27)) (justify left bottom))
-    )
-    (property "Sheet file" "Path LEDs.kicad_sch" (id 1) (at 60.325 108.5346 0)
-      (effects (font (size 1.27 1.27)) (justify left top) hide)
-    )
-  )
-  (sheet (at 225.425 77.47) (size 30.48 30.48) (fields_autoplaced)
-    (stroke (width 0.1524) (type solid) (color 0 0 0 0))
-    (fill (color 255 229 191 1.0000))
-    (property "Sheet name" "Battery indicator LED" (id 0) (at 225.425 76.7584 0)
-      (effects (font (size 1.27 1.27)) (justify left bottom))
-    )
-    (property "Sheet file" "Battery indicator LED.kicad_sch" (id 1) (at 225.425 108.5346 0)
-      (effects (font (size 1.27 1.27)) (justify left top) hide)
-    )
-  )
 )
