File: KiCad files/BoardGame/USB.kicad_sch (KiCad schematic)
At the start: 12 parts

Commit message: update
Parts:
- C? (x2): footprint (none) -> Capacitor_SMD:C_0603_1608Metric
- C?: footprint (none) -> Capacitor_SMD:C_0603_1608Metric; Basic/Extended Basic -> (none); JLCPCB Part # C1710 -> (none); U labosu? Ne -> (none)
- C?: footprint (none) -> Capacitor_Tantalum_SMD:CP_EIA-3528-21_Kemet-B
- FB?, R? (x4): footprint (none) -> Resistor_SMD:R_0603_1608Metric
- U?: footprint (none) -> Package_SO:SOIC-16_3.9x9.9mm_P1.27mm
Other:
- title: (none) -> BoardGame
- moved on the sheet: R?
Changed lines of the file:
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@@
 (kicad_sch (version 20211123) (generator eeschema)
   (paper "A4")
+  (title_block
+    (title "BoardGame")
+    (date "2022-09-21")
+    (rev "1")
+  )
   (junction (at 59.055 82.55) (diameter 0) (color 0 0 0 0)
   )
@@
     (stroke (width 0) (type default) (color 0 0 0 0))
   )
-  (wire (pts (xy 239.395 81.28) (xy 238.125 81.28))
+  (wire (pts (xy 238.125 81.28) (xy 238.76 81.28))
+    (stroke (width 0) (type default) (color 0 0 0 0))
+  )
+  (wire (pts (xy 239.395 78.74) (xy 238.76 78.74))
     (stroke (width 0) (type default) (color 0 0 0 0))
   )
@@
   )
   (wire (pts (xy 81.28 82.55) (xy 81.28 83.82))
+    (stroke (width 0) (type default) (color 0 0 0 0))
+  )
+  (wire (pts (xy 238.76 78.74) (xy 238.76 81.28))
     (stroke (width 0) (type default) (color 0 0 0 0))
   )
@@
     )
   )
-  (global_label "RX" (shape input) (at 244.475 81.28 0) (fields_autoplaced)
-    (effects (font (size 1.27 1.27)) (justify left))
-    (property "Intersheet References" "${INTERSHEET_REFS}" (id 0) (at 86.995 7.62 0)
+  (global_label "RX" (shape input) (at 244.475 78.74 0) (fields_autoplaced)
+    (effects (font (size 1.27 1.27)) (justify left))
+    (property "Intersheet References" "${INTERSHEET_REFS}" (id 0) (at 86.995 5.08 0)
       (effects (font (size 1.27 1.27)) hide)
     )
@@
       (effects (font (size 1.27 1.27)) (justify left))
     )
-    (property "Footprint" "" (id 2) (at 255.905 78.74 0)
+    (property "Footprint" "Capacitor_SMD:C_0603_1608Metric" (id 2) (at 255.905 78.74 0)
       (effects (font (size 1.27 1.27)) hide)
     )
@@
   (symbol (lib_id "Device:C_Small") (at 243.205 99.06 270) (unit 1)
     (in_bom yes) (on_board yes)
-    (property "Reference" "C?" (id 0) (at 243.205 93.2434 90))
-    (property "Value" "100n" (id 1) (at 243.205 95.5548 90))
-    (property "Footprint" "" (id 2) (at 243.205 99.06 0)
+    (property "Reference" "C?" (id 0) (at 243.205 95.885 90))
+    (property "Value" "100n" (id 1) (at 243.205 102.235 90))
+    (property "Footprint" "Capacitor_SMD:C_0603_1608Metric" (id 2) (at 243.205 99.06 0)
       (effects (font (size 1.27 1.27)) hide)
     )
@@
       (effects (font (size 1.27 1.27)) (justify left))
     )
-    (property "Value" "1k" (id 1) (at 240.665 86.36 90)
-      (effects (font (size 0.9906 0.9906)) (justify left))
-    )
-    (property "Footprint" "" (id 2) (at 241.935 86.36 0)
+    (property "Value" "1k" (id 1) (at 240.665 88.265 90)
+      (effects (font (size 1.27 1.27)) (justify left))
+    )
+    (property "Footprint" "Resistor_SMD:R_0603_1608Metric" (id 2) (at 241.935 86.36 0)
       (effects (font (size 1.27 1.27)) hide)
     )
@@
       (effects (font (size 1.27 1.27)) (justify left))
     )
-    (property "Footprint" "" (id 2) (at 204.47 78.74 0)
+    (property "Footprint" "Capacitor_SMD:C_0603_1608Metric" (id 2) (at 204.47 78.74 0)
       (effects (font (size 1.27 1.27)) hide)
     )
     (property "Datasheet" "~" (id 3) (at 204.47 78.74 0)
-      (effects (font (size 1.27 1.27)) hide)
-    )
-    (property "Basic/Extended" "Basic" (id 4) (at 204.47 78.74 0)
-      (effects (font (size 1.27 1.27)) hide)
-    )
-    (property "JLCPCB Part #" "C1710" (id 5) (at 204.47 78.74 0)
-      (effects (font (size 1.27 1.27)) hide)
-    )
-    (property "U labosu?" "Ne" (id 6) (at 204.47 78.74 0)
       (effects (font (size 1.27 1.27)) hide)
     )
@@
   (symbol (lib_id "Device:R_Small") (at 81.28 80.01 0) (unit 1)
     (in_bom yes) (on_board yes)
-    (property "Reference" "R?" (id 0) (at 82.55 80.01 0)
-      (effects (font (size 1.27 1.27)) (justify left))
-    )
-    (property "Value" "5k1" (id 1) (at 81.28 81.28 90)
-      (effects (font (size 0.9906 0.9906)) (justify left))
-    )
-    (property "Footprint" "" (id 2) (at 81.28 80.01 0)
+    (property "Reference" "R?" (id 0) (at 82.55 78.74 0)
+      (effects (font (size 1.27 1.27)) (justify left))
+    )
+    (property "Value" "5k1" (id 1) (at 82.55 80.645 0)
+      (effects (font (size 1.27 1.27)) (justify left))
+    )
+    (property "Footprint" "Resistor_SMD:R_0603_1608Metric" (id 2) (at 81.28 80.01 0)
       (effects (font (size 1.27 1.27)) hide)
     )
@@
   (symbol (lib_id "Device:R_Small") (at 87.63 80.01 0) (unit 1)
     (in_bom yes) (on_board yes)
-    (property "Reference" "R?" (id 0) (at 88.9 80.01 0)
-      (effects (font (size 1.27 1.27)) (justify left))
-    )
-    (property "Value" "5k1" (id 1) (at 87.63 81.28 90)
-      (effects (font (size 0.9906 0.9906)) (justify left))
-    )
-    (property "Footprint" "" (id 2) (at 87.63 80.01 0)
+    (property "Reference" "R?" (id 0) (at 88.9 78.74 0)
+      (effects (font (size 1.27 1.27)) (justify left))
+    )
+    (property "Value" "5k1" (id 1) (at 88.9 80.645 0)
+      (effects (font (size 1.27 1.27)) (justify left))
+    )
+    (property "Footprint" "Resistor_SMD:R_0603_1608Metric" (id 2) (at 87.63 80.01 0)
       (effects (font (size 1.27 1.27)) hide)
     )
@@
     (property "Reference" "U?" (id 0) (at 221.615 77.47 0))
     (property "Value" "CH340C" (id 1) (at 232.41 105.41 0))
-    (property "Footprint" "" (id 2) (at 229.235 105.41 0)
+    (property "Footprint" "Package_SO:SOIC-16_3.9x9.9mm_P1.27mm" (id 2) (at 229.235 105.41 0)
       (effects (font (size 1.27 1.27)) (justify left) hide)
     )
@@
       (effects (font (size 1.27 1.27)) (justify left))
     )
-    (property "Footprint" "" (id 2) (at 267.335 78.74 0)
+    (property "Footprint" "Capacitor_Tantalum_SMD:CP_EIA-3528-21_Kemet-B" (id 2) (at 267.335 78.74 0)
       (effects (font (size 1.27 1.27)) hide)
     )
@@
     (pin "2")
   )
-  (symbol (lib_id "Device:R_Small") (at 241.935 81.28 270) (unit 1)
-    (in_bom yes) (on_board yes)
-    (property "Reference" "R?" (id 0) (at 240.665 79.375 90)
-      (effects (font (size 1.27 1.27)) (justify left))
-    )
-    (property "Value" "1k" (id 1) (at 240.665 81.28 90)
-      (effects (font (size 0.9906 0.9906)) (justify left))
-    )
-    (property "Footprint" "" (id 2) (at 241.935 81.28 0)
-      (effects (font (size 1.27 1.27)) hide)
-    )
-    (property "Datasheet" "~" (id 3) (at 241.935 81.28 0)
+  (symbol (lib_id "Device:R_Small") (at 241.935 78.74 270) (unit 1)
+    (in_bom yes) (on_board yes)
+    (property "Reference" "R?" (id 0) (at 240.665 76.835 90)
+      (effects (font (size 1.27 1.27)) (justify left))
+    )
+    (property "Value" "1k" (id 1) (at 240.665 80.645 90)
+      (effects (font (size 1.27 1.27)) (justify left))
+    )
+    (property "Footprint" "Resistor_SMD:R_0603_1608Metric" (id 2) (at 241.935 78.74 0)
+      (effects (font (size 1.27 1.27)) hide)
+    )
+    (property "Datasheet" "~" (id 3) (at 241.935 78.74 0)
       (effects (font (size 1.27 1.27)) hide)
     )
@@
     (property "Reference" "FB?" (id 0) (at 65.9892 62.2386 90))
     (property "Value" "100 @ 100MHz" (id 1) (at 65.9892 64.7755 90))
-    (property "Footprint" "" (id 2) (at 66.04 70.358 90)
-      (effects (font (size 1.27 1.27)) hide)
-    )
+    (property "Footprint" "Resistor_SMD:R_0603_1608Metric" (id 2) (at 66.04 70.358 90)
+      (effects (font (size 1.27 1.27)) hide)
+    )

Commit message: update
Parts:
- J1: renamed from J?; footprint (none) -> Footprints:USB_C_Receptacle_HRO_TYPE-C-31-M-12
- gave numbers to parts that had none: 11
Changed lines of the file:
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@@
   (symbol (lib_id "Connector:USB_C_Receptacle_USB2.0") (at 39.37 83.82 0) (unit 1)
     (in_bom yes) (on_board yes)
-    (property "Reference" "J?" (id 0) (at 30.48 64.643 0))
+    (property "Reference" "J1" (id 0) (at 30.48 64.643 0))
     (property "Value" "USB_C_Receptacle_USB2.0" (id 1) (at 42.0878 64.1096 0)
       (effects (font (size 1.27 1.27)) hide)
     )
-    (property "Footprint" "" (id 2) (at 43.18 83.82 0)
+    (property "Footprint" "Footprints:USB_C_Receptacle_HRO_TYPE-C-31-M-12" (id 2) (at 43.18 83.82 0)
       (effects (font (size 1.27 1.27)) hide)
     )
@@
   (symbol (lib_id "power:VBUS") (at 267.335 73.66 0) (unit 1)
     (in_bom yes) (on_board yes)
-    (property "Reference" "#PWR?" (id 0) (at 267.335 77.47 0)
+    (property "Reference" "#PWR05" (id 0) (at 267.335 77.47 0)
       (effects (font (size 1.27 1.27)) hide)
     )
@@
   (symbol (lib_id "power:GND") (at 267.335 82.55 0) (unit 1)
     (in_bom yes) (on_board yes)
-    (property "Reference" "#PWR?" (id 0) (at 267.335 88.9 0)
+    (property "Reference" "#PWR09" (id 0) (at 267.335 88.9 0)
       (effects (font (size 1.27 1.27)) hide)
     )
@@
   (symbol (lib_id "power:GND") (at 255.905 82.55 0) (unit 1)
     (in_bom yes) (on_board yes)
-    (property "Reference" "#PWR?" (id 0) (at 255.905 88.9 0)
+    (property "Reference" "#PWR08" (id 0) (at 255.905 88.9 0)
       (effects (font (size 1.27 1.27)) hide)
     )
@@
   (symbol (lib_id "Device:C_Small") (at 255.905 78.74 0) (unit 1)
     (in_bom yes) (on_board yes)
-    (property "Reference" "C?" (id 0) (at 258.2418 77.5716 0)
+    (property "Reference" "C2" (id 0) (at 258.2418 77.5716 0)
       (effects (font (size 1.27 1.27)) (justify left))
     )
@@
   (symbol (lib_id "Device:C_Small") (at 243.205 99.06 270) (unit 1)
     (in_bom yes) (on_board yes)
-    (property "Reference" "C?" (id 0) (at 243.205 95.885 90))
+    (property "Reference" "C4" (id 0) (at 243.205 95.885 90))
     (property "Value" "100n" (id 1) (at 243.205 102.235 90))
     (property "Footprint" "Capacitor_SMD:C_0603_1608Metric" (id 2) (at 243.205 99.06 0)
@@
   (symbol (lib_id "Device:R_Small") (at 241.935 86.36 270) (unit 1)
     (in_bom yes) (on_board yes)
-    (property "Reference" "R?" (id 0) (at 240.665 84.455 90)
+    (property "Reference" "R4" (id 0) (at 240.665 84.455 90)
       (effects (font (size 1.27 1.27)) (justify left))
     )
@@
   (symbol (lib_id "power:VBUS") (at 168.91 76.2 0) (unit 1)
     (in_bom yes) (on_board yes)
-    (property "Reference" "#PWR?" (id 0) (at 168.91 80.01 0)
+    (property "Reference" "#PWR06" (id 0) (at 168.91 80.01 0)
       (effects (font (size 1.27 1.27)) hide)
     )
@@
   (symbol (lib_id "power:GND") (at 84.455 85.09 0) (unit 1)
     (in_bom yes) (on_board yes)
-    (property "Reference" "#PWR?" (id 0) (at 84.455 91.44 0)
+    (property "Reference" "#PWR010" (id 0) (at 84.455 91.44 0)
       (effects (font (size 1.27 1.27)) hide)
     )
@@
   (symbol (lib_id "Device:C_Small") (at 204.47 78.74 0) (unit 1)
     (in_bom yes) (on_board yes)
-    (property "Reference" "C?" (id 0) (at 206.8068 77.5716 0)
+    (property "Reference" "C1" (id 0) (at 206.8068 77.5716 0)
       (effects (font (size 1.27 1.27)) (justify left))
     )
@@
   (symbol (lib_id "power:VBUS") (at 76.2 66.04 0) (unit 1)
     (in_bom yes) (on_board yes)
-    (property "Reference" "#PWR?" (id 0) (at 76.2 69.85 0)
+    (property "Reference" "#PWR04" (id 0) (at 76.2 69.85 0)
       (effects (font (size 1.27 1.27)) hide)
     )
@@
   (symbol (lib_id "Device:R_Small") (at 81.28 80.01 0) (unit 1)
     (in_bom yes) (on_board yes)
-    (property "Reference" "R?" (id 0) (at 82.55 78.74 0)
+    (property "Reference" "R2" (id 0) (at 82.55 78.74 0)
       (effects (font (size 1.27 1.27)) (justify left))
     )
@@
   (symbol (lib_id "Device:R_Small") (at 87.63 80.01 0) (unit 1)
     (in_bom yes) (on_board yes)
-    (property "Reference" "R?" (id 0) (at 88.9 78.74 0)
+    (property "Reference" "R3" (id 0) (at 88.9 78.74 0)
       (effects (font (size 1.27 1.27)) (justify left))
     )
@@
   (symbol (lib_id "Interface_USB:CH340C") (at 227.965 91.44 0) (unit 1)
     (in_bom yes) (on_board yes)
-    (property "Reference" "U?" (id 0) (at 221.615 77.47 0))
+    (property "Reference" "U2" (id 0) (at 221.615 77.47 0))
     (property "Value" "CH340C" (id 1) (at 232.41 105.41 0))
     (property "Footprint" "Package_SO:SOIC-16_3.9x9.9mm_P1.27mm" (id 2) (at 229.235 105.41 0)
@@
   (symbol (lib_id "power:GND") (at 39.37 106.68 0) (unit 1)
     (in_bom yes) (on_board yes)
-    (property "Reference" "#PWR?" (id 0) (at 39.37 113.03 0)
+    (property "Reference" "#PWR012" (id 0) (at 39.37 113.03 0)
       (effects (font (size 1.27 1.27)) hide)
     )
@@
   (symbol (lib_id "Device:C_Polarized_Small") (at 267.335 78.74 0) (unit 1)
     (in_bom yes) (on_board yes) (fields_autoplaced)
-    (property "Reference" "C?" (id 0) (at 269.494 77.3592 0)
+    (property "Reference" "C3" (id 0) (at 269.494 77.3592 0)
       (effects (font (size 1.27 1.27)) (justify left))
     )
@@
   (symbol (lib_id "Device:R_Small") (at 241.935 78.74 270) (unit 1)
     (in_bom yes) (on_board yes)
-    (property "Reference" "R?" (id 0) (at 240.665 76.835 90)
+    (property "Reference" "R1" (id 0) (at 240.665 76.835 90)
       (effects (font (size 1.27 1.27)) (justify left))
     )
@@
   (symbol (lib_id "Device:FerriteBead") (at 66.04 68.58 90) (unit 1)
     (in_bom yes) (on_board yes) (fields_autoplaced)
-    (property "Reference" "FB?" (id 0) (at 65.9892 62.2386 90))
+    (property "Reference" "FB1" (id 0) (at 65.9892 62.2386 90))
     (property "Value" "100 @ 100MHz" (id 1) (at 65.9892 64.7755 90))
     (property "Footprint" "Resistor_SMD:R_0603_1608Metric" (id 2) (at 66.04 70.358 90)
@@
   (symbol (lib_id "power:GND") (at 227.965 106.68 0) (unit 1)
     (in_bom yes) (on_board yes)
-    (property "Reference" "#PWR?" (id 0) (at 227.965 113.03 0)
+    (property "Reference" "#PWR013" (id 0) (at 227.965 113.03 0)
       (effects (font (size 1.27 1.27)) hide)
     )
@@
   (symbol (lib_id "power:GND") (at 168.91 96.52 0) (unit 1)
     (in_bom yes) (on_board yes)
-    (property "Reference" "#PWR?" (id 0) (at 168.91 102.87 0)
+    (property "Reference" "#PWR011" (id 0) (at 168.91 102.87 0)
       (effects (font (size 1.27 1.27)) hide)
     )
@@
   (symbol (lib_id "Power_Protection:USBLC6-2SC6") (at 168.91 86.36 0) (unit 1)
     (in_bom yes) (on_board yes)
-    (property "Reference" "U?" (id 0) (at 161.29 77.47 0)
+    (property "Reference" "U1" (id 0) (at 161.29 77.47 0)
       (effects (font (size 1.27 1.27)) (justify left))
     )
@@
   (symbol (lib_id "power:GND") (at 204.47 82.55 0) (unit 1)
     (in_bom yes) (on_board yes)
-    (property "Reference" "#PWR?" (id 0) (at 204.47 88.9 0)
-      (effects (font (size 1.27 1.27)) hide)
-    )
+    (property "Reference" "#PWR07" (id 0) (at 204.47 88.9 0)
+      (effects (font (size 1.27 1.27)) hide)
+    )

Commit message: update
Parts:
- renumbered C1 to C201, C2 to C202, C3 to C203, C4 to C204, FB1 to FB201, J1 to J201, R1 to R201, R2 to R202, R3 to R203, R4 to R204, U1 to U201, U2 to U202
Changed lines of the file:
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@@
   (symbol (lib_id "Connector:USB_C_Receptacle_USB2.0") (at 39.37 83.82 0) (unit 1)
     (in_bom yes) (on_board yes)
-    (property "Reference" "J1" (id 0) (at 30.48 64.643 0))
+    (property "Reference" "J201" (id 0) (at 30.48 64.643 0))
     (property "Value" "USB_C_Receptacle_USB2.0" (id 1) (at 42.0878 64.1096 0)
       (effects (font (size 1.27 1.27)) hide)
@@
   (symbol (lib_id "power:VBUS") (at 267.335 73.66 0) (unit 1)
     (in_bom yes) (on_board yes)
-    (property "Reference" "#PWR05" (id 0) (at 267.335 77.47 0)
+    (property "Reference" "#PWR0202" (id 0) (at 267.335 77.47 0)
       (effects (font (size 1.27 1.27)) hide)
     )
@@
   (symbol (lib_id "power:GND") (at 267.335 82.55 0) (unit 1)
     (in_bom yes) (on_board yes)
-    (property "Reference" "#PWR09" (id 0) (at 267.335 88.9 0)
+    (property "Reference" "#PWR0206" (id 0) (at 267.335 88.9 0)
       (effects (font (size 1.27 1.27)) hide)
     )
@@
   (symbol (lib_id "power:GND") (at 255.905 82.55 0) (unit 1)
     (in_bom yes) (on_board yes)
-    (property "Reference" "#PWR08" (id 0) (at 255.905 88.9 0)
+    (property "Reference" "#PWR0205" (id 0) (at 255.905 88.9 0)
       (effects (font (size 1.27 1.27)) hide)
     )
@@
   (symbol (lib_id "Device:C_Small") (at 255.905 78.74 0) (unit 1)
     (in_bom yes) (on_board yes)
-    (property "Reference" "C2" (id 0) (at 258.2418 77.5716 0)
+    (property "Reference" "C202" (id 0) (at 258.2418 77.5716 0)
       (effects (font (size 1.27 1.27)) (justify left))
     )
@@
   (symbol (lib_id "Device:C_Small") (at 243.205 99.06 270) (unit 1)
     (in_bom yes) (on_board yes)
-    (property "Reference" "C4" (id 0) (at 243.205 95.885 90))
+    (property "Reference" "C204" (id 0) (at 243.205 95.885 90))
     (property "Value" "100n" (id 1) (at 243.205 102.235 90))
     (property "Footprint" "Capacitor_SMD:C_0603_1608Metric" (id 2) (at 243.205 99.06 0)
@@
   (symbol (lib_id "Device:R_Small") (at 241.935 86.36 270) (unit 1)
     (in_bom yes) (on_board yes)
-    (property "Reference" "R4" (id 0) (at 240.665 84.455 90)
+    (property "Reference" "R204" (id 0) (at 240.665 84.455 90)
       (effects (font (size 1.27 1.27)) (justify left))
     )
@@
   (symbol (lib_id "power:VBUS") (at 168.91 76.2 0) (unit 1)
     (in_bom yes) (on_board yes)
-    (property "Reference" "#PWR06" (id 0) (at 168.91 80.01 0)
+    (property "Reference" "#PWR0203" (id 0) (at 168.91 80.01 0)
       (effects (font (size 1.27 1.27)) hide)
     )
@@
   (symbol (lib_id "power:GND") (at 84.455 85.09 0) (unit 1)
     (in_bom yes) (on_board yes)
-    (property "Reference" "#PWR010" (id 0) (at 84.455 91.44 0)
+    (property "Reference" "#PWR0207" (id 0) (at 84.455 91.44 0)
       (effects (font (size 1.27 1.27)) hide)
     )
@@
   (symbol (lib_id "Device:C_Small") (at 204.47 78.74 0) (unit 1)
     (in_bom yes) (on_board yes)
-    (property "Reference" "C1" (id 0) (at 206.8068 77.5716 0)
+    (property "Reference" "C201" (id 0) (at 206.8068 77.5716 0)
       (effects (font (size 1.27 1.27)) (justify left))
     )
@@
   (symbol (lib_id "power:VBUS") (at 76.2 66.04 0) (unit 1)
     (in_bom yes) (on_board yes)
-    (property "Reference" "#PWR04" (id 0) (at 76.2 69.85 0)
+    (property "Reference" "#PWR0201" (id 0) (at 76.2 69.85 0)
       (effects (font (size 1.27 1.27)) hide)
     )
@@
   (symbol (lib_id "Device:R_Small") (at 81.28 80.01 0) (unit 1)
     (in_bom yes) (on_board yes)
-    (property "Reference" "R2" (id 0) (at 82.55 78.74 0)
+    (property "Reference" "R202" (id 0) (at 82.55 78.74 0)
       (effects (font (size 1.27 1.27)) (justify left))
     )
@@
   (symbol (lib_id "Device:R_Small") (at 87.63 80.01 0) (unit 1)
     (in_bom yes) (on_board yes)
-    (property "Reference" "R3" (id 0) (at 88.9 78.74 0)
+    (property "Reference" "R203" (id 0) (at 88.9 78.74 0)
       (effects (font (size 1.27 1.27)) (justify left))
     )
@@
   (symbol (lib_id "Interface_USB:CH340C") (at 227.965 91.44 0) (unit 1)
     (in_bom yes) (on_board yes)
-    (property "Reference" "U2" (id 0) (at 221.615 77.47 0))
+    (property "Reference" "U202" (id 0) (at 221.615 77.47 0))
     (property "Value" "CH340C" (id 1) (at 232.41 105.41 0))
     (property "Footprint" "Package_SO:SOIC-16_3.9x9.9mm_P1.27mm" (id 2) (at 229.235 105.41 0)
@@
   (symbol (lib_id "power:GND") (at 39.37 106.68 0) (unit 1)
     (in_bom yes) (on_board yes)
-    (property "Reference" "#PWR012" (id 0) (at 39.37 113.03 0)
+    (property "Reference" "#PWR0209" (id 0) (at 39.37 113.03 0)
       (effects (font (size 1.27 1.27)) hide)
     )
@@
   (symbol (lib_id "Device:C_Polarized_Small") (at 267.335 78.74 0) (unit 1)
     (in_bom yes) (on_board yes) (fields_autoplaced)
-    (property "Reference" "C3" (id 0) (at 269.494 77.3592 0)
+    (property "Reference" "C203" (id 0) (at 269.494 77.3592 0)
       (effects (font (size 1.27 1.27)) (justify left))
     )
@@
   (symbol (lib_id "Device:R_Small") (at 241.935 78.74 270) (unit 1)
     (in_bom yes) (on_board yes)
-    (property "Reference" "R1" (id 0) (at 240.665 76.835 90)
+    (property "Reference" "R201" (id 0) (at 240.665 76.835 90)
       (effects (font (size 1.27 1.27)) (justify left))
     )
@@
   (symbol (lib_id "Device:FerriteBead") (at 66.04 68.58 90) (unit 1)
     (in_bom yes) (on_board yes) (fields_autoplaced)
-    (property "Reference" "FB1" (id 0) (at 65.9892 62.2386 90))
+    (property "Reference" "FB201" (id 0) (at 65.9892 62.2386 90))
     (property "Value" "100 @ 100MHz" (id 1) (at 65.9892 64.7755 90))
     (property "Footprint" "Resistor_SMD:R_0603_1608Metric" (id 2) (at 66.04 70.358 90)
@@
   (symbol (lib_id "power:GND") (at 227.965 106.68 0) (unit 1)
     (in_bom yes) (on_board yes)
-    (property "Reference" "#PWR013" (id 0) (at 227.965 113.03 0)
+    (property "Reference" "#PWR0210" (id 0) (at 227.965 113.03 0)
       (effects (font (size 1.27 1.27)) hide)
     )
@@
   (symbol (lib_id "power:GND") (at 168.91 96.52 0) (unit 1)
     (in_bom yes) (on_board yes)
-    (property "Reference" "#PWR011" (id 0) (at 168.91 102.87 0)
+    (property "Reference" "#PWR0208" (id 0) (at 168.91 102.87 0)
       (effects (font (size 1.27 1.27)) hide)
     )
@@
   (symbol (lib_id "Power_Protection:USBLC6-2SC6") (at 168.91 86.36 0) (unit 1)
     (in_bom yes) (on_board yes)
-    (property "Reference" "U1" (id 0) (at 161.29 77.47 0)
+    (property "Reference" "U201" (id 0) (at 161.29 77.47 0)
       (effects (font (size 1.27 1.27)) (justify left))
     )
@@
   (symbol (lib_id "power:GND") (at 204.47 82.55 0) (unit 1)
     (in_bom yes) (on_board yes)
-    (property "Reference" "#PWR07" (id 0) (at 204.47 88.9 0)
-      (effects (font (size 1.27 1.27)) hide)
-    )
+    (property "Reference" "#PWR0204" (id 0) (at 204.47 88.9 0)
+      (effects (font (size 1.27 1.27)) hide)
+    )
