File: KiCad files/BoardGame/USB.kicad_sch (KiCad schematic)
At the start: 12 parts, among them J201 USB_C_Receptacle_USB2.0, U201 USBLC6-2SC6, U202 CH340C

Commit message: update
Parts:
- C201: JLCPCB Part # (none) -> C113803; U labosu? (none) -> ne
- C202, C204: JLCPCB Part # C49678 -> C113803; U labosu? Da -> ne
- C203: JLCPCB Part # (none) -> C2798040; U labosu? (none) -> ne
- FB201: JLCPCB Part # (none) -> C107332; U labosu? (none) -> ne
- J201: Ostalo https://www.aliexpress.com/item/32976750426.html?spm=a2g0o.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 -> 32976750426; U labosu? Da -> da
- R201, R204, U202: U labosu? (none) -> da
- R202, R203: JLCPCB Part # (none) -> C3017721; U labosu? (none) -> ne
- U201: JLCPCB Part # (none) -> C3029034; U labosu? (none) -> ne
Changed lines of the file:
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@@
       (effects (font (size 1.27 1.27)) hide)
     )
-    (property "Ostalo" "https://www.aliexpress.com/item/32976750426.html?spm=a2g0o.9042311.0.0.39c14c4dXFSZYC" (id 6) (at 39.37 83.82 0)
-      (effects (font (size 1.27 1.27)) hide)
-    )
-    (property "U labosu?" "Da" (id 7) (at 39.37 83.82 0)
+    (property "Ostalo" "32976750426" (id 6) (at 39.37 83.82 0)
+      (effects (font (size 1.27 1.27)) hide)
+    )
+    (property "U labosu?" "da" (id 7) (at 39.37 83.82 0)
       (effects (font (size 1.27 1.27)) hide)
     )
@@
       (effects (font (size 1.27 1.27)) hide)
     )
-    (property "JLCPCB Part #" "C49678" (id 5) (at 255.905 78.74 0)
-      (effects (font (size 1.27 1.27)) hide)
-    )
-    (property "U labosu?" "Da" (id 6) (at 255.905 78.74 0)
+    (property "JLCPCB Part #" "C113803" (id 5) (at 255.905 78.74 0)
+      (effects (font (size 1.27 1.27)) hide)
+    )
+    (property "U labosu?" "ne" (id 6) (at 255.905 78.74 0)
       (effects (font (size 1.27 1.27)) hide)
     )
@@
       (effects (font (size 1.27 1.27)) hide)
     )
-    (property "JLCPCB Part #" "C49678" (id 5) (at 243.205 99.06 0)
-      (effects (font (size 1.27 1.27)) hide)
-    )
-    (property "U labosu?" "Da" (id 6) (at 243.205 99.06 0)
+    (property "JLCPCB Part #" "C113803" (id 5) (at 243.205 99.06 0)
+      (effects (font (size 1.27 1.27)) hide)
+    )
+    (property "U labosu?" "ne" (id 6) (at 243.205 99.06 0)
       (effects (font (size 1.27 1.27)) hide)
     )
@@
     )
     (property "Datasheet" "~" (id 3) (at 241.935 86.36 0)
+      (effects (font (size 1.27 1.27)) hide)
+    )
+    (property "U labosu?" "da" (id 4) (at 241.935 86.36 0)
       (effects (font (size 1.27 1.27)) hide)
     )
@@
       (effects (font (size 1.27 1.27)) hide)
     )
+    (property "U labosu?" "ne" (id 4) (at 204.47 78.74 0)
+      (effects (font (size 1.27 1.27)) hide)
+    )
+    (property "JLCPCB Part #" "C113803" (id 5) (at 204.47 78.74 0)
+      (effects (font (size 1.27 1.27)) hide)
+    )
     (pin "1")
     (pin "2")
@@
       (effects (font (size 1.27 1.27)) hide)
     )
+    (property "JLCPCB Part #" "C3017721" (id 4) (at 81.28 80.01 0)
+      (effects (font (size 1.27 1.27)) hide)
+    )
+    (property "U labosu?" "ne" (id 5) (at 81.28 80.01 0)
+      (effects (font (size 1.27 1.27)) hide)
+    )
     (pin "1")
     (pin "2")
@@
     )
     (property "Datasheet" "~" (id 3) (at 87.63 80.01 0)
+      (effects (font (size 1.27 1.27)) hide)
+    )
+    (property "JLCPCB Part #" "C3017721" (id 4) (at 87.63 80.01 0)
+      (effects (font (size 1.27 1.27)) hide)
+    )
+    (property "U labosu?" "ne" (id 5) (at 87.63 80.01 0)
       (effects (font (size 1.27 1.27)) hide)
     )
@@
     )
     (property "Datasheet" "https://datasheet.lcsc.com/szlcsc/Jiangsu-Qin-Heng-CH340C_C84681.pdf" (id 3) (at 219.075 71.12 0)
+      (effects (font (size 1.27 1.27)) hide)
+    )
+    (property "U labosu?" "da" (id 4) (at 227.965 91.44 0)
       (effects (font (size 1.27 1.27)) hide)
     )
@@
       (effects (font (size 1.27 1.27)) hide)
     )
+    (property "JLCPCB Part #" "C2798040" (id 4) (at 267.335 78.74 0)
+      (effects (font (size 1.27 1.27)) hide)
+    )
+    (property "U labosu?" "ne" (id 5) (at 267.335 78.74 0)
+      (effects (font (size 1.27 1.27)) hide)
+    )
     (pin "1")
     (pin "2")
@@
     )
     (property "Datasheet" "~" (id 3) (at 241.935 78.74 0)
+      (effects (font (size 1.27 1.27)) hide)
+    )
+    (property "U labosu?" "da" (id 4) (at 241.935 78.74 0)
       (effects (font (size 1.27 1.27)) hide)
     )
@@
       (effects (font (size 1.27 1.27)) hide)
     )
+    (property "JLCPCB Part #" "C107332" (id 4) (at 66.04 68.58 0)
+      (effects (font (size 1.27 1.27)) hide)
+    )
+    (property "U labosu?" "ne" (id 5) (at 66.04 68.58 0)
+      (effects (font (size 1.27 1.27)) hide)
+    )
     (pin "1")
     (pin "2")
@@
       (effects (font (size 1.27 1.27)) hide)
     )
+    (property "JLCPCB Part #" "C3029034" (id 4) (at 168.91 86.36 0)
+      (effects (font (size 1.27 1.27)) hide)
+    )
+    (property "U labosu?" "ne" (id 5) (at 168.91 86.36 0)
+      (effects (font (size 1.27 1.27)) hide)
+    )

Commit message: layout_v2
Connections:
- net USB: now reaches FB201.1, J201.A4 (VBUS), J201.A9 (VBUS), J201.B4 (VBUS), J201.B9 (VBUS)
Changed lines of the file:
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@@
+    (effects (font (size 1.27 1.27)) (justify left bottom))
+  )
+  (label "USB" (at 55.245 68.58 0)
     (effects (font (size 1.27 1.27)) (justify left bottom))
   )

Commit message: update
Connections:
- net USB_CONN_D+: now also U201.3 (I/O2); no longer U201.6 (I/O1)
- net USB_CONN_D-: now also U201.1 (I/O1); no longer U201.4 (I/O2)
- net USB_D+: now also U201.4 (I/O2); no longer U201.1 (I/O1)
- net USB_D-: now also U201.6 (I/O1); no longer U201.3 (I/O2)
Changed lines of the file:
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@@
     (effects (font (size 1.27 1.27)) (justify left bottom))
   )
-  (global_label "USB_CONN_D+" (shape input) (at 158.75 83.82 180) (fields_autoplaced)
-    (effects (font (size 1.27 1.27)) (justify right))
-    (property "Intersheet References" "${INTERSHEET_REFS}" (id 0) (at 142.4879 83.8994 0)
-      (effects (font (size 1.27 1.27)) (justify right) hide)
+  (global_label "USB_CONN_D+" (shape input) (at 179.07 88.9 0) (fields_autoplaced)
+    (effects (font (size 1.27 1.27)) (justify left))
+    (property "Intersheet References" "${INTERSHEET_REFS}" (id 0) (at 195.3321 88.8206 0)
+      (effects (font (size 1.27 1.27)) (justify left) hide)
     )
   )
@@
     )
   )
-  (global_label "USB_CONN_D-" (shape input) (at 179.07 83.82 0) (fields_autoplaced)
-    (effects (font (size 1.27 1.27)) (justify left))
-    (property "Intersheet References" "${INTERSHEET_REFS}" (id 0) (at 195.3321 83.7406 0)
-      (effects (font (size 1.27 1.27)) (justify left) hide)
+  (global_label "USB_CONN_D-" (shape input) (at 158.75 88.9 180) (fields_autoplaced)
+    (effects (font (size 1.27 1.27)) (justify right))
+    (property "Intersheet References" "${INTERSHEET_REFS}" (id 0) (at 142.4879 88.9794 0)
+      (effects (font (size 1.27 1.27)) (justify right) hide)
     )
   )
@@
     )
   )
-  (global_label "USB_D+" (shape input) (at 158.75 88.9 180) (fields_autoplaced)
-    (effects (font (size 1.27 1.27)) (justify right))
-    (property "Intersheet References" "${INTERSHEET_REFS}" (id 0) (at 148.7169 88.8206 0)
-      (effects (font (size 1.27 1.27)) (justify right) hide)
+  (global_label "USB_D+" (shape input) (at 179.07 83.82 0) (fields_autoplaced)
+    (effects (font (size 1.27 1.27)) (justify left))
+    (property "Intersheet References" "${INTERSHEET_REFS}" (id 0) (at 189.1031 83.8994 0)
+      (effects (font (size 1.27 1.27)) (justify left) hide)
     )
   )
@@
     )
   )
-  (global_label "USB_D-" (shape input) (at 179.07 88.9 0) (fields_autoplaced)
-    (effects (font (size 1.27 1.27)) (justify left))
-    (property "Intersheet References" "${INTERSHEET_REFS}" (id 0) (at 189.1031 88.8206 0)
-      (effects (font (size 1.27 1.27)) (justify left) hide)
+  (global_label "USB_D-" (shape input) (at 158.75 83.82 180) (fields_autoplaced)
+    (effects (font (size 1.27 1.27)) (justify right))
+    (property "Intersheet References" "${INTERSHEET_REFS}" (id 0) (at 148.7169 83.8994 0)
+      (effects (font (size 1.27 1.27)) (justify right) hide)
     )
   )

Commit message: update
Changed lines of the file:
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@@
     (effects (font (size 1.27 1.27)) (justify left bottom))
   )
-  (text "CH340C USB-UART IC" (at 219.075 71.12 0)
-    (effects (font (size 1.27 1.27)) (justify left bottom))
+  (text "CH340C USB-UART IC" (at 210.185 64.77 0)
+    (effects (font (size 3 3) (thickness 0.6) bold) (justify left bottom))
   )
   (text "ESD protection IC" (at 161.29 105.41 0)

Commit message: Schematic update
Other:
- moved on the sheet: R203
Changed lines of the file:
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@@
     (stroke (width 0) (type default) (color 0 0 0 0))
   )
-  (wire (pts (xy 84.455 83.82) (xy 87.63 83.82))
+  (wire (pts (xy 84.455 83.82) (xy 88.9 83.82))
     (stroke (width 0) (type default) (color 0 0 0 0))
   )
@@
     (stroke (width 0) (type default) (color 0 0 0 0))
   )
-  (wire (pts (xy 54.61 73.66) (xy 87.63 73.66))
+  (wire (pts (xy 54.61 73.66) (xy 88.9 73.66))
     (stroke (width 0) (type default) (color 0 0 0 0))
   )
@@
     (stroke (width 0) (type default) (color 0 0 0 0))
   )
-  (wire (pts (xy 87.63 83.82) (xy 87.63 82.55))
+  (wire (pts (xy 88.9 83.82) (xy 88.9 82.55))
     (stroke (width 0) (type default) (color 0 0 0 0))
   )
@@
     (stroke (width 0) (type default) (color 0 0 0 0))
   )
-  (wire (pts (xy 87.63 73.66) (xy 87.63 77.47))
+  (wire (pts (xy 88.9 73.66) (xy 88.9 77.47))
     (stroke (width 0) (type default) (color 0 0 0 0))
   )
@@
     )
   )
-  (global_label "RESET" (shape input) (at 247.65 99.06 0) (fields_autoplaced)
-    (effects (font (size 1.27 1.27)) (justify left))
-    (property "Intersheet References" "${INTERSHEET_REFS}" (id 0) (at 86.995 7.62 0)
-      (effects (font (size 1.27 1.27)) hide)
-    )
-  )
   (global_label "USB_CONN_D-" (shape input) (at 60.96 82.55 0) (fields_autoplaced)
     (effects (font (size 1.27 1.27)) (justify left))
     (property "Intersheet References" "${INTERSHEET_REFS}" (id 0) (at 77.2221 82.4706 0)
       (effects (font (size 1.27 1.27)) (justify left) hide)
-    )
-  )
-  (global_label "RX" (shape input) (at 244.475 78.74 0) (fields_autoplaced)
-    (effects (font (size 1.27 1.27)) (justify left))
-    (property "Intersheet References" "${INTERSHEET_REFS}" (id 0) (at 86.995 5.08 0)
-      (effects (font (size 1.27 1.27)) hide)
     )
   )
@@
     )
   )
-  (global_label "TX" (shape input) (at 244.475 86.36 0) (fields_autoplaced)
-    (effects (font (size 1.27 1.27)) (justify left))
-    (property "Intersheet References" "${INTERSHEET_REFS}" (id 0) (at 86.995 7.62 0)
-      (effects (font (size 1.27 1.27)) hide)
-    )
-  )
   (global_label "USB_D-" (shape input) (at 158.75 83.82 180) (fields_autoplaced)
     (effects (font (size 1.27 1.27)) (justify right))
@@
       (effects (font (size 1.27 1.27)) (justify right) hide)
     )
+  )
+  (hierarchical_label "RX" (shape output) (at 244.475 78.74 0)
+    (effects (font (size 1.27 1.27)) (justify left))
+  )
+  (hierarchical_label "RESET" (shape output) (at 247.65 99.06 0)
+    (effects (font (size 1.27 1.27)) (justify left))
+  )
+  (hierarchical_label "TX" (shape input) (at 244.475 86.36 0)
+    (effects (font (size 1.27 1.27)) (justify left))
   )
   (symbol (lib_id "Connector:USB_C_Receptacle_USB2.0") (at 39.37 83.82 0) (unit 1)
@@
     (pin "2")
   )
-  (symbol (lib_id "Device:R_Small") (at 87.63 80.01 0) (unit 1)
-    (in_bom yes) (on_board yes)
-    (property "Reference" "R203" (id 0) (at 88.9 78.74 0)
-      (effects (font (size 1.27 1.27)) (justify left))
-    )
-    (property "Value" "5k1" (id 1) (at 88.9 80.645 0)
-      (effects (font (size 1.27 1.27)) (justify left))
-    )
-    (property "Footprint" "Resistor_SMD:R_0603_1608Metric" (id 2) (at 87.63 80.01 0)
-      (effects (font (size 1.27 1.27)) hide)
-    )
-    (property "Datasheet" "~" (id 3) (at 87.63 80.01 0)
-      (effects (font (size 1.27 1.27)) hide)
-    )
-    (property "JLCPCB Part #" "C3017721" (id 4) (at 87.63 80.01 0)
-      (effects (font (size 1.27 1.27)) hide)
-    )
-    (property "U labosu?" "ne" (id 5) (at 87.63 80.01 0)
-      (effects (font (size 1.27 1.27)) hide)
-    )
+  (symbol (lib_id "Device:R_Small") (at 88.9 80.01 0) (unit 1)
+    (in_bom yes) (on_board yes)
+    (property "Reference" "R203" (id 0) (at 90.17 78.74 0)
+      (effects (font (size 1.27 1.27)) (justify left))
+    )
+    (property "Value" "5k1" (id 1) (at 90.17 80.645 0)
+      (effects (font (size 1.27 1.27)) (justify left))
+    )
+    (property "Footprint" "Resistor_SMD:R_0603_1608Metric" (id 2) (at 88.9 80.01 0)
+      (effects (font (size 1.27 1.27)) hide)
+    )
+    (property "Datasheet" "~" (id 3) (at 88.9 80.01 0)
+      (effects (font (size 1.27 1.27)) hide)
+    )
+    (property "JLCPCB Part #" "C3017721" (id 4) (at 88.9 80.01 0)
+      (effects (font (size 1.27 1.27)) hide)
+    )
+    (property "U labosu?" "ne" (id 5) (at 88.9 80.01 0)
+      (effects (font (size 1.27 1.27)) hide)
+    )
