File: KiCad files/BoardGame/USB.kicad_sch (KiCad schematic)
At the start: 12 parts, among them J201 USB_C_Receptacle_USB2.0, U201 USBLC6-2SC6, U202 CH340C

Commit message: update
Changed lines of the file:
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@@
 (kicad_sch
-	(version 20231120)
+	(version 20250114)
 	(generator "eeschema")
-	(generator_version "8.0")
+	(generator_version "9.0")
 	(paper "A4")
 	(title_block
@@
 		(rev "1")
 	)
+	(text "Shield is grounded at the host side (PC) so NC here."
+		(exclude_from_sim no)
+		(at 17.78 116.84 0)
+		(effects
+			(font
+				(size 1.27 1.27)
+			)
+			(justify left bottom)
+		)
+	)
+	(text "CH340C USB-UART IC"
+		(exclude_from_sim no)
+		(at 210.185 64.77 0)
+		(effects
+			(font
+				(size 3 3)
+				(thickness 0.6)
+				(bold yes)
+			)
+			(justify left bottom)
+		)
+	)
+	(text "ESD protection IC"
+		(exclude_from_sim no)
+		(at 161.29 105.41 0)
+		(effects
+			(font
+				(size 1.27 1.27)
+			)
+			(justify left bottom)
+		)
+	)
+	(text "The device must have 5.1k pull-down on the its port CC pin (on both pins).\n\nOnce the C-C cable is connected between two link partners, the DFP (host)\nwill sense the drag by 5.1k resistor (from device side). As result, it will turn the VBUS on.\nThis is how a host recognizes that a connection has been made.\nThe connect event is essentially controlled by sink side having 5.1k Rd."
+		(exclude_from_sim no)
+		(at 30.48 57.15 0)
+		(effects
+			(font
+				(size 1.27 1.27)
+			)
+			(justify left bottom)
+		)
+	)
+	(text "SBU1/SBU2: these are low-speed lines used only for\nAlternate Mode and accessory mode. For example, with\nDisplayPort, AUX+/AUX– transmit over the SBU lines. For\naudio adapter accessory mode, these lines are used for\nthe microphone input and analog GND."
+		(exclude_from_sim no)
+		(at 58.42 104.14 0)
+		(effects
+			(font
+				(size 1.27 1.27)
+			)
+			(justify left bottom)
+		)
+	)
+	(text "Ferrite bead needs to be placed close to USB connector on PCB"
+		(exclude_from_sim no)
+		(at 85.09 67.31 0)
+		(effects
+			(font
+				(size 1.27 1.27)
+			)
+			(justify left bottom)
+		)
+	)
 	(junction
 		(at 59.055 82.55)
@@
 		)
 	)
-	(text "Shield is grounded at the host side (PC) so NC here."
-		(exclude_from_sim no)
-		(at 17.78 116.84 0)
-		(effects
-			(font
-				(size 1.27 1.27)
-			)
-			(justify left bottom)
-		)
-	)
-	(text "CH340C USB-UART IC"
-		(exclude_from_sim no)
-		(at 210.185 64.77 0)
-		(effects
-			(font
-				(size 3 3)
-				(thickness 0.6)
-				(bold yes)
-			)
-			(justify left bottom)
-		)
-	)
-	(text "ESD protection IC"
-		(exclude_from_sim no)
-		(at 161.29 105.41 0)
-		(effects
-			(font
-				(size 1.27 1.27)
-			)
-			(justify left bottom)
-		)
-	)
-	(text "The device must have 5.1k pull-down on the its port CC pin (on both pins).\n\nOnce the C-C cable is connected between two link partners, the DFP (host)\nwill sense the drag by 5.1k resistor (from device side). As result, it will turn the VBUS on.\nThis is how a host recognizes that a connection has been made.\nThe connect event is essentially controlled by sink side having 5.1k Rd."
-		(exclude_from_sim no)
-		(at 30.48 57.15 0)
-		(effects
-			(font
-				(size 1.27 1.27)
-			)
-			(justify left bottom)
-		)
-	)
-	(text "SBU1/SBU2: these are low-speed lines used only for\nAlternate Mode and accessory mode. For example, with\nDisplayPort, AUX+/AUX– transmit over the SBU lines. For\naudio adapter accessory mode, these lines are used for\nthe microphone input and analog GND."
-		(exclude_from_sim no)
-		(at 58.42 104.14 0)
-		(effects
-			(font
-				(size 1.27 1.27)
-			)
-			(justify left bottom)
-		)
-	)
-	(text "Ferrite bead needs to be placed close to USB connector on PCB"
-		(exclude_from_sim no)
-		(at 85.09 67.31 0)
-		(effects
-			(font
-				(size 1.27 1.27)
-			)
-			(justify left bottom)
-		)
-	)
 	(label "USB"
 		(at 55.245 68.58 0)
-		(fields_autoplaced yes)
 		(effects
 			(font
@@
 		(shape output)
 		(at 244.475 78.74 0)
-		(fields_autoplaced yes)
 		(effects
 			(font
@@
 		(shape output)
 		(at 247.65 99.06 0)
-		(fields_autoplaced yes)
 		(effects
 			(font
@@
 		(shape input)
 		(at 244.475 86.36 0)
-		(fields_autoplaced yes)
-		(effects
-			(font
+		(effects
+			(font
