File: KiCad files/BoardGame/Boost Converter.kicad_sch (KiCad schematic)
At the start: 7 parts

Commit message: update
Parts:
- gave numbers to parts that had none: 7
Changed lines of the file:
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@@
   (symbol (lib_id "Regulator_Switching:MT3608") (at 139.7 80.645 0) (unit 1)
     (in_bom yes) (on_board yes)
-    (property "Reference" "U?" (id 0) (at 135.89 74.295 0))
+    (property "Reference" "U6" (id 0) (at 135.89 74.295 0))
     (property "Value" "MT3608" (id 1) (at 144.145 86.995 0))
     (property "Footprint" "Package_TO_SOT_SMD:SOT-23-6" (id 2) (at 140.97 86.995 0)
@@
   (symbol (lib_id "Device:R_Small") (at 159.385 87.63 0) (unit 1)
     (in_bom yes) (on_board yes)
-    (property "Reference" "R?" (id 0) (at 160.655 86.36 0)
+    (property "Reference" "R19" (id 0) (at 160.655 86.36 0)
       (effects (font (size 1.27 1.27)) (justify left))
     )
@@
   (symbol (lib_id "power:+5V") (at 170.815 67.31 0) (unit 1)
     (in_bom yes) (on_board yes) (fields_autoplaced)
-    (property "Reference" "#PWR?" (id 0) (at 170.815 71.12 0)
+    (property "Reference" "#PWR058" (id 0) (at 170.815 71.12 0)
       (effects (font (size 1.27 1.27)) hide)
     )
@@
   (symbol (lib_id "power:VBUS") (at 118.745 67.31 0) (unit 1)
     (in_bom yes) (on_board yes) (fields_autoplaced)
-    (property "Reference" "#PWR?" (id 0) (at 118.745 71.12 0)
+    (property "Reference" "#PWR057" (id 0) (at 118.745 71.12 0)
       (effects (font (size 1.27 1.27)) hide)
     )
@@
   (symbol (lib_id "Device:D_Schottky_Small") (at 153.035 68.58 180) (unit 1)
     (in_bom yes) (on_board yes)
-    (property "Reference" "D?" (id 0) (at 153.035 66.04 0))
+    (property "Reference" "D4" (id 0) (at 153.035 66.04 0))
     (property "Value" "SS12" (id 1) (at 153.035 71.12 0))
     (property "Footprint" "Diode_SMD:D_SMA" (id 2) (at 153.035 68.58 90)
@@
   (symbol (lib_id "Device:R_Small") (at 159.385 76.2 0) (unit 1)
     (in_bom yes) (on_board yes)
-    (property "Reference" "R?" (id 0) (at 160.655 74.93 0)
+    (property "Reference" "R18" (id 0) (at 160.655 74.93 0)
       (effects (font (size 1.27 1.27)) (justify left))
     )
@@
   (symbol (lib_id "Device:C_Small") (at 118.745 80.645 0) (unit 1)
     (in_bom yes) (on_board yes)
-    (property "Reference" "C?" (id 0) (at 120.65 79.375 0)
+    (property "Reference" "C14" (id 0) (at 120.65 79.375 0)
       (effects (font (size 1.27 1.27)) (justify left))
     )
@@
   (symbol (lib_id "Device:L_Small") (at 139.7 68.58 90) (unit 1)
     (in_bom yes) (on_board yes)
-    (property "Reference" "L?" (id 0) (at 139.7 66.675 90))
+    (property "Reference" "L2" (id 0) (at 139.7 66.675 90))
     (property "Value" "4R7" (id 1) (at 139.7 70.485 90))
     (property "Footprint" "Footprints:Inductor_4mm(5x5mm pads)" (id 2) (at 139.7 68.58 0)
@@
   (symbol (lib_id "Device:C_Small") (at 170.815 80.645 0) (unit 1)
     (in_bom yes) (on_board yes) (fields_autoplaced)
-    (property "Reference" "C?" (id 0) (at 173.1391 79.8166 0)
+    (property "Reference" "C15" (id 0) (at 173.1391 79.8166 0)
       (effects (font (size 1.27 1.27)) (justify left))
     )
@@
   (symbol (lib_id "power:GND") (at 139.7 94.615 0) (unit 1)
     (in_bom yes) (on_board yes) (fields_autoplaced)
-    (property "Reference" "#PWR?" (id 0) (at 139.7 100.965 0)
+    (property "Reference" "#PWR059" (id 0) (at 139.7 100.965 0)
       (effects (font (size 1.27 1.27)) hide)
     )

Commit message: update
Parts:
- renumbered C14 to C601, C15 to C602, D4 to D601, L2 to L601, R18 to R601, R19 to R602, U6 to U601
Changed lines of the file:
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@@
   (symbol (lib_id "Regulator_Switching:MT3608") (at 139.7 80.645 0) (unit 1)
     (in_bom yes) (on_board yes)
-    (property "Reference" "U6" (id 0) (at 135.89 74.295 0))
+    (property "Reference" "U601" (id 0) (at 135.89 74.295 0))
     (property "Value" "MT3608" (id 1) (at 144.145 86.995 0))
     (property "Footprint" "Package_TO_SOT_SMD:SOT-23-6" (id 2) (at 140.97 86.995 0)
@@
   (symbol (lib_id "Device:R_Small") (at 159.385 87.63 0) (unit 1)
     (in_bom yes) (on_board yes)
-    (property "Reference" "R19" (id 0) (at 160.655 86.36 0)
+    (property "Reference" "R602" (id 0) (at 160.655 86.36 0)
       (effects (font (size 1.27 1.27)) (justify left))
     )
@@
   (symbol (lib_id "power:+5V") (at 170.815 67.31 0) (unit 1)
     (in_bom yes) (on_board yes) (fields_autoplaced)
-    (property "Reference" "#PWR058" (id 0) (at 170.815 71.12 0)
+    (property "Reference" "#PWR0602" (id 0) (at 170.815 71.12 0)
       (effects (font (size 1.27 1.27)) hide)
     )
@@
   (symbol (lib_id "power:VBUS") (at 118.745 67.31 0) (unit 1)
     (in_bom yes) (on_board yes) (fields_autoplaced)
-    (property "Reference" "#PWR057" (id 0) (at 118.745 71.12 0)
+    (property "Reference" "#PWR0601" (id 0) (at 118.745 71.12 0)
       (effects (font (size 1.27 1.27)) hide)
     )
@@
   (symbol (lib_id "Device:D_Schottky_Small") (at 153.035 68.58 180) (unit 1)
     (in_bom yes) (on_board yes)
-    (property "Reference" "D4" (id 0) (at 153.035 66.04 0))
+    (property "Reference" "D601" (id 0) (at 153.035 66.04 0))
     (property "Value" "SS12" (id 1) (at 153.035 71.12 0))
     (property "Footprint" "Diode_SMD:D_SMA" (id 2) (at 153.035 68.58 90)
@@
   (symbol (lib_id "Device:R_Small") (at 159.385 76.2 0) (unit 1)
     (in_bom yes) (on_board yes)
-    (property "Reference" "R18" (id 0) (at 160.655 74.93 0)
+    (property "Reference" "R601" (id 0) (at 160.655 74.93 0)
       (effects (font (size 1.27 1.27)) (justify left))
     )
@@
   (symbol (lib_id "Device:C_Small") (at 118.745 80.645 0) (unit 1)
     (in_bom yes) (on_board yes)
-    (property "Reference" "C14" (id 0) (at 120.65 79.375 0)
+    (property "Reference" "C601" (id 0) (at 120.65 79.375 0)
       (effects (font (size 1.27 1.27)) (justify left))
     )
@@
   (symbol (lib_id "Device:L_Small") (at 139.7 68.58 90) (unit 1)
     (in_bom yes) (on_board yes)
-    (property "Reference" "L2" (id 0) (at 139.7 66.675 90))
+    (property "Reference" "L601" (id 0) (at 139.7 66.675 90))
     (property "Value" "4R7" (id 1) (at 139.7 70.485 90))
     (property "Footprint" "Footprints:Inductor_4mm(5x5mm pads)" (id 2) (at 139.7 68.58 0)
@@
   (symbol (lib_id "Device:C_Small") (at 170.815 80.645 0) (unit 1)
     (in_bom yes) (on_board yes) (fields_autoplaced)
-    (property "Reference" "C15" (id 0) (at 173.1391 79.8166 0)
+    (property "Reference" "C602" (id 0) (at 173.1391 79.8166 0)
       (effects (font (size 1.27 1.27)) (justify left))
     )
@@
   (symbol (lib_id "power:GND") (at 139.7 94.615 0) (unit 1)
     (in_bom yes) (on_board yes) (fields_autoplaced)
-    (property "Reference" "#PWR059" (id 0) (at 139.7 100.965 0)
+    (property "Reference" "#PWR0603" (id 0) (at 139.7 100.965 0)
       (effects (font (size 1.27 1.27)) hide)
     )

Commit message: update
Parts:
- C601, C602: JLCPCB Part # (none) -> C337451; U labosu? (none) -> ne
- D601: JLCPCB Part # (none) -> C2985002; U labosu? (none) -> ne
- L601, R601: U labosu? (none) -> da
- R602: JLCPCB Part # (none) -> C185373; U labosu? (none) -> ne
- U601: JLCPCB Part # (none) -> C2932326; U labosu? (none) -> da
Changed lines of the file:
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@@
+      (effects (font (size 1.27 1.27)) hide)
+    )
+    (property "JLCPCB Part #" "C2932326" (id 4) (at 139.7 80.645 0)
+      (effects (font (size 1.27 1.27)) hide)
+    )
+    (property "U labosu?" "da" (id 5) (at 139.7 80.645 0)
       (effects (font (size 1.27 1.27)) hide)
     )
@@
     )
     (property "Datasheet" "~" (id 3) (at 159.385 87.63 0)
+      (effects (font (size 1.27 1.27)) hide)
+    )
+    (property "JLCPCB Part #" "C185373" (id 4) (at 159.385 87.63 0)
+      (effects (font (size 1.27 1.27)) hide)
+    )
+    (property "U labosu?" "ne" (id 5) (at 159.385 87.63 0)
       (effects (font (size 1.27 1.27)) hide)
     )
@@
       (effects (font (size 1.27 1.27)) hide)
     )
+    (property "JLCPCB Part #" "C2985002" (id 4) (at 153.035 68.58 0)
+      (effects (font (size 1.27 1.27)) hide)
+    )
+    (property "U labosu?" "ne" (id 5) (at 153.035 68.58 0)
+      (effects (font (size 1.27 1.27)) hide)
+    )
     (pin "1")
     (pin "2")
@@
     )
     (property "Datasheet" "~" (id 3) (at 159.385 76.2 0)
+      (effects (font (size 1.27 1.27)) hide)
+    )
+    (property "U labosu?" "da" (id 4) (at 159.385 76.2 0)
       (effects (font (size 1.27 1.27)) hide)
     )
@@
       (effects (font (size 1.27 1.27)) hide)
     )
+    (property "JLCPCB Part #" "C337451" (id 4) (at 118.745 80.645 0)
+      (effects (font (size 1.27 1.27)) hide)
+    )
+    (property "U labosu?" "ne" (id 5) (at 118.745 80.645 0)
+      (effects (font (size 1.27 1.27)) hide)
+    )
     (pin "1")
     (pin "2")
@@
     )
     (property "Datasheet" "~" (id 3) (at 139.7 68.58 0)
+      (effects (font (size 1.27 1.27)) hide)
+    )
+    (property "U labosu?" "da" (id 4) (at 139.7 68.58 0)
       (effects (font (size 1.27 1.27)) hide)
     )
@@
       (effects (font (size 1.27 1.27)) hide)
     )
+    (property "JLCPCB Part #" "C337451" (id 4) (at 170.815 80.645 0)
+      (effects (font (size 1.27 1.27)) hide)
+    )
+    (property "U labosu?" "ne" (id 5) (at 170.815 80.645 0)
+      (effects (font (size 1.27 1.27)) hide)
+    )

Commit message: update
Connections:
- net VBUS: now also U601.4 (EN)
- net L_OUT: now reaches D601.2 (A), L601.2, U601.1 (SW)
- net FB: now reaches R601.2, R602.1, U601.3 (FB)
- no-connect marks 1 -> 0
Changed lines of the file:
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@@
     (rev "1")
+  )
+  (junction (at 131.445 78.105) (diameter 0) (color 0 0 0 0)
   )
   (junction (at 170.815 68.58) (diameter 0) (color 0 0 0 0)
@@
   (junction (at 131.445 68.58) (diameter 0) (color 0 0 0 0)
   )
-  (no_connect (at 132.08 83.185))
   (wire (pts (xy 159.385 68.58) (xy 170.815 68.58))
     (stroke (width 0) (type default) (color 0 0 0 0))
@@
     (stroke (width 0) (type default) (color 0 0 0 0))
   )
+  (wire (pts (xy 131.445 83.185) (xy 132.08 83.185))
+    (stroke (width 0) (type default) (color 0 0 0 0))
+  )
   (wire (pts (xy 132.08 78.105) (xy 131.445 78.105))
     (stroke (width 0) (type default) (color 0 0 0 0))
   )
   (wire (pts (xy 131.445 78.105) (xy 131.445 68.58))
+    (stroke (width 0) (type default) (color 0 0 0 0))
+  )
+  (wire (pts (xy 131.445 78.105) (xy 131.445 83.185))
     (stroke (width 0) (type default) (color 0 0 0 0))
   )
@@
     (effects (font (size 1.27 1.27)) (justify left bottom))
   )
+  (label "L_OUT" (at 142.875 68.58 0)
+    (effects (font (size 1.27 1.27)) (justify left bottom))
+  )
+  (label "FB" (at 147.32 83.185 0)
+    (effects (font (size 1.27 1.27)) (justify left bottom))
+  )

Commit message: Documentation
Other:
- note removed: "For best performance of the MT3608, the following guidelines must be strictly followed: - Input and Output capacitors should be placed close to the IC and connected to ground plane to reduce noise coupling - The GND should be connected to a strong ground plane for heat sinking and noise protection - Keep the main current traces as possible as short and wide - SW node of DC-DC converter is with hi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"
Changed lines of the file:
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@@
-    (effects (font (size 1.27 1.27)) (justify left bottom))
-  )
-  (text "For best performance of the MT3608, the following\nguidelines must be strictly followed:\n\n- Input and Output capacitors should be placed\nclose to the IC and connected to ground plane\nto reduce noise coupling\n\n- The GND should be connected to a strong\nground plane for heat sinking and noise\nprotection\n\n- Keep the main current traces as possible as\nshort and wide\n\n- SW node of DC-DC converter is with high\nfrequency voltage swing. It should be kept at a\nsmall area\n\n- Place the feedback components as close as\npossible to the IC and keep away from the\nnoisy devices"
-    (at 26.67 160.655 0)
     (effects (font (size 1.27 1.27)) (justify left bottom))
   )
