File: KiCad files/BoardGame/Finish LEDs.kicad_sch (KiCad schematic)
At the start: 17 parts

Commit message: Schematic update
Changed lines of the file:
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@@
     (stroke (width 0) (type default) (color 0 0 0 0))
   )
-  (global_label "NP_1" (shape input) (at 74.93 77.47 180) (fields_autoplaced)
+  (hierarchical_label "NP_1" (shape input) (at 74.93 77.47 180)
     (effects (font (size 1.27 1.27)) (justify right))
-    (property "Intersheet References" "${INTERSHEET_REFS}" (id 0) (at 67.8282 77.3906 0)
-      (effects (font (size 1.27 1.27)) (justify right) hide)
-    )
   )
   (symbol (lib_id "power:GND") (at 106.045 85.09 0) (unit 1)
