File: KiCad files/BoardGame/Finish LEDs.kicad_sch (KiCad schematic)
At the start: 17 parts

Commit message: update
Other:
- note added: "Finish LEDs"
Changed lines of the file:
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@@
     (stroke (width 0) (type default))
+  )
+  (text "Finish LEDs" (at 95.885 43.18 0)
+    (effects (font (size 3 3) (thickness 0.6) bold) (justify left bottom))
   )
   (hierarchical_label "NP_1" (shape input) (at 74.93 77.47 180) (fields_autoplaced)
