File: KiCad files/BoardGame/Path LEDs.kicad_sch (KiCad schematic)
At the start: 53 parts

Commit message: Schematic update
Changed lines of the file:
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@@
     (stroke (width 0) (type default) (color 0 0 0 0))
   )
-  (global_label "NP_2" (shape input) (at 53.975 38.1 180) (fields_autoplaced)
+  (hierarchical_label "NP_2" (shape input) (at 53.975 38.1 180)
     (effects (font (size 1.27 1.27)) (justify right))
-    (property "Intersheet References" "${INTERSHEET_REFS}" (id 0) (at 46.8732 38.0206 0)
-      (effects (font (size 1.27 1.27)) (justify right) hide)
-    )
   )
   (symbol (lib_id "power:GND") (at 234.95 155.575 0) (unit 1)
