File: KiCad files/BoardGame/Path LEDs.kicad_sch (KiCad schematic)
At the start: 53 parts

Commit message: update
Other:
- note added: "Path LEDs"
Changed lines of the file:
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@@
     (stroke (width 0) (type default))
+  )
+  (text "Path LEDs" (at 25.4 22.86 0)
+    (effects (font (size 3 3) (thickness 0.6) bold) (justify left bottom))
   )
   (hierarchical_label "NP_2" (shape input) (at 53.975 38.1 180) (fields_autoplaced)
