File: KiCad files/BoardGame/Touchpad LEDs.kicad_sch (KiCad schematic)
At the start: 13 parts

Commit message: Schematic update
Changed lines of the file:
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@@
     (stroke (width 0) (type default) (color 0 0 0 0))
   )
-  (global_label "NP_5" (shape input) (at 63.5 83.185 180) (fields_autoplaced)
+  (hierarchical_label "NP_5" (shape input) (at 63.5 83.185 180)
     (effects (font (size 1.27 1.27)) (justify right))
-    (property "Intersheet References" "${INTERSHEET_REFS}" (id 0) (at 56.3982 83.1056 0)
-      (effects (font (size 1.27 1.27)) (justify right) hide)
-    )
   )
   (symbol (lib_id "LED:WS2812B") (at 94.615 83.185 0) (unit 1)
