File: KiCad files/BoardGame/Touchpad LEDs.kicad_sch (KiCad schematic)
At the start: 13 parts

Commit message: update
Other:
- note added: "Touchpads LEDs"
Changed lines of the file:
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@@
     (stroke (width 0) (type default))
+  )
+  (text "Touchpads LEDs" (at 81.28 44.45 0)
+    (effects (font (size 3 3) (thickness 0.6) bold) (justify left bottom))
   )
   (hierarchical_label "NP_5" (shape input) (at 63.5 83.185 180) (fields_autoplaced)
