File: KiCad files/BoardGame/Battery indicator LED.kicad_sch (KiCad schematic)
At the start: 2 parts

Commit message: update
Other:
- note added: "Battery LED"
Changed lines of the file:
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@@
     (stroke (width 0) (type default))
+  )
+  (text "Battery LED" (at 86.995 43.18 0)
+    (effects (font (size 3 3) (thickness 0.6) bold) (justify left bottom))
   )
   (hierarchical_label "NP_6" (shape input) (at 112.395 73.025 180) (fields_autoplaced)
