File: KiCad files/BoardGame/Dice LEDs.kicad_sch (KiCad schematic)
At the start: 19 parts

Commit message: update
Other:
- note added: "Dice LEDs"
Changed lines of the file:
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@@
     (stroke (width 0) (type default))
+  )
+  (text "Dice LEDs" (at 67.31 32.385 0)
+    (effects (font (size 3 3) (thickness 0.6) bold) (justify left bottom))
   )
   (hierarchical_label "NP_3" (shape input) (at 57.15 64.135 180) (fields_autoplaced)
