File: KiCad files/BoardGame/Safehouse LEDs.kicad_sch (KiCad schematic)
At the start: 17 parts

Commit message: update
Other:
- note added: "Safehouse LEDs"
Changed lines of the file:
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@@
     (stroke (width 0) (type default))
+  )
+  (text "Safehouse LEDs" (at 90.17 40.64 0)
+    (effects (font (size 3 3) (thickness 0.6) bold) (justify left bottom))
   )
   (hierarchical_label "NP_4" (shape input) (at 75.565 76.835 180) (fields_autoplaced)
