File: KiCad files/Touchpad/Touchpad.kicad_pcb (KiCad board)
At the start: 2 copper layers, 56 x 16 mm, 13 parts, among them J1 Conn_02x03_Counter_Clockwise, U1 TTP223-BA6, U2 TTP223-BA6, U3 TTP223-BA6

Commit message: Schematic update
Other:
- outline, holes or cut-outs redrawn
