File: KiCad files/Dice/Dice.kicad_sch (KiCad schematic)
At the start: 4 parts, among them J1 Conn_01x02_Male, J2 Conn_01x02_Male, J3 Conn_01x02_Male, J4 Conn_01x02_Male

Commit message: Schematic update
Parts:
- added C1: 100n, Capacitor_SMD:C_0603_1608Metric, symbol Device:C_Small
- added C2: 0-50 pF, Capacitor_SMD:C_0603_1608Metric, symbol Device:C_Small
- added U1: TTP223-BA6, Package_TO_SOT_SMD:SOT-23-6, symbol Symbols:TTP223-BA6
- renumbered J3 to J1, J1 to J3
Connections:
- removed net TOUCHPAD: J1.1 (Pin_1), J1.2 (Pin_2), J2.1 (Pin_1), J2.2 (Pin_2), J3.1 (Pin_1), J3.2 (Pin_2), J4.1 (Pin_1), J4.2 (Pin_2)
- new net +5V: C1.1, J3.1 (Pin_1), J3.2 (Pin_2), U1.5 (VDD)
- new net GND: C1.2, C2.2, J4.1 (Pin_1), J4.2 (Pin_2), U1.2 (VSS)
- new net TP: C2.1, U1.3 (I)
- new net TP_OUT: J2.1 (Pin_1), J2.2 (Pin_2), U1.1 (Q)
- no-connect marks 0 -> 4
Other:
- moved on the sheet: J1, J2, J3, J4
