File: KiCad files/Dice/Dice.kicad_pcb (KiCad board)
At the start: 2 copper layers, 26 x 26 mm, 7 parts, among them J1 Conn_01x02_Male, J2 Conn_01x02_Male, J3 Conn_01x02_Male, J4 Conn_01x02_Male, U1 TTP223-BA6

Commit message: update
Routing:
- added copper zone on B.Cu, net /TP
